File: Canal_Aux.kicad_sch (KiCad schematic)
At the start: 0 parts

Commit message: Add files via upload
Connections:
- no-connect marks 1 -> 0
Changed lines of the file:
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@@
 	(generator_version "10.0")
 	(paper "A4")
-	(no_connect
-		(at -88.9 46.99)
-	)
 	(wire
 		(pts

Commit message: Add files via upload
Other:
- sheet Vehicule_Aux ports: added none; removed Injection_Aux_Fault
Changed lines of the file:
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@@
-	(wire
-		(pts
-			(xy 49.53 27.94) (xy 58.42 27.94)
-		)
-		(stroke
-			(width 0)
-			(type default)
-		)
-	)
 	(wire
 		(pts
@@
 	(wire
 		(pts
-			(xy 53.34 46.99) (xy 53.34 41.91)
-		)
-		(stroke
-			(width 0)
-			(type default)
-		)
-	)
-	(wire
-		(pts
-			(xy 48.26 36.83) (xy 58.42 36.83)
-		)
-		(stroke
-			(width 0)
-			(type default)
-		)
-	)
-	(wire
-		(pts
-			(xy 48.26 30.48) (xy 58.42 30.48)
-		)
-		(stroke
-			(width 0)
-			(type default)
-		)
-	)
-	(wire
-		(pts
-			(xy 39.37 41.91) (xy 48.26 41.91)
-		)
-		(stroke
-			(width 0)
-			(type default)
-		)
-	)
-	(wire
-		(pts
-			(xy 39.37 46.99) (xy 53.34 46.99)
-		)
-		(stroke
-			(width 0)
-			(type default)
-		)
-	)
-	(wire
-		(pts
-			(xy 48.26 25.4) (xy 48.26 30.48)
-		)
-		(stroke
-			(width 0)
-			(type default)
-		)
-	)
-	(wire
-		(pts
-			(xy 53.34 41.91) (xy 58.42 41.91)
-		)
-		(stroke
-			(width 0)
-			(type default)
-		)
-	)
-	(wire
-		(pts
-			(xy 50.8 39.37) (xy 50.8 44.45)
-		)
-		(stroke
-			(width 0)
-			(type default)
-		)
-	)
-	(wire
-		(pts
-			(xy 50.8 39.37) (xy 58.42 39.37)
-		)
-		(stroke
-			(width 0)
-			(type default)
-		)
-	)
-	(wire
-		(pts
-			(xy 38.1 21.59) (xy 49.53 21.59)
-		)
-		(stroke
-			(width 0)
-			(type default)
-		)
-	)
-	(wire
-		(pts
-			(xy 38.1 25.4) (xy 48.26 25.4)
-		)
-		(stroke
-			(width 0)
-			(type default)
-		)
-	)
-	(wire
-		(pts
-			(xy 39.37 54.61) (xy 41.91 54.61)
-		)
-		(stroke
-			(width 0)
-			(type default)
-		)
-	)
-	(wire
-		(pts
-			(xy 49.53 21.59) (xy 49.53 27.94)
-		)
-		(stroke
-			(width 0)
-			(type default)
-		)
-	)
-	(wire
-		(pts
-			(xy 39.37 44.45) (xy 50.8 44.45)
-		)
-		(stroke
-			(width 0)
-			(type default)
-		)
-	)
-	(wire
-		(pts
-			(xy 38.1 32.385) (xy 40.64 32.385)
-		)
-		(stroke
-			(width 0)
-			(type default)
-		)
-	)
-	(wire
-		(pts
-			(xy 48.26 36.83) (xy 48.26 41.91)
+			(xy 39.37 41.91) (xy 52.07 41.91)
+		)
+		(stroke
+			(width 0)
+			(type default)
+		)
+	)
+	(wire
+		(pts
+			(xy 39.37 46.99) (xy 52.07 46.99)
+		)
+		(stroke
+			(width 0)
+			(type default)
+		)
+	)
+	(wire
+		(pts
+			(xy 97.79 69.85) (xy 99.06 69.85)
+		)
+		(stroke
+			(width 0)
+			(type default)
+		)
+	)
+	(wire
+		(pts
+			(xy 38.1 21.59) (xy 52.07 21.59)
+		)
+		(stroke
+			(width 0)
+			(type default)
+		)
+	)
+	(wire
+		(pts
+			(xy 38.1 25.4) (xy 52.07 25.4)
+		)
+		(stroke
+			(width 0)
+			(type default)
+		)
+	)
+	(wire
+		(pts
+			(xy 39.37 49.53) (xy 41.91 49.53)
+		)
+		(stroke
+			(width 0)
+			(type default)
+		)
+	)
+	(wire
+		(pts
+			(xy 39.37 44.45) (xy 52.07 44.45)
 		)
 		(stroke
@@
 	(hierarchical_label "Trail_Aux"
 		(shape input)
-		(at 41.91 54.61 0)
-		(effects
-			(font
-				(size 0.762 0.762)
-			)
-			(justify left)
-		)
-	)
-	(hierarchical_label "Injection_Aux_Fault"
-		(shape input)
-		(at 40.64 32.385 0)
+		(at 41.91 49.53 0)
 		(effects
 			(font
@@
 			)
 		)
-		(pin "Injection_Aux_Fault" input
-			(at 38.1 32.385 0)
-			(effects
-				(font
-					(size 0.762 0.762)
-				)
-				(justify right)
-			)
-		)
 		(instances
 			(project "TrailerDiagnosticSystem"
@@
 	(sheet
 		(at 17.78 39.37)
-		(size 21.59 19.05)
+		(size 21.59 12.7)
 		(exclude_from_sim no)
 		(in_bom yes)
@@
 		)
 		(property "Sheetfile" "Trailer_Aux.kicad_sch"
-			(at 17.78 58.8014 0)
+			(at 17.78 52.4514 0)
 			(show_name no)
 			(do_not_autoplace no)
@@
 		)
 		(pin "Trail_Aux" input
-			(at 39.37 54.61 0)
+			(at 39.37 49.53 0)
 			(effects
 				(font
@@
 	)
 	(sheet
-		(at 58.42 24.13)
-		(size 25.4 22.86)
+		(at 52.07 19.05)
+		(size 25.4 33.02)
 		(exclude_from_sim no)
 		(in_bom yes)
@@
 		)
 		(property "Sheetname" "Bloc_Test_Aux"
-			(at 58.42 23.6724 0)
+			(at 52.07 18.5924 0)
 			(show_name no)
 			(do_not_autoplace no)
@@
 		)
 		(property "Sheetfile" "Bloc_Test_Aux.kicad_sch"
-			(at 58.42 47.3714 0)
+			(at 52.07 52.4514 0)
 			(show_name no)
 			(do_not_autoplace no)
@@
 		)
 		(pin "Court_Aux_Trailer" input
-			(at 58.42 39.37 180)
+			(at 52.07 44.45 180)
 			(effects
 				(font
@@
 		)
 		(pin "Ouvert_Aux_Vehic" input
-			(at 58.42 27.94 180)
+			(at 52.07 21.59 180)
 			(effects
 				(font
@@
 		)
 		(pin "Btn_Aux_Etat" input
-			(at 58.42 41.91 180)
+			(at 52.07 46.99 180)
 			(effects
 				(font
@@
 		)
 		(pin "Ouvert_Aux_Trailer" input
-			(at 58.42 36.83 180)
+			(at 52.07 41.91 180)
 			(effects
 				(font
@@
 		)
 		(pin "Court_Aux_Vehic" input
-			(at 58.42 30.48 180)
-			(effects
-				(font
+			(at 52.07 25.4 180)
+			(effects
+				(font
