File: Canal_Brake.kicad_sch (KiCad schematic)
At the start: 0 parts

Commit message: Add files via upload
Changed lines of the file:
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@@
 	(paper "A4")
 	(sheet
-		(at 39.37 34.29)
+		(at 19.05 12.7)
 		(size 40.64 44.45)
 		(exclude_from_sim no)
@@
 		)
 		(property "Sheetname" "Vehicule_Brake"
-			(at 39.37 33.8324 0)
+			(at 19.05 12.2424 0)
 			(show_name no)
 			(do_not_autoplace no)
@@
 		)
 		(property "Sheetfile" "Vehicule_Brake.kicad_sch"
-			(at 39.37 79.1214 0)
+			(at 19.05 57.5314 0)
 			(show_name no)
 			(do_not_autoplace no)
@@
 	)
 	(sheet
-		(at 90.17 35.56)
+		(at 20.32 62.23)
 		(size 35.56 43.18)
 		(exclude_from_sim no)
@@
 		)
 		(property "Sheetname" "Trailer_Brake"
-			(at 90.17 35.1024 0)
+			(at 20.32 61.7724 0)
 			(show_name no)
 			(do_not_autoplace no)
@@
 		)
 		(property "Sheetfile" "Trailer_Brake.kicad_sch"
-			(at 90.17 79.1214 0)
+			(at 20.32 105.7914 0)
 			(show_name no)
 			(do_not_autoplace no)
@@
 	)
 	(sheet
-		(at 138.43 35.56)
+		(at 91.44 29.21)
 		(size 33.02 43.18)
 		(exclude_from_sim no)
@@
 		)
 		(property "Sheetname" "Bloc_Test_Brake"
-			(at 138.43 35.1024 0)
+			(at 91.44 28.7524 0)
 			(show_name no)
 			(do_not_autoplace no)
@@
 		)
 		(property "Sheetfile" "Bloc_Test_Brake.kicad_sch"
-			(at 138.43 79.1214 0)
+			(at 91.44 72.7714 0)
 			(show_name no)
 			(do_not_autoplace no)
@@
 		)
 		(pin "Ouvert_Brake_Trailer" input
-			(at 138.43 45.72 180)
+			(at 91.44 39.37 180)
 			(effects
 				(font
@@
 		)
 		(pin "Ouvert_Brake_Vehic" input
-			(at 138.43 50.8 180)
+			(at 91.44 44.45 180)
 			(effects
 				(font
@@
 		)
 		(pin "Btn_Brake_Etat" input
-			(at 138.43 55.88 180)
+			(at 91.44 49.53 180)
 			(effects
 				(font
@@
 		)
 		(pin "Court_Brake_Trailer" input
-			(at 138.43 59.69 180)
+			(at 91.44 53.34 180)
 			(effects
 				(font
@@
 		)
 		(pin "Court_Brake_Vehic" input
-			(at 138.43 64.77 180)
+			(at 91.44 58.42 180)
 			(effects
 				(font

Commit message: Add files via upload
Other:
- sheet Trailer_Brake ports: added Btn_Brake_Etat, Court_Brake_Trailer, Ouvert_Brake_Trailer, Trail_Brake; removed none
- sheet Vehicule_Brake ports: added Court_Brake_Vehic, Ouvert_Brake_Vehic, Veh_Brake; removed none

Commit message: Add files via upload
Other:
- sheet Vehicule_Brake ports: added Injection_Brake_Fault; removed none
Changed lines of the file:
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@@
+	(wire
+		(pts
+			(xy 38.1 40.005) (xy 40.64 40.005)
+		)
+		(stroke
+			(width 0)
+			(type default)
+		)
+	)
 	(wire
 		(pts
@@
 		)
 	)
+	(hierarchical_label "Injection_Brake_Fault"
+		(shape input)
+		(at 40.64 40.005 0)
+		(effects
+			(font
+				(size 1.27 1.27)
+			)
+			(justify left)
+		)
+	)
 	(hierarchical_label "Trail_Brake"
 		(shape input)
@@
 	(sheet
 		(at 17.78 20.32)
-		(size 20.32 19.05)
+		(size 20.32 22.86)
 		(exclude_from_sim no)
 		(in_bom yes)
@@
 		)
 		(property "Sheetfile" "Vehicule_Brake.kicad_sch"
-			(at 17.78 39.7514 0)
+			(at 17.78 43.5614 0)
 			(show_name no)
 			(do_not_autoplace no)
@@
 				)
 				(justify right)
+			)
+		)
+		(pin "Injection_Brake_Fault" input
+			(at 38.1 40.005 0)
+			(effects
+				(font
+					(size 1.016 1.016)
+				)
+				(justify right)

Commit message: Add files via upload
Other:
- sheet Vehicule_Brake ports: added none; removed Injection_Brake_Fault
Changed lines of the file:
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@@
-	(wire
-		(pts
-			(xy 38.1 40.005) (xy 40.64 40.005)
-		)
-		(stroke
-			(width 0)
-			(type default)
-		)
-	)
 	(wire
 		(pts
@@
 		)
 	)
-	(hierarchical_label "Injection_Brake_Fault"
-		(shape input)
-		(at 40.64 40.005 0)
-		(effects
-			(font
-				(size 1.27 1.27)
-			)
-			(justify left)
-		)
-	)
 	(hierarchical_label "Trail_Brake"
 		(shape input)
@@
 	(sheet
 		(at 17.78 20.32)
-		(size 20.32 22.86)
+		(size 20.32 19.05)
 		(exclude_from_sim no)
 		(in_bom yes)
@@
 		)
 		(property "Sheetfile" "Vehicule_Brake.kicad_sch"
-			(at 17.78 43.5614 0)
+			(at 17.78 39.7514 0)
 			(show_name no)
 			(do_not_autoplace no)
@@
 				)
 				(justify right)
-			)
-		)
-		(pin "Injection_Brake_Fault" input
-			(at 38.1 40.005 0)
-			(effects
-				(font
-					(size 1.016 1.016)
-				)
-				(justify right)
