File: Canal_Tail.kicad_sch (KiCad schematic)
At the start: 0 parts

Commit message: Add files via upload
Other:
- sheet Vehicule_Tail ports: added none; removed Injection_Tail_Fault
Changed lines of the file:
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@@
 	(wire
 		(pts
-			(xy 59.69 55.88) (xy 64.77 55.88)
-		)
-		(stroke
-			(width 0)
-			(type default)
-		)
-	)
-	(wire
-		(pts
-			(xy 63.5 53.34) (xy 63.5 20.32)
+			(xy 59.69 53.34) (xy 64.77 53.34)
+		)
+		(stroke
+			(width 0)
+			(type default)
+		)
+	)
+	(wire
+		(pts
+			(xy 63.5 50.8) (xy 63.5 20.32)
 		)
 		(stroke
@@
 	(wire
 		(pts
-			(xy 59.69 50.8) (xy 62.23 50.8)
+			(xy 59.69 48.26) (xy 62.23 48.26)
 		)
 		(stroke
@@
 	(wire
 		(pts
-			(xy 59.69 87.63) (xy 64.77 87.63)
+			(xy 59.69 69.85) (xy 64.77 69.85)
 		)
 		(stroke
@@
 	(wire
 		(pts
-			(xy 35.56 31.75) (xy 35.56 85.09)
-		)
-		(stroke
-			(width 0)
-			(type default)
-		)
-	)
-	(wire
-		(pts
-			(xy 59.69 60.325) (xy 64.77 60.325)
-		)
-		(stroke
-			(width 0)
-			(type default)
-		)
-	)
-	(wire
-		(pts
-			(xy 39.37 82.55) (xy 39.37 35.56)
-		)
-		(stroke
-			(width 0)
-			(type default)
-		)
-	)
-	(wire
-		(pts
-			(xy 43.18 82.55) (xy 39.37 82.55)
-		)
-		(stroke
-			(width 0)
-			(type default)
-		)
-	)
-	(wire
-		(pts
-			(xy 43.18 90.17) (xy 31.75 90.17)
-		)
-		(stroke
-			(width 0)
-			(type default)
-		)
-	)
-	(wire
-		(pts
-			(xy 62.23 50.8) (xy 62.23 24.13)
+			(xy 35.56 31.75) (xy 35.56 67.31)
+		)
+		(stroke
+			(width 0)
+			(type default)
+		)
+	)
+	(wire
+		(pts
+			(xy 39.37 64.77) (xy 39.37 35.56)
+		)
+		(stroke
+			(width 0)
+			(type default)
+		)
+	)
+	(wire
+		(pts
+			(xy 43.18 64.77) (xy 39.37 64.77)
+		)
+		(stroke
+			(width 0)
+			(type default)
+		)
+	)
+	(wire
+		(pts
+			(xy 43.18 72.39) (xy 31.75 72.39)
+		)
+		(stroke
+			(width 0)
+			(type default)
+		)
+	)
+	(wire
+		(pts
+			(xy 62.23 48.26) (xy 62.23 24.13)
 		)
 		(stroke
@@
 	(wire
 		(pts
-			(xy 31.75 90.17) (xy 31.75 27.94)
-		)
-		(stroke
-			(width 0)
-			(type default)
-		)
-	)
-	(wire
-		(pts
-			(xy 35.56 85.09) (xy 43.18 85.09)
-		)
-		(stroke
-			(width 0)
-			(type default)
-		)
-	)
-	(wire
-		(pts
-			(xy 59.69 53.34) (xy 63.5 53.34)
-		)
-		(stroke
-			(width 0)
-			(type default)
-		)
-	)
-	(hierarchical_label "Injection_Tail_Fault"
+			(xy 31.75 72.39) (xy 31.75 27.94)
+		)
+		(stroke
+			(width 0)
+			(type default)
+		)
+	)
+	(wire
+		(pts
+			(xy 35.56 67.31) (xy 43.18 67.31)
+		)
+		(stroke
+			(width 0)
+			(type default)
+		)
+	)
+	(wire
+		(pts
+			(xy 59.69 50.8) (xy 63.5 50.8)
+		)
+		(stroke
+			(width 0)
+			(type default)
+		)
+	)
+	(hierarchical_label "Trail_Tail"
 		(shape input)
-		(at 64.77 60.325 0)
+		(at 64.77 69.85 0)
 		(effects
 			(font
@@
 		)
 	)
-	(hierarchical_label "Trail_Tail"
+	(hierarchical_label "Veh_Tail"
 		(shape input)
-		(at 64.77 87.63 0)
+		(at 64.77 53.34 0)
 		(effects
 			(font
@@
 		)
 	)
-	(hierarchical_label "Veh_Tail"
-		(shape input)
-		(at 64.77 55.88 0)
-		(effects
-			(font
-				(size 1.27 1.27)
-			)
-			(justify left)
-		)
-	)
 	(sheet
-		(at 43.18 80.01)
-		(size 16.51 22.86)
+		(at 43.18 62.23)
+		(size 16.51 12.446)
 		(exclude_from_sim no)
 		(in_bom yes)
@@
 		)
 		(property "Sheetname" "Trailer_Tail"
-			(at 43.18 79.5524 0)
+			(at 43.18 61.7724 0)
 			(show_name no)
 			(do_not_autoplace no)
@@
 		)
 		(property "Sheetfile" "Trailer_Tail.kicad_sch"
-			(at 43.18 103.2514 0)
+			(at 43.18 75.0574 0)
 			(show_name no)
 			(do_not_autoplace no)
@@
 		)
 		(pin "Trail_Tail" input
-			(at 59.69 87.63 0)
+			(at 59.69 69.85 0)
 			(effects
 				(font
@@
 		)
 		(pin "Ouvert_Tail_Trailer" input
-			(at 43.18 90.17 180)
+			(at 43.18 72.39 180)
 			(effects
 				(font
@@
 		)
 		(pin "Court_Tail_Trailer" input
-			(at 43.18 85.09 180)
+			(at 43.18 67.31 180)
 			(effects
 				(font
@@
 		)
 		(pin "Btn_Tail_Etat" input
-			(at 43.18 82.55 180)
+			(at 43.18 64.77 180)
 			(effects
 				(font
@@
 	)
 	(sheet
-		(at 43.18 48.26)
-		(size 16.51 24.13)
+		(at 43.18 45.72)
+		(size 16.51 9.652)
 		(exclude_from_sim no)
 		(in_bom yes)
@@
 		)
 		(property "Sheetname" "Vehicule_Tail"
-			(at 43.18 47.8024 0)
+			(at 43.18 45.2624 0)
 			(show_name no)
 			(do_not_autoplace no)
@@
 		)
 		(property "Sheetfile" "Vehicule_Tail.kicad_sch"
-			(at 43.18 72.7714 0)
+			(at 43.18 55.7534 0)
 			(show_name no)
 			(do_not_autoplace no)
@@
 		)
 		(pin "Ouvert_Tail_Vehic" input
+			(at 59.69 48.26 0)
+			(effects
+				(font
+					(size 0.762 0.762)
+				)
+				(justify right)
+			)
+		)
+		(pin "Court_Tail_Vehic" input
 			(at 59.69 50.8 0)
 			(effects
@@
 			)
 		)
-		(pin "Court_Tail_Vehic" input
+		(pin "Veh_Tail" input
 			(at 59.69 53.34 0)
 			(effects
 				(font
-					(size 0.762 0.762)
-				)
-				(justify right)
-			)
-		)
-		(pin "Veh_Tail" input
-			(at 59.69 55.88 0)
-			(effects
-				(font
-					(size 0.762 0.762)
-				)
-				(justify right)
-			)
-		)
-		(pin "Injection_Tail_Fault" input
-			(at 59.69 60.325 0)
-			(effects
-				(font
