File: TrailerDiagnosticSystem.kicad_sch (KiCad schematic)
At the start: 2 parts, among them J3 Conn_01x10, J4 Conn_01x10

Commit message: Add files via upload
Parts:
- removed J3, J4: Conn_01x10, symbol Connector_Generic:Conn_01x10
- added BMS3s1: (no value), symbol TrailerDiagSymols:BMS_3S
- added BT1, BT2, BT3: Battery_Cell, symbol Device:Battery_Cell
Connections:
- new net: BMS3s1.C2, BT2.2 (-), BT3.1 (+)
- new net: BMS3s1.B-, BT3.2 (-)
- new net: BMS3s1.B+, BT1.1 (+)
- new net: BMS3s1.C1, BT1.2 (-), BT2.1 (+)
- new net Batt_Interne_GND: BMS3s1.P-
- new net Batt_Interne_Pos: BMS3s1.P+
- no-connect marks 4 -> 0
Other:
- removed sheet Alimentation
- removed sheet Canal_Brake
- removed sheet Canal_Left
- removed sheet Canal_Tail
- removed sheet Mode_Coherence
- note added: "BMS 3S"

Commit message: Add files via upload
Parts:
- removed BMS3s1: (no value), symbol TrailerDiagSymols:BMS_3S
- removed BT1, BT2, BT3: Battery_Cell, symbol Device:Battery_Cell
- added J3, J4: Conn_01x10, symbol Connector_Generic:Conn_01x10
Connections:
- new net Detect_Trailer: J4.8 (Pin_8)
- new net Detect_Vehicule: J3.8 (Pin_8)
- new net GND: J3.1 (Pin_1), J4.1 (Pin_1)
- new net Trail_Aux: J4.7 (Pin_7)
- new net Trail_Backup: J4.6 (Pin_6)
- new net Trail_Brake: J4.3 (Pin_3)
- new net Trail_Left: J4.4 (Pin_4)
- new net Trail_Right: J4.5 (Pin_5)
- new net Trail_Tail: J4.2 (Pin_2)
- new net Veh_Aux: J3.7 (Pin_7)
- new net Veh_Backup: J3.6 (Pin_6)
- new net Veh_Brake: J3.3 (Pin_3)
- new net Veh_Left: J3.4 (Pin_4)
- new net Veh_Right: J3.5 (Pin_5)
- new net Veh_Tail: J3.2 (Pin_2)
- no-connect marks 0 -> 4
Other:
- added sheet Alimentation (Alimentation.kicad_sch)
- added sheet Canal_Aux (Canal_Aux.kicad_sch)
- added sheet Canal_Backup (Canal_Backup.kicad_sch)
- added sheet Canal_Brake (Canal_Brake.kicad_sch)
- added sheet Canal_Left (Canal_Left.kicad_sch)
- added sheet Canal_Right (Canal_Right.kicad_sch)
- added sheet Canal_Tail (Canal_Tail.kicad_sch)
- added sheet Mode_Coherence (mode_coherence.kicad_sch)
- note removed: "BMS 3S"

Commit message: Add files via upload
Connections:
- net Masse_Sense_Veh: now reaches J3.9 (Pin_9)
- net Masse_Sense_Trail: now reaches J4.9 (Pin_9)
- no-connect marks 4 -> 2
Other:
- added sheet Detection_De_Masse (MassDetection.kicad_sch)
- moved on the sheet: J3, J4

Commit message: Add files via upload
Other:
- added sheet Alarmes_Buzzer (Alarmes_Buzzer_sch.kicad_sch)
Changed lines of the file:
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@@
+	)
+	(sheet
+		(at 30.48 163.83)
+		(size 19.05 6.35)
+		(exclude_from_sim no)
+		(in_bom yes)
+		(on_board yes)
+		(dnp no)
+		(fields_autoplaced yes)
+		(stroke
+			(width 0.1524)
+			(type solid)
+		)
+		(fill
+			(color 0 0 0 0)
+		)
+		(property "Sheetname" "Alarmes_Buzzer"
+			(at 30.48 163.1184 0)
+			(show_name no)
+			(do_not_autoplace no)
+			(effects
+				(font
+					(size 1.27 1.27)
+				)
+				(justify left bottom)
+			)
+		)
+		(property "Sheetfile" "Alarmes_Buzzer_sch.kicad_sch"
+			(at 30.48 170.7646 0)
+			(show_name no)
+			(do_not_autoplace no)
+			(effects
+				(font
+					(size 1.27 1.27)
+				)
+				(justify left top)
+			)
+		)
+		(instances
+			(project "TrailerDiagnosticSystem"
+				(path "/d4e407a7-3e32-4226-ae57-831ecdb3edf4"
+					(page "29")
+				)
+			)
+		)
 	)
 	(sheet

Commit message: Add files via upload
Other:
- sheet Alarmes_Buzzer ports: added Alerte_Incoherence, Buzzer_Trigger, Court_Bus_Fault, Injection_Aux_Fault, Injection_Backup_Fault, Injection_Brake_Fault, Injection_Left_Fault, Injection_Right_Fault, Injection_Tail_Fault, Masse_Fault, Surtension_Fault; removed none
- sheet Alimentation ports: added Buzzer_Trigger, Court_Bus_Fault, Surtension_Fault; removed none

Commit message: Add files via upload
Other:
- sheet Detection_De_Masse ports: added Masse_Fault; removed none

Commit message: Add files via upload
Other:
- sheet Canal_Aux ports: added Injection_Aux_Fault; removed none
- sheet Canal_Backup ports: added Injection_Backup_Fault; removed none
- sheet Canal_Brake ports: added Injection_Brake_Fault; removed none
- sheet Canal_Left ports: added Injection_Left_Fault; removed none
- sheet Canal_Right ports: added Injection_Right_Fault; removed none
- sheet Canal_Tail ports: added Injection_Tail_Fault; removed none

Commit message: Add files via upload
Other:
- sheet Alarmes_Buzzer renamed Alertes
- sheet Alertes: file Alarmes_Buzzer_sch.kicad_sch -> Alertes.kicad_sch
- sheet Alertes ports: added none; removed Alerte_Incoherence, Buzzer_Trigger, Court_Bus_Fault, Injection_Aux_Fault, Injection_Backup_Fault, Injection_Brake_Fault, Injection_Left_Fault, Injection_Right_Fault, Injection_Tail_Fault, Masse_Fault, Surtension_Fault
- sheet Alimentation ports: added none; removed Buzzer_Trigger, Court_Bus_Fault, Surtension_Fault
- sheet Canal_Aux ports: added none; removed Injection_Aux_Fault
- sheet Canal_Backup ports: added none; removed Injection_Backup_Fault
- sheet Canal_Brake ports: added none; removed Injection_Brake_Fault
- sheet Canal_Left ports: added none; removed Injection_Left_Fault
- sheet Canal_Right ports: added none; removed Injection_Right_Fault
- sheet Canal_Tail ports: added none; removed Injection_Tail_Fault
- sheet Detection_De_Masse ports: added none; removed Masse_Fault
