File: TrailerDiagnosticSystem.kicad_sch (KiCad schematic)
At the start: 10 parts, among them J3 Conn_01x10, J4 Conn_01x10, SW9 CKS1503

Commit message: Add files via upload
Parts:
- added R252: 1k, Resistor_THT:R_Axial_DIN0309_L9.0mm_D3.2mm_P12.70mm_Horizontal, symbol PCM_SL_Resistors:Resistor
Connections:
- net Trail_Aux: now also R252.2
- net at SW9.8: now also R252.1
- no-connect marks 7 -> 6
Changed lines of the file:
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@@
 		(at 101.6 107.95)
 	)
-	(no_connect
-		(at 171.45 83.82)
-	)
 	(wire
 		(pts
@@
 	(wire
 		(pts
+			(xy 171.45 83.82) (xy 176.53 83.82)
+		)
+		(stroke
+			(width 0)
+			(type default)
+		)
+	)
+	(wire
+		(pts
 			(xy 101.6 95.25) (xy 106.68 95.25)
 		)
@@
 		(pts
 			(xy 49.53 94.615) (xy 52.07 94.615)
+		)
+		(stroke
+			(width 0)
+			(type default)
+		)
+	)
+	(wire
+		(pts
+			(xy 184.15 83.82) (xy 187.96 83.82)
 		)
 		(stroke
@@
 		)
 	)
+	(label "Trail_Aux"
+		(at 187.96 83.82 0)
+		(effects
+			(font
+				(size 1.27 1.27)
+			)
+			(justify left bottom)
+		)
+	)
 	(label "Trail_Backup"
 		(at 53.34 105.41 0)
@@
 		)
 	)
+	(symbol
+		(lib_id "PCM_SL_Resistors:Resistor")
+		(at 180.34 83.82 0)
+		(unit 1)
+		(body_style 1)
+		(exclude_from_sim no)
+		(in_bom yes)
+		(on_board yes)
+		(in_pos_files yes)
+		(dnp no)
+		(fields_autoplaced yes)
+		(property "Reference" "R252"
+			(at 180.34 77.47 0)
+			(hide yes)
+			(show_name no)
+			(do_not_autoplace no)
+			(effects
+				(font
+					(size 1.27 1.27)
+				)
+			)
+		)
+		(property "Value" "1k"
+			(at 180.34 80.01 0)
+			(hide yes)
+			(show_name no)
+			(do_not_autoplace no)
+			(effects
+				(font
+					(size 1.27 1.27)
+				)
+			)
+		)
+		(property "Footprint" "Resistor_THT:R_Axial_DIN0309_L9.0mm_D3.2mm_P12.70mm_Horizontal"
+			(at 181.229 88.138 0)
+			(hide yes)
+			(show_name no)
+			(do_not_autoplace no)
+			(effects
+				(font
+					(size 1.27 1.27)
+				)
+			)
+		)
+		(property "Datasheet" ""
+			(at 180.848 83.82 0)
+			(hide yes)
+			(show_name no)
+			(do_not_autoplace no)
+			(effects
+				(font
+					(size 1.27 1.27)
+				)
+			)
+		)
+		(property "Description" "1/2W Resistor"
+			(at 180.34 83.82 0)
+			(hide yes)
+			(show_name no)
+			(do_not_autoplace no)
+			(effects
+				(font
+					(size 1.27 1.27)
+				)
+			)
+		)
+		(pin "1"
+		)
+		(pin "2"
+		)
+		(instances
+			(project "TrailerDiagnosticSystem"
+				(path "/d4e407a7-3e32-4226-ae57-831ecdb3edf4"
+					(reference "R252")
+					(unit 1)
+				)
+			)
+		)
+	)

Commit message: Add files via upload
Parts:
- removed R235, R236, R237, R238, R240, R241: 1K, Resistor_THT:R_Axial_DIN0309_L9.0mm_D3.2mm_P12.70mm_Horizontal, symbol PCM_SL_Resistors:Resistor
- removed R239, R252: 1k, Resistor_THT:R_Axial_DIN0309_L9.0mm_D3.2mm_P12.70mm_Horizontal, symbol PCM_SL_Resistors:Resistor
- removed SW9: CKS1503, symbol Switch:SW_Rotary_1x12
Connections:
- no-connect marks 6 -> 2
Other:
- sheet Alarmes_Buzzer renamed Alertes
- sheet Alertes: file Alarmes_Buzzer_sch.kicad_sch -> Alertes.kicad_sch
- sheet Alertes ports: added none; removed Alerte_Incoherence, Buzzer_Trigger, Court_Bus_Fault, Injection_Aux_Fault, Injection_Backup_Fault, Injection_Brake_Fault, Injection_Left_Fault, Injection_Right_Fault, Injection_Tail_Fault, Masse_Fault, Surtension_Fault
- sheet Alimentation ports: added none; removed Buzzer_Trigger, Court_Bus_Fault, Surtension_Fault, VM_Mesure
- sheet Canal_Aux ports: added none; removed Injection_Aux_Fault
- sheet Canal_Backup ports: added none; removed Injection_Backup_Fault
- sheet Canal_Brake ports: added none; removed Injection_Brake_Fault
- sheet Canal_Left ports: added none; removed Injection_Left_Fault
- sheet Canal_Right ports: added none; removed Injection_Right_Fault
- sheet Canal_Tail ports: added none; removed Injection_Tail_Fault
- sheet Detection_De_Masse ports: added none; removed Masse_Fault

Commit message: Add files via upload
Parts:
- added R235, R236, R237, R238, R240, R241: 1K, Resistor_THT:R_Axial_DIN0309_L9.0mm_D3.2mm_P12.70mm_Horizontal, symbol PCM_SL_Resistors:Resistor
- added R239, R252: 1k, Resistor_THT:R_Axial_DIN0309_L9.0mm_D3.2mm_P12.70mm_Horizontal, symbol PCM_SL_Resistors:Resistor
- added SW9: CKS1503, symbol Switch:SW_Rotary_1x12
Connections:
- net Trail_Aux: now also R252.2
- net V12_Rail: now also R235.2
- net Veh_Aux: now also R239.2
- net Veh_Backup: now also R240.2
- net Veh_Brake: now also R241.2
- net Veh_Left: now also R237.2
- net Veh_Right: now also R238.2
- net Veh_Tail: now also R236.2
- new net: R252.1, SW9.8
- new net: R235.1, SW9.2
- new net: R240.1, SW9.6
- new net: R241.1, SW9.1
- new net: R236.1, SW9.3
- new net: R237.1, SW9.4
- new net: R238.1, SW9.5
- new net: R239.1, SW9.7
- new net VM_Mesure: SW9.13
- no-connect marks 2 -> 6
Other:
- sheet Alertes renamed Alarmes_Buzzer
- sheet Alarmes_Buzzer: file Alertes.kicad_sch -> Alarmes_Buzzer_sch.kicad_sch
- sheet Alarmes_Buzzer ports: added Alerte_Incoherence, Buzzer_Trigger, Court_Bus_Fault, Injection_Aux_Fault, Injection_Backup_Fault, Injection_Brake_Fault, Injection_Left_Fault, Injection_Right_Fault, Injection_Tail_Fault, Masse_Fault, Surtension_Fault; removed none
- sheet Alimentation ports: added Buzzer_Trigger, Court_Bus_Fault, Surtension_Fault, VM_Mesure; removed none
- sheet Canal_Aux ports: added Injection_Aux_Fault; removed none
- sheet Canal_Backup ports: added Injection_Backup_Fault; removed none
- sheet Canal_Brake ports: added Injection_Brake_Fault; removed none
- sheet Canal_Left ports: added Injection_Left_Fault; removed none
- sheet Canal_Right ports: added Injection_Right_Fault; removed none
- sheet Canal_Tail ports: added Injection_Tail_Fault; removed none
- sheet Detection_De_Masse ports: added Masse_Fault; removed none

Commit message: Add files via upload
Parts:
- added R308, R309: 1k, Resistor_THT:R_Axial_DIN0207_L6.3mm_D2.5mm_P10.16mm_Horizontal, symbol PCM_SL_Resistors:1k
Changed lines of the file:
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@@
 		(effects
 			(font
-				(size 1.27 1.27)
+				(size 1.016 1.016)
 			)
 			(justify left bottom)
@@
 		(effects
 			(font
-				(size 1.27 1.27)
+				(size 1.016 1.016)
 			)
 			(justify left bottom)
@@
 		(effects
 			(font
-				(size 1.27 1.27)
+				(size 1.016 1.016)
 			)
 			(justify left bottom)
@@
 	)
 	(symbol
+		(lib_id "PCM_SL_Resistors:1k")
+		(at 195.58 93.98 0)
+		(unit 1)
+		(body_style 1)
+		(exclude_from_sim no)
+		(in_bom yes)
+		(on_board yes)
+		(in_pos_files yes)
+		(dnp no)
+		(property "Reference" "R309"
+			(at 195.58 88.9 0)
+			(show_name no)
+			(do_not_autoplace no)
+			(effects
+				(font
+					(size 1.27 1.27)
+				)
+			)
+		)
+		(property "Value" "1k"
+			(at 195.58 91.44 0)
+			(show_name no)
+			(do_not_autoplace no)
+			(effects
+				(font
+					(size 1.27 1.27)
+				)
+			)
+		)
+		(property "Footprint" "Resistor_THT:R_Axial_DIN0207_L6.3mm_D2.5mm_P10.16mm_Horizontal"
+			(at 196.469 98.298 0)
+			(hide yes)
+			(show_name no)
+			(do_not_autoplace no)
+			(effects
+				(font
+					(size 1.27 1.27)
+				)
+			)
+		)
+		(property "Datasheet" ""
+			(at 196.088 93.98 0)
+			(hide yes)
+			(show_name no)
+			(do_not_autoplace no)
+			(effects
+				(font
+					(size 1.27 1.27)
+				)
+			)
+		)
+		(property "Description" "1kΩ, 1/4W Resistor"
+			(at 195.58 93.98 0)
+			(hide yes)
+			(show_name no)
+			(do_not_autoplace no)
+			(effects
+				(font
+					(size 1.27 1.27)
+				)
+			)
+		)
+		(pin "1"
+		)
+		(pin "2"
+		)
+		(instances
+			(project "TrailerDiagnosticSystem"
+				(path "/d4e407a7-3e32-4226-ae57-831ecdb3edf4"
+					(reference "R309")
+					(unit 1)
+				)
+			)
+		)
+	)
+	(symbol
 		(lib_id "power:GND")
 		(at 96.52 85.09 270)
@@
 					(unit 1)
 				)
+			)
+		)
+	)
+	(symbol
+		(lib_id "PCM_SL_Resistors:1k")
+		(at 186.69 95.25 0)
+		(unit 1)
+		(body_style 1)
+		(exclude_from_sim no)
+		(in_bom yes)
+		(on_board yes)
+		(in_pos_files yes)
+		(dnp no)
+		(property "Reference" "R308"
+			(at 186.69 90.17 0)
+			(show_name no)
+			(do_not_autoplace no)
+			(effects
+				(font
+					(size 1.27 1.27)
+				)
+			)
+		)
+		(property "Value" "1k"
+			(at 186.69 92.71 0)
+			(show_name no)
+			(do_not_autoplace no)
+			(effects
+				(font
+					(size 1.27 1.27)
+				)
+			)
+		)
+		(property "Footprint" "Resistor_THT:R_Axial_DIN0207_L6.3mm_D2.5mm_P10.16mm_Horizontal"
+			(at 187.579 99.568 0)
+			(hide yes)
+			(show_name no)
+			(do_not_autoplace no)
+			(effects
+				(font
+					(size 1.27 1.27)
+				)
+			)
+		)
+		(property "Datasheet" ""
+			(at 187.198 95.25 0)
+			(hide yes)
+			(show_name no)
+			(do_not_autoplace no)
+			(effects
+				(font
+					(size 1.27 1.27)
+				)
+			)
+		)
+		(property "Description" "1kΩ, 1/4W Resistor"
+			(at 186.69 95.25 0)
+			(hide yes)
+			(show_name no)
+			(do_not_autoplace no)
+			(effects
+				(font
+					(size 1.27 1.27)
+				)
+			)
+		)
+		(pin "1"
+		)
+		(pin "2"
+		)
+		(instances
+			(project "TrailerDiagnosticSystem"
+				(path "/d4e407a7-3e32-4226-ae57-831ecdb3edf4"
+					(reference "R308")
+					(unit 1)
+				)

Commit message: Add files via upload
Connections:
- net at R309.1: now also SW9.10
- net Pince_Trail: now reaches R309.2
- net at SW9.9: now also R308.1
- net Pince_Veh: now reaches R308.2
- no-connect marks 6 -> 4
Other:
- sheet Detection_De_Masse ports: added Pince_Trail, Pince_Veh; removed Masse_Sense_Trail, Masse_Sense_Veh
Changed lines of the file:
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@@
 	(paper "B")
 	(no_connect
-		(at 171.45 86.36)
-	)
-	(no_connect
 		(at 171.45 91.44)
 	)
 	(no_connect
-		(at 171.45 88.9)
-	)
-	(no_connect
 		(at 100.33 72.39)
 	)
@@
 	(wire
 		(pts
-			(xy 49.53 132.715) (xy 52.07 132.715)
+			(xy 49.53 133.35) (xy 52.07 133.35)
 		)
 		(stroke
@@
 	(wire
 		(pts
+			(xy 171.45 88.9) (xy 176.53 88.9)
+		)
+		(stroke
+			(width 0)
+			(type default)
+		)
+	)
+	(wire
+		(pts
 			(xy 49.53 66.04) (xy 54.61 66.04)
 		)
@@
 	(wire
 		(pts
-			(xy 49.53 74.295) (xy 54.61 74.295)
+			(xy 49.53 74.93) (xy 54.61 74.93)
 		)
 		(stroke
@@
 	(wire
 		(pts
+			(xy 184.15 86.36) (xy 187.96 86.36)
+		)
+		(stroke
+			(width 0)
+			(type default)
+		)
+	)
+	(wire
+		(pts
 			(xy 49.53 40.64) (xy 54.61 40.64)
 		)
@@
 	(wire
 		(pts
-			(xy 49.53 109.855) (xy 53.34 109.855)
+			(xy 49.53 110.49) (xy 53.34 110.49)
 		)
 		(stroke
@@
 	(wire
 		(pts
-			(xy 49.53 76.835) (xy 54.61 76.835)
+			(xy 49.53 77.47) (xy 54.61 77.47)
 		)
 		(stroke
@@
 	(wire
 		(pts
-			(xy 62.23 154.305) (xy 67.31 154.305)
+			(xy 62.23 154.94) (xy 67.31 154.94)
+		)
+		(stroke
+			(width 0)
+			(type default)
+		)
+	)
+	(wire
+		(pts
+			(xy 171.45 86.36) (xy 176.53 86.36)
 		)
 		(stroke
@@
 	(wire
 		(pts
-			(xy 62.23 150.495) (xy 67.31 150.495)
+			(xy 62.23 151.13) (xy 67.31 151.13)
 		)
 		(stroke
@@
 	(wire
 		(pts
-			(xy 49.53 94.615) (xy 52.07 94.615)
+			(xy 49.53 95.25) (xy 52.07 95.25)
 		)
 		(stroke
@@
 	(wire
 		(pts
+			(xy 184.15 88.9) (xy 187.96 88.9)
+		)
+		(stroke
+			(width 0)
+			(type default)
+		)
+	)
+	(wire
+		(pts
 			(xy 184.15 73.66) (xy 187.96 73.66)
 		)
@@
 	(wire
 		(pts
-			(xy 49.53 79.375) (xy 54.61 79.375)
+			(xy 49.53 80.01) (xy 54.61 80.01)
 		)
 		(stroke
@@
 		)
 	)
+	(label "Pince_Veh"
+		(at 187.96 86.36 0)
+		(effects
+			(font
+				(size 1.27 1.27)
+			)
+			(justify left bottom)
+		)
+	)
 	(label "Veh_Left"
 		(at 100.33 57.15 180)
@@
 	)
 	(label "Veh_Left"
-		(at 54.61 74.295 0)
+		(at 54.61 74.93 0)
 		(effects
 			(font
@@
 		)
 	)
-	(label "Masse_Sense_Trail"
-		(at 67.31 154.305 0)
+	(label "Pince_Trail"
+		(at 67.31 154.94 0)
 		(effects
 			(font
@@
 		)
 	)
-	(label "Masse_Sense_Veh"
-		(at 67.31 150.495 0)
+	(label "Pince_Veh"
+		(at 67.31 151.13 0)
 		(effects
 			(font
@@
 	)
 	(label "Injection_Left_Fault"
-		(at 54.61 79.375 0)
+		(at 54.61 80.01 0)
 		(effects
 			(font
@@
 	)
 	(label "Trail_Left"
-		(at 54.61 76.835 0)
+		(at 54.61 77.47 0)
 		(effects
 			(font
@@
 		)
 	)
+	(label "Pince_Trail"
+		(at 187.96 88.9 0)
+		(effects
+			(font
+				(size 1.27 1.27)
+			)
+			(justify left bottom)
+		)
+	)
 	(label "Injection_Tail_Fault"
 		(at 67.31 165.1 0)
@@
 	)
 	(label "Injection_Right_Fault"
-		(at 52.07 94.615 0)
+		(at 52.07 95.25 0)
 		(effects
 			(font
@@
 	)
 	(label "Injection_Backup_Fault"
-		(at 53.34 109.855 0)
+		(at 53.34 110.49 0)
 		(effects
 			(font
@@
 	)
 	(label "Injection_Brake_Fault"
-		(at 52.07 132.715 0)
+		(at 52.07 133.35 0)
 		(effects
 			(font
@@
 	(symbol
 		(lib_id "PCM_SL_Resistors:1k")
-		(at 195.58 93.98 0)
+		(at 180.34 88.9 0)
 		(unit 1)
 		(body_style 1)
@@
 		(dnp no)
 		(property "Reference" "R309"
-			(at 195.58 88.9 0)
+			(at 180.34 83.82 0)
+			(hide yes)
 			(show_name no)
 			(do_not_autoplace no)
@@
 		)
 		(property "Value" "1k"
-			(at 195.58 91.44 0)
+			(at 180.34 86.36 0)
+			(hide yes)
 			(show_name no)
 			(do_not_autoplace no)
@@
 		)
 		(property "Footprint" "Resistor_THT:R_Axial_DIN0207_L6.3mm_D2.5mm_P10.16mm_Horizontal"
-			(at 196.469 98.298 0)
+			(at 181.229 93.218 0)
 			(hide yes)
 			(show_name no)
@@
 		)
 		(property "Datasheet" ""
-			(at 196.088 93.98 0)
+			(at 180.848 88.9 0)
 			(hide yes)
 			(show_name no)
@@
 		)
 		(property "Description" "1kΩ, 1/4W Resistor"
-			(at 195.58 93.98 0)
+			(at 180.34 88.9 0)
 			(hide yes)
 			(show_name no)
@@
 	(symbol
 		(lib_id "PCM_SL_Resistors:1k")
-		(at 186.69 95.25 0)
+		(at 180.34 86.36 0)
 		(unit 1)
 		(body_style 1)
@@
 		(dnp no)
 		(property "Reference" "R308"
-			(at 186.69 90.17 0)
+			(at 180.34 81.28 0)
+			(hide yes)
 			(show_name no)
 			(do_not_autoplace no)
@@
 		)
 		(property "Value" "1k"
-			(at 186.69 92.71 0)
+			(at 180.34 83.82 0)
+			(hide yes)
 			(show_name no)
 			(do_not_autoplace no)
@@
 		)
 		(property "Footprint" "Resistor_THT:R_Axial_DIN0207_L6.3mm_D2.5mm_P10.16mm_Horizontal"
-			(at 187.579 99.568 0)
+			(at 181.229 90.678 0)
 			(hide yes)
 			(show_name no)
@@
 		)
 		(property "Datasheet" ""
-			(at 187.198 95.25 0)
+			(at 180.848 86.36 0)
 			(hide yes)
 			(show_name no)
@@
 		)
 		(property "Description" "1kΩ, 1/4W Resistor"
-			(at 186.69 95.25 0)
+			(at 180.34 86.36 0)
 			(hide yes)
 			(show_name no)
@@
 	)
 	(sheet
-		(at 30.48 130.175)
-		(size 19.05 10.795)
+		(at 30.48 130.81)
+		(size 19.05 10.16)
 		(exclude_from_sim no)
 		(in_bom yes)
@@
 		)
 		(property "Sheetname" "Canal_Brake"
-			(at 30.48 129.7174 0)
+			(at 30.48 130.3524 0)
 			(show_name no)
 			(do_not_autoplace no)
@@
 		)
 		(property "Sheetfile" "Canal_Brake.kicad_sch"
-			(at 30.48 141.3514 0)
+			(at 30.48 141.9864 0)
 			(show_name no)
 			(do_not_autoplace no)
@@
 		)
 		(pin "Injection_Brake_Fault" input
-			(at 49.53 132.715 0)
+			(at 49.53 133.35 0)
 			(effects
 				(font
@@
 	(sheet
 		(at 30.48 144.78)
-		(size 31.75 12.065)
+		(size 31.75 12.7)
 		(exclude_from_sim no)
 		(in_bom yes)
@@
 			)
 		)
-		(pin "Masse_Sense_Veh" input
-			(at 62.23 150.495 0)
+		(pin "Masse_Fault" input
+			(at 62.23 146.05 0)
 			(effects
 				(font
@@
 			)
 		)
-		(pin "Masse_Sense_Trail" input
-			(at 62.23 154.305 0)
+		(pin "Pince_Trail" input
+			(at 62.23 154.94 0)
 			(effects
 				(font
@@
 			)
 		)
-		(pin "Masse_Fault" input
-			(at 62.23 146.05 0)
+		(pin "Pince_Veh" input
+			(at 62.23 151.13 0)
 			(effects
 				(font
@@
 		)
 		(pin "Injection_Right_Fault" input
-			(at 49.53 94.615 0)
+			(at 49.53 95.25 0)
 			(effects
 				(font
@@
 	(sheet
 		(at 30.48 57.15)
-		(size 19.05 10.795)
+		(size 19.05 11.43)
 		(exclude_from_sim no)
 		(in_bom yes)
@@
 		)
 		(pin "Injection_Backup_Fault" input
-			(at 49.53 109.855 0)
+			(at 49.53 110.49 0)
 			(effects
 				(font
@@
 		)
 		(pin "Trail_Left" input
-			(at 49.53 76.835 0)
+			(at 49.53 77.47 0)
 			(effects
 				(font
@@
 		)
 		(pin "Veh_Left" input
-			(at 49.53 74.295 0)
+			(at 49.53 74.93 0)
 			(effects
 				(font
@@
 		)
 		(pin "Injection_Left_Fault" input
-			(at 49.53 79.375 0)
+			(at 49.53 80.01 0)
 			(effects
 				(font
@@
 	)
 	(sheet
-		(at 30.48 33.274)
-		(size 19.05 18.796)
+		(at 30.48 33.02)
+		(size 19.05 19.05)
 		(exclude_from_sim no)
 		(in_bom yes)
@@
 		)
 		(property "Sheetname" "Mode_Coherence"
-			(at 30.48 32.8164 0)
+			(at 30.48 32.5624 0)
 			(show_name yes)
 			(do_not_autoplace no)
@@
 		)
 		(property "Sheetfile" "mode_coherence.kicad_sch"
-			(at 30.48 52.4514 0)
+			(at 30.48 52.1974 0)
 			(show_name yes)
 			(do_not_autoplace no)

Commit message: Add files via upload
Connections:
- net Masse_Sense_Trail is gone; now on net Pince_Trail: J4.9 (Pin_9)
- net Masse_Sense_Veh is gone; now on net Pince_Veh: J3.9 (Pin_9)
Changed lines of the file:
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@@
 		)
 	)
-	(label "Masse_Sense_Veh"
+	(label "Pince_Veh"
 		(at 100.33 69.85 180)
 		(effects
@@
 		)
 	)
-	(label "Masse_Sense_Trail"
+	(label "Pince_Trail"
 		(at 101.6 105.41 180)
 		(effects

Commit message: Add files via upload
Parts:
- removed R235: 1K, Resistor_THT:R_Axial_DIN0309_L9.0mm_D3.2mm_P12.70mm_Horizontal, symbol PCM_SL_Resistors:Resistor
Other:
- sheet Alarmes_Buzzer ports: added none; removed Buzzer_Trigger
- sheet Alimentation ports: added none; removed Buzzer_Trigger
Changed lines of the file:
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@@
-	(wire
-		(pts
-			(xy 62.23 203.2) (xy 67.31 203.2)
-		)
-		(stroke
-			(width 0)
-			(type default)
-		)
-	)
 	(wire
 		(pts
@@
 	(wire
 		(pts
-			(xy 184.15 66.04) (xy 187.96 66.04)
-		)
-		(stroke
-			(width 0)
-			(type default)
-		)
-	)
-	(wire
-		(pts
 			(xy 106.68 97.79) (xy 101.6 97.79)
 		)
@@
 		(pts
 			(xy 138.43 78.74) (xy 140.97 78.74)
-		)
-		(stroke
-			(width 0)
-			(type default)
-		)
-	)
-	(wire
-		(pts
-			(xy 49.53 19.05) (xy 54.61 19.05)
 		)
 		(stroke
@@
 		)
 	)
-	(label "Buzzer_Trigger"
-		(at 67.31 203.2 0)
-		(effects
-			(font
-				(size 1.27 1.27)
-			)
-			(justify left bottom)
-		)
-	)
 	(label "Surtension_Fault"
 		(at 67.31 187.96 0)
@@
 		)
 	)
-	(label "V12_Rail"
-		(at 187.96 66.04 0)
-		(effects
-			(font
-				(size 1.016 1.016)
-			)
-			(justify left bottom)
-		)
-	)
 	(label "Veh_Right"
 		(at 100.33 59.69 180)
@@
 			)
 			(justify right bottom)
-		)
-	)
-	(label "Buzzer_Trigger"
-		(at 54.61 19.05 0)
-		(effects
-			(font
-				(size 1.27 1.27)
-			)
-			(justify left bottom)
 		)
 	)
@@
 	(symbol
 		(lib_id "PCM_SL_Resistors:Resistor")
-		(at 180.34 66.04 0)
-		(unit 1)
-		(body_style 1)
-		(exclude_from_sim no)
-		(in_bom yes)
-		(on_board yes)
-		(in_pos_files yes)
-		(dnp no)
-		(fields_autoplaced yes)
-		(property "Reference" "R235"
-			(at 180.34 59.69 0)
-			(hide yes)
-			(show_name no)
-			(do_not_autoplace no)
-			(effects
-				(font
-					(size 1.27 1.27)
-				)
-			)
-		)
-		(property "Value" "1K"
-			(at 180.34 62.23 0)
-			(hide yes)
-			(show_name no)
-			(do_not_autoplace no)
-			(effects
-				(font
-					(size 1.27 1.27)
-				)
-			)
-		)
-		(property "Footprint" "Resistor_THT:R_Axial_DIN0309_L9.0mm_D3.2mm_P12.70mm_Horizontal"
-			(at 181.229 70.358 0)
-			(hide yes)
-			(show_name no)
-			(do_not_autoplace no)
-			(effects
-				(font
-					(size 1.27 1.27)
-				)
-			)
-		)
-		(property "Datasheet" ""
-			(at 180.848 66.04 0)
-			(hide yes)
-			(show_name no)
-			(do_not_autoplace no)
-			(effects
-				(font
-					(size 1.27 1.27)
-				)
-			)
-		)
-		(property "Description" "1/2W Resistor"
-			(at 180.34 66.04 0)
-			(hide yes)
-			(show_name no)
-			(do_not_autoplace no)
-			(effects
-				(font
-					(size 1.27 1.27)
-				)
-			)
-		)
-		(pin "1"
-		)
-		(pin "2"
-		)
-		(instances
-			(project "TrailerDiagnosticSystem"
-				(path "/d4e407a7-3e32-4226-ae57-831ecdb3edf4"
-					(reference "R235")
-					(unit 1)
-				)
-			)
-		)
-	)
-	(symbol
-		(lib_id "PCM_SL_Resistors:Resistor")
 		(at 180.34 76.2 0)
 		(unit 1)
@@
 			)
 		)
-		(pin "Buzzer_Trigger" input
-			(at 49.53 19.05 0)
-			(effects
-				(font
-					(size 1.27 1.27)
-				)
-				(justify right)
-			)
-		)
 		(pin "Court_Bus_Fault" input
 			(at 49.53 24.13 0)
@@
 			(effects
 				(font
-					(size 1.27 1.27)
-				)
-				(justify right)
-			)
-		)
-		(pin "Buzzer_Trigger" input
-			(at 62.23 203.2 0)
-			(effects
-				(font

Commit message: Add files via upload
Other:
- sheet Alimentation ports: added V12_PostShunt; removed none
Changed lines of the file:
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@@
+	(wire
+		(pts
+			(xy 49.53 20.32) (xy 54.61 20.32)
+		)
+		(stroke
+			(width 0)
+			(type default)
+		)
+	)
 	(wire
 		(pts
@@
 	(wire
 		(pts
-			(xy 49.53 24.13) (xy 54.61 24.13)
+			(xy 49.53 25.4) (xy 54.61 25.4)
 		)
 		(stroke
@@
 	(wire
 		(pts
-			(xy 49.53 21.59) (xy 54.61 21.59)
+			(xy 49.53 22.86) (xy 54.61 22.86)
 		)
 		(stroke
@@
 	(wire
 		(pts
-			(xy 49.53 16.51) (xy 54.61 16.51)
+			(xy 49.53 17.78) (xy 54.61 17.78)
 		)
 		(stroke
@@
 	)
 	(label "V12_Rail"
-		(at 54.61 21.59 0)
+		(at 54.61 22.86 0)
 		(effects
 			(font
@@
 	)
 	(label "Surtension_Fault"
-		(at 54.61 16.51 0)
+		(at 54.61 17.78 0)
+		(effects
+			(font
+				(size 1.27 1.27)
+			)
+			(justify left bottom)
+		)
+	)
+	(label "V12_PostShunt"
+		(at 54.61 20.32 0)
 		(effects
 			(font
@@
 	)
 	(label "Court_Bus_Fault"
-		(at 54.61 24.13 0)
+		(at 54.61 25.4 0)
 		(effects
 			(font
@@
 	)
 	(sheet
-		(at 30.48 13.97)
-		(size 19.05 15.24)
+		(at 30.48 15.24)
+		(size 19.05 13.97)
 		(exclude_from_sim no)
 		(in_bom yes)
@@
 		)
 		(property "Sheetname" "Alimentation"
-			(at 30.48 13.5124 0)
+			(at 30.48 14.7824 0)
 			(show_name yes)
 			(do_not_autoplace no)
@@
 		)
 		(pin "V12_Rail" input
-			(at 49.53 21.59 0)
+			(at 49.53 22.86 0)
 			(effects
 				(font
@@
 		)
 		(pin "Surtension_Fault" input
-			(at 49.53 16.51 0)
+			(at 49.53 17.78 0)
 			(effects
 				(font
@@
 		)
 		(pin "Court_Bus_Fault" input
-			(at 49.53 24.13 0)
+			(at 49.53 25.4 0)
 			(effects
 				(font
@@
 				)
 				(justify right)
+			)
+		)
+		(pin "V12_PostShunt" input
+			(at 49.53 20.32 0)
+			(effects
+				(font
+					(size 1.27 1.27)
+					(italic yes)
+				)
+				(justify right)
