File: Alimentation.kicad_sch (KiCad schematic)
At the start: 33 parts, among them J2 Screw_Terminal_2_P3.50mm, P1 Conn_Plug_2P, Q1 IRLZ44N, Q55 2N3906, Q56 2N7000, Q57 2N7000, SW1 SW_DPDT_x2, U1 LM74610QDGKRQ1, U16 LM339, U6 LM7805CT

Commit message: Add files via upload
Connections:
- net GND: now also U16.7 (+)
- net V_Ref: now also R222.2, U16.6 (-)
- no-connect marks 5 -> 6
Other:
- moved on the sheet: R216

Commit message: Add files via upload
Connections:
- net GND: no longer U16.7 (+)
- net V_Ref: no longer R222.2, U16.6 (-)
- no-connect marks 6 -> 5
Other:
- moved on the sheet: R216

Commit message: Add files via upload
Parts:
- added D25: OSX10201-GYR1, OSX10201-GYR1:DIP760W45P254L2550H815Q20B, symbol OSX10201-GYR1.kicad_sym:OSX10201-GYR1
- added Q64: IRLZ44N, PCM_Package_TO_SOT_THT_AKL:TO-220-3_Vertical_GDS, symbol PCM_Transistor_MOSFET_AKL:IRLZ44N
- added Q65: 2N7000, PCM_Package_TO_SOT_THT_AKL:TO-92_Inline_Wide_SGD, symbol PCM_Transistor_MOSFET_AKL:2N7000
- added R230, R231: 4.7kΩ, Resistor_THT:R_Axial_DIN0207_L6.3mm_D2.5mm_P10.16mm_Horizontal, symbol PCM_SL_Resistors:4.7k
- added U17: LM3914N, Package_DIP:DIP-18_W7.62mm, symbol Driver_LED:LM3914N
Connections:
- net Court_Bus_Fault: now also R231.1
- net GND: now also U16.7 (+), Q65.1 (S)
- net V12_Rail: now also Q64.3 (S); no longer R221.2
- net V_Ref: now also R222.2, U16.6 (-), R230.2
- new net: Q64.1 (G), Q65.3 (D), R230.1
- new net: Q65.2 (G), R231.2
- new net V12_PostShunt: Q64.2 (D), R221.2
- no-connect marks 5 -> 6
Other:
- note added: "Coupure de V12_Rail sur court-circuit"
- moved on the sheet: R216

Commit message: Add files via upload
Parts:
- added C6: SR205E104MARAP1, SR205E104MARAP1:CAPRR254W50L508T317H508, symbol TrailerDiagSymbols:SR205E104MARAP1
- added R232: 18k, Resistor_THT:R_Axial_DIN0207_L6.3mm_D2.5mm_P10.16mm_Horizontal, symbol PCM_SL_Resistors:18k
- added R233: 10k, Resistor_THT:R_Axial_DIN0207_L6.3mm_D2.5mm_P10.16mm_Horizontal, symbol PCM_SL_Resistors:10k
- added R234: 68ohm, Resistor_THT:R_Axial_Power_L25.0mm_W9.0mm_P27.94mm, symbol PCM_SL_Devices:Resistor_5W
- added R36: 1.5k, Resistor_THT:R_Axial_DIN0207_L6.3mm_D2.5mm_P10.16mm_Horizontal, symbol PCM_SL_Resistors:1.5k
- added R53: 3.9k, Resistor_THT:R_Axial_DIN0207_L6.3mm_D2.5mm_P10.16mm_Horizontal, symbol PCM_SL_Resistors:3.9k
- added VR1: 3296W-1-102LF, 3296W-1-102LF:TRIM_3296W-1-102LF, symbol 3296-1-102lf:3296W-1-102LF
Connections:
- net Batt_Externe_Pos: no longer F1.1
- net Batt_Interne_Pos: now also R232.2
- net GND: now also U17.2 (V-), C6.1, R53.1, VR1.2, VR1.3
- net V12_Rail: now also U17.3 (V+), U17.9 (MODE), R234.1
- net VLed_Jauge: now reaches D25.1
- net VLed_Jauge: now also D25.10, D25.2, D25.3, D25.4, D25.5, D25.6, D25.7, D25.8, D25.9, C6.2, R234.2
- net at D25.11: now also U17.1 (LED1)
- net at D25.12: now also U17.18 (LED2)
- net at D25.13: now also U17.17 (LED3)
- net at D25.14: now also U17.16 (LED4)
- net at D25.15: now also U17.15 (LED5)
- net at D25.16: now also U17.14 (LED6)
- net at D25.17: now also U17.13 (LED7)
- net at D25.18: now also U17.12 (LED8)
- net at D25.19: now also U17.11 (LED9)
- net at D25.20: now also U17.10 (LED10)
- net at U17.4 (RLO): now also U17.8 (REFADJ), R36.1, R53.2
- net Sig_Jauge: now reaches U17.5 (SIG)
- net Sig_Jauge: now also R232.1, R233.1
- net at U17.6 (RHI): now also U17.7 (REFOUT), R36.2
- new net: R233.2, VR1.1
Other:
- moved on the sheet: D25, U17

Commit message: Add files via upload
Parts:
- removed C6: SR205E104MARAP1, SR205E104MARAP1:CAPRR254W50L508T317H508, symbol TrailerDiagSymbols:SR205E104MARAP1
- removed D25: OSX10201-GYR1, OSX10201-GYR1:DIP760W45P254L2550H815Q20B, symbol OSX10201-GYR1.kicad_sym:OSX10201-GYR1
- removed Q64: IRLZ44N, PCM_Package_TO_SOT_THT_AKL:TO-220-3_Vertical_GDS, symbol PCM_Transistor_MOSFET_AKL:IRLZ44N
- removed Q65: 2N7000, PCM_Package_TO_SOT_THT_AKL:TO-92_Inline_Wide_SGD, symbol PCM_Transistor_MOSFET_AKL:2N7000
- removed R230, R231: 4.7kΩ, Resistor_THT:R_Axial_DIN0207_L6.3mm_D2.5mm_P10.16mm_Horizontal, symbol PCM_SL_Resistors:4.7k
- removed R232: 18k, Resistor_THT:R_Axial_DIN0207_L6.3mm_D2.5mm_P10.16mm_Horizontal, symbol PCM_SL_Resistors:18k
- removed R233: 10k, Resistor_THT:R_Axial_DIN0207_L6.3mm_D2.5mm_P10.16mm_Horizontal, symbol PCM_SL_Resistors:10k
- removed R234: 68ohm, Resistor_THT:R_Axial_Power_L25.0mm_W9.0mm_P27.94mm, symbol PCM_SL_Devices:Resistor_5W
- removed R36: 1.5k, Resistor_THT:R_Axial_DIN0207_L6.3mm_D2.5mm_P10.16mm_Horizontal, symbol PCM_SL_Resistors:1.5k
- removed R53: 3.9k, Resistor_THT:R_Axial_DIN0207_L6.3mm_D2.5mm_P10.16mm_Horizontal, symbol PCM_SL_Resistors:3.9k
- removed U17: LM3914N, Package_DIP:DIP-18_W7.62mm, symbol Driver_LED:LM3914N
- removed VR1: 3296W-1-102LF, 3296W-1-102LF:TRIM_3296W-1-102LF, symbol 3296-1-102lf:3296W-1-102LF
Connections:
- net V12_PostShunt is gone; now on net V12_Rail: R221.2
- net Batt_Externe_Pos: now also F1.1
- net GND: no longer U16.7 (+)
- net V_Ref: no longer R222.2, U16.6 (-)
- no-connect marks 6 -> 5
Other:
- note removed: "Coupure de V12_Rail sur court-circuit"
- moved on the sheet: R216

Commit message: Add files via upload
Parts:
- added C6: SR205E104MARAP1, SR205E104MARAP1:CAPRR254W50L508T317H508, symbol TrailerDiagSymbols:SR205E104MARAP1
- added C7: SR655C106KAR, CAPRR508W50L762T381H762:CAPRR508W50L762T381H762, symbol SR655C106KAR:SR655C106KAR
- added C8: FG26X7R1E106KRT06, FG26X7R1E106KRT06:CAPRB500W50L550T350H600, symbol FG26X7R1E106KRT06:FG26X7R1E106KRT06
- added D25: OSX10201-GYR1, OSX10201-GYR1:DIP760W45P254L2550H815Q20B, symbol OSX10201-GYR1:OSX10201-GYR1
- added J1: Conn_01x05, symbol Connector_Generic:Conn_01x05
- added PS1: TMR_2-1211WIN, TMR 2-1211WIN:CONV_TMR_2-1211WIN, symbol TMR 2-1211WIN:TMR_2-1211WIN
- added Q64: IRLZ44N, PCM_Package_TO_SOT_THT_AKL:TO-220-3_Vertical_GDS, symbol PCM_Transistor_MOSFET_AKL:IRLZ44N
- added Q65: 2N7000, PCM_Package_TO_SOT_THT_AKL:TO-92_Inline_Wide_SGD, symbol PCM_Transistor_MOSFET_AKL:2N7000
- added R230, R231: 4.7kΩ, Resistor_THT:R_Axial_DIN0207_L6.3mm_D2.5mm_P10.16mm_Horizontal, symbol PCM_SL_Resistors:4.7k
- added R232: 18k, Resistor_THT:R_Axial_DIN0207_L6.3mm_D2.5mm_P10.16mm_Horizontal, symbol PCM_SL_Resistors:18k
- added R233: 10k, Resistor_THT:R_Axial_DIN0207_L6.3mm_D2.5mm_P10.16mm_Horizontal, symbol PCM_SL_Resistors:10k
- added R234: 68ohm, Resistor_THT:R_Axial_Power_L25.0mm_W9.0mm_P27.94mm, symbol PCM_SL_Devices:Resistor_5W
- added R242: 50A/75mV, symbol Device:R_Shunt
- added R36: 1.5k, Resistor_THT:R_Axial_DIN0207_L6.3mm_D2.5mm_P10.16mm_Horizontal, symbol PCM_SL_Resistors:1.5k
- added R53: 3.9k, Resistor_THT:R_Axial_DIN0207_L6.3mm_D2.5mm_P10.16mm_Horizontal, symbol PCM_SL_Resistors:3.9k
- added U17: LM3914N, Package_DIP:DIP-18_W7.62mm, symbol Driver_LED:LM3914N
- added VR1: 3296W-1-102LF, 3296W-1-102LF:TRIM_3296W-1-102LF, symbol 3296-1-102lf:3296W-1-102LF
- R216: footprint 3296W1103LF:TRIM_3296W1103LF -> TRIM_3296W1103LF:TRIM_3296W1103LF
Connections:
- net Batt_Interne_Pos: now also R232.2
- net Court_Bus_Fault: now also R231.1
- net GND: now also U16.7 (+), C6.1, C7.2, PS1.1 (-VIN_(GND)), Q65.1 (S), R242.4, R53.1, U17.2 (V-), VR1.2, VR1.3; no longer BMS3s1.P-, J2.2, P1.2 (N)
- net V12_Rail: now also C7.1, PS1.2 (+VIN_(VCC)), Q64.3 (S), R234.1, U17.3 (V+), U17.9 (MODE); no longer R221.2
- net V_Ref: now also R222.2, U16.6 (-), R230.2
- new net: Q64.1 (G), Q65.3 (D), R230.1
- new net: R233.2, VR1.1
- new net: D25.11, U17.1 (LED1)
- new net: D25.12, U17.18 (LED2)
- new net: D25.13, U17.17 (LED3)
- new net: D25.14, U17.16 (LED4)
- new net: D25.15, U17.15 (LED5)
- new net: D25.16, U17.14 (LED6)
- new net: D25.17, U17.13 (LED7)
- new net: D25.18, U17.12 (LED8)
- new net: D25.19, U17.11 (LED9)
- new net: D25.20, U17.10 (LED10)
- new net: R36.1, R53.2, U17.4 (RLO), U17.8 (REFADJ)
- new net: R36.2, U17.6 (RHI), U17.7 (REFOUT)
- new net: Q65.2 (G), R231.2
- new net Batt_Neg: BMS3s1.P-, J2.2, P1.2 (N), R242.1
- new net Sig_Jauge: R232.1, R233.1, U17.5 (SIG)
- new net V12_PostShunt: Q64.2 (D), R221.2
- new net VLed_Jauge: C6.2, D25.1, D25.10, D25.2, D25.3, D25.4, D25.5, D25.6, D25.7, D25.8, D25.9, R234.2
- new net VM_0V_Iso: C8.2, J1.2 (Pin_2), PS1.7 (-VOUT)
- new net VM_5V_Iso: C8.1, J1.1 (Pin_1), PS1.6 (+VOUT)
- new net VM_Mesure: J1.3 (Pin_3)
- new net VM_Shunt_Batt: J1.4 (Pin_4), R242.2
- new net VM_Shunt_Gnd: J1.5 (Pin_5), R242.3
- no-connect marks 5 -> 7
Other:
- note added: "Coupure de V12_Rail sur court-circuit"
- note added: "Module du voltmetre/ampèremetre"
- moved on the sheet: R216

Commit message: Add files via upload
Parts:
- removed C6: SR205E104MARAP1, SR205E104MARAP1:CAPRR254W50L508T317H508, symbol TrailerDiagSymbols:SR205E104MARAP1
- removed C7: SR655C106KAR, CAPRR508W50L762T381H762:CAPRR508W50L762T381H762, symbol SR655C106KAR:SR655C106KAR
- removed C8: FG26X7R1E106KRT06, FG26X7R1E106KRT06:CAPRB500W50L550T350H600, symbol FG26X7R1E106KRT06:FG26X7R1E106KRT06
- removed D25: OSX10201-GYR1, OSX10201-GYR1:DIP760W45P254L2550H815Q20B, symbol OSX10201-GYR1:OSX10201-GYR1
- removed J1: Conn_01x05, symbol Connector_Generic:Conn_01x05
- removed PS1: TMR_2-1211WIN, TMR 2-1211WIN:CONV_TMR_2-1211WIN, symbol TMR 2-1211WIN:TMR_2-1211WIN
- removed Q64: IRLZ44N, PCM_Package_TO_SOT_THT_AKL:TO-220-3_Vertical_GDS, symbol PCM_Transistor_MOSFET_AKL:IRLZ44N
- removed Q65: 2N7000, PCM_Package_TO_SOT_THT_AKL:TO-92_Inline_Wide_SGD, symbol PCM_Transistor_MOSFET_AKL:2N7000
- removed R230, R231: 4.7kΩ, Resistor_THT:R_Axial_DIN0207_L6.3mm_D2.5mm_P10.16mm_Horizontal, symbol PCM_SL_Resistors:4.7k
- removed R232: 18k, Resistor_THT:R_Axial_DIN0207_L6.3mm_D2.5mm_P10.16mm_Horizontal, symbol PCM_SL_Resistors:18k
- removed R233: 10k, Resistor_THT:R_Axial_DIN0207_L6.3mm_D2.5mm_P10.16mm_Horizontal, symbol PCM_SL_Resistors:10k
- removed R234: 68ohm, Resistor_THT:R_Axial_Power_L25.0mm_W9.0mm_P27.94mm, symbol PCM_SL_Devices:Resistor_5W
- removed R242: 50A/75mV, symbol Device:R_Shunt
- removed R36: 1.5k, Resistor_THT:R_Axial_DIN0207_L6.3mm_D2.5mm_P10.16mm_Horizontal, symbol PCM_SL_Resistors:1.5k
- removed R53: 3.9k, Resistor_THT:R_Axial_DIN0207_L6.3mm_D2.5mm_P10.16mm_Horizontal, symbol PCM_SL_Resistors:3.9k
- removed U17: LM3914N, Package_DIP:DIP-18_W7.62mm, symbol Driver_LED:LM3914N
- removed VR1: 3296W-1-102LF, 3296W-1-102LF:TRIM_3296W-1-102LF, symbol 3296-1-102lf:3296W-1-102LF
- R216: footprint TRIM_3296W1103LF:TRIM_3296W1103LF -> 3296W1103LF:TRIM_3296W1103LF
Connections:
- net Batt_Neg is gone; now on net GND: BMS3s1.P-, J2.2, P1.2 (N)
- net V12_PostShunt is gone; now on net V12_Rail: R221.2
- net GND: no longer U16.7 (+)
- net V_Ref: no longer R222.2, U16.6 (-)
- no-connect marks 7 -> 5
Other:
- note removed: "Coupure de V12_Rail sur court-circuit"
- note removed: "Module du voltmetre/ampèremetre"
- moved on the sheet: R216

Commit message: Add files via upload
Parts:
- added C6: SR205E104MARAP1, SR205E104MARAP1:CAPRR254W50L508T317H508, symbol TrailerDiagSymbols:SR205E104MARAP1
- added D25: OSX10201-GYR1, OSX10201-GYR1:DIP760W45P254L2550H815Q20B, symbol OSX10201-GYR1.kicad_sym:OSX10201-GYR1
- added Q64: IRLZ44N, PCM_Package_TO_SOT_THT_AKL:TO-220-3_Vertical_GDS, symbol PCM_Transistor_MOSFET_AKL:IRLZ44N
- added Q65: 2N7000, PCM_Package_TO_SOT_THT_AKL:TO-92_Inline_Wide_SGD, symbol PCM_Transistor_MOSFET_AKL:2N7000
- added R230, R231: 4.7kΩ, Resistor_THT:R_Axial_DIN0207_L6.3mm_D2.5mm_P10.16mm_Horizontal, symbol PCM_SL_Resistors:4.7k
- added R232: 18k, Resistor_THT:R_Axial_DIN0207_L6.3mm_D2.5mm_P10.16mm_Horizontal, symbol PCM_SL_Resistors:18k
- added R233: 10k, Resistor_THT:R_Axial_DIN0207_L6.3mm_D2.5mm_P10.16mm_Horizontal, symbol PCM_SL_Resistors:10k
- added R234: 68ohm, Resistor_THT:R_Axial_Power_L25.0mm_W9.0mm_P27.94mm, symbol PCM_SL_Devices:Resistor_5W
- added R36: 1.5k, Resistor_THT:R_Axial_DIN0207_L6.3mm_D2.5mm_P10.16mm_Horizontal, symbol PCM_SL_Resistors:1.5k
- added R53: 3.9k, Resistor_THT:R_Axial_DIN0207_L6.3mm_D2.5mm_P10.16mm_Horizontal, symbol PCM_SL_Resistors:3.9k
- added U17: LM3914N, Package_DIP:DIP-18_W7.62mm, symbol Driver_LED:LM3914N
- added VR1: 3296W-1-102LF, 3296W-1-102LF:TRIM_3296W-1-102LF, symbol 3296-1-102lf:3296W-1-102LF
- R216: footprint 3296W1103LF:TRIM_3296W1103LF -> TRIM_3296W1103LF:TRIM_3296W1103LF
Connections:
- net Batt_Externe_Pos: no longer F1.1
- net Batt_Interne_Pos: now also R232.2
- net Court_Bus_Fault: now also R231.1
- net GND: now also U16.7 (+), C6.1, Q65.1 (S), R53.1, U17.2 (V-), VR1.2, VR1.3
- net V12_Rail: now also Q64.3 (S), R234.1, U17.3 (V+), U17.9 (MODE); no longer R221.2
- net V_Ref: now also R222.2, U16.6 (-), R230.2
- new net: Q64.1 (G), Q65.3 (D), R230.1
- new net: R233.2, VR1.1
- new net: D25.11, U17.1 (LED1)
- new net: D25.12, U17.18 (LED2)
- new net: D25.13, U17.17 (LED3)
- new net: D25.14, U17.16 (LED4)
- new net: D25.15, U17.15 (LED5)
- new net: D25.16, U17.14 (LED6)
- new net: D25.17, U17.13 (LED7)
- new net: D25.18, U17.12 (LED8)
- new net: D25.19, U17.11 (LED9)
- new net: D25.20, U17.10 (LED10)
- new net: R36.1, R53.2, U17.4 (RLO), U17.8 (REFADJ)
- new net: R36.2, U17.6 (RHI), U17.7 (REFOUT)
- new net: Q65.2 (G), R231.2
- new net Sig_Jauge: R232.1, R233.1, U17.5 (SIG)
- new net V12_PostShunt: Q64.2 (D), R221.2
- new net VLed_Jauge: C6.2, D25.1, D25.10, D25.2, D25.3, D25.4, D25.5, D25.6, D25.7, D25.8, D25.9, R234.2
- no-connect marks 5 -> 6
Other:
- note added: "Coupure de V12_Rail sur court-circuit"
- moved on the sheet: R216
