File: Alimentation.kicad_sch (KiCad schematic)
At the start: 46 parts, among them J2 Screw_Terminal_2_P3.50mm, P1 Conn_Plug_2P, Q1 IRLZ44N, Q55 2N3906, Q56 2N7000, Q57 2N7000, Q64 IRLZ44N, Q65 2N7000, SW1 SW_DPDT_x2, U1 LM74610QDGKRQ1, U16 LM339, U17 LM3914N, U6 LM7805CT

Commit message: Add files via upload
Connections:
- net Batt_Externe_Pos: now also F1.1
Changed lines of the file:
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@@
+	(wire
+		(pts
+			(xy 76.2 35.56) (xy 78.74 35.56)
+		)
+		(stroke
+			(width 0)
+			(type default)
+		)
+	)
 	(wire
 		(pts
@@
 		(effects
 			(font
+				(size 1.27 1.27)
+			)
+			(justify left bottom)
+		)
+	)
+	(label "Batt_Externe_Pos"
+		(at 78.74 35.56 0)
+		(effects
+			(font

Commit message: Add files via upload
Changed lines of the file:
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@@
+		)
+	)
+	(label "Batt_Interne_Pos"
+		(at 50.8 69.85 0)
+		(effects
+			(font
+				(size 1.27 1.27)
+			)
+			(justify left bottom)
 		)
 	)
@@
 		)
 	)
+	(label "Batt_Interne_Pos"
+		(at 127 67.31 180)
+		(effects
+			(font
+				(size 1.27 1.27)
+			)
+			(justify right bottom)
+		)
+	)
+	(label "Batt_Interne_Pos"
+		(at 73.66 172.72 0)
+		(effects
+			(font
+				(size 1.27 1.27)
+			)
+			(justify left bottom)
+		)
+	)
 	(label "V12_PostShunt"
 		(at 188.722 123.19 0)
@@
 		)
 	)
-	(hierarchical_label "Batt_Interne_Pos"
-		(shape input)
-		(at 50.8 69.85 0)
+	(hierarchical_label "V12_Rail"
+		(shape input)
+		(at 68.58 185.42 180)
+		(effects
+			(font
+				(size 1.27 1.27)
+			)
+			(justify right)
+		)
+	)
+	(hierarchical_label "Court_Bus_Fault"
+		(shape input)
+		(at 378.46 147.32 180)
+		(effects
+			(font
+				(size 1.27 1.27)
+			)
+			(justify right)
+		)
+	)
+	(hierarchical_label "Surtension_Fault"
+		(shape input)
+		(at 386.08 46.99 0)
 		(effects
 			(font
@@
 	(hierarchical_label "V12_Rail"
 		(shape input)
-		(at 68.58 185.42 180)
-		(effects
-			(font
-				(size 1.27 1.27)
-			)
-			(justify right)
-		)
-	)
-	(hierarchical_label "Court_Bus_Fault"
-		(shape input)
-		(at 378.46 147.32 180)
-		(effects
-			(font
-				(size 1.27 1.27)
-			)
-			(justify right)
-		)
-	)
-	(hierarchical_label "Surtension_Fault"
-		(shape input)
-		(at 386.08 46.99 0)
-		(effects
-			(font
-				(size 1.27 1.27)
-			)
-			(justify left)
+		(at 29.21 119.38 180)
+		(effects
+			(font
+				(size 1.27 1.27)
+			)
+			(justify right)
 		)
 	)
 	(hierarchical_label "V12_Rail"
 		(shape input)
-		(at 29.21 119.38 180)
-		(effects
-			(font
-				(size 1.27 1.27)
-			)
-			(justify right)
-		)
-	)
-	(hierarchical_label "Batt_Interne_Pos"
-		(shape input)
-		(at 73.66 172.72 0)
-		(effects
-			(font
-				(size 1.27 1.27)
-			)
-			(justify left)
-		)
-	)
-	(hierarchical_label "V12_Rail"
-		(shape input)
 		(at 314.96 36.83 180)
 		(effects
 			(font
-				(size 1.27 1.27)
-			)
-			(justify right)
-		)
-	)
-	(hierarchical_label "Batt_Interne_Pos"
-		(shape input)
-		(at 127 67.31 180)
-		(effects
-			(font

Commit message: Add files via upload
Changed lines of the file:
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@@
 	)
 	(symbol
-		(lib_name "IRLZ44N_1")
 		(lib_id "PCM_Transistor_MOSFET_AKL:IRLZ44N")
 		(at 207.264 178.816 0)
@@
 	)
 	(symbol
-		(lib_name "2N7000_1")
 		(lib_id "PCM_Transistor_MOSFET_AKL:2N7000")
 		(at 379.73 167.64 0)
@@
 	)
 	(symbol
-		(lib_name "2N7000_2")
 		(lib_id "PCM_Transistor_MOSFET_AKL:2N7000")
 		(at 258.064 171.196 0)

Commit message: Add files via upload
Parts:
- D25: symbol OSX10201-GYR1.kicad_sym:OSX10201-GYR1 -> OSX10201-GYR1:OSX10201-GYR1
Changed lines of the file:
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@@
 	)
 	(symbol
-		(lib_id "OSX10201-GYR1.kicad_sym:OSX10201-GYR1")
+		(lib_id "OSX10201-GYR1:OSX10201-GYR1")
 		(at 130.81 220.98 0)
 		(unit 1)

Commit message: Add files via upload
Parts:
- U16: footprint (none) -> Package_DIP:DIP-14_W7.62mm_Socket
- U17: footprint Package_DIP:DIP-18_W7.62mm -> Package_DIP:DIP-18_W7.62mm_Socket
Changed lines of the file:
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@@
 			)
 		)
-		(property "Footprint" ""
+		(property "Footprint" "Package_DIP:DIP-14_W7.62mm_Socket"
 			(at 356.87 53.34 0)
 			(hide yes)
@@
 			)
 		)
-		(property "Footprint" ""
+		(property "Footprint" "Package_DIP:DIP-14_W7.62mm_Socket"
 			(at 359.41 104.14 0)
 			(hide yes)
@@
 			)
 		)
-		(property "Footprint" "Package_DIP:DIP-18_W7.62mm"
+		(property "Footprint" "Package_DIP:DIP-18_W7.62mm_Socket"
 			(at 86.36 232.41 0)
 			(hide yes)
@@
 			)
 		)
-		(property "Footprint" ""
+		(property "Footprint" "Package_DIP:DIP-14_W7.62mm_Socket"
 			(at 356.87 69.85 0)
 			(hide yes)
@@
 			)
 		)
-		(property "Footprint" ""
+		(property "Footprint" "Package_DIP:DIP-14_W7.62mm_Socket"
 			(at 356.87 86.36 0)
 			(hide yes)
@@
 			)
 		)
-		(property "Footprint" ""
+		(property "Footprint" "Package_DIP:DIP-14_W7.62mm_Socket"
 			(at 356.87 36.83 0)
 			(hide yes)

Commit message: Add files via upload
Parts:
- U16: footprint Package_DIP:DIP-14_W7.62mm_Socket -> (none)
- U17: footprint Package_DIP:DIP-18_W7.62mm_Socket -> Package_DIP:DIP-18_W7.62mm
Changed lines of the file:
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@@
 		)
 	)
+	(hierarchical_label "VM_Mesure"
+		(shape input)
+		(at 205.74 134.62 0)
+		(effects
+			(font
+				(size 1.27 1.27)
+			)
+			(justify left)
+		)
+	)
 	(hierarchical_label "Court_Bus_Fault"
 		(shape input)
@@
 			)
 		)
-		(property "Footprint" "Package_DIP:DIP-14_W7.62mm_Socket"
+		(property "Footprint" ""
 			(at 356.87 53.34 0)
 			(hide yes)
@@
 			)
 		)
-		(property "Footprint" "Package_DIP:DIP-14_W7.62mm_Socket"
+		(property "Footprint" ""
 			(at 359.41 104.14 0)
 			(hide yes)
@@
 			)
 		)
-		(property "Footprint" "Package_DIP:DIP-18_W7.62mm_Socket"
+		(property "Footprint" "Package_DIP:DIP-18_W7.62mm"
 			(at 86.36 232.41 0)
 			(hide yes)
@@
 			)
 		)
-		(property "Footprint" "Package_DIP:DIP-14_W7.62mm_Socket"
+		(property "Footprint" ""
 			(at 356.87 69.85 0)
 			(hide yes)
@@
 			)
 		)
-		(property "Footprint" "Package_DIP:DIP-14_W7.62mm_Socket"
+		(property "Footprint" ""
 			(at 356.87 86.36 0)
 			(hide yes)
@@
 			)
 		)
-		(property "Footprint" "Package_DIP:DIP-14_W7.62mm_Socket"
+		(property "Footprint" ""
 			(at 356.87 36.83 0)
 			(hide yes)

Commit message: Add files via upload
Parts:
- removed C6: SR205E104MARAP1, SR205E104MARAP1:CAPRR254W50L508T317H508, symbol TrailerDiagSymbols:SR205E104MARAP1
- removed D25: OSX10201-GYR1, OSX10201-GYR1:DIP760W45P254L2550H815Q20B, symbol OSX10201-GYR1:OSX10201-GYR1
- removed Q64: IRLZ44N, PCM_Package_TO_SOT_THT_AKL:TO-220-3_Vertical_GDS, symbol PCM_Transistor_MOSFET_AKL:IRLZ44N
- removed Q65: 2N7000, PCM_Package_TO_SOT_THT_AKL:TO-92_Inline_Wide_SGD, symbol PCM_Transistor_MOSFET_AKL:2N7000
- removed R230, R231: 4.7kΩ, Resistor_THT:R_Axial_DIN0207_L6.3mm_D2.5mm_P10.16mm_Horizontal, symbol PCM_SL_Resistors:4.7k
- removed R232: 18k, Resistor_THT:R_Axial_DIN0207_L6.3mm_D2.5mm_P10.16mm_Horizontal, symbol PCM_SL_Resistors:18k
- removed R233: 10k, Resistor_THT:R_Axial_DIN0207_L6.3mm_D2.5mm_P10.16mm_Horizontal, symbol PCM_SL_Resistors:10k
- removed R234: 68ohm, Resistor_THT:R_Axial_Power_L25.0mm_W9.0mm_P27.94mm, symbol PCM_SL_Devices:Resistor_5W
- removed R36: 1.5k, Resistor_THT:R_Axial_DIN0207_L6.3mm_D2.5mm_P10.16mm_Horizontal, symbol PCM_SL_Resistors:1.5k
- removed R53: 3.9k, Resistor_THT:R_Axial_DIN0207_L6.3mm_D2.5mm_P10.16mm_Horizontal, symbol PCM_SL_Resistors:3.9k
- removed U17: LM3914N, Package_DIP:DIP-18_W7.62mm, symbol Driver_LED:LM3914N
- removed VR1: 3296W-1-102LF, 3296W-1-102LF:TRIM_3296W-1-102LF, symbol 3296-1-102lf:3296W-1-102LF
- R216: footprint TRIM_3296W1103LF:TRIM_3296W1103LF -> 3296W1103LF:TRIM_3296W1103LF
Connections:
- net V12_PostShunt is gone; now on net V12_Rail: R221.2
- net GND: no longer U16.7 (+)
- net V_Ref: no longer R222.2, U16.6 (-)
- no-connect marks 6 -> 5
Other:
- note removed: "Coupure de V12_Rail sur court-circuit"
- moved on the sheet: R216
