File: Trailer_Brake.kicad_sch (KiCad schematic)
At the start: 11 parts, among them Q52 IRLZ44N, SW8 SW_SPST, U14 LM339

Commit message: Add files via upload
Parts:
- R201: footprint PCM_SL_Devices:Resistor_5W -> Resistor_THT:R_Axial_Power_L25.0mm_W9.0mm_P27.94mm
Changed lines of the file:
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@@
 			)
 		)
-		(property "Footprint" "PCM_SL_Devices:Resistor_5W"
+		(property "Footprint" "Resistor_THT:R_Axial_Power_L25.0mm_W9.0mm_P27.94mm"
 			(at 106.299 66.548 0)
 			(hide yes)

Commit message: Add files via upload
Parts:
- R202, R203: footprint (none) -> TRIM_3296W1103LF:TRIM_3296W1103LF
Changed lines of the file:
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@@
 			)
 		)
-		(property "Footprint" ""
+		(property "Footprint" "TRIM_3296W1103LF:TRIM_3296W1103LF"
 			(at 111.76 52.07 0)
 			(hide yes)
@@
 			)
 		)
-		(property "Footprint" ""
+		(property "Footprint" "TRIM_3296W1103LF:TRIM_3296W1103LF"
 			(at 123.19 73.66 0)
 			(hide yes)

Commit message: Add files via upload
Parts:
- removed Q52: IRLZ44N, PCM_Package_TO_SOT_THT_AKL:TO-220-3_Vertical_GDS, symbol PCM_Transistor_MOSFET_AKL:IRLZ44N
- removed R200: 10k, Resistor_THT:R_Axial_DIN0207_L6.3mm_D2.5mm_P10.16mm_Horizontal, symbol PCM_SL_Resistors:10k
- removed R201: .1 ohm, Resistor_THT:R_Axial_Power_L25.0mm_W9.0mm_P27.94mm, symbol PCM_SL_Resistors:4.7k
- added D172: MUR1520G, Package_TO_SOT_THT:TO-220-2_Vertical, symbol Device:D
- added DZ3: 1N5242B, PCM_Diode_THT_AKL:D_DO-35_SOD27_P7.62mm_Horizontal_Zener, symbol PCM_Diode_Zener_AKL:1N5242B
- added Q52: IRF4905PBF, Package_TO_SOT_THT:TO-220-3_Vertical, symbol Transistor_FET:IRF4905
- added Q71: 2N7000, PCM_Package_TO_SOT_THT_AKL:TO-92_Inline_Wide_SGD, symbol PCM_Transistor_MOSFET_AKL:2N7000
- added Q72: 2N3906, PCM_Package_TO_SOT_THT_AKL:TO-92_Inline_Wide_EBC, symbol PCM_Transistor_BJT_AKL:2N3906
- added R200: 10k, Resistor_THT:R_Axial_DIN0207_L6.3mm_D2.5mm_P10.16mm_Horizontal, symbol PCM_SL_Resistors:4.7k
- added R201: 12 Ohm - 1W, Resistor_THT:R_Axial_DIN0414_L11.9mm_D4.5mm_P15.24mm_Horizontal, symbol PCM_SL_Devices:Resistor_5W
- added R260, R262: 1k, Resistor_THT:R_Axial_DIN0207_L6.3mm_D2.5mm_P10.16mm_Horizontal, symbol PCM_SL_Resistors:1k
- added R261, R263, R266: 10k, Resistor_THT:R_Axial_DIN0207_L6.3mm_D2.5mm_P10.16mm_Horizontal, symbol PCM_SL_Resistors:10k
- added R264: 2.7k, Resistor_THT:R_Axial_DIN0207_L6.3mm_D2.5mm_P10.16mm_Horizontal, symbol PCM_SL_Resistors:2.7k
- added R265: 39kΩ, Resistor_THT:R_Axial_DIN0207_L6.3mm_D2.5mm_P10.16mm_Horizontal, symbol PCM_SL_Resistors:10k
- R202: Etiquette Pot_Brake_Ouvert -> (none)
- R203: Etiquette Pot2_Brake_Court -> (none)
Connections:
- net Btn_Brake_Etat: now also Q71.2 (G), R200.2
- net GND: now also R203.1, Q71.1 (S), R200.1, R264.2, R266.2; no longer R203.3
- net Trail_Brake: now also D172.1 (K), R201.2, R262.1, R265.2
- net V_Ref: now also R203.3; no longer R203.1
- net Brake_Trailer_Shunt_Haut renamed Court_Sense_Brake
- net Court_Sense_Brake: now also R265.1, R266.1; no longer U14.6 (-)
- net Q52.2_Drain: no longer names the net of F7.2
- net Q52.2_Drain: now also DZ3.1 (K), Q52.3 (S), R261.2
- new net: Q71.3 (D), R260.1
- new net: DZ3.2 (A), Q52.1 (G), R260.2, R261.1
- new net: Q72.3 (C), R263.1
- new net: Q72.2 (B), R262.2
- new net: D172.2 (A), Q52.2 (D), Q72.1 (E), R201.1
- new net I_Present_Brake: R263.2, R264.1, U14.6 (-)

Commit message: Add files via upload
Parts:
- D146: value SMBJ33A -> P6KE39A; footprint PCM_Diode_SMD_AKL:D_SMB -> PCM_Diode_THT_AKL:D_DO-15_P10.16mm_Horizontal_Zener; symbol PCM_Diode_TVS_AKL:SMBJ33A -> PCM_Diode_TVS_AKL:P6KE39A
Changed lines of the file:
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@@
 	)
 	(symbol
-		(lib_id "PCM_Diode_TVS_AKL:SMBJ33A")
+		(lib_id "PCM_Diode_TVS_AKL:P6KE39A")
 		(at 199.39 109.22 0)
 		(unit 1)
@@
 			)
 		)
-		(property "Value" "SMBJ33A"
+		(property "Value" "P6KE39A"
 			(at 199.39 105.41 0)
 			(show_name no)
@@
 			)
 		)
-		(property "Footprint" "PCM_Diode_SMD_AKL:D_SMB"
+		(property "Footprint" "PCM_Diode_THT_AKL:D_DO-15_P10.16mm_Horizontal_Zener"
 			(at 199.39 109.22 0)
 			(hide yes)
@@
 			)
 		)
-		(property "Datasheet" "https://www.tme.eu/Document/0b6222bec7e12d83185b51d73cb6a54d/SMBJ_ser.pdf"
+		(property "Datasheet" "https://www.tme.eu/Document/6b488a936123e1f9ccf03f4f9186b150/P6KE_ser.pdf"
 			(at 199.39 109.22 0)
 			(hide yes)
@@
 			)
 		)
-		(property "Description" "SMB Unidirectional TVS diode, 33V, 600W, Alternate KiCAD Library"
+		(property "Description" "DO-15 Unidirectional TVS diode, 39V, 600W, Alternate KiCAD Library"
 			(at 199.39 109.22 0)
 			(hide yes)

Commit message: Add files via upload
Parts:
- F7: value Polyfuse -> MF-R300
- U14: footprint (none) -> Package_DIP:DIP-14_W7.62mm_Socket
Changed lines of the file:
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@@
 			)
 		)
-		(property "Footprint" ""
+		(property "Footprint" "Package_DIP:DIP-14_W7.62mm_Socket"
 			(at 236.22 124.46 0)
 			(hide yes)
@@
 			)
 		)
-		(property "Footprint" ""
+		(property "Footprint" "Package_DIP:DIP-14_W7.62mm_Socket"
 			(at 240.03 83.82 0)
 			(hide yes)
@@
 			)
 		)
-		(property "Footprint" ""
+		(property "Footprint" "Package_DIP:DIP-14_W7.62mm_Socket"
 			(at 240.03 62.23 0)
 			(hide yes)
@@
 			)
 		)
-		(property "Footprint" ""
+		(property "Footprint" "Package_DIP:DIP-14_W7.62mm_Socket"
 			(at 241.3 104.14 0)
 			(hide yes)
@@
 			)
 		)
-		(property "Value" "Polyfuse"
+		(property "Value" "MF-R300"
 			(at 115.57 74.93 90)
 			(show_name no)
@@
 			)
 		)
-		(property "Footprint" ""
+		(property "Footprint" "Package_DIP:DIP-14_W7.62mm_Socket"
 			(at 240.03 40.64 0)
 			(hide yes)

Commit message: Add files via upload
Parts:
- F7: footprint (none) -> PTC_Bourns_MF-R:PTC_Bourns_MF-R_P5.10mm_W12.0mm
Changed lines of the file:
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@@
 			)
 		)
-		(property "Footprint" ""
+		(property "Footprint" "PTC_Bourns_MF-R:PTC_Bourns_MF-R_P5.10mm_W12.0mm"
 			(at 110.49 77.47 0)
 			(hide yes)

Commit message: Add files via upload
Parts:
- SW8: value SW_SPST -> SW_SPDT; symbol Switch:SW_SPST -> Switch:SW_SPDT
Connections:
- net GND: now also SW8.3 (C)
Other:
- moved on the sheet: R200
Changed lines of the file:
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@@
 	)
 	(junction
+		(at 68.58 76.2)
+		(diameter 0)
+		(color 0 0 0 0)
+	)
+	(junction
 		(at 207.01 95.25)
 		(diameter 0)
@@
 		(color 0 0 0 0)
 	)
-	(junction
-		(at 68.58 76.2)
-		(diameter 0)
-		(color 0 0 0 0)
-	)
 	(no_connect
 		(at 250.19 106.68)
@@
 	(wire
 		(pts
-			(xy 57.15 76.2) (xy 68.58 76.2)
+			(xy 63.5 76.2) (xy 68.58 76.2)
 		)
 		(stroke
@@
 	(wire
 		(pts
+			(xy 55.88 76.2) (xy 52.07 76.2)
+		)
+		(stroke
+			(width 0)
+			(type default)
+		)
+	)
+	(wire
+		(pts
 			(xy 233.68 60.96) (xy 233.68 62.23)
 		)
@@
 	(wire
 		(pts
-			(xy 52.07 63.5) (xy 55.88 63.5)
+			(xy 52.07 60.96) (xy 55.88 60.96)
 		)
 		(stroke
@@
 	(wire
 		(pts
+			(xy 52.07 66.04) (xy 55.88 66.04)
+		)
+		(stroke
+			(width 0)
+			(type default)
+		)
+	)
+	(wire
+		(pts
 			(xy 107.95 58.42) (xy 176.53 58.42)
 		)
@@
 	(global_label "GND"
 		(shape input)
-		(at 49.53 76.2 180)
+		(at 52.07 66.04 180)
 		(fields_autoplaced yes)
 		(effects
@@
 		)
 		(property "Intersheetrefs" "${INTERSHEET_REFS}"
-			(at 42.6743 76.2 0)
+			(at 45.2143 66.04 0)
+			(hide yes)
+			(show_name no)
+			(do_not_autoplace no)
+			(effects
+				(font
+					(size 1.27 1.27)
+				)
+				(justify right)
+			)
+		)
+	)
+	(global_label "GND"
+		(shape input)
+		(at 52.07 76.2 180)
+		(fields_autoplaced yes)
+		(effects
+			(font
+				(size 1.27 1.27)
+			)
+			(justify right)
+		)
+		(property "Intersheetrefs" "${INTERSHEET_REFS}"
+			(at 45.2143 76.2 0)
 			(hide yes)
 			(show_name no)
@@
 	(global_label "V_Ref"
 		(shape input)
-		(at 52.07 63.5 180)
+		(at 52.07 60.96 180)
 		(fields_autoplaced yes)
 		(effects
@@
 		)
 		(property "Intersheetrefs" "${INTERSHEET_REFS}"
-			(at 43.9443 63.5 0)
+			(at 43.9443 60.96 0)
 			(hide yes)
 			(show_name no)
@@
 	)
 	(symbol
-		(lib_id "Switch:SW_SPST")
+		(lib_id "Switch:SW_SPDT")
 		(at 60.96 63.5 0)
+		(mirror y)
 		(unit 1)
 		(body_style 1)
@@
 		(in_pos_files yes)
 		(dnp no)
-		(fields_autoplaced yes)
 		(property "Reference" "SW8"
-			(at 60.96 57.15 0)
+			(at 60.96 56.388 0)
 			(show_name no)
 			(do_not_autoplace no)
@@
 			)
 		)
-		(property "Value" "SW_SPST"
-			(at 60.96 59.69 0)
+		(property "Value" "SW_SPDT"
+			(at 60.96 58.42 0)
 			(show_name no)
 			(do_not_autoplace no)
@@
 			)
 		)
-		(property "Description" "Single Pole Single Throw (SPST) switch"
+		(property "Description" "Switch, single pole double throw"
 			(at 60.96 63.5 0)
 			(hide yes)
@@
 		(pin "2"
 		)
+		(pin "3"
+		)
 		(instances
 			(project "TrailerDiagnosticSystem"
@@
 	(symbol
 		(lib_id "PCM_SL_Resistors:4.7k")
-		(at 53.34 76.2 0)
+		(at 59.69 76.2 0)
 		(unit 1)
 		(body_style 1)
@@
 		(fields_autoplaced yes)
 		(property "Reference" "R200"
-			(at 53.34 69.85 0)
+			(at 59.69 69.85 0)
 			(show_name no)
 			(do_not_autoplace no)
@@
 		)
 		(property "Value" "10k"
-			(at 53.34 72.39 0)
+			(at 59.69 72.39 0)
 			(show_name no)
 			(do_not_autoplace no)
@@
 		)
 		(property "Footprint" "Resistor_THT:R_Axial_DIN0207_L6.3mm_D2.5mm_P10.16mm_Horizontal"
-			(at 54.229 80.518 0)
+			(at 60.579 80.518 0)
 			(hide yes)
 			(show_name no)
@@
 		)
 		(property "Datasheet" ""
-			(at 53.848 76.2 0)
+			(at 60.198 76.2 0)
 			(hide yes)
 			(show_name no)
@@
 		)
 		(property "Description" "10kΩ, 1/4W Resistor"
-			(at 53.34 76.2 0)
+			(at 59.69 76.2 0)
 			(hide yes)
 			(show_name no)

Commit message: Add files via upload
Parts:
- R200, R261, R263, R266: value 10k -> 10kΩ
- R204, R205: value 4.7k -> 4.7kΩ
- R260, R262: value 1k -> 1kΩ
- R264: value 2.7k -> 2.7kΩ
Changed lines of the file:
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@@
 			)
 		)
-		(property "Value" "1k"
+		(property "Value" "1kΩ"
 			(at 91.44 59.69 0)
 			(show_name no)
@@
 			)
 		)
-		(property "Value" "10k"
+		(property "Value" "10kΩ"
 			(at 182.88 88.9 0)
 			(show_name no)
@@
 			)
 		)
-		(property "Value" "2.7k"
+		(property "Value" "2.7kΩ"
 			(at 135.89 90.17 0)
 			(show_name no)
@@
 			)
 		)
-		(property "Value" "4.7k"
+		(property "Value" "4.7kΩ"
 			(at 256.54 60.96 0)
 			(show_name no)
@@
 			)
 		)
-		(property "Value" "10k"
+		(property "Value" "10kΩ"
 			(at 102.87 71.12 0)
 			(show_name no)
@@
 			)
 		)
-		(property "Value" "10k"
+		(property "Value" "10kΩ"
 			(at 152.4 40.64 0)
 			(show_name no)
@@
 			)
 		)
-		(property "Value" "1k"
+		(property "Value" "1kΩ"
 			(at 163.83 78.74 0)
 			(show_name no)
@@
 			)
 		)
-		(property "Value" "4.7k"
+		(property "Value" "4.7kΩ"
 			(at 256.54 82.55 0)
 			(show_name no)
@@
 			)
 		)
-		(property "Value" "10k"
+		(property "Value" "10kΩ"
 			(at 59.69 72.39 0)
 			(show_name no)
