File: Trailer_Right.kicad_sch (KiCad schematic)
At the start: 11 parts, among them Q20 IRLZ44N, SW4 SW_SPST, U5 LM339

Commit message: Add files via upload
Parts:
- removed D50: SMBJ33A, PCM_Diode_SMD_AKL:D_SMB, symbol PCM_Diode_TVS_AKL:SMBJ33A
- removed F3: Polyfuse, symbol Device:Polyfuse
- removed Q20: IRLZ44N, PCM_Package_TO_SOT_THT_AKL:TO-220-3_Vertical_GDS, symbol PCM_Transistor_MOSFET_AKL:IRLZ44N
- removed R67: .1 ohm, Resistor_THT:R_Axial_DIN0207_L6.3mm_D2.5mm_P10.16mm_Horizontal, symbol PCM_SL_Resistors:4.7k
- removed R68, R69: Potentiometer, symbol Simulation_SPICE:Potentiometer
- removed R70, R71: 4.7k, Resistor_THT:R_Axial_DIN0207_L6.3mm_D2.5mm_P10.16mm_Horizontal, symbol PCM_SL_Resistors:4.7k
- removed R72: 10k, Resistor_THT:R_Axial_DIN0207_L6.3mm_D2.5mm_P10.16mm_Horizontal, symbol PCM_SL_Resistors:10k
- removed SW4: SW_SPST, symbol Switch:SW_SPST
- removed U5: LM339, symbol Comparator:LM339
- added D74: SMBJ33A, PCM_Diode_SMD_AKL:D_SMB, symbol PCM_Diode_TVS_AKL:SMBJ33A
- added F4: Polyfuse, symbol Device:Polyfuse
- added Q28: IRLZ44N, PCM_Package_TO_SOT_THT_AKL:TO-220-3_Vertical_GDS, symbol PCM_Transistor_MOSFET_AKL:IRLZ44N
- added R101: 10k, Resistor_THT:R_Axial_DIN0207_L6.3mm_D2.5mm_P10.16mm_Horizontal, symbol PCM_SL_Resistors:10k
- added R102: .1 ohm, Resistor_THT:R_Axial_DIN0207_L6.3mm_D2.5mm_P10.16mm_Horizontal, symbol PCM_SL_Resistors:4.7k
- added R103, R104: Potentiometer, symbol Simulation_SPICE:Potentiometer
- added R105, R106: 4.7k, Resistor_THT:R_Axial_DIN0207_L6.3mm_D2.5mm_P10.16mm_Horizontal, symbol PCM_SL_Resistors:4.7k
- added SW5: SW_SPST, symbol Switch:SW_SPST
- added U8: LM339, symbol Comparator:LM339
Connections:
- net GND: now also D74.2 (A), R101.2, R103.3, R104.3, U8.12 (V-), U8.5 (+), U8.9 (+)
- net V_Arm_Trailer: now also F4.1
- net V_Ref: now also R103.1, R104.1, R105.2, R106.2, SW5.1 (A), U8.3 (V+), U8.4 (-), U8.8 (-)
- new net: R104.2, U8.11 (+)
- new net: R103.2, U8.7 (+)
- new net Btn_Right_Etat: Q28.1 (G), R101.1, SW5.2 (B)
- new net Court_Right_Trailer: R106.1, U8.13
- new net Ouvert_Right_Trailer: R105.1, U8.1
- new net Q28.2_Drain: F4.2, Q28.2 (D)
- new net Right_Trailer_Shunt_Haut: Q28.3 (S), R102.2, U8.10 (-), U8.6 (-)
- new net Trail_Right: D74.1 (K), R102.1

Commit message: Add files via upload
Other:
- moved on the sheet: D74, F4, Q28, R101, R102, R103, R104, R105, R106, SW5, U8A, U8B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

Commit message: Add files via upload
Parts:
- R102: footprint Resistor_THT:R_Axial_DIN0207_L6.3mm_D2.5mm_P10.16mm_Horizontal -> PCM_SL_Devices:Resistor_5W
Changed lines of the file:
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@@
 			)
 		)
-		(property "Footprint" "Resistor_THT:R_Axial_DIN0207_L6.3mm_D2.5mm_P10.16mm_Horizontal"
+		(property "Footprint" "PCM_SL_Devices:Resistor_5W"
 			(at 93.599 65.278 0)
 			(hide yes)

Commit message: Add files via upload
Parts:
- R102: footprint PCM_SL_Devices:Resistor_5W -> Resistor_THT:R_Axial_Power_L25.0mm_W9.0mm_P27.94mm
Changed lines of the file:
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@@
 			)
 		)
-		(property "Footprint" "PCM_SL_Devices:Resistor_5W"
+		(property "Footprint" "Resistor_THT:R_Axial_Power_L25.0mm_W9.0mm_P27.94mm"
 			(at 93.599 65.278 0)
 			(hide yes)

Commit message: Add files via upload
Parts:
- R103, R104: footprint (none) -> TRIM_3296W1103LF:TRIM_3296W1103LF
Changed lines of the file:
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@@
 			)
 		)
-		(property "Footprint" ""
+		(property "Footprint" "TRIM_3296W1103LF:TRIM_3296W1103LF"
 			(at 99.06 50.8 0)
 			(hide yes)
@@
 			)
 		)
-		(property "Footprint" ""
+		(property "Footprint" "TRIM_3296W1103LF:TRIM_3296W1103LF"
 			(at 110.49 72.39 0)
 			(hide yes)

Commit message: Add files via upload
Parts:
- U8: footprint (none) -> Package_DIP:DIP-14_W7.62mm_Socket
Changed lines of the file:
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@@
 			)
 		)
-		(property "Footprint" ""
+		(property "Footprint" "Package_DIP:DIP-14_W7.62mm_Socket"
 			(at 139.7 68.58 0)
 			(hide yes)
@@
 			)
 		)
-		(property "Footprint" ""
+		(property "Footprint" "Package_DIP:DIP-14_W7.62mm_Socket"
 			(at 139.7 27.94 0)
 			(hide yes)
@@
 			)
 		)
-		(property "Footprint" ""
+		(property "Footprint" "Package_DIP:DIP-14_W7.62mm_Socket"
 			(at 128.27 106.68 0)
 			(hide yes)
@@
 			)
 		)
-		(property "Footprint" ""
+		(property "Footprint" "Package_DIP:DIP-14_W7.62mm_Socket"
 			(at 139.7 46.99 0)
 			(hide yes)
@@
 			)
 		)
-		(property "Footprint" ""
+		(property "Footprint" "Package_DIP:DIP-14_W7.62mm_Socket"
 			(at 140.97 86.36 0)
 			(hide yes)

Commit message: Add files via upload
Parts:
- U8: footprint Package_DIP:DIP-14_W7.62mm_Socket -> (none)
Changed lines of the file:
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@@
 			)
 		)
-		(property "Footprint" "Package_DIP:DIP-14_W7.62mm_Socket"
+		(property "Footprint" ""
 			(at 139.7 68.58 0)
 			(hide yes)
@@
 			)
 		)
-		(property "Footprint" "Package_DIP:DIP-14_W7.62mm_Socket"
+		(property "Footprint" ""
 			(at 139.7 27.94 0)
 			(hide yes)
@@
 			)
 		)
-		(property "Footprint" "Package_DIP:DIP-14_W7.62mm_Socket"
+		(property "Footprint" ""
 			(at 128.27 106.68 0)
 			(hide yes)
@@
 			)
 		)
-		(property "Footprint" "Package_DIP:DIP-14_W7.62mm_Socket"
+		(property "Footprint" ""
 			(at 139.7 46.99 0)
 			(hide yes)
@@
 			)
 		)
-		(property "Footprint" "Package_DIP:DIP-14_W7.62mm_Socket"
+		(property "Footprint" ""
 			(at 140.97 86.36 0)
 			(hide yes)

Commit message: Add files via upload
Parts:
- R102: footprint Resistor_THT:R_Axial_Power_L25.0mm_W9.0mm_P27.94mm -> Resistor_THT:R_Axial_DIN0207_L6.3mm_D2.5mm_P10.16mm_Horizontal
- R103, R104: footprint TRIM_3296W1103LF:TRIM_3296W1103LF -> (none)
Changed lines of the file:
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@@
 			)
 		)
-		(property "Footprint" "TRIM_3296W1103LF:TRIM_3296W1103LF"
+		(property "Footprint" ""
 			(at 99.06 50.8 0)
 			(hide yes)
@@
 			)
 		)
-		(property "Footprint" "TRIM_3296W1103LF:TRIM_3296W1103LF"
+		(property "Footprint" ""
 			(at 110.49 72.39 0)
 			(hide yes)
@@
 			)
 		)
-		(property "Footprint" "Resistor_THT:R_Axial_Power_L25.0mm_W9.0mm_P27.94mm"
+		(property "Footprint" "Resistor_THT:R_Axial_DIN0207_L6.3mm_D2.5mm_P10.16mm_Horizontal"
 			(at 93.599 65.278 0)
 			(hide yes)
