File: Trailer_Right.kicad_sch (KiCad schematic)
At the start: 11 parts, among them Q28 IRLZ44N, SW5 SW_SPST, U8 LM339

Commit message: Add files via upload
Parts:
- R102: footprint Resistor_THT:R_Axial_DIN0207_L6.3mm_D2.5mm_P10.16mm_Horizontal -> Resistor_THT:R_Axial_Power_L25.0mm_W9.0mm_P27.94mm
- R103, R104: footprint (none) -> TRIM_3296W1103LF:TRIM_3296W1103LF
Changed lines of the file:
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@@
 			)
 		)
-		(property "Footprint" ""
+		(property "Footprint" "TRIM_3296W1103LF:TRIM_3296W1103LF"
 			(at 99.06 50.8 0)
 			(hide yes)
@@
 			)
 		)
-		(property "Footprint" ""
+		(property "Footprint" "TRIM_3296W1103LF:TRIM_3296W1103LF"
 			(at 110.49 72.39 0)
 			(hide yes)
@@
 			)
 		)
-		(property "Footprint" "Resistor_THT:R_Axial_DIN0207_L6.3mm_D2.5mm_P10.16mm_Horizontal"
+		(property "Footprint" "Resistor_THT:R_Axial_Power_L25.0mm_W9.0mm_P27.94mm"
 			(at 93.599 65.278 0)
 			(hide yes)

Commit message: Add files via upload
Other:
- moved on the sheet: R102
Changed lines of the file:
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@@
 	)
 	(junction
-		(at 120.65 60.96)
+		(at 93.98 60.96)
 		(diameter 0)
 		(color 0 0 0 0)
@@
 	(wire
 		(pts
-			(xy 120.65 60.96) (xy 133.35 60.96)
-		)
-		(stroke
-			(width 0)
-			(type default)
-		)
-	)
-	(wire
-		(pts
-			(xy 85.09 60.96) (xy 88.9 60.96)
+			(xy 88.9 60.96) (xy 93.98 60.96)
+		)
+		(stroke
+			(width 0)
+			(type default)
+		)
+	)
+	(wire
+		(pts
+			(xy 77.47 60.96) (xy 81.28 60.96)
 		)
 		(stroke
@@
 	(wire
 		(pts
-			(xy 96.52 60.96) (xy 120.65 60.96)
+			(xy 93.98 60.96) (xy 133.35 60.96)
 		)
 		(stroke
@@
 	(wire
 		(pts
-			(xy 120.65 64.77) (xy 120.65 60.96)
-		)
-		(stroke
-			(width 0)
-			(type default)
-		)
-	)
-	(wire
-		(pts
 			(xy 46.99 85.09) (xy 46.99 88.9)
 		)
@@
 	(wire
 		(pts
-			(xy 93.98 64.77) (xy 120.65 64.77)
-		)
-		(stroke
-			(width 0)
-			(type default)
-		)
-	)
-	(wire
-		(pts
 			(xy 127 116.84) (xy 130.81 116.84)
 		)
@@
 	(wire
 		(pts
-			(xy 93.98 72.39) (xy 93.98 64.77)
+			(xy 93.98 60.96) (xy 93.98 72.39)
 		)
 		(stroke
@@
 	(hierarchical_label "Trail_Right"
 		(shape input)
-		(at 85.09 60.96 180)
+		(at 77.47 60.96 180)
 		(effects
 			(font
@@
 		(dnp no)
 		(property "Reference" "R103"
-			(at 94.488 50.038 0)
+			(at 95.504 50.8 0)
 			(show_name no)
 			(do_not_autoplace no)
@@
 			(at 96.52 52.07 0)
 			(hide yes)
-			(show_name yes)
+			(show_name no)
 			(do_not_autoplace no)
 			(effects
@@
 		(property "Etiquette" "Pot_Right_Ouvert"
 			(at 92.964 51.562 0)
+			(hide yes)
 			(show_name no)
 			(do_not_autoplace no)
@@
 		(dnp no)
 		(property "Reference" "R104"
-			(at 107.95 71.7549 0)
+			(at 107.188 72.39 0)
 			(show_name no)
 			(do_not_autoplace no)
@@
 		(property "Etiquette" "Pot2_Right_Court"
 			(at 104.394 73.66 0)
+			(hide yes)
 			(show_name no)
 			(do_not_autoplace no)
@@
 	(symbol
 		(lib_id "PCM_SL_Resistors:4.7k")
-		(at 92.71 60.96 0)
+		(at 85.09 60.96 0)
 		(unit 1)
 		(body_style 1)
@@
 		(fields_autoplaced yes)
 		(property "Reference" "R102"
-			(at 92.71 54.61 0)
+			(at 85.09 54.61 0)
 			(show_name no)
 			(do_not_autoplace no)
@@
 		)
 		(property "Value" ".1 ohm"
-			(at 92.71 57.15 0)
+			(at 85.09 57.15 0)
 			(show_name no)
 			(do_not_autoplace no)
@@
 		)
 		(property "Footprint" "Resistor_THT:R_Axial_Power_L25.0mm_W9.0mm_P27.94mm"
-			(at 93.599 65.278 0)
+			(at 85.979 65.278 0)
 			(hide yes)
 			(show_name no)
@@
 		)
 		(property "Datasheet" ""
-			(at 93.218 60.96 0)
+			(at 85.598 60.96 0)
 			(hide yes)
 			(show_name no)
@@
 		)
 		(property "Description" ".1 ohm , 2"
-			(at 92.71 60.96 0)
-			(hide yes)
-			(show_name no)
+			(at 85.09 60.96 0)
+			(hide yes)
+			(show_name no)

Commit message: Add files via upload
Parts:
- removed Q28: IRLZ44N, PCM_Package_TO_SOT_THT_AKL:TO-220-3_Vertical_GDS, symbol PCM_Transistor_MOSFET_AKL:IRLZ44N
- removed R101: 10k, Resistor_THT:R_Axial_DIN0207_L6.3mm_D2.5mm_P10.16mm_Horizontal, symbol PCM_SL_Resistors:10k
- removed R102: .1 ohm, Resistor_THT:R_Axial_Power_L25.0mm_W9.0mm_P27.94mm, symbol PCM_SL_Resistors:4.7k
- added D176: MUR1520G, Package_TO_SOT_THT:TO-220-2_Vertical, symbol Device:D
- added DZ5: 1N5242B, PCM_Diode_THT_AKL:D_DO-35_SOD27_P7.62mm_Horizontal_Zener, symbol PCM_Diode_Zener_AKL:1N5242B
- added Q28: IRF4905PBF, Package_TO_SOT_THT:TO-220-3_Vertical, symbol Transistor_FET:IRF4905
- added Q75: 2N7000, PCM_Package_TO_SOT_THT_AKL:TO-92_Inline_Wide_SGD, symbol PCM_Transistor_MOSFET_AKL:2N7000
- added Q76: 2N3906, PCM_Package_TO_SOT_THT_AKL:TO-92_Inline_Wide_EBC, symbol PCM_Transistor_BJT_AKL:2N3906
- added R101: 10k, Resistor_THT:R_Axial_DIN0207_L6.3mm_D2.5mm_P10.16mm_Horizontal, symbol PCM_SL_Resistors:4.7k
- added R102: 12 Ohm - 1W, Resistor_THT:R_Axial_DIN0414_L11.9mm_D4.5mm_P15.24mm_Horizontal, symbol PCM_SL_Devices:Resistor_5W
- added R274, R276: 1k, Resistor_THT:R_Axial_DIN0207_L6.3mm_D2.5mm_P10.16mm_Horizontal, symbol PCM_SL_Resistors:1k
- added R275, R277, R280: 10k, Resistor_THT:R_Axial_DIN0207_L6.3mm_D2.5mm_P10.16mm_Horizontal, symbol PCM_SL_Resistors:10k
- added R278: 2.7k, Resistor_THT:R_Axial_DIN0207_L6.3mm_D2.5mm_P10.16mm_Horizontal, symbol PCM_SL_Resistors:2.7k
- added R279: 39kΩ, Resistor_THT:R_Axial_DIN0207_L6.3mm_D2.5mm_P10.16mm_Horizontal, symbol PCM_SL_Resistors:10k
- R103: Etiquette Pot_Right_Ouvert -> (none)
- R104: Etiquette Pot2_Right_Court -> (none)
Connections:
- net Btn_Right_Etat: now also Q75.2 (G), R101.2
- net GND: now also R104.1, Q75.1 (S), R101.1, R278.2, R280.2; no longer R104.3
- net Trail_Right: now also D176.1 (K), R102.2, R276.1, R279.2
- net V_Ref: now also R104.3; no longer R104.1
- net Q28.2_Drain: no longer names the net of F4.2
- net Q28.2_Drain: now also DZ5.1 (K), Q28.3 (S), R275.2
- net Right_Trailer_Shunt_Haut renamed Court_Sense_Right
- net Court_Sense_Right: now also R279.1, R280.1; no longer U8.6 (-)
- new net: D176.2 (A), Q28.2 (D), Q76.1 (E), R102.1
- new net: Q76.2 (B), R276.2
- new net: Q76.3 (C), R277.1
- new net: Q75.3 (D), R274.1
- new net: DZ5.2 (A), Q28.1 (G), R274.2, R275.1
- new net I_Present_Right: R277.2, R278.1, U8.6 (-)

Commit message: Add files via upload
Parts:
- removed D176: MUR1520G, Package_TO_SOT_THT:TO-220-2_Vertical, symbol Device:D
- removed D74: SMBJ33A, PCM_Diode_SMD_AKL:D_SMB, symbol PCM_Diode_TVS_AKL:SMBJ33A
- removed DZ5: 1N5242B, PCM_Diode_THT_AKL:D_DO-35_SOD27_P7.62mm_Horizontal_Zener, symbol PCM_Diode_Zener_AKL:1N5242B
- removed Q28: IRF4905PBF, Package_TO_SOT_THT:TO-220-3_Vertical, symbol Transistor_FET:IRF4905
- removed Q75: 2N7000, PCM_Package_TO_SOT_THT_AKL:TO-92_Inline_Wide_SGD, symbol PCM_Transistor_MOSFET_AKL:2N7000
- removed Q76: 2N3906, PCM_Package_TO_SOT_THT_AKL:TO-92_Inline_Wide_EBC, symbol PCM_Transistor_BJT_AKL:2N3906
- removed R101: 10k, Resistor_THT:R_Axial_DIN0207_L6.3mm_D2.5mm_P10.16mm_Horizontal, symbol PCM_SL_Resistors:4.7k
- removed R102: 12 Ohm - 1W, Resistor_THT:R_Axial_DIN0414_L11.9mm_D4.5mm_P15.24mm_Horizontal, symbol PCM_SL_Devices:Resistor_5W
- removed R274, R276: 1k, Resistor_THT:R_Axial_DIN0207_L6.3mm_D2.5mm_P10.16mm_Horizontal, symbol PCM_SL_Resistors:1k
- removed R275, R277, R280: 10k, Resistor_THT:R_Axial_DIN0207_L6.3mm_D2.5mm_P10.16mm_Horizontal, symbol PCM_SL_Resistors:10k
- removed R278: 2.7k, Resistor_THT:R_Axial_DIN0207_L6.3mm_D2.5mm_P10.16mm_Horizontal, symbol PCM_SL_Resistors:2.7k
- removed R279: 39kΩ, Resistor_THT:R_Axial_DIN0207_L6.3mm_D2.5mm_P10.16mm_Horizontal, symbol PCM_SL_Resistors:10k
- added D74: P6KE39A, PCM_Diode_THT_AKL:D_DO-15_P10.16mm_Horizontal_Zener, symbol PCM_Diode_TVS_AKL:P6KE39A
- added Q28: IRLZ44N, PCM_Package_TO_SOT_THT_AKL:TO-220-3_Vertical_GDS, symbol PCM_Transistor_MOSFET_AKL:IRLZ44N
- added R101: 10k, Resistor_THT:R_Axial_DIN0207_L6.3mm_D2.5mm_P10.16mm_Horizontal, symbol PCM_SL_Resistors:10k
- added R102: .1 ohm, Resistor_THT:R_Axial_Power_L25.0mm_W9.0mm_P27.94mm, symbol PCM_SL_Resistors:4.7k
- R103: Etiquette (none) -> Pot_Right_Ouvert
- R104: Etiquette (none) -> Pot2_Right_Court
Connections:
- net I_Present_Right is gone; now on net Right_Trailer_Shunt_Haut: U8.6 (-)
- net Btn_Right_Etat: now also Q28.1 (G), R101.1
- net GND: now also R104.3, D74.2 (A), R101.2; no longer R104.1
- net Trail_Right: now also D74.1 (K), R102.1
- net V_Ref: now also R104.1; no longer R104.3
- net Q28.2_Drain: now reaches F4.2
- net Q28.2_Drain: now also Q28.2 (D)
- net Court_Sense_Right renamed Right_Trailer_Shunt_Haut
- net Right_Trailer_Shunt_Haut: now also Q28.3 (S), R102.2

Commit message: Add files via upload
Parts:
- removed D74: P6KE39A, PCM_Diode_THT_AKL:D_DO-15_P10.16mm_Horizontal_Zener, symbol PCM_Diode_TVS_AKL:P6KE39A
- removed Q28: IRLZ44N, PCM_Package_TO_SOT_THT_AKL:TO-220-3_Vertical_GDS, symbol PCM_Transistor_MOSFET_AKL:IRLZ44N
- removed R101: 10k, Resistor_THT:R_Axial_DIN0207_L6.3mm_D2.5mm_P10.16mm_Horizontal, symbol PCM_SL_Resistors:10k
- removed R102: .1 ohm, Resistor_THT:R_Axial_Power_L25.0mm_W9.0mm_P27.94mm, symbol PCM_SL_Resistors:4.7k
- added D176: MUR1520G, Package_TO_SOT_THT:TO-220-2_Vertical, symbol Device:D
- added D74: SMBJ33A, PCM_Diode_SMD_AKL:D_SMB, symbol PCM_Diode_TVS_AKL:SMBJ33A
- added DZ5: 1N5242B, PCM_Diode_THT_AKL:D_DO-35_SOD27_P7.62mm_Horizontal_Zener, symbol PCM_Diode_Zener_AKL:1N5242B
- added Q28: IRF4905PBF, Package_TO_SOT_THT:TO-220-3_Vertical, symbol Transistor_FET:IRF4905
- added Q75: 2N7000, PCM_Package_TO_SOT_THT_AKL:TO-92_Inline_Wide_SGD, symbol PCM_Transistor_MOSFET_AKL:2N7000
- added Q76: 2N3906, PCM_Package_TO_SOT_THT_AKL:TO-92_Inline_Wide_EBC, symbol PCM_Transistor_BJT_AKL:2N3906
- added R101: 10k, Resistor_THT:R_Axial_DIN0207_L6.3mm_D2.5mm_P10.16mm_Horizontal, symbol PCM_SL_Resistors:4.7k
- added R102: 12 Ohm - 1W, Resistor_THT:R_Axial_DIN0414_L11.9mm_D4.5mm_P15.24mm_Horizontal, symbol PCM_SL_Devices:Resistor_5W
- added R274, R276: 1k, Resistor_THT:R_Axial_DIN0207_L6.3mm_D2.5mm_P10.16mm_Horizontal, symbol PCM_SL_Resistors:1k
- added R275, R277, R280: 10k, Resistor_THT:R_Axial_DIN0207_L6.3mm_D2.5mm_P10.16mm_Horizontal, symbol PCM_SL_Resistors:10k
- added R278: 2.7k, Resistor_THT:R_Axial_DIN0207_L6.3mm_D2.5mm_P10.16mm_Horizontal, symbol PCM_SL_Resistors:2.7k
- added R279: 39kΩ, Resistor_THT:R_Axial_DIN0207_L6.3mm_D2.5mm_P10.16mm_Horizontal, symbol PCM_SL_Resistors:10k
- R103: Etiquette Pot_Right_Ouvert -> (none)
- R104: Etiquette Pot2_Right_Court -> (none)
Connections:
- net Btn_Right_Etat: now also Q75.2 (G), R101.2
- net GND: now also R104.1, D74.2 (A), Q75.1 (S), R101.1, R278.2, R280.2; no longer R104.3
- net Trail_Right: now also D176.1 (K), D74.1 (K), R102.2, R276.1, R279.2
- net V_Ref: now also R104.3; no longer R104.1
- net Q28.2_Drain: no longer names the net of F4.2
- net Q28.2_Drain: now also DZ5.1 (K), Q28.3 (S), R275.2
- net Right_Trailer_Shunt_Haut renamed Court_Sense_Right
- net Court_Sense_Right: now also R279.1, R280.1; no longer U8.6 (-)
- new net: D176.2 (A), Q28.2 (D), Q76.1 (E), R102.1
- new net: Q76.2 (B), R276.2
- new net: Q76.3 (C), R277.1
- new net: Q75.3 (D), R274.1
- new net: DZ5.2 (A), Q28.1 (G), R274.2, R275.1
- new net I_Present_Right: R277.2, R278.1, U8.6 (-)

Commit message: Add files via upload
Parts:
- D74: value SMBJ33A -> P6KE39A; footprint PCM_Diode_SMD_AKL:D_SMB -> PCM_Diode_THT_AKL:D_DO-15_P10.16mm_Horizontal_Zener; symbol PCM_Diode_TVS_AKL:SMBJ33A -> PCM_Diode_TVS_AKL:P6KE39A

Commit message: Add files via upload
Parts:
- F4: value Polyfuse -> MF-R700
- U8: footprint (none) -> Package_DIP:DIP-14_W7.62mm_Socket
Changed lines of the file:
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@@
 			)
 		)
-		(property "Footprint" ""
+		(property "Footprint" "Package_DIP:DIP-14_W7.62mm_Socket"
 			(at 233.68 40.64 0)
 			(hide yes)
@@
 			)
 		)
-		(property "Footprint" ""
+		(property "Footprint" "Package_DIP:DIP-14_W7.62mm_Socket"
 			(at 236.22 128.27 0)
 			(hide yes)
@@
 			)
 		)
-		(property "Footprint" ""
+		(property "Footprint" "Package_DIP:DIP-14_W7.62mm_Socket"
 			(at 233.68 83.82 0)
 			(hide yes)
@@
 			)
 		)
-		(property "Footprint" ""
+		(property "Footprint" "Package_DIP:DIP-14_W7.62mm_Socket"
 			(at 233.68 62.23 0)
 			(hide yes)
@@
 			)
 		)
-		(property "Value" "Polyfuse"
+		(property "Value" "MF-R700"
 			(at 115.57 74.93 90)
 			(show_name no)
@@
 			)
 		)
-		(property "Footprint" ""
+		(property "Footprint" "Package_DIP:DIP-14_W7.62mm_Socket"
 			(at 234.95 104.14 0)
 			(hide yes)

Commit message: Add files via upload
Parts:
- F4: footprint (none) -> PTC_Bourns_MF-R:PTC_Bourns_MF-R_P10.20mm_W24.2mm
Changed lines of the file:
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@@
 			)
 		)
-		(property "Footprint" ""
+		(property "Footprint" "PTC_Bourns_MF-R:PTC_Bourns_MF-R_P10.20mm_W24.2mm"
 			(at 110.49 77.47 0)
 			(hide yes)
