File: Trailer_Tail.kicad_sch (KiCad schematic)
At the start: 22 parts, among them Q12 IRF4905PBF, Q69 2N7000, Q70 2N3906, SW3 SW_SPST, U3 LM339

Commit message: Add files via upload
Parts:
- removed D170: MUR1520G, Package_TO_SOT_THT:TO-220-2_Vertical, symbol Device:D
- removed DZ2: 1N5242B, PCM_Diode_THT_AKL:D_DO-35_SOD27_P7.62mm_Horizontal_Zener, symbol PCM_Diode_Zener_AKL:1N5242B
- removed Q69: 2N7000, PCM_Package_TO_SOT_THT_AKL:TO-92_Inline_Wide_SGD, symbol PCM_Transistor_MOSFET_AKL:2N7000
- removed Q70: 2N3906, PCM_Package_TO_SOT_THT_AKL:TO-92_Inline_Wide_EBC, symbol PCM_Transistor_BJT_AKL:2N3906
- removed R253, R255: 1k, Resistor_THT:R_Axial_DIN0207_L6.3mm_D2.5mm_P10.16mm_Horizontal, symbol PCM_SL_Resistors:1k
- removed R254, R256, R259: 10k, Resistor_THT:R_Axial_DIN0207_L6.3mm_D2.5mm_P10.16mm_Horizontal, symbol PCM_SL_Resistors:10k
- removed R257: 2.7k, Resistor_THT:R_Axial_DIN0207_L6.3mm_D2.5mm_P10.16mm_Horizontal, symbol PCM_SL_Resistors:2.7k
- removed R258: 39kΩ, Resistor_THT:R_Axial_DIN0207_L6.3mm_D2.5mm_P10.16mm_Horizontal, symbol PCM_SL_Resistors:10k
- Q12: value IRF4905PBF -> IRLZ44N; footprint Package_TO_SOT_THT:TO-220-3_Vertical -> PCM_Package_TO_SOT_THT_AKL:TO-220-3_Vertical_GDS; symbol Transistor_FET:IRF4905 -> PCM_Transistor_MOSFET_AKL:IRLZ44N; Etiquette Q_Sortie_Tail_Trail -> (none)
- R31, R32: footprint TRIM_3296W1103LF:TRIM_3296W1103LF -> (none)
- R33: value 12 Ohm - 1W -> .1 Ohm - 2W; footprint Resistor_THT:R_Axial_DIN0414_L11.9mm_D4.5mm_P15.24mm_Horizontal -> Resistor_THT:R_Axial_Power_L25.0mm_W9.0mm_P27.94mm
Connections:
- net Court_Sense_Tail is gone; now on net Trail_Tail: U3.10 (-)
- net I_Present_Tail is gone; now on net Trail_Tail: U3.6 (-)
- net Btn_Tail_Etat: now also Q12.1 (G)
- net at R33.1: now also Q12.3 (S); no longer Q12.2 (D)
- net at F2.2: now also Q12.2 (D); no longer Q12.3 (S)
Other:
- moved on the sheet: D148, F2, R31, R32, R33, R34, R35, R73, SW3, U3A, U3B, U3C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

Commit message: Add files via upload
Parts:
- R31, R32: footprint (none) -> TRIM_3296W1103LF:TRIM_3296W1103LF
Changed lines of the file:
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@@
 			)
 		)
-		(property "Footprint" ""
+		(property "Footprint" "TRIM_3296W1103LF:TRIM_3296W1103LF"
 			(at 83.82 76.2 0)
 			(hide yes)
@@
 			)
 		)
-		(property "Footprint" ""
+		(property "Footprint" "TRIM_3296W1103LF:TRIM_3296W1103LF"
 			(at 83.82 57.15 0)
 			(hide yes)

Commit message: Add files via upload
Parts:
- U3: footprint (none) -> Package_DIP:DIP-14_W7.62mm_Socket
Changed lines of the file:
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@@
 			)
 		)
-		(property "Footprint" ""
+		(property "Footprint" "Package_DIP:DIP-14_W7.62mm_Socket"
 			(at 96.52 80.01 0)
 			(hide yes)
@@
 			)
 		)
-		(property "Footprint" ""
+		(property "Footprint" "Package_DIP:DIP-14_W7.62mm_Socket"
 			(at 97.79 100.33 0)
 			(hide yes)
@@
 			)
 		)
-		(property "Footprint" ""
+		(property "Footprint" "Package_DIP:DIP-14_W7.62mm_Socket"
 			(at 96.52 36.83 0)
 			(hide yes)
@@
 			)
 		)
-		(property "Footprint" ""
+		(property "Footprint" "Package_DIP:DIP-14_W7.62mm_Socket"
 			(at 99.06 124.46 0)
 			(hide yes)
@@
 			)
 		)
-		(property "Footprint" ""
+		(property "Footprint" "Package_DIP:DIP-14_W7.62mm_Socket"
 			(at 96.52 58.42 0)
 			(hide yes)

Commit message: Add files via upload
Parts:
- U3: footprint Package_DIP:DIP-14_W7.62mm_Socket -> (none)
Changed lines of the file:
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@@
 			)
 		)
-		(property "Footprint" "Package_DIP:DIP-14_W7.62mm_Socket"
+		(property "Footprint" ""
 			(at 96.52 80.01 0)
 			(hide yes)
@@
 			)
 		)
-		(property "Footprint" "Package_DIP:DIP-14_W7.62mm_Socket"
+		(property "Footprint" ""
 			(at 97.79 100.33 0)
 			(hide yes)
@@
 			)
 		)
-		(property "Footprint" "Package_DIP:DIP-14_W7.62mm_Socket"
+		(property "Footprint" ""
 			(at 96.52 36.83 0)
 			(hide yes)
@@
 			)
 		)
-		(property "Footprint" "Package_DIP:DIP-14_W7.62mm_Socket"
+		(property "Footprint" ""
 			(at 99.06 124.46 0)
 			(hide yes)
@@
 			)
 		)
-		(property "Footprint" "Package_DIP:DIP-14_W7.62mm_Socket"
+		(property "Footprint" ""
 			(at 96.52 58.42 0)
 			(hide yes)

Commit message: Add files via upload
Parts:
- R31, R32: footprint TRIM_3296W1103LF:TRIM_3296W1103LF -> (none)
Changed lines of the file:
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@@
 			)
 		)
-		(property "Footprint" "TRIM_3296W1103LF:TRIM_3296W1103LF"
+		(property "Footprint" ""
 			(at 83.82 76.2 0)
 			(hide yes)
@@
 			)
 		)
-		(property "Footprint" "TRIM_3296W1103LF:TRIM_3296W1103LF"
+		(property "Footprint" ""
 			(at 83.82 57.15 0)
 			(hide yes)
