File: Trailer_Tail.kicad_sch (KiCad schematic)
At the start: 11 parts, among them Q12 IRLZ44N, SW3 SW_SPST, U3 LM339

Commit message: Add files via upload
Parts:
- removed D25: D_TVS, symbol Device:D_TVS
- added D148: SMBJ33A, PCM_Diode_SMD_AKL:D_SMB, symbol PCM_Diode_TVS_AKL:SMBJ33A
- R34: value 4.7k -> 10k
Connections:
- net Btn_Tail_Etat: now also Q12.1 (G), SW3.2 (B)
- net GND: now also D148.2 (A)
- net Trail_Tail: now also D148.1 (K)
Other:
- moved on the sheet: R34, SW3

Commit message: Add files via upload
Parts:
- added D170: MUR1520G, Package_TO_SOT_THT:TO-220-2_Vertical, symbol Device:D
- added DZ2: 1N5242B, PCM_Diode_THT_AKL:D_DO-35_SOD27_P7.62mm_Horizontal_Zener, symbol PCM_Diode_Zener_AKL:1N5242B
- added Q69: 2N7000, PCM_Package_TO_SOT_THT_AKL:TO-92_Inline_Wide_SGD, symbol PCM_Transistor_MOSFET_AKL:2N7000
- added Q70: 2N3906, PCM_Package_TO_SOT_THT_AKL:TO-92_Inline_Wide_EBC, symbol PCM_Transistor_BJT_AKL:2N3906
- added R253, R255: 1k, Resistor_THT:R_Axial_DIN0207_L6.3mm_D2.5mm_P10.16mm_Horizontal, symbol PCM_SL_Resistors:1k
- added R254, R256, R259: 10k, Resistor_THT:R_Axial_DIN0207_L6.3mm_D2.5mm_P10.16mm_Horizontal, symbol PCM_SL_Resistors:10k
- added R257: 2.7k, Resistor_THT:R_Axial_DIN0207_L6.3mm_D2.5mm_P10.16mm_Horizontal, symbol PCM_SL_Resistors:2.7k
- added R258: 10kΩ, Resistor_THT:R_Axial_DIN0207_L6.3mm_D2.5mm_P10.16mm_Horizontal, symbol PCM_SL_Resistors:10k
- Q12: value IRLZ44N -> IRF4905PBF; footprint PCM_Package_TO_SOT_THT_AKL:TO-220-3_Vertical_GDS -> Package_TO_SOT_THT:TO-220-3_Vertical; symbol PCM_Transistor_MOSFET_AKL:IRLZ44N -> Transistor_FET:IRF4905; Etiquette (none) -> Q_Sortie_Tail_Trail
- R31, R32: footprint (none) -> TRIM_3296W1103LF:TRIM_3296W1103LF
- R33: value .1 Ohm - 2W -> 12 Ohm - 1W; footprint Resistor_THT:R_Axial_Power_L25.0mm_W9.0mm_P27.94mm -> Resistor_THT:R_Axial_DIN0414_L11.9mm_D4.5mm_P15.24mm_Horizontal
Connections:
- net Btn_Tail_Etat: now also Q69.2 (G); no longer Q12.1 (G)
- net GND: now also Q69.1 (S), R257.2, R259.2
- net Trail_Tail: now also D170.1 (K), R255.1, R258.2; no longer U3.10 (-), U3.6 (-)
- net at R33.1: now also Q12.2 (D), D170.2 (A), Q70.1 (E); no longer Q12.3 (S)
- net at F2.2: now also Q12.3 (S), DZ2.1 (K), R254.2; no longer Q12.2 (D)
- new net: Q69.3 (D), R253.1
- new net: DZ2.2 (A), Q12.1 (G), R253.2, R254.1
- new net: Q70.3 (C), R256.1
- new net: Q70.2 (B), R255.2
- new net Court_Sense_Tail: R258.1, R259.1, U3.10 (-)
- new net I_Present_Tail: R256.2, R257.1, U3.6 (-)
Other:
- moved on the sheet: D148, F2, R31, R32, R33, R34, R35, R73, SW3, U3A, U3B, U3C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

Commit message: Add files via upload
Parts:
- R258: value 10kΩ -> 39kΩ
Changed lines of the file:
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@@
 			)
 		)
-		(property "Value" "10kΩ"
+		(property "Value" "39kΩ"
 			(at 198.12 45.72 0)
 			(show_name no)
@@
 			)
 		)
-		(property "Description" "10kΩ, 1/4W Resistor"
+		(property "Description" "39kΩ, 1/4W Resistor"
 			(at 198.12 48.26 0)
 			(hide yes)

Commit message: Add files via upload
Parts:
- D148: value SMBJ33A -> P6KE39A; footprint PCM_Diode_SMD_AKL:D_SMB -> PCM_Diode_THT_AKL:D_DO-15_P10.16mm_Horizontal_Zener; symbol PCM_Diode_TVS_AKL:SMBJ33A -> PCM_Diode_TVS_AKL:P6KE39A
Changed lines of the file:
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@@
 	)
 	(symbol
-		(lib_id "PCM_Diode_TVS_AKL:SMBJ33A")
+		(lib_id "PCM_Diode_TVS_AKL:P6KE39A")
 		(at 199.39 109.22 0)
 		(unit 1)
@@
 			)
 		)
-		(property "Value" "SMBJ33A"
+		(property "Value" "P6KE39A"
 			(at 199.39 105.41 0)
 			(show_name no)
@@
 			)
 		)
-		(property "Footprint" "PCM_Diode_SMD_AKL:D_SMB"
+		(property "Footprint" "PCM_Diode_THT_AKL:D_DO-15_P10.16mm_Horizontal_Zener"
 			(at 199.39 109.22 0)
 			(hide yes)
@@
 			)
 		)
-		(property "Datasheet" "https://www.tme.eu/Document/0b6222bec7e12d83185b51d73cb6a54d/SMBJ_ser.pdf"
+		(property "Datasheet" "https://www.tme.eu/Document/6b488a936123e1f9ccf03f4f9186b150/P6KE_ser.pdf"
 			(at 199.39 109.22 0)
 			(hide yes)
@@
 			)
 		)
-		(property "Description" "SMB Unidirectional TVS diode, 33V, 600W, Alternate KiCAD Library"
+		(property "Description" "DO-15 Unidirectional TVS diode, 39V, 600W, Alternate KiCAD Library"
 			(at 199.39 109.22 0)
 			(hide yes)

Commit message: Add files via upload
Parts:
- F2: value Polyfuse -> MF-R700
- U3: footprint (none) -> Package_DIP:DIP-14_W7.62mm_Socket
Changed lines of the file:
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@@
 			)
 		)
-		(property "Footprint" ""
+		(property "Footprint" "Package_DIP:DIP-14_W7.62mm_Socket"
 			(at 233.68 83.82 0)
 			(hide yes)
@@
 			)
 		)
-		(property "Footprint" ""
+		(property "Footprint" "Package_DIP:DIP-14_W7.62mm_Socket"
 			(at 234.95 104.14 0)
 			(hide yes)
@@
 			)
 		)
-		(property "Value" "Polyfuse"
+		(property "Value" "MF-R700"
 			(at 115.57 74.93 90)
 			(show_name no)
@@
 			)
 		)
-		(property "Footprint" ""
+		(property "Footprint" "Package_DIP:DIP-14_W7.62mm_Socket"
 			(at 233.68 40.64 0)
 			(hide yes)
@@
 			)
 		)
-		(property "Footprint" ""
+		(property "Footprint" "Package_DIP:DIP-14_W7.62mm_Socket"
 			(at 236.22 128.27 0)
 			(hide yes)
@@
 			)
 		)
-		(property "Footprint" ""
+		(property "Footprint" "Package_DIP:DIP-14_W7.62mm_Socket"
 			(at 233.68 62.23 0)
 			(hide yes)

Commit message: Add files via upload
Parts:
- F2: footprint (none) -> PTC_Bourns_MF-R:PTC_Bourns_MF-R_P10.20mm_W24.2mm
Changed lines of the file:
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@@
 			)
 		)
-		(property "Footprint" ""
+		(property "Footprint" "PTC_Bourns_MF-R:PTC_Bourns_MF-R_P10.20mm_W24.2mm"
 			(at 110.49 77.47 0)
 			(hide yes)

Commit message: Add files via upload
Parts:
- SW3: value SW_SPST -> SW_SPDT; symbol Switch:SW_SPST -> Switch:SW_SPDT
Connections:
- net GND: now also SW3.3 (C)
Other:
- moved on the sheet: R34
Changed lines of the file:
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@@
 	)
 	(junction
-		(at 97.79 63.5)
+		(at 68.58 76.2)
 		(diameter 0)
 		(color 0 0 0 0)
 	)
 	(junction
-		(at 245.11 64.77)
+		(at 97.79 63.5)
 		(diameter 0)
 		(color 0 0 0 0)
 	)
 	(junction
-		(at 68.58 76.2)
+		(at 245.11 64.77)
 		(diameter 0)
 		(color 0 0 0 0)
@@
 	(wire
 		(pts
-			(xy 52.07 63.5) (xy 55.88 63.5)
+			(xy 50.8 60.96) (xy 55.88 60.96)
 		)
 		(stroke
@@
 	(wire
 		(pts
-			(xy 57.15 76.2) (xy 68.58 76.2)
+			(xy 58.42 76.2) (xy 68.58 76.2)
 		)
 		(stroke
@@
 	(wire
 		(pts
+			(xy 50.8 66.04) (xy 55.88 66.04)
+		)
+		(stroke
+			(width 0)
+			(type default)
+		)
+	)
+	(wire
+		(pts
 			(xy 176.53 87.63) (xy 176.53 91.44)
 		)
@@
 	(global_label "V_Ref"
 		(shape input)
-		(at 52.07 63.5 180)
+		(at 50.8 60.96 180)
 		(fields_autoplaced yes)
 		(effects
@@
 		)
 		(property "Intersheetrefs" "${INTERSHEET_REFS}"
-			(at 43.9443 63.5 0)
+			(at 42.6743 60.96 0)
 			(hide yes)
 			(show_name no)
@@
 	(global_label "GND"
 		(shape input)
+		(at 50.8 66.04 180)
+		(fields_autoplaced yes)
+		(effects
+			(font
+				(size 1.27 1.27)
+			)
+			(justify right)
+		)
+		(property "Intersheetrefs" "${INTERSHEET_REFS}"
+			(at 43.9443 66.04 0)
+			(hide yes)
+			(show_name no)
+			(do_not_autoplace no)
+			(effects
+				(font
+					(size 1.27 1.27)
+				)
+				(justify right)
+			)
+		)
+	)
+	(global_label "GND"
+		(shape input)
 		(at 191.77 109.22 180)
 		(fields_autoplaced yes)
@@
 	(global_label "GND"
 		(shape input)
-		(at 49.53 76.2 180)
+		(at 50.8 76.2 180)
 		(fields_autoplaced yes)
 		(effects
@@
 		)
 		(property "Intersheetrefs" "${INTERSHEET_REFS}"
-			(at 42.6743 76.2 0)
+			(at 43.9443 76.2 0)
 			(hide yes)
 			(show_name no)
@@
 	(symbol
 		(lib_id "PCM_SL_Resistors:4.7k")
-		(at 53.34 76.2 0)
+		(at 54.61 76.2 0)
 		(unit 1)
 		(body_style 1)
@@
 		(fields_autoplaced yes)
 		(property "Reference" "R34"
-			(at 53.34 69.85 0)
+			(at 54.61 69.85 0)
 			(show_name no)
 			(do_not_autoplace no)
@@
 		)
 		(property "Value" "10k"
-			(at 53.34 72.39 0)
+			(at 54.61 72.39 0)
 			(show_name no)
 			(do_not_autoplace no)
@@
 		)
 		(property "Footprint" "Resistor_THT:R_Axial_DIN0207_L6.3mm_D2.5mm_P10.16mm_Horizontal"
-			(at 54.229 80.518 0)
+			(at 55.499 80.518 0)
 			(hide yes)
 			(show_name no)
@@
 		)
 		(property "Datasheet" ""
-			(at 53.848 76.2 0)
+			(at 55.118 76.2 0)
 			(hide yes)
 			(show_name no)
@@
 		)
 		(property "Description" "10kΩ, 1/4W Resistor"
-			(at 53.34 76.2 0)
+			(at 54.61 76.2 0)
 			(hide yes)
 			(show_name no)
@@
 	)
 	(symbol
-		(lib_id "Switch:SW_SPST")
+		(lib_id "Switch:SW_SPDT")
 		(at 60.96 63.5 0)
+		(mirror y)
 		(unit 1)
 		(body_style 1)
@@
 		(in_pos_files yes)
 		(dnp no)
-		(fields_autoplaced yes)
 		(property "Reference" "SW3"
-			(at 60.96 57.15 0)
+			(at 60.96 56.134 0)
 			(show_name no)
 			(do_not_autoplace no)
@@
 			)
 		)
-		(property "Value" "SW_SPST"
-			(at 60.96 59.69 0)
+		(property "Value" "SW_SPDT"
+			(at 60.96 57.912 0)
 			(show_name no)
 			(do_not_autoplace no)
@@
 			)
 		)
-		(property "Description" "Single Pole Single Throw (SPST) switch"
+		(property "Description" "Switch, single pole double throw"
 			(at 60.96 63.5 0)
 			(hide yes)
@@
 		(pin "2"
 		)
+		(pin "3"
+		)
 		(instances

Commit message: Add files via upload
Parts:
- R253, R255: value 1k -> 1kΩ
- R254, R256, R259, R34: value 10k -> 10kΩ
- R257: value 2.7k -> 2.7kΩ
- R35, R73: value 4.7k -> 4.7kΩ
Changed lines of the file:
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@@
 			)
 		)
-		(property "Value" "1k"
+		(property "Value" "1kΩ"
 			(at 91.44 59.69 0)
 			(show_name no)
@@
 			)
 		)
-		(property "Value" "10k"
+		(property "Value" "10kΩ"
 			(at 182.88 88.9 0)
 			(show_name no)
@@
 			)
 		)
-		(property "Value" "1k"
+		(property "Value" "1kΩ"
 			(at 163.83 78.74 0)
 			(show_name no)
@@
 			)
 		)
-		(property "Value" "2.7k"
+		(property "Value" "2.7kΩ"
 			(at 135.89 90.17 0)
 			(show_name no)
@@
 			)
 		)
-		(property "Value" "4.7k"
+		(property "Value" "4.7kΩ"
 			(at 250.19 82.55 0)
 			(show_name no)
@@
 			)
 		)
-		(property "Value" "10k"
+		(property "Value" "10kΩ"
 			(at 152.4 40.64 0)
 			(show_name no)
@@
 			)
 		)
-		(property "Value" "10k"
+		(property "Value" "10kΩ"
 			(at 54.61 72.39 0)
 			(show_name no)
@@
 			)
 		)
-		(property "Value" "4.7k"
+		(property "Value" "4.7kΩ"
 			(at 250.19 60.96 0)
 			(show_name no)
@@
 			)
 		)
-		(property "Value" "10k"
+		(property "Value" "10kΩ"
 			(at 102.87 71.12 0)
 			(show_name no)
