File: Canal_Right.kicad_sch (KiCad schematic)
At the start: 0 parts

Commit message: Add files via upload
Other:
- sheet Vehicule_Right ports: added none; removed Injection_Right_Fault
Changed lines of the file:
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@@
 	(wire
 		(pts
-			(xy 85.09 60.96) (xy 85.09 50.8)
-		)
-		(stroke
-			(width 0)
-			(type default)
-		)
-	)
-	(wire
-		(pts
-			(xy 63.5 71.12) (xy 92.71 71.12)
-		)
-		(stroke
-			(width 0)
-			(type default)
-		)
-	)
-	(wire
-		(pts
-			(xy 92.71 59.69) (xy 95.25 59.69)
+			(xy 63.5 71.12) (xy 95.25 71.12)
 		)
 		(stroke
@@
 	(wire
 		(pts
-			(xy 85.09 50.8) (xy 95.25 50.8)
-		)
-		(stroke
-			(width 0)
-			(type default)
-		)
-	)
-	(wire
-		(pts
-			(xy 63.5 36.83) (xy 88.9 36.83)
-		)
-		(stroke
-			(width 0)
-			(type default)
-		)
-	)
-	(wire
-		(pts
-			(xy 63.5 60.96) (xy 85.09 60.96)
-		)
-		(stroke
-			(width 0)
-			(type default)
-		)
-	)
-	(wire
-		(pts
-			(xy 88.9 36.83) (xy 88.9 41.91)
-		)
-		(stroke
-			(width 0)
-			(type default)
-		)
-	)
-	(wire
-		(pts
-			(xy 85.09 45.72) (xy 95.25 45.72)
+			(xy 63.5 36.83) (xy 95.25 36.83)
+		)
+		(stroke
+			(width 0)
+			(type default)
+		)
+	)
+	(wire
+		(pts
+			(xy 63.5 60.96) (xy 95.25 60.96)
 		)
 		(stroke
@@
 	(wire
 		(pts
-			(xy 85.09 40.64) (xy 85.09 45.72)
-		)
-		(stroke
-			(width 0)
-			(type default)
-		)
-	)
-	(wire
-		(pts
-			(xy 63.5 33.655) (xy 68.58 33.655)
-		)
-		(stroke
-			(width 0)
-			(type default)
-		)
-	)
-	(wire
-		(pts
-			(xy 63.5 66.04) (xy 88.9 66.04)
-		)
-		(stroke
-			(width 0)
-			(type default)
-		)
-	)
-	(wire
-		(pts
-			(xy 88.9 41.91) (xy 95.25 41.91)
-		)
-		(stroke
-			(width 0)
-			(type default)
-		)
-	)
-	(wire
-		(pts
-			(xy 92.71 71.12) (xy 92.71 59.69)
-		)
-		(stroke
-			(width 0)
-			(type default)
-		)
-	)
-	(wire
-		(pts
-			(xy 63.5 40.64) (xy 85.09 40.64)
-		)
-		(stroke
-			(width 0)
-			(type default)
-		)
-	)
-	(wire
-		(pts
-			(xy 88.9 54.61) (xy 95.25 54.61)
-		)
-		(stroke
-			(width 0)
-			(type default)
-		)
-	)
-	(wire
-		(pts
-			(xy 88.9 66.04) (xy 88.9 54.61)
-		)
-		(stroke
-			(width 0)
-			(type default)
-		)
-	)
-	(hierarchical_label "Injection_Right_Fault"
-		(shape input)
-		(at 68.58 33.655 0)
-		(effects
-			(font
-				(size 1.27 1.27)
-			)
-			(justify left)
+			(xy 63.5 66.04) (xy 95.25 66.04)
+		)
+		(stroke
+			(width 0)
+			(type default)
+		)
+	)
+	(wire
+		(pts
+			(xy 63.5 40.64) (xy 95.25 40.64)
+		)
+		(stroke
+			(width 0)
+			(type default)
 		)
 	)
@@
 	)
 	(sheet
-		(at 95.25 39.37)
-		(size 46.99 35.56)
+		(at 95.25 30.48)
+		(size 46.99 44.45)
 		(exclude_from_sim no)
 		(in_bom yes)
@@
 		)
 		(property "Sheetname" "Bloc_Test_Right"
-			(at 95.25 38.9124 0)
+			(at 95.25 30.0224 0)
 			(show_name no)
 			(do_not_autoplace no)
@@
 		)
 		(pin "Btn_Right_Etat" input
-			(at 95.25 59.69 180)
+			(at 95.25 71.12 180)
 			(effects
 				(font
@@
 		)
 		(pin "Court_Right_Trailer" input
-			(at 95.25 50.8 180)
+			(at 95.25 60.96 180)
 			(effects
 				(font
@@
 		)
 		(pin "Court_Right_Vehic" input
-			(at 95.25 41.91 180)
+			(at 95.25 36.83 180)
 			(effects
 				(font
@@
 		)
 		(pin "Ouvert_Right_Trailer" input
-			(at 95.25 54.61 180)
+			(at 95.25 66.04 180)
 			(effects
 				(font
@@
 		)
 		(pin "Ouvert_Right_Vehic" input
-			(at 95.25 45.72 180)
+			(at 95.25 40.64 180)
 			(effects
 				(font
@@
 			(effects
 				(font
-					(size 1.016 1.016)
-				)
-				(justify right)
-			)
-		)
-		(pin "Injection_Right_Fault" input
-			(at 63.5 33.655 0)
-			(effects
-				(font
