File: Vehicule_Brake.kicad_sch (KiCad schematic)
At the start: 0 parts

Commit message: Add files via upload
Parts:
- added OC11, OC12: PC817, PCM_Package_DIP_AKL:DIP-4_W7.62mm_LongPads, symbol PCM_Optocoupler_AKL:PC817
- added Q51: IRLZ44N, PCM_Package_TO_SOT_THT_AKL:TO-220-3_Vertical_GDS, symbol PCM_Transistor_MOSFET_AKL:IRLZ44N
- added R188: 3 Ohm - 5W, Resistor_THT:R_Axial_Power_L25.0mm_W9.0mm_P27.94mm, symbol PCM_SL_Devices:Resistor_5W
- added R189: .05R Shunt, Resistor_THT:R_Axial_Power_L25.0mm_W9.0mm_P27.94mm, symbol PCM_SL_Devices:Resistor_5W
- added R190, R191, R192: 4.7k, Resistor_THT:R_Axial_DIN0207_L6.3mm_D2.5mm_P10.16mm_Horizontal, symbol PCM_SL_Resistors:4.7k
- added R193, R194: 1k, Resistor_THT:R_Axial_DIN0207_L6.3mm_D2.5mm_P10.16mm_Horizontal, symbol PCM_SL_Resistors:4.7k
- added R195: 100k, Resistor_THT:R_Axial_DIN0207_L6.3mm_D2.5mm_P10.16mm_Horizontal, symbol PCM_SL_Resistors:100k
- added R196: 10k, Resistor_THT:R_Axial_DIN0207_L6.3mm_D2.5mm_P10.16mm_Horizontal, symbol PCM_SL_Resistors:10k
- added R197, R198, R199: Potentiometer, symbol Simulation_SPICE:Potentiometer
- added U13: LM339, symbol Comparator:LM339
Connections:
- new net: R190.1, U13.2
- new net: OC11.1, R193.2
- new net: OC12.1, R194.2
- new net: R188.2, R189.1, U13.11 (+), U13.6 (-)
- new net: R191.1, U13.1
- new net: R195.2, R196.1, U13.5 (+)
- new net: R192.1, U13.13
- new net Court_Brake_Vehic: OC11.4
- new net GND: OC11.3, OC12.3, R189.2, R196.2, R197.3, R198.3, R199.3, U13.12 (V-), U13.9 (+)
- new net Ouvert_Brake_Vehic: OC12.4
- new net Q51_Source: Q51.3 (S), R188.1
- new net Seuil_Court_Brake: R199.2, U13.10 (-)
- new net Seuil_Injection_Brake: R197.2, U13.4 (-)
- new net Seuil_Ouvert_Brake: R198.2, U13.7 (+)
- new net V_Ref: OC11.2, OC12.2, Q51.1 (G), R190.2, R191.2, R192.2, R193.1, R194.1, R197.1, R198.1, R199.1, U13.3 (V+), U13.8 (-)
- new net Veh_Brake: Q51.2 (D), R195.1
- no-connect marks 0 -> 1
Other:
- note added: "Brake_Vehic_Shunt_Haut"
- note added: "Court-circuit"
- note added: "Injection"
- note added: "Non_Utilisé"
- note added: "Ouvvert"

Commit message: Add files via upload
Parts:
- added D147: LED_1.8mm_Amber, PCM_LED_THT_AKL:LED_D1.8mm_W3.3mm_H2.4mm, symbol PCM_LED_AKL:LED_1.8mm_Amber
- added Q53, Q54: 2N7000, Package_TO_SOT_THT:TO-92_Inline, symbol Transistor_FET:2N7000
- added R206: 100k, Resistor_THT:R_Axial_DIN0207_L6.3mm_D2.5mm_P10.16mm_Horizontal, symbol PCM_SL_Resistors:100k
- added R207: 330ohm, Resistor_THT:R_Axial_DIN0207_L6.3mm_D2.5mm_P10.16mm_Horizontal, symbol PCM_SL_Resistors:100k
- added TH1: SW_SPST_Temperature_NC, symbol Switch:SW_SPST_Temperature_NC
Connections:
- net GND: now also Q53.1 (S), Q54.1 (S), TH1.2
- net V_Ref: now also D147.2 (A), Q54.3 (D), R206.1
- new net: Q53.3 (D), R207.1
- new net: D147.1 (K), R207.2
- new net Surchauffe_Brake: Q53.2 (G), Q54.2 (G), R206.2, TH1.1
Other:
- note added: "Protection Thermique (Brake applied)"
- moved on the sheet: OC11, OC12, Q51, R188, R189, R190, R191, R192, R193, R194, R195, R196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

Commit message: Add files via upload
Connections:
- net V_Ref: no longer Q51.1 (G), Q54.3 (D)
- net Veh_Brake_Inject_Cmd: now reaches R190.1, U13.2
- net Veh_Brake_Inject_Cmd: now also Q51.1 (G), Q54.3 (D)
Other:
- moved on the sheet: D147, OC11, OC12, Q51, Q53, Q54, R188, R189, R190, R191, R192, R193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

Commit message: Add files via upload
Parts:
- R188: value 3 Ohm - 5W -> 12 Ohm - 25W; footprint Resistor_THT:R_Axial_Power_L25.0mm_W9.0mm_P27.94mm -> TerminalBlock_Phoenix:TerminalBlock_Phoenix_PT-1,5-2-3.5-H_1x02_P3.50mm_Horizontal
- R189: value .05R Shunt -> 0.2 Ohm Shunt
- R197, R198, R199: footprint (none) -> TRIM_3296W1103LF:TRIM_3296W1103LF
Connections:
- net Veh_Brake_Inject_Cmd renamed Injection_Brake_Fault
Other:
- note removed: "Court-circuit"
- note removed: "Injection"
- note removed: "Non_Utilisé"
- note removed: "Ouvvert"
Changed lines of the file:
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@@
 		)
 	)
-	(text "Ouvvert\n"
-		(exclude_from_sim no)
-		(at 83.82 67.31 0)
-		(effects
-			(font
-				(size 0.762 0.762)
-			)
-		)
-	)
-	(text "Court-circuit\n"
-		(exclude_from_sim no)
-		(at 83.82 83.82 0)
-		(effects
-			(font
-				(size 0.762 0.762)
-			)
-		)
-	)
-	(text "Injection"
-		(exclude_from_sim no)
-		(at 80.01 49.53 0)
-		(effects
-			(font
-				(size 0.762 0.762)
-			)
-		)
-	)
-	(text "Non_Utilisé"
-		(exclude_from_sim no)
-		(at 82.55 99.06 0)
-		(effects
-			(font
-				(size 0.762 0.762)
-			)
-		)
-	)
 	(text "Brake_Vehic_Shunt_Haut"
 		(exclude_from_sim no)
@@
 	)
 	(junction
+		(at 99.695 40.64)
+		(diameter 0)
+		(color 0 0 0 0)
+	)
+	(junction
 		(at 135.89 33.02)
 		(diameter 0)
@@
 	(wire
 		(pts
+			(xy 99.695 33.02) (xy 99.695 40.64)
+		)
+		(stroke
+			(width 0)
+			(type default)
+		)
+	)
+	(wire
+		(pts
 			(xy 212.09 158.75) (xy 212.09 162.56)
 		)
@@
 	(wire
 		(pts
+			(xy 95.25 33.02) (xy 99.695 33.02)
+		)
+		(stroke
+			(width 0)
+			(type default)
+		)
+	)
+	(wire
+		(pts
 			(xy 43.18 127) (xy 48.26 127)
 		)
@@
 	(wire
 		(pts
+			(xy 99.695 40.64) (xy 90.17 40.64)
+		)
+		(stroke
+			(width 0)
+			(type default)
+		)
+	)
+	(wire
+		(pts
 			(xy 48.26 127) (xy 48.26 116.84)
 		)
@@
 	(wire
 		(pts
-			(xy 115.57 40.64) (xy 90.17 40.64)
+			(xy 115.57 40.64) (xy 99.695 40.64)
 		)
 		(stroke
@@
 		)
 	)
-	(label "Veh_Brake_Inject_Cmd"
-		(at 90.17 40.64 180)
-		(effects
-			(font
-				(size 1.016 1.016)
-			)
-			(justify right bottom)
-		)
-	)
 	(label "Surchauffe_Brake"
 		(at 152.4 153.67 180)
@@
 		)
 	)
-	(label "Veh_Brake_Inject_Cmd"
+	(label "Injection_Brake_Fault"
 		(at 210.82 147.32 180)
 		(effects
@@
 		)
 	)
+	(hierarchical_label "Injection_Brake_Fault"
+		(shape input)
+		(at 95.25 33.02 180)
+		(effects
+			(font
+				(size 1.27 1.27)
+			)
+			(justify right)
+		)
+	)
 	(hierarchical_label "Veh_Brake"
 		(shape input)
@@
 			)
 		)
-		(property "Value" "3 Ohm - 5W"
+		(property "Value" "12 Ohm - 25W"
 			(at 39.37 113.03 0)
 			(show_name no)
@@
 			)
 		)
-		(property "Footprint" "Resistor_THT:R_Axial_Power_L25.0mm_W9.0mm_P27.94mm"
+		(property "Footprint" "TerminalBlock_Phoenix:TerminalBlock_Phoenix_PT-1,5-2-3.5-H_1x02_P3.50mm_Horizontal"
 			(at 40.259 121.158 0)
 			(hide yes)
@@
 			)
 		)
-		(property "Description" "5W Resistor"
+		(property "Description" "25W Resistor"
 			(at 39.37 116.84 0)
 			(hide yes)
@@
 			)
 		)
-		(property "Footprint" ""
+		(property "Footprint" "TRIM_3296W1103LF:TRIM_3296W1103LF"
 			(at 176.53 49.53 0)
 			(hide yes)
@@
 			)
 		)
-		(property "Footprint" ""
+		(property "Footprint" "TRIM_3296W1103LF:TRIM_3296W1103LF"
 			(at 176.53 31.75 0)
 			(hide yes)
@@
 			)
 		)
-		(property "Value" ".05R Shunt"
+		(property "Value" "0.2 Ohm Shunt"
 			(at 39.37 123.19 0)
 			(show_name no)
@@
 			)
 		)
-		(property "Footprint" ""
+		(property "Footprint" "TRIM_3296W1103LF:TRIM_3296W1103LF"
 			(at 176.53 68.58 0)
 			(hide yes)

Commit message: Add files via upload
Connections:
- net V_Ref: no longer OC11.2, OC12.2
- net Veh_Brake: now also R188.1; no longer Q51.2 (D)
- net Brake_Vehic_Shunt_Haut: now reaches R189.1, U13.11 (+), U13.6 (-)
- net Brake_Vehic_Shunt_Haut: now also Q51.3 (S); no longer R188.2
- net Opto_Ouvert_Brake: now reaches R191.1, U13.1
- net Opto_Ouvert_Brake: now also OC12.2
- net Opto_Court_Brake: now reaches R192.1, U13.13
- net Opto_Court_Brake: now also OC11.2
- removed net Q51_Source: Q51.3 (S), R188.1
- new net Q51_Drain: Q51.2 (D), R188.2
Other:
- note removed: "Brake_Vehic_Shunt_Haut"
- moved on the sheet: R188, R195, R196

Commit message: Add files via upload
Parts:
- U13: footprint (none) -> Package_DIP:DIP-14_W7.62mm_Socket
Changed lines of the file:
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@@
 			)
 		)
-		(property "Footprint" ""
+		(property "Footprint" "Package_DIP:DIP-14_W7.62mm_Socket"
 			(at 78.74 69.85 0)
 			(hide yes)
@@
 			)
 		)
-		(property "Footprint" ""
+		(property "Footprint" "Package_DIP:DIP-14_W7.62mm_Socket"
 			(at 78.74 52.07 0)
 			(hide yes)
@@
 			)
 		)
-		(property "Footprint" ""
+		(property "Footprint" "Package_DIP:DIP-14_W7.62mm_Socket"
 			(at 78.74 101.6 0)
 			(hide yes)
@@
 			)
 		)
-		(property "Footprint" ""
+		(property "Footprint" "Package_DIP:DIP-14_W7.62mm_Socket"
 			(at 78.74 86.36 0)
 			(hide yes)
@@
 			)
 		)
-		(property "Footprint" ""
+		(property "Footprint" "Package_DIP:DIP-14_W7.62mm_Socket"
 			(at 76.2 119.38 0)
 			(hide yes)

Commit message: Add files via upload
Parts:
- TH1: footprint (none) -> TerminalBlock_Phoenix:TerminalBlock_Phoenix_PT-1,5-2-3.5-H_1x02_P3.50mm_Horizontal
Changed lines of the file:
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@@
 			)
 		)
-		(property "Footprint" ""
+		(property "Footprint" "TerminalBlock_Phoenix:TerminalBlock_Phoenix_PT-1,5-2-3.5-H_1x02_P3.50mm_Horizontal"
 			(at 116.84 156.21 0)
 			(hide yes)

Commit message: Add files via upload
Changed lines of the file:
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@@
+		)
+	)
+	(label "Injection_Brake_Fault"
+		(at 95.25 33.02 180)
+		(effects
+			(font
+				(size 1.27 1.27)
+			)
+			(justify right bottom)
 		)
 	)
@@
 		)
 	)
-	(hierarchical_label "Injection_Brake_Fault"
-		(shape input)
-		(at 95.25 33.02 180)
-		(effects
-			(font
-				(size 1.27 1.27)
-			)
-			(justify right)
-		)
-	)
