File: Bloc_Test_Aux.kicad_sch (KiCad schematic)
At the start: 45 parts, among them Q45 2N7000, Q46 2N7000, Q47 2N7000, Q48 2N7000, Q49 2N7000, Q50 2N7000

Commit message: Add files via upload
Parts:
- R174, R177, R181: value 4.7k -> 470kΩ
- R175, R178: value 4.7k -> 100kΩ
Connections:
- net GND: no longer R184.2
- net V_Ref: now also R184.2
Changed lines of the file:
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@@
 		)
 	)
-	(global_label "GND"
+	(global_label "V_Ref"
 		(shape input)
 		(at 242.57 58.42 0)
@@
 		)
 		(property "Intersheetrefs" "${INTERSHEET_REFS}"
-			(at 249.4257 58.42 0)
+			(at 250.6957 58.42 0)
 			(hide yes)
 			(show_name no)
@@
 			)
 		)
-		(property "Value" "4.7k"
+		(property "Value" "100kΩ"
 			(at 48.26 97.79 0)
 			(show_name no)
@@
 			)
 		)
-		(property "Value" "4.7k"
+		(property "Value" "470kΩ"
 			(at 148.59 152.4 0)
 			(show_name no)
@@
 			)
 		)
-		(property "Value" "4.7k"
+		(property "Value" "470kΩ"
 			(at 40.64 151.13 0)
 			(show_name no)
@@
 			)
 		)
-		(property "Value" "4.7k"
+		(property "Value" "100kΩ"
 			(at 87.63 97.79 0)
 			(show_name no)
@@
 			)
 		)
-		(property "Value" "4.7k"
+		(property "Value" "470kΩ"
 			(at 86.36 156.21 0)
 			(show_name no)

Commit message: Add files via upload
Parts:
- R173, R176, R179, R180, R182, R183, R184: value 4.7k -> 4.7kΩ
- R185, R186, R187: value 330ohm -> 330Ω
Changed lines of the file:
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@@
 			)
 		)
-		(property "Value" "330ohm"
+		(property "Value" "330Ω"
 			(at 234.95 122.174 0)
 			(show_name no)
@@
 			)
 		)
-		(property "Value" "330ohm"
+		(property "Value" "330Ω"
 			(at 234.95 100.584 0)
 			(show_name no)
@@
 			)
 		)
-		(property "Value" "4.7k"
+		(property "Value" "4.7kΩ"
 			(at 110.49 55.88 0)
 			(show_name no)
@@
 			)
 		)
-		(property "Value" "4.7k"
+		(property "Value" "4.7kΩ"
 			(at 205.74 43.18 0)
 			(show_name no)
@@
 			)
 		)
-		(property "Value" "330ohm"
+		(property "Value" "330Ω"
 			(at 234.95 142.494 0)
 			(show_name no)
@@
 			)
 		)
-		(property "Value" "4.7k"
+		(property "Value" "4.7kΩ"
 			(at 152.4 58.42 0)
 			(show_name no)
@@
 			)
 		)
-		(property "Value" "4.7k"
+		(property "Value" "4.7kΩ"
 			(at 31.75 53.34 0)
 			(show_name no)
@@
 			)
 		)
-		(property "Value" "4.7k"
+		(property "Value" "4.7kΩ"
 			(at 69.85 53.34 0)
 			(show_name no)
@@
 			)
 		)
-		(property "Value" "4.7k"
+		(property "Value" "4.7kΩ"
 			(at 95.25 176.53 0)
 			(show_name no)
@@
 			)
 		)
-		(property "Value" "4.7k"
+		(property "Value" "4.7kΩ"
 			(at 233.68 55.88 0)
 			(show_name no)
