File: Bloc_Test_Tail.kicad_sch (KiCad schematic)
At the start: 44 parts, among them Q10 2N7000, Q5 2N7000, Q6 2N7000, Q7 2N7000, Q8 2N7000, Q9 2N7000

Commit message: Add files via upload
Connections:
- net Court_V_Actif: now also D7.2 (A)
- net Mode_Vehicule: no longer D3.1 (K)
- new net Court_Tail_Vehic: D3.1 (K)
Changed lines of the file:
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@@
-	(wire
-		(pts
-			(xy 67.31 26.67) (xy 67.31 36.83)
-		)
-		(stroke
-			(width 0)
-			(type default)
-		)
-	)
 	(wire
 		(pts
@@
 	)
 	(label "Court_V_Actif"
-		(at 39.37 154.94 180)
-		(effects
-			(font
+		(at 62.23 158.75 180)
+		(effects
+			(font

Commit message: Add files via upload
Connections:
- net Bleu_Tail: now also D16.1 (K), D17.1 (K), R13.1
- net Court_T_Actif: now also D5.2 (A), D6.2 (A), R7.1
- net Court_Tail: now also D7.1 (K), D8.1 (K), R8.1
- net Court_V_Actif: now also D3.2 (A), D4.2 (A), R6.1
- net Ouvert_T_Actif: now also D11.2 (A), D12.2 (A), D13.2 (A), R10.1
- net Ouvert_Tail: now also D14.1 (K), D15.1 (K), R11.2
- net Ouvert_V_Actif: now also D10.2 (A), D9.2 (A), R9.1
- net Fault_Actif: now reaches D20.1 (K), D21.1 (K), D22.1 (K), Q10.2 (G), R16.1
- net Vert_Enable: now reaches Q10.3 (D), R20.2
- net Vert_Enable: now also Q7.2 (G)
Other:
- note removed: "Vert_Enable"
- moved on the sheet: D10, D11, D12, D13, D14, D15, D16, D17, D7, D8, D9, Q7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

Commit message: Add files via upload
Changed lines of the file:
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@@
 	)
 	(label "Court_Tail"
-		(at 64.77 187.96 180)
+		(at 58.42 187.96 180)
 		(effects
 			(font

Commit message: Add files via upload
Parts:
- added D171: 1N4148, PCM_Diode_THT_AKL:D_DO-35_SOD27_P7.62mm_Horizontal, symbol PCM_Diode_AKL:1N4148
Connections:
- net Court_T_Actif: now also D171.2 (A)
- net Not_Btn_Tail: now also D171.1 (K)
Changed lines of the file:
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@@
 	(wire
 		(pts
+			(xy 110.49 123.19) (xy 115.57 123.19)
+		)
+		(stroke
+			(width 0)
+			(type default)
+		)
+	)
+	(wire
+		(pts
 			(xy 81.28 116.84) (xy 76.2 116.84)
 		)
@@
 	(wire
 		(pts
+			(xy 99.06 123.19) (xy 102.87 123.19)
+		)
+		(stroke
+			(width 0)
+			(type default)
+		)
+	)
+	(wire
+		(pts
 			(xy 114.3 191.77) (xy 121.92 191.77)
 		)
@@
 		)
 	)
+	(label "Not_Btn_Tail"
+		(at 115.57 123.19 0)
+		(effects
+			(font
+				(size 1.27 1.27)
+			)
+			(justify left bottom)
+		)
+	)
 	(label "Ouvert_Tail"
 		(at 153.67 25.4 180)
@@
 		)
 	)
+	(label "Court_T_Actif"
+		(at 99.06 123.19 180)
+		(effects
+			(font
+				(size 1.27 1.27)
+			)
+			(justify right bottom)
+		)
+	)
 	(label "Fault_Actif"
 		(at 220.98 125.73 0)
@@
 					(unit 1)
 				)
+			)
+		)
+	)
+	(symbol
+		(lib_id "PCM_Diode_AKL:1N4148")
+		(at 106.68 123.19 0)
+		(unit 1)
+		(body_style 1)
+		(exclude_from_sim no)
+		(in_bom yes)
+		(on_board yes)
+		(in_pos_files yes)
+		(dnp no)
+		(property "Reference" "D171"
+			(at 106.68 117.856 0)
+			(show_name no)
+			(do_not_autoplace no)
+			(effects
+				(font
+					(size 1.27 1.27)
+				)
+			)
+		)
+		(property "Value" "1N4148"
+			(at 106.68 120.142 0)
+			(show_name no)
+			(do_not_autoplace no)
+			(effects
+				(font
+					(size 1.27 1.27)
+				)
+			)
+		)
+		(property "Footprint" "PCM_Diode_THT_AKL:D_DO-35_SOD27_P7.62mm_Horizontal"
+			(at 106.68 123.19 0)
+			(hide yes)
+			(show_name no)
+			(do_not_autoplace no)
+			(effects
+				(font
+					(size 1.27 1.27)
+				)
+			)
+		)
+		(property "Datasheet" "https://datasheet.octopart.com/1N4148TR-ON-Semiconductor-datasheet-42765246.pdf"
+			(at 106.68 123.19 0)
+			(hide yes)
+			(show_name no)
+			(do_not_autoplace no)
+			(effects
+				(font
+					(size 1.27 1.27)
+				)
+			)
+		)
+		(property "Description" "DO-35 Diode, Small Signal, Fast Switching, 75V, 150mA, 4ns, Alternate KiCad Library"
+			(at 106.68 123.19 0)
+			(hide yes)
+			(show_name no)
+			(do_not_autoplace no)
+			(effects
+				(font
+					(size 1.27 1.27)
+				)
+			)
+		)
+		(pin "2"
+		)
+		(pin "1"
+		)
+		(instances
+			(project "TrailerDiagnosticSystem"
+				(path "/d4e407a7-3e32-4226-ae57-831ecdb3edf4/891824ea-a79b-4938-b55f-b811c31e662c/16a46d25-c71f-43e3-999b-a92ed112d481"
+					(reference "D171")
+					(unit 1)
+				)

Commit message: Add files via upload
Connections:
- net Btn_Tail_Etat: now also D171.1 (K)
- net Not_Btn_Tail: no longer D171.1 (K)
Other:
- moved on the sheet: D171
Changed lines of the file:
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@@
 	(wire
 		(pts
-			(xy 110.49 123.19) (xy 115.57 123.19)
+			(xy 118.11 115.57) (xy 123.19 115.57)
 		)
 		(stroke
@@
 	(wire
 		(pts
-			(xy 99.06 123.19) (xy 102.87 123.19)
+			(xy 106.68 115.57) (xy 110.49 115.57)
 		)
 		(stroke
@@
 		)
 	)
-	(label "Not_Btn_Tail"
-		(at 115.57 123.19 0)
-		(effects
-			(font
-				(size 1.27 1.27)
-			)
-			(justify left bottom)
-		)
-	)
 	(label "Ouvert_Tail"
 		(at 153.67 25.4 180)
@@
 	)
 	(label "Court_T_Actif"
-		(at 99.06 123.19 180)
+		(at 106.68 115.57 180)
 		(effects
 			(font
@@
 		)
 	)
+	(hierarchical_label "Btn_Tail_Etat"
+		(shape input)
+		(at 123.19 115.57 0)
+		(effects
+			(font
+				(size 1.27 1.27)
+			)
+			(justify left)
+		)
+	)
 	(hierarchical_label "Court_Tail_Vehic"
 		(shape input)
@@
 	(symbol
 		(lib_id "PCM_Diode_AKL:1N4148")
-		(at 106.68 123.19 0)
+		(at 114.3 115.57 0)
 		(unit 1)
 		(body_style 1)
@@
 		(dnp no)
 		(property "Reference" "D171"
-			(at 106.68 117.856 0)
+			(at 114.3 110.236 0)
 			(show_name no)
 			(do_not_autoplace no)
@@
 		)
 		(property "Value" "1N4148"
-			(at 106.68 120.142 0)
+			(at 114.3 112.522 0)
 			(show_name no)
 			(do_not_autoplace no)
@@
 		)
 		(property "Footprint" "PCM_Diode_THT_AKL:D_DO-35_SOD27_P7.62mm_Horizontal"
-			(at 106.68 123.19 0)
+			(at 114.3 115.57 0)
 			(hide yes)
 			(show_name no)
@@
 		)
 		(property "Datasheet" "https://datasheet.octopart.com/1N4148TR-ON-Semiconductor-datasheet-42765246.pdf"
-			(at 106.68 123.19 0)
+			(at 114.3 115.57 0)
 			(hide yes)
 			(show_name no)
@@
 		)
 		(property "Description" "DO-35 Diode, Small Signal, Fast Switching, 75V, 150mA, 4ns, Alternate KiCad Library"
-			(at 106.68 123.19 0)
+			(at 114.3 115.57 0)
 			(hide yes)
 			(show_name no)

Commit message: Add files via upload
Parts:
- R11, R8: value 4.7k -> 100kΩ
- R14, R16, R19: value 4.7k -> 470kΩ
Connections:
- net Bleu_Tail: now also D16.2 (A), D17.2 (A); no longer D16.1 (K), D17.1 (K)
- net GND: no longer Q8.2 (G)
- net Mode_Trailer: now also D16.1 (K); no longer D16.2 (A)
- net Not_Btn_Tail: now also D17.1 (K); no longer D17.2 (A)
- net Ouvert_Ou_Bleu_Tail: now reaches D18.1 (K), D19.1 (K), Q9.3 (D), R14.1
- net Ouvert_Ou_Bleu_Tail: now also Q8.2 (G)
Changed lines of the file:
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@@
 	)
 	(junction
+		(at 165.1 49.53)
+		(diameter 0)
+		(color 0 0 0 0)
+	)
+	(junction
 		(at 121.92 185.42)
 		(diameter 0)
@@
 	)
 	(junction
-		(at 165.1 64.77)
-		(diameter 0)
-		(color 0 0 0 0)
-	)
-	(junction
 		(at 214.63 85.09)
 		(diameter 0)
@@
 	(wire
 		(pts
+			(xy 151.13 81.28) (xy 153.67 81.28)
+		)
+		(stroke
+			(width 0)
+			(type default)
+		)
+	)
+	(wire
+		(pts
 			(xy 165.1 36.83) (xy 165.1 46.99)
 		)
@@
 	(wire
 		(pts
+			(xy 200.66 147.32) (xy 203.2 147.32)
+		)
+		(stroke
+			(width 0)
+			(type default)
+		)
+	)
+	(wire
+		(pts
 			(xy 156.21 86.36) (xy 161.29 86.36)
 		)
@@
 	(wire
 		(pts
+			(xy 165.1 49.53) (xy 167.64 49.53)
+		)
+		(stroke
+			(width 0)
+			(type default)
+		)
+	)
+	(wire
+		(pts
 			(xy 99.06 64.77) (xy 99.06 74.93)
 		)
@@
 	(wire
 		(pts
+			(xy 165.1 49.53) (xy 165.1 50.8)
+		)
+		(stroke
+			(width 0)
+			(type default)
+		)
+	)
+	(wire
+		(pts
 			(xy 101.6 26.67) (xy 104.14 26.67)
 		)
@@
 	(wire
 		(pts
-			(xy 153.67 71.12) (xy 165.1 71.12)
+			(xy 58.42 78.74) (xy 58.42 86.36)
 		)
 		(stroke
@@
 	(wire
 		(pts
-			(xy 58.42 78.74) (xy 58.42 86.36)
+			(xy 107.95 185.42) (xy 110.49 185.42)
 		)
 		(stroke
@@
 	(wire
 		(pts
-			(xy 165.1 71.12) (xy 165.1 64.77)
-		)
-		(stroke
-			(width 0)
-			(type default)
-		)
-	)
-	(wire
-		(pts
 			(xy 59.69 173.99) (xy 62.23 173.99)
 		)
@@
 	(wire
 		(pts
+			(xy 67.31 128.27) (xy 68.58 128.27)
+		)
+		(stroke
+			(width 0)
+			(type default)
+		)
+	)
+	(wire
+		(pts
 			(xy 81.28 116.84) (xy 76.2 116.84)
 		)
@@
 	(wire
 		(pts
+			(xy 151.13 46.99) (xy 153.67 46.99)
+		)
+		(stroke
+			(width 0)
+			(type default)
+		)
+	)
+	(wire
+		(pts
 			(xy 58.42 92.71) (xy 66.04 92.71)
 		)
@@
 	(wire
 		(pts
-			(xy 214.63 125.73) (xy 214.63 134.62)
+			(xy 67.31 116.84) (xy 68.58 116.84)
 		)
 		(stroke
@@
 	(wire
 		(pts
-			(xy 58.42 187.96) (xy 74.93 187.96)
+			(xy 214.63 125.73) (xy 214.63 134.62)
 		)
 		(stroke
@@
 	(wire
 		(pts
-			(xy 165.1 64.77) (xy 158.75 64.77)
+			(xy 58.42 187.96) (xy 74.93 187.96)
 		)
 		(stroke
@@
 	(wire
 		(pts
-			(xy 74.93 181.61) (xy 74.93 187.96)
+			(xy 165.1 64.77) (xy 158.75 64.77)
 		)
 		(stroke
@@
 	(wire
 		(pts
-			(xy 121.92 163.83) (xy 121.92 191.77)
+			(xy 74.93 181.61) (xy 74.93 187.96)
 		)
 		(stroke
@@
 	(wire
 		(pts
-			(xy 99.06 100.33) (xy 106.68 100.33)
+			(xy 121.92 163.83) (xy 121.92 191.77)
 		)
 		(stroke
@@
 	(wire
 		(pts
-			(xy 58.42 68.58) (xy 58.42 78.74)
+			(xy 99.06 100.33) (xy 106.68 100.33)
 		)
 		(stroke
@@
 	(wire
 		(pts
-			(xy 166.37 110.49) (xy 166.37 115.57)
+			(xy 58.42 68.58) (xy 58.42 78.74)
 		)
 		(stroke
@@
 	(wire
 		(pts
-			(xy 153.67 81.28) (xy 153.67 71.12)
+			(xy 166.37 110.49) (xy 166.37 115.57)
 		)
 		(stroke
@@
 	(wire
 		(pts
-			(xy 165.1 46.99) (xy 165.1 50.8)
+			(xy 165.1 46.99) (xy 165.1 49.53)
 		)
 		(stroke
@@
 	)
 	(label "Not_Btn_Tail"
-		(at 68.58 128.27 180)
+		(at 67.31 128.27 180)
 		(effects
 			(font
@@
 		)
 	)
+	(label "Ouvert_Ou_Bleu_Tail"
+		(at 151.13 81.28 180)
+		(effects
+			(font
+				(size 1.27 1.27)
+			)
+			(justify right bottom)
+		)
+	)
 	(label "Not_Btn_Tail"
 		(at 162.56 115.57 180)
@@
 		)
 	)
+	(label "Ouvert_Ou_Bleu_Tail"
+		(at 167.64 49.53 0)
+		(effects
+			(font
+				(size 1.27 1.27)
+			)
+			(justify left bottom)
+		)
+	)
 	(label "Court_V_Actif"
 		(at 62.23 50.8 0)
@@
 	(global_label "Mode_Trailer"
 		(shape input)
-		(at 68.58 116.84 180)
+		(at 67.31 116.84 180)
 		(fields_autoplaced yes)
 		(effects
@@
 		)
 		(property "Intersheetrefs" "${INTERSHEET_REFS}"
-			(at 83.4184 116.84 0)
+			(at 82.1484 116.84 0)
 			(hide yes)
 			(show_name no)
@@
 	(global_label "GND"
 		(shape input)
-		(at 110.49 185.42 180)
+		(at 107.95 185.42 180)
 		(fields_autoplaced yes)
 		(effects
@@
 		)
 		(property "Intersheetrefs" "${INTERSHEET_REFS}"
-			(at 103.6343 185.42 0)
+			(at 101.0943 185.42 0)
 			(hide yes)
 			(show_name no)
@@
 	(global_label "GND"
 		(shape input)
-		(at 153.67 46.99 180)
+		(at 151.13 46.99 180)
 		(fields_autoplaced yes)
 		(effects
@@
 		)
 		(property "Intersheetrefs" "${INTERSHEET_REFS}"
-			(at 146.8143 46.99 0)
+			(at 144.2743 46.99 0)
 			(hide yes)
 			(show_name no)
@@
 	(global_label "GND"
 		(shape input)
-		(at 203.2 147.32 180)
+		(at 200.66 147.32 180)
 		(fields_autoplaced yes)
 		(effects
@@
 		)
 		(property "Intersheetrefs" "${INTERSHEET_REFS}"
-			(at 196.3443 147.32 0)
+			(at 193.8043 147.32 0)
 			(hide yes)
 			(show_name no)
@@
 			)
 		)
-		(property "Value" "4.7k"
+		(property "Value" "470kΩ"
 			(at 207.01 143.51 0)
 			(show_name no)
@@
 			)
 		)
-		(property "Description" "4.7kΩ, 1/4W Resistor"
+		(property "Description" "470kΩ, 1/4W Resistor"
 			(at 207.01 147.32 0)
 			(hide yes)
@@
 			)
 		)
-		(property "Value" "4.7k"
+		(property "Value" "470kΩ"
 			(at 218.44 87.63 0)
 			(show_name no)
@@
 			)
 		)
-		(property "Description" "4.7kΩ, 1/4W Resistor"
+		(property "Description" "470kΩ, 1/4W Resistor"
 			(at 218.44 91.44 0)
 			(hide yes)
@@
 			)
 		)
-		(property "Value" "4.7k"
+		(property "Value" "100kΩ"
 			(at 114.3 181.61 0)
 			(show_name no)
@@
 			)
 		)
-		(property "Description" "4.7kΩ, 1/4W Resistor"
+		(property "Description" "100kΩ, 1/4W Resistor"
 			(at 114.3 185.42 0)
 			(hide yes)
@@
 		(lib_id "PCM_Diode_AKL:1N4148")
 		(at 72.39 128.27 0)
+		(mirror y)
 		(unit 1)
 		(body_style 1)
@@
 		(lib_id "PCM_Diode_AKL:1N4148")
 		(at 72.39 116.84 0)
+		(mirror y)
 		(unit 1)
 		(body_style 1)
@@
 			)
 		)
-		(property "Value" "4.7k"
+		(property "Value" "100kΩ"
 			(at 64.77 179.07 0)
 			(show_name no)
@@
 			)
 		)
-		(property "Description" "4.7kΩ, 1/4W Resistor"
+		(property "Description" "100kΩ, 1/4W Resistor"
 			(at 64.77 181.61 0)
 			(hide yes)
@@
 			)
 		)
-		(property "Value" "4.7k"
+		(property "Value" "470kΩ"
 			(at 157.48 43.18 0)
 			(show_name no)
@@
 			)
 		)
-		(property "Description" "4.7kΩ, 1/4W Resistor"
+		(property "Description" "470kΩ, 1/4W Resistor"
 			(at 157.48 46.99 0)
 			(hide yes)

Commit message: Add files via upload
Parts:
- R10, R12, R13, R20, R6, R7, R9: value 4.7k -> 4.7kΩ
- R15, R17, R18: value 330ohm -> 330Ω
Changed lines of the file:
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@@
 			)
 		)
-		(property "Value" "4.7k"
+		(property "Value" "4.7kΩ"
 			(at 62.23 83.82 0)
 			(show_name no)
@@
 			)
 		)
-		(property "Value" "4.7k"
+		(property "Value" "4.7kΩ"
 			(at 107.95 42.926 0)
 			(show_name no)
@@
 			)
 		)
-		(property "Value" "330ohm"
+		(property "Value" "330Ω"
 			(at 219.71 21.59 0)
 			(show_name no)
@@
 			)
 		)
-		(property "Value" "4.7k"
+		(property "Value" "4.7kΩ"
 			(at 72.39 135.89 0)
 			(show_name no)
@@
 			)
 		)
-		(property "Value" "4.7k"
+		(property "Value" "4.7kΩ"
 			(at 102.87 92.71 0)
 			(show_name no)
@@
 			)
 		)
-		(property "Value" "4.7k"
+		(property "Value" "4.7kΩ"
 			(at 162.56 106.68 0)
 			(show_name no)
@@
 			)
 		)
-		(property "Value" "330ohm"
+		(property "Value" "330Ω"
 			(at 170.18 69.85 0)
 			(show_name no)
@@
 			)
 		)
-		(property "Value" "4.7k"
+		(property "Value" "4.7kΩ"
 			(at 64.77 43.18 0)
 			(show_name no)
@@
 			)
 		)
-		(property "Value" "4.7k"
+		(property "Value" "4.7kΩ"
 			(at 245.11 152.4 0)
 			(show_name no)
@@
 			)
 		)
-		(property "Value" "330ohm"
+		(property "Value" "330Ω"
 			(at 237.49 63.5 0)
 			(show_name no)

Commit message: Add files via upload
Connections:
- net Fac_Tail_G: now reaches Q7.3 (D), R17.1
- net R_Lim_B renamed Fac_Tail_B
- net R_Lim_R renamed Fac_Tail_R
Changed lines of the file:
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@@
 	(rectangle
 		(start 191.77 55.88)
-		(end 250.19 93.98)
+		(end 259.588 93.98)
 		(stroke
 			(width 0)
@@
 	)
 	(junction
+		(at 214.63 25.4)
+		(diameter 0)
+		(color 0 0 0 0)
+	)
+	(junction
 		(at 241.3 146.05)
 		(diameter 0)
@@
 	)
 	(junction
+		(at 173.99 73.66)
+		(diameter 0)
+		(color 0 0 0 0)
+	)
+	(junction
 		(at 214.63 120.65)
 		(diameter 0)
@@
 		(color 0 0 0 0)
 	)
+	(junction
+		(at 243.84 67.31)
+		(diameter 0)
+		(color 0 0 0 0)
+	)
 	(wire
 		(pts
@@
 	(wire
 		(pts
+			(xy 243.84 67.31) (xy 241.3 67.31)
+		)
+		(stroke
+			(width 0)
+			(type default)
+		)
+	)
+	(wire
+		(pts
 			(xy 55.88 36.83) (xy 59.69 36.83)
 		)
@@
 	(wire
 		(pts
+			(xy 173.99 66.04) (xy 173.99 73.66)
+		)
+		(stroke
+			(width 0)
+			(type default)
+		)
+	)
+	(wire
+		(pts
 			(xy 101.6 26.67) (xy 104.14 26.67)
 		)
@@
 	(wire
 		(pts
+			(xy 176.53 73.66) (xy 173.99 73.66)
+		)
+		(stroke
+			(width 0)
+			(type default)
+		)
+	)
+	(wire
+		(pts
 			(xy 99.06 74.93) (xy 99.06 85.09)
 		)
@@
 	(wire
 		(pts
+			(xy 246.38 60.96) (xy 243.84 60.96)
+		)
+		(stroke
+			(width 0)
+			(type default)
+		)
+	)
+	(wire
+		(pts
 			(xy 151.13 46.99) (xy 153.67 46.99)
 		)
@@
 	(wire
 		(pts
+			(xy 209.55 25.4) (xy 214.63 25.4)
+		)
+		(stroke
+			(width 0)
+			(type default)
+		)
+	)
+	(wire
+		(pts
 			(xy 106.68 115.57) (xy 110.49 115.57)
 		)
@@
 	(wire
 		(pts
+			(xy 173.99 66.04) (xy 179.07 66.04)
+		)
+		(stroke
+			(width 0)
+			(type default)
+		)
+	)
+	(wire
+		(pts
 			(xy 166.37 129.54) (xy 165.1 129.54)
 		)
@@
 	(wire
 		(pts
+			(xy 246.38 67.31) (xy 243.84 67.31)
+		)
+		(stroke
+			(width 0)
+			(type default)
+		)
+	)
+	(wire
+		(pts
+			(xy 243.84 60.96) (xy 243.84 67.31)
+		)
+		(stroke
+			(width 0)
+			(type default)
+		)
+	)
+	(wire
+		(pts
 			(xy 241.3 143.51) (xy 241.3 146.05)
 		)
@@
 	)
 	(label "R_Lim_R"
-		(at 241.3 67.31 0)
+		(at 246.38 67.31 0)
 		(effects
 			(font
@@
 	)
 	(label "R_Lim_B"
-		(at 173.99 73.66 0)
+		(at 176.53 73.66 0)
 		(effects
 			(font
@@
 		)
 	)
+	(global_label "Fac_Tail_G"
+		(shape input)
+		(at 209.55 25.4 180)
+		(fields_autoplaced yes)
+		(effects
+			(font
+				(size 1.27 1.27)
+			)
+			(justify right)
+		)
+		(property "Intersheetrefs" "${INTERSHEET_REFS}"
+			(at 196.6468 25.4 0)
+			(hide yes)
+			(show_name no)
+			(do_not_autoplace no)
+			(effects
+				(font
+					(size 1.27 1.27)
+				)
+				(justify right)
+			)
+		)
+	)
 	(global_label "GND"
 		(shape input)
@@
 		)
 	)
+	(global_label "Fac_Tail_B"
+		(shape input)
+		(at 179.07 66.04 0)
+		(fields_autoplaced yes)
+		(effects
+			(font
+				(size 1.27 1.27)
+			)
+			(justify left)
+		)
+		(property "Intersheetrefs" "${INTERSHEET_REFS}"
+			(at 191.9732 66.04 0)
+			(hide yes)
+			(show_name no)
+			(do_not_autoplace no)
+			(effects
+				(font
+					(size 1.27 1.27)
+				)
+				(justify left)
+			)
+		)
+	)
 	(global_label "GND"
 		(shape input)
@@
 		)
 	)
+	(global_label "Fac_Tail_R"
+		(shape input)
+		(at 246.38 60.96 0)
+		(fields_autoplaced yes)
+		(effects
+			(font
+				(size 1.27 1.27)
+			)
+			(justify left)
+		)
+		(property "Intersheetrefs" "${INTERSHEET_REFS}"
+			(at 259.2832 60.96 0)
+			(hide yes)
+			(show_name no)
+			(do_not_autoplace no)
+			(effects
+				(font
+					(size 1.27 1.27)
+				)
+				(justify left)
+			)
+		)
+	)
 	(global_label "Mode_Trailer"
 		(shape input)
@@
 		(in_pos_files yes)
 		(dnp no)
-		(fields_autoplaced yes)
 		(property "Reference" "R15"
-			(at 170.18 67.31 0)
+			(at 170.18 67.818 0)
 			(show_name no)
 			(do_not_autoplace no)
