File: Trailer_Aux.kicad_sch (KiCad schematic)
At the start: 11 parts, among them Q44 IRLZ44N, SW7 SW_SPST, U12 LM339

Commit message: Add files via upload
Parts:
- U12: footprint (none) -> Package_DIP:DIP-14_W7.62mm_Socket
Changed lines of the file:
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@@
 			)
 		)
-		(property "Footprint" ""
+		(property "Footprint" "Package_DIP:DIP-14_W7.62mm_Socket"
 			(at 158.75 102.87 0)
 			(hide yes)
@@
 			)
 		)
-		(property "Footprint" ""
+		(property "Footprint" "Package_DIP:DIP-14_W7.62mm_Socket"
 			(at 157.48 44.45 0)
 			(hide yes)
@@
 			)
 		)
-		(property "Footprint" ""
+		(property "Footprint" "Package_DIP:DIP-14_W7.62mm_Socket"
 			(at 146.05 123.19 0)
 			(hide yes)
@@
 			)
 		)
-		(property "Footprint" ""
+		(property "Footprint" "Package_DIP:DIP-14_W7.62mm_Socket"
 			(at 157.48 85.09 0)
 			(hide yes)
@@
 			)
 		)
-		(property "Footprint" ""
+		(property "Footprint" "Package_DIP:DIP-14_W7.62mm_Socket"
 			(at 157.48 63.5 0)
 			(hide yes)

Commit message: Add files via upload
Parts:
- U12: footprint Package_DIP:DIP-14_W7.62mm_Socket -> (none)
Changed lines of the file:
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@@
 			)
 		)
-		(property "Footprint" "Package_DIP:DIP-14_W7.62mm_Socket"
+		(property "Footprint" ""
 			(at 158.75 102.87 0)
 			(hide yes)
@@
 			)
 		)
-		(property "Footprint" "Package_DIP:DIP-14_W7.62mm_Socket"
+		(property "Footprint" ""
 			(at 157.48 44.45 0)
 			(hide yes)
@@
 			)
 		)
-		(property "Footprint" "Package_DIP:DIP-14_W7.62mm_Socket"
+		(property "Footprint" ""
 			(at 146.05 123.19 0)
 			(hide yes)
@@
 			)
 		)
-		(property "Footprint" "Package_DIP:DIP-14_W7.62mm_Socket"
+		(property "Footprint" ""
 			(at 157.48 85.09 0)
 			(hide yes)
@@
 			)
 		)
-		(property "Footprint" "Package_DIP:DIP-14_W7.62mm_Socket"
+		(property "Footprint" ""
 			(at 157.48 63.5 0)
 			(hide yes)

Commit message: Add files via upload
Parts:
- Q44: value IRLZ44N -> IRF4905PBF; footprint PCM_Package_TO_SOT_THT_AKL:TO-220-3_Vertical_GDS -> Package_TO_SOT_THT:TO-220-3_Vertical; symbol PCM_Transistor_MOSFET_AKL:IRLZ44N -> Transistor_FET:IRF4905
Connections:
- net Aux_Trailer_Shunt_Haut: no longer Q44.3 (S)
- net Q44.2_Drain: no longer F6.2, Q44.2 (D)
- new net: F6.2, Q44.3 (S)
Changed lines of the file:
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@@
+	(wire
+		(pts
+			(xy 36.83 119.38) (xy 64.77 119.38)
+		)
+		(stroke
+			(width 0)
+			(type default)
+		)
+	)
 	(wire
 		(pts
@@
 	(wire
 		(pts
-			(xy 60.96 73.66) (xy 64.77 73.66)
-		)
-		(stroke
-			(width 0)
-			(type default)
-		)
-	)
-	(wire
-		(pts
 			(xy 166.37 87.63) (xy 168.91 87.63)
 		)
@@
 	(wire
 		(pts
+			(xy 36.83 119.38) (xy 36.83 73.66)
+		)
+		(stroke
+			(width 0)
+			(type default)
+		)
+	)
+	(wire
+		(pts
 			(xy 168.91 87.63) (xy 170.18 87.63)
 		)
@@
 	(wire
 		(pts
+			(xy 36.83 73.66) (xy 64.77 73.66)
+		)
+		(stroke
+			(width 0)
+			(type default)
+		)
+	)
+	(wire
+		(pts
 			(xy 168.91 93.98) (xy 172.72 93.98)
 		)
@@
 	(wire
 		(pts
-			(xy 60.96 119.38) (xy 64.77 119.38)
-		)
-		(stroke
-			(width 0)
-			(type default)
-		)
-	)
-	(wire
-		(pts
 			(xy 111.76 88.9) (xy 111.76 81.28)
 		)
@@
 	(wire
 		(pts
-			(xy 54.61 111.76) (xy 58.42 111.76)
+			(xy 53.34 110.49) (xy 57.15 110.49)
 		)
 		(stroke
@@
 		)
 	)
-	(label "Aux_Trailer_Shunt_Haut"
-		(at 60.96 119.38 180)
-		(effects
-			(font
-				(size 1.27 1.27)
-			)
-			(justify right bottom)
-		)
-	)
 	(label "Q44.2_Drain"
-		(at 60.96 73.66 180)
-		(effects
-			(font
-				(size 1.27 1.27)
-			)
-			(justify right bottom)
-		)
-	)
-	(label "Q44.2_Drain"
-		(at 64.77 101.6 180)
+		(at 26.67 99.06 180)
 		(effects
 			(font
@@
 		)
 	)
+	(label "Q44.2_Drain"
+		(at 26.67 102.87 180)
+		(effects
+			(font
+				(size 1.27 1.27)
+			)
+			(justify right bottom)
+		)
+	)
 	(global_label "GND"
 		(shape input)
@@
 	(hierarchical_label "Btn_Aux_Etat"
 		(shape input)
-		(at 54.61 111.76 180)
+		(at 53.34 110.49 180)
 		(effects
 			(font
@@
 	)
 	(symbol
-		(lib_id "PCM_Transistor_MOSFET_AKL:IRLZ44N")
+		(lib_id "Transistor_FET:IRF4905")
 		(at 62.23 110.49 0)
 		(unit 1)
@@
 			)
 		)
-		(property "Value" "IRLZ44N"
+		(property "Value" "IRF4905PBF"
 			(at 68.58 111.7599 0)
 			(show_name no)
@@
 			)
 		)
-		(property "Footprint" "PCM_Package_TO_SOT_THT_AKL:TO-220-3_Vertical_GDS"
+		(property "Footprint" "Package_TO_SOT_THT:TO-220-3_Vertical"
 			(at 67.31 107.95 0)
 			(hide yes)
@@
 			)
 		)
-		(property "Datasheet" "https://www.tme.eu/Document/71cf1899624764088671ce6de5d15eb4/irlz44n.pdf"
+		(property "Datasheet" "https://www.mouser.com/datasheet/2/196/Infineon_IRF4905_DataSheet_v01_01_EN-3362811.pdf"
 			(at 62.23 110.49 0)
 			(hide yes)
@@
 			)
 		)
-		(property "Description" "TO-220 N-MOSFET enchancement mode transistor, 55V, 47A, 110W, Alternate KiCAD Library"
+		(property "Description" "P-Channel MOSFET, -55V, -74A, 20mOhm, TO-220AB"
 			(at 62.23 110.49 0)
 			(hide yes)

Commit message: Add files via upload
Parts:
- added Q68: 2N7000, PCM_Package_TO_SOT_THT_AKL:TO-92_Inline_Wide_SGD, symbol PCM_Transistor_MOSFET_AKL:2N7000
- added R247: 1 kΩ, Resistor_THT:R_Axial_DIN0207_L6.3mm_D2.5mm_P10.16mm_Horizontal, symbol PCM_SL_Resistors:4.7k
- added SW11: KSD9700, symbol Switch:SW_SPST_Temperature_NC
- R168: value .1 ohm -> 12 Ohm; footprint Resistor_THT:R_Axial_Power_L25.0mm_W9.0mm_P27.94mm -> TerminalBlock_Phoenix:TerminalBlock_Phoenix_PT-1,5-2-3.5-H_1x02_P3.50mm_Horizontal
Connections:
- net Aux_Trailer_Shunt_Haut: no longer R168.2
- net Btn_Aux_Etat: now also Q68.2 (G); no longer Q44.1 (G)
- net GND: now also Q68.1 (S)
- net at Q44.2 (D): now also SW11.1
- new net: Q68.3 (D), R247.2
- new net: Q44.1 (G), R247.1
- new net: R168.2, SW11.2
Other:
- moved on the sheet: D122, F6, Q44, R167, R168, R169, R170, R171, R172, SW7, U12A, U12B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

Commit message: Add files via upload
Parts:
- added DZ1: 1N5242B, PCM_Diode_THT_AKL:D_DO-35_SOD27_P7.62mm_Horizontal_Zener, symbol PCM_Diode_Zener_AKL:1N5242B
- added R248, R250: 10k, Resistor_THT:R_Axial_DIN0207_L6.3mm_D2.5mm_P10.16mm_Horizontal, symbol PCM_SL_Resistors:10k
- added R249: 39 kΩ, Resistor_THT:R_Axial_DIN0207_L6.3mm_D2.5mm_P10.16mm_Horizontal, symbol PCM_SL_Resistors:10k
- R168: value 12 Ohm -> 12 Ohm, 50W
Connections:
- net GND: now also R250.1
- net Trail_Aux: now also R249.1
- net at Q44.1 (G), R247.1: now also DZ1.2 (A), R248.1
- net at F6.2, Q44.3 (S): now also DZ1.1 (K), R248.2
- net at R169.2: now also U12.6 (-); no longer U12.7 (+)
- net Aux_Trailer_Shunt_Haut renamed Mesure_Aux_Trailer
- net Mesure_Aux_Trailer: now also U12.7 (+), R249.2, R250.2; no longer U12.6 (-)
Other:
- moved on the sheet: D122, Q44, R168, R169, R170, SW11

Commit message: Add files via upload
Parts:
- added R251: 100 kΩ, Resistor_THT:R_Axial_DIN0207_L6.3mm_D2.5mm_P10.16mm_Horizontal, symbol PCM_SL_Resistors:10k
- F6: value Polyfuse -> MF-R160
Connections:
- net V_Ref: now also R251.2; no longer R170.1
- new net: R170.1, R251.1

Commit message: Add files via upload
Parts:
- removed DZ1: 1N5242B, PCM_Diode_THT_AKL:D_DO-35_SOD27_P7.62mm_Horizontal_Zener, symbol PCM_Diode_Zener_AKL:1N5242B
- removed Q68: 2N7000, PCM_Package_TO_SOT_THT_AKL:TO-92_Inline_Wide_SGD, symbol PCM_Transistor_MOSFET_AKL:2N7000
- removed R247: 1 kΩ, Resistor_THT:R_Axial_DIN0207_L6.3mm_D2.5mm_P10.16mm_Horizontal, symbol PCM_SL_Resistors:4.7k
- removed R248, R250: 10k, Resistor_THT:R_Axial_DIN0207_L6.3mm_D2.5mm_P10.16mm_Horizontal, symbol PCM_SL_Resistors:10k
- removed R249: 39 kΩ, Resistor_THT:R_Axial_DIN0207_L6.3mm_D2.5mm_P10.16mm_Horizontal, symbol PCM_SL_Resistors:10k
- removed R251: 100 kΩ, Resistor_THT:R_Axial_DIN0207_L6.3mm_D2.5mm_P10.16mm_Horizontal, symbol PCM_SL_Resistors:10k
- removed SW11: KSD9700, symbol Switch:SW_SPST_Temperature_NC
- F6: value MF-R160 -> Polyfuse
- Q44: value IRF4905PBF -> IRLZ44N; footprint Package_TO_SOT_THT:TO-220-3_Vertical -> PCM_Package_TO_SOT_THT_AKL:TO-220-3_Vertical_GDS; symbol Transistor_FET:IRF4905 -> PCM_Transistor_MOSFET_AKL:IRLZ44N
- R168: value 12 Ohm, 50W -> .1 ohm; footprint TerminalBlock_Phoenix:TerminalBlock_Phoenix_PT-1,5-2-3.5-H_1x02_P3.50mm_Horizontal -> Resistor_THT:R_Axial_DIN0207_L6.3mm_D2.5mm_P10.16mm_Horizontal
- R169, R170: footprint TRIM_3296W1103LF:TRIM_3296W1103LF -> (none)
Connections:
- net Btn_Aux_Etat: now also Q44.1 (G)
- net V_Ref: now also R170.1
- net Q44.2_Drain: now reaches Q44.2 (D)
- net Q44.2_Drain: now also F6.2
- net Aux_Trailer_Shunt_Haut: now reaches Q44.3 (S)
- net Aux_Trailer_Shunt_Haut: now also R168.2, U12.10 (-), U12.6 (-); no longer F6.2
- net at R169.2: now also U12.7 (+); no longer U12.6 (-)
- removed net Mesure_Aux_Trailer: U12.10 (-), U12.7 (+)
Other:
- moved on the sheet: D122, F6, R167, R168, R169, R171, R172, SW7, U12A, U12B, U12C, U12D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

Commit message: Add files via upload
Parts:
- added DZ1: 1N5242B, PCM_Diode_THT_AKL:D_DO-35_SOD27_P7.62mm_Horizontal_Zener, symbol PCM_Diode_Zener_AKL:1N5242B
- added Q68: 2N7000, PCM_Package_TO_SOT_THT_AKL:TO-92_Inline_Wide_SGD, symbol PCM_Transistor_MOSFET_AKL:2N7000
- added R247: 1 kΩ, Resistor_THT:R_Axial_DIN0207_L6.3mm_D2.5mm_P10.16mm_Horizontal, symbol PCM_SL_Resistors:4.7k
- added R248, R250: 10k, Resistor_THT:R_Axial_DIN0207_L6.3mm_D2.5mm_P10.16mm_Horizontal, symbol PCM_SL_Resistors:10k
- added R249: 39 kΩ, Resistor_THT:R_Axial_DIN0207_L6.3mm_D2.5mm_P10.16mm_Horizontal, symbol PCM_SL_Resistors:10k
- added R251: 100 kΩ, Resistor_THT:R_Axial_DIN0207_L6.3mm_D2.5mm_P10.16mm_Horizontal, symbol PCM_SL_Resistors:10k
- added SW11: KSD9700, symbol Switch:SW_SPST_Temperature_NC
- F6: value Polyfuse -> MF-R160
- Q44: value IRLZ44N -> IRF4905PBF; footprint PCM_Package_TO_SOT_THT_AKL:TO-220-3_Vertical_GDS -> Package_TO_SOT_THT:TO-220-3_Vertical; symbol PCM_Transistor_MOSFET_AKL:IRLZ44N -> Transistor_FET:IRF4905
- R168: value .1 ohm -> 12 Ohm, 50W; footprint Resistor_THT:R_Axial_DIN0207_L6.3mm_D2.5mm_P10.16mm_Horizontal -> TerminalBlock_Phoenix:TerminalBlock_Phoenix_PT-1,5-2-3.5-H_1x02_P3.50mm_Horizontal
- R169, R170: footprint (none) -> TRIM_3296W1103LF:TRIM_3296W1103LF
Connections:
- net Btn_Aux_Etat: now also Q68.2 (G); no longer Q44.1 (G)
- net GND: now also Q68.1 (S), R250.1
- net Trail_Aux: now also R249.1
- net V_Ref: now also R251.2; no longer R170.1
- net at R169.2: now also U12.6 (-); no longer U12.7 (+)
- removed net Aux_Trailer_Shunt_Haut: Q44.3 (S), R168.2, U12.10 (-), U12.6 (-)
- net Q44.2_Drain: no longer names the net of Q44.2 (D)
- net Q44.2_Drain: now also SW11.1; no longer F6.2
- new net: Q68.3 (D), R247.2
- new net: DZ1.2 (A), Q44.1 (G), R247.1, R248.1
- new net: DZ1.1 (K), F6.2, Q44.3 (S), R248.2
- new net: R168.2, SW11.2
- new net: R170.1, R251.1
- new net Mesure_Aux_Trailer: R249.2, R250.2, U12.10 (-), U12.7 (+)
Other:
- moved on the sheet: D122, F6, R167, R168, R169, R171, R172, SW7, U12A, U12B, U12C, U12D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
