File: Trailer_Aux.kicad_sch (KiCad schematic)
At the start: 19 parts, among them Q44 IRF4905PBF, Q68 2N7000, SW11 KSD9700, SW7 SW_SPST, U12 LM339

Commit message: Add files via upload
Parts:
- D122: value SMBJ33A -> P6KE39A; footprint PCM_Diode_SMD_AKL:D_SMB -> PCM_Diode_THT_AKL:D_DO-15_P10.16mm_Horizontal_Zener; symbol PCM_Diode_TVS_AKL:SMBJ33A -> PCM_Diode_TVS_AKL:P6KE39A
Changed lines of the file:
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@@
 	)
 	(symbol
-		(lib_id "PCM_Diode_TVS_AKL:SMBJ33A")
+		(lib_id "PCM_Diode_TVS_AKL:P6KE39A")
 		(at 129.54 134.62 0)
 		(unit 1)
@@
 			)
 		)
-		(property "Value" "SMBJ33A"
+		(property "Value" "P6KE39A"
 			(at 129.54 130.81 0)
 			(show_name no)
@@
 			)
 		)
-		(property "Footprint" "PCM_Diode_SMD_AKL:D_SMB"
+		(property "Footprint" "PCM_Diode_THT_AKL:D_DO-15_P10.16mm_Horizontal_Zener"
 			(at 129.54 134.62 0)
 			(hide yes)
@@
 			)
 		)
-		(property "Datasheet" "https://www.tme.eu/Document/0b6222bec7e12d83185b51d73cb6a54d/SMBJ_ser.pdf"
+		(property "Datasheet" "https://www.tme.eu/Document/6b488a936123e1f9ccf03f4f9186b150/P6KE_ser.pdf"
 			(at 129.54 134.62 0)
 			(hide yes)
@@
 			)
 		)
-		(property "Description" "SMB Unidirectional TVS diode, 33V, 600W, Alternate KiCAD Library"
+		(property "Description" "DO-15 Unidirectional TVS diode, 39V, 600W, Alternate KiCAD Library"
 			(at 129.54 134.62 0)
 			(hide yes)

Commit message: Add files via upload
Parts:
- U12: footprint (none) -> Package_DIP:DIP-14_W7.62mm_Socket
Changed lines of the file:
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@@
 			)
 		)
-		(property "Footprint" ""
+		(property "Footprint" "Package_DIP:DIP-14_W7.62mm_Socket"
 			(at 190.5 102.87 0)
 			(hide yes)
@@
 			)
 		)
-		(property "Footprint" ""
+		(property "Footprint" "Package_DIP:DIP-14_W7.62mm_Socket"
 			(at 189.23 44.45 0)
 			(hide yes)
@@
 			)
 		)
-		(property "Footprint" ""
+		(property "Footprint" "Package_DIP:DIP-14_W7.62mm_Socket"
 			(at 177.8 123.19 0)
 			(hide yes)
@@
 			)
 		)
-		(property "Footprint" ""
+		(property "Footprint" "Package_DIP:DIP-14_W7.62mm_Socket"
 			(at 189.23 85.09 0)
 			(hide yes)
@@
 			)
 		)
-		(property "Footprint" ""
+		(property "Footprint" "Package_DIP:DIP-14_W7.62mm_Socket"
 			(at 189.23 63.5 0)
 			(hide yes)

Commit message: Add files via upload
Parts:
- F6: footprint (none) -> PTC_Bourns_MF-R:PTC_Bourns_MF-R_P5.10mm_W12.0mm
- SW11: footprint (none) -> TerminalBlock_Phoenix:TerminalBlock_Phoenix_PT-1,5-2-3.5-H_1x02_P3.50mm_Horizontal
Changed lines of the file:
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@@
 			)
 		)
-		(property "Footprint" ""
+		(property "Footprint" "TerminalBlock_Phoenix:TerminalBlock_Phoenix_PT-1,5-2-3.5-H_1x02_P3.50mm_Horizontal"
 			(at 83.82 96.52 0)
 			(hide yes)
@@
 			)
 		)
-		(property "Footprint" ""
+		(property "Footprint" "PTC_Bourns_MF-R:PTC_Bourns_MF-R_P5.10mm_W12.0mm"
 			(at 66.04 67.31 0)
 			(hide yes)

Commit message: Add files via upload
Parts:
- SW7: value SW_SPST -> SW_SPDT; symbol Switch:SW_SPST -> Switch:SW_SPDT
Connections:
- net GND: now also SW7.3 (C)
Other:
- moved on the sheet: R167
Changed lines of the file:
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@@
 	)
 	(junction
+		(at 48.26 44.45)
+		(diameter 0)
+		(color 0 0 0 0)
+	)
+	(junction
 		(at 57.15 106.68)
 		(diameter 0)
@@
 	)
 	(junction
-		(at 48.26 31.75)
-		(diameter 0)
-		(color 0 0 0 0)
-	)
-	(junction
 		(at 72.39 128.27)
 		(diameter 0)
@@
 	(wire
 		(pts
-			(xy 48.26 31.75) (xy 48.26 39.37)
+			(xy 48.26 31.75) (xy 48.26 44.45)
 		)
 		(stroke
@@
 	(wire
 		(pts
+			(xy 33.02 44.45) (xy 36.83 44.45)
+		)
+		(stroke
+			(width 0)
+			(type default)
+		)
+	)
+	(wire
+		(pts
 			(xy 153.67 80.01) (xy 157.48 80.01)
 		)
@@
 	(wire
 		(pts
-			(xy 33.02 31.75) (xy 36.83 31.75)
+			(xy 33.02 29.21) (xy 36.83 29.21)
 		)
 		(stroke
@@
 	(wire
 		(pts
-			(xy 142.24 80.01) (xy 142.24 81.28)
+			(xy 48.26 44.45) (xy 48.26 49.53)
 		)
 		(stroke
@@
 	(wire
 		(pts
-			(xy 53.34 31.75) (xy 48.26 31.75)
+			(xy 142.24 80.01) (xy 142.24 81.28)
 		)
 		(stroke
@@
 	(wire
 		(pts
+			(xy 33.02 34.29) (xy 36.83 34.29)
+		)
+		(stroke
+			(width 0)
+			(type default)
+		)
+	)
+	(wire
+		(pts
 			(xy 59.69 128.27) (xy 57.15 128.27)
 		)
@@
 	(wire
 		(pts
-			(xy 48.26 39.37) (xy 52.07 39.37)
+			(xy 48.26 44.45) (xy 44.45 44.45)
 		)
 		(stroke
@@
 	(wire
 		(pts
+			(xy 33.02 49.53) (xy 48.26 49.53)
+		)
+		(stroke
+			(width 0)
+			(type default)
+		)
+	)
+	(wire
+		(pts
 			(xy 57.15 128.27) (xy 57.15 118.11)
 		)
@@
 	(global_label "GND"
 		(shape input)
-		(at 59.69 39.37 0)
+		(at 33.02 44.45 180)
 		(fields_autoplaced yes)
 		(effects
@@
 				(size 1.27 1.27)
 			)
-			(justify left)
+			(justify right)
 		)
 		(property "Intersheetrefs" "${INTERSHEET_REFS}"
-			(at 66.5457 39.37 0)
+			(at 26.1643 44.45 0)
 			(hide yes)
 			(show_name no)
@@
 					(size 1.27 1.27)
 				)
-				(justify left)
+				(justify right)
 			)
 		)
@@
 	(global_label "V_Ref"
 		(shape input)
-		(at 33.02 31.75 180)
+		(at 33.02 29.21 180)
 		(fields_autoplaced yes)
 		(effects
@@
 		)
 		(property "Intersheetrefs" "${INTERSHEET_REFS}"
-			(at 24.8943 31.75 0)
+			(at 24.8943 29.21 0)
 			(hide yes)
 			(show_name no)
@@
 		)
 	)
-	(global_label "V_Ref"
+	(global_label "GND"
 		(shape input)
-		(at 157.48 80.01 0)
+		(at 33.02 34.29 180)
 		(fields_autoplaced yes)
 		(effects
@@
 				(size 1.27 1.27)
 			)
-			(justify left)
+			(justify right)
 		)
 		(property "Intersheetrefs" "${INTERSHEET_REFS}"
-			(at 165.6057 80.01 0)
+			(at 26.1643 34.29 0)
 			(hide yes)
 			(show_name no)
@@
 					(size 1.27 1.27)
 				)
-				(justify left)
+				(justify right)
 			)
 		)
 	)
-	(hierarchical_label "Btn_Aux_Etat"
+	(global_label "V_Ref"
 		(shape input)
-		(at 53.34 31.75 0)
+		(at 157.48 80.01 0)
+		(fields_autoplaced yes)
 		(effects
 			(font
@@
 			(justify left)
 		)
+		(property "Intersheetrefs" "${INTERSHEET_REFS}"
+			(at 165.6057 80.01 0)
+			(hide yes)
+			(show_name no)
+			(do_not_autoplace no)
+			(effects
+				(font
+					(size 1.27 1.27)
+				)
+				(justify left)
+			)
+		)
 	)
 	(hierarchical_label "Trail_Aux"
@@
 		)
 	)
+	(hierarchical_label "Btn_Aux_Etat"
+		(shape input)
+		(at 33.02 49.53 180)
+		(effects
+			(font
+				(size 1.27 1.27)
+			)
+			(justify right)
+		)
+	)
 	(symbol
 		(lib_id "PCM_Transistor_MOSFET_AKL:2N7000")
@@
 	)
 	(symbol
-		(lib_id "Switch:SW_SPST")
+		(lib_id "Switch:SW_SPDT")
 		(at 41.91 31.75 0)
+		(mirror y)
 		(unit 1)
 		(body_style 1)
@@
 		(in_pos_files yes)
 		(dnp no)
-		(fields_autoplaced yes)
 		(property "Reference" "SW7"
-			(at 41.91 25.4 0)
+			(at 41.91 24.638 0)
 			(show_name no)
 			(do_not_autoplace no)
@@
 			)
 		)
-		(property "Value" "SW_SPST"
-			(at 41.91 27.94 0)
+		(property "Value" "SW_SPDT"
+			(at 41.91 26.924 0)
 			(show_name no)
 			(do_not_autoplace no)
@@
 			)
 		)
-		(property "Description" "Single Pole Single Throw (SPST) switch"
+		(property "Description" "Switch, single pole double throw"
 			(at 41.91 31.75 0)
 			(hide yes)
@@
 		(pin "2"
 		)
+		(pin "3"
+		)
 		(instances
 			(project "TrailerDiagnosticSystem"
@@
 	(symbol
 		(lib_id "PCM_SL_Resistors:10k")
-		(at 55.88 39.37 0)
+		(at 40.64 44.45 0)
+		(mirror y)
 		(unit 1)
 		(body_style 1)
@@
 		(dnp no)
 		(property "Reference" "R167"
-			(at 55.88 35.052 0)
+			(at 40.64 40.132 0)
 			(show_name no)
 			(do_not_autoplace no)
@@
 		)
 		(property "Value" "10k"
-			(at 55.88 36.83 0)
+			(at 40.64 41.91 0)
 			(show_name no)
 			(do_not_autoplace no)
@@
 		)
 		(property "Footprint" "Resistor_THT:R_Axial_DIN0207_L6.3mm_D2.5mm_P10.16mm_Horizontal"
-			(at 56.769 43.688 0)
+			(at 39.751 48.768 0)
 			(hide yes)
 			(show_name no)
@@
 		)
 		(property "Datasheet" ""
-			(at 56.388 39.37 0)
+			(at 40.132 44.45 0)
 			(hide yes)
 			(show_name no)
@@
 		)
 		(property "Description" "10kΩ, 1/4W Resistor"
-			(at 55.88 39.37 0)
+			(at 40.64 44.45 0)
 			(hide yes)
 			(show_name no)

Commit message: Add files via upload
Parts:
- R167, R248, R250: value 10k -> 10kΩ
- R171, R172: value 4.7k -> 4.7kΩ
- R251: value 100 kΩ -> 100kΩ
Changed lines of the file:
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@@
 			)
 		)
-		(property "Value" "10k"
+		(property "Value" "10kΩ"
 			(at 63.5 115.57 0)
 			(show_name no)
@@
 			)
 		)
-		(property "Value" "4.7k"
+		(property "Value" "4.7kΩ"
 			(at 205.74 62.23 0)
 			(show_name no)
@@
 			)
 		)
-		(property "Value" "4.7k"
+		(property "Value" "4.7kΩ"
 			(at 205.74 83.82 0)
 			(show_name no)
@@
 			)
 		)
-		(property "Value" "100 kΩ"
+		(property "Value" "100kΩ"
 			(at 149.86 77.47 0)
 			(show_name no)
@@
 			)
 		)
-		(property "Value" "10k"
+		(property "Value" "10kΩ"
 			(at 129.54 116.84 0)
 			(show_name no)
@@
 			)
 		)
-		(property "Value" "10k"
+		(property "Value" "10kΩ"
 			(at 40.64 41.91 0)
 			(show_name no)

Commit message: Add files via upload
Parts:
- R247: value 1 kΩ -> 1kΩ
- R249: value 39 kΩ -> 39kΩ
Changed lines of the file:
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@@
 			)
 		)
-		(property "Value" "1 kΩ"
+		(property "Value" "1kΩ"
 			(at 48.26 104.14 0)
 			(show_name no)
@@
 			)
 		)
-		(property "Value" "39 kΩ"
+		(property "Value" "39kΩ"
 			(at 129.54 107.95 0)
 			(show_name no)

Commit message: Add files via upload
Connections:
- net Btn_Aux_Etat renamed Fac_Btn_Aux
Changed lines of the file:
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@@
+	)
+	(junction
+		(at 48.26 31.75)
+		(diameter 0)
+		(color 0 0 0 0)
 	)
 	(junction
@@
 	(wire
 		(pts
+			(xy 48.26 31.75) (xy 55.88 31.75)
+		)
+		(stroke
+			(width 0)
+			(type default)
+		)
+	)
+	(wire
+		(pts
 			(xy 41.91 107.95) (xy 41.91 106.68)
 		)
@@
 			)
 		)
+	)
+	(global_label "Fac_Btn_Aux"
+		(shape input)
+		(at 55.88 31.75 0)
+		(fields_autoplaced yes)
+		(effects
+			(font
+				(size 1.27 1.27)
+			)
+			(justify left)
+		)
+		(property "Intersheetrefs" "${INTERSHEET_REFS}"
+			(at 70.537 31.75 0)
+			(hide yes)
+			(show_name no)
+			(do_not_autoplace no)
+			(effects
+				(font
+					(size 1.27 1.27)
+				)
+				(justify left)
+			)
+		)
