File: Vehicule_Backup.kicad_sch (KiCad schematic)
At the start: 16 parts, among them Q27 IRLZ44N, U7 LM339

Commit message: Add files via upload
Parts:
- removed OC5, OC6: PC817, PCM_Package_DIP_AKL:DIP-4_W7.62mm_LongPads, symbol PCM_Optocoupler_AKL:PC817
- removed Q27: IRLZ44N, PCM_Package_TO_SOT_THT_AKL:TO-220-3_Vertical_GDS, symbol PCM_Transistor_MOSFET_AKL:IRLZ44N
- removed R100, R98, R99: Potentiometer, symbol Simulation_SPICE:Potentiometer
- removed R89: 3 Ohm - 5W, Resistor_THT:R_Axial_Power_L25.0mm_W9.0mm_P27.94mm, symbol PCM_SL_Devices:Resistor_5W
- removed R90: .05R Shunt, Resistor_THT:R_Axial_Power_L25.0mm_W9.0mm_P27.94mm, symbol PCM_SL_Devices:Resistor_5W
- removed R91, R92, R93: 4.7k, Resistor_THT:R_Axial_DIN0207_L6.3mm_D2.5mm_P10.16mm_Horizontal, symbol PCM_SL_Resistors:4.7k
- removed R94, R95: 1k, Resistor_THT:R_Axial_DIN0207_L6.3mm_D2.5mm_P10.16mm_Horizontal, symbol PCM_SL_Resistors:4.7k
- removed R96: 100k, Resistor_THT:R_Axial_DIN0207_L6.3mm_D2.5mm_P10.16mm_Horizontal, symbol PCM_SL_Resistors:100k
- removed R97: 10k, Resistor_THT:R_Axial_DIN0207_L6.3mm_D2.5mm_P10.16mm_Horizontal, symbol PCM_SL_Resistors:10k
- removed U7: LM339, symbol Comparator:LM339
- added OC7, OC8: PC817, PCM_Package_DIP_AKL:DIP-4_W7.62mm_LongPads, symbol PCM_Optocoupler_AKL:PC817
- added Q35: IRLZ44N, PCM_Package_TO_SOT_THT_AKL:TO-220-3_Vertical_GDS, symbol PCM_Transistor_MOSFET_AKL:IRLZ44N
- added R122: 3 Ohm - 5W, Resistor_THT:R_Axial_Power_L25.0mm_W9.0mm_P27.94mm, symbol PCM_SL_Devices:Resistor_5W
- added R123: .05R Shunt, Resistor_THT:R_Axial_Power_L25.0mm_W9.0mm_P27.94mm, symbol PCM_SL_Devices:Resistor_5W
- added R124, R125, R126: 4.7k, Resistor_THT:R_Axial_DIN0207_L6.3mm_D2.5mm_P10.16mm_Horizontal, symbol PCM_SL_Resistors:4.7k
- added R127, R128: 1k, Resistor_THT:R_Axial_DIN0207_L6.3mm_D2.5mm_P10.16mm_Horizontal, symbol PCM_SL_Resistors:4.7k
- added R129: 100k, Resistor_THT:R_Axial_DIN0207_L6.3mm_D2.5mm_P10.16mm_Horizontal, symbol PCM_SL_Resistors:100k
- added R130: 10k, Resistor_THT:R_Axial_DIN0207_L6.3mm_D2.5mm_P10.16mm_Horizontal, symbol PCM_SL_Resistors:10k
- added R131, R132, R133: Potentiometer, symbol Simulation_SPICE:Potentiometer
- added U9: LM339, symbol Comparator:LM339
Connections:
- net GND: now also OC7.3, OC8.3, R123.2, R130.2, R131.3, R132.3, R133.3, U9.12 (V-), U9.9 (+)
- net V_Ref: now also OC7.2, OC8.2, R125.2, R126.2, R127.1, R128.1, R131.1, R132.1, R133.1, U9.3 (V+), U9.8 (-)
- new net: R125.1, U9.1
- new net: R122.2, R123.1, U9.11 (+), U9.6 (-)
- new net: OC8.1, R128.2
- new net: OC7.1, R127.2
- new net: R126.1, U9.13
- new net: Q35.1 (G), R124.2
- new net: R124.1, U9.2
- new net: R129.2, R130.1, U9.5 (+)
- new net Court_Backup_Vehic: OC7.4
- new net Ouvert_Backup_Vehic: OC8.4
- new net Q35_Source: Q35.3 (S), R122.1
- new net Seuil_Court_Backup: R133.2, U9.10 (-)
- new net Seuil_Injection_Backup: R131.2, U9.4 (-)
- new net Seuil_Ouvert_Backup: R132.2, U9.7 (+)
- new net Veh_Backup: Q35.2 (D), R129.1
Other:
- note added: "Backup_Vehic_Shunt_Haut"
- note removed: "Right_Vehic_Shunt_Haut"

Commit message: Add files via upload
Connections:
- net V_Ref: now also Q35.1 (G), R124.2
Changed lines of the file:
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@@
+	)
+	(junction
+		(at 113.03 87.63)
+		(diameter 0)
+		(color 0 0 0 0)
 	)
 	(junction
@@
 	(wire
 		(pts
-			(xy 116.84 87.63) (xy 114.3 87.63)
-		)
-		(stroke
-			(width 0)
-			(type default)
-		)
-	)
-	(wire
-		(pts
 			(xy 101.6 105.41) (xy 96.52 105.41)
 		)
@@
 		)
 		(stroke
+			(width 0)
+			(type default)
+		)
+	)
+	(wire
+		(pts
+			(xy 113.03 87.63) (xy 116.84 87.63)
+		)
+		(stroke

Commit message: Add files via upload
Connections:
- net V_Ref: no longer Q35.1 (G)
- net Veh_Backup_Inject_Cmd: now reaches R124.1, U9.2
- net Veh_Backup_Inject_Cmd: now also Q35.1 (G)
Changed lines of the file:
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@@
-	)
-	(junction
-		(at 113.03 87.63)
-		(diameter 0)
-		(color 0 0 0 0)
 	)
 	(junction
@@
 		(color 0 0 0 0)
 	)
+	(junction
+		(at 99.06 87.63)
+		(diameter 0)
+		(color 0 0 0 0)
+	)
 	(no_connect
 		(at 96.52 137.16)
@@
 	(wire
 		(pts
-			(xy 101.6 87.63) (xy 96.52 87.63)
+			(xy 101.6 87.63) (xy 99.06 87.63)
 		)
 		(stroke
@@
 	(wire
 		(pts
+			(xy 99.06 73.66) (xy 99.06 87.63)
+		)
+		(stroke
+			(width 0)
+			(type default)
+		)
+	)
+	(wire
+		(pts
 			(xy 119.38 101.6) (xy 119.38 105.41)
 		)
@@
 	(wire
 		(pts
+			(xy 99.06 87.63) (xy 96.52 87.63)
+		)
+		(stroke
+			(width 0)
+			(type default)
+		)
+	)
+	(wire
+		(pts
 			(xy 144.78 66.04) (xy 144.78 52.07)
 		)
@@
 	(wire
 		(pts
+			(xy 99.06 73.66) (xy 124.46 73.66)
+		)
+		(stroke
+			(width 0)
+			(type default)
+		)
+	)
+	(wire
+		(pts
 			(xy 182.88 60.96) (xy 185.42 60.96)
 		)
@@
 	(wire
 		(pts
-			(xy 124.46 73.66) (xy 113.03 73.66)
-		)
-		(stroke
-			(width 0)
-			(type default)
-		)
-	)
-	(wire
-		(pts
 			(xy 182.88 63.5) (xy 182.88 60.96)
 		)
@@
 	(wire
 		(pts
-			(xy 113.03 87.63) (xy 116.84 87.63)
-		)
-		(stroke
-			(width 0)
-			(type default)
-		)
-	)
-	(wire
-		(pts
-			(xy 113.03 73.66) (xy 113.03 87.63)
-		)
-		(stroke
-			(width 0)
-			(type default)
-		)
-	)
-	(wire
-		(pts
-			(xy 113.03 87.63) (xy 109.22 87.63)
+			(xy 109.22 87.63) (xy 116.84 87.63)
 		)
 		(stroke
@@
 		)
 	)
+	(label "Veh_Backup_Inject_Cmd"
+		(at 99.06 73.66 180)
+		(effects
+			(font
+				(size 1.016 1.016)
+			)
+			(justify right bottom)
+		)
+	)

Commit message: Add files via upload
Connections:
- net Veh_Backup_Inject_Cmd renamed Injection_Backup_Fault
Changed lines of the file:
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@@
+	)
+	(junction
+		(at 111.125 73.66)
+		(diameter 0)
+		(color 0 0 0 0)
 	)
 	(junction
@@
 	(wire
 		(pts
+			(xy 111.125 59.69) (xy 111.125 73.66)
+		)
+		(stroke
+			(width 0)
+			(type default)
+		)
+	)
+	(wire
+		(pts
 			(xy 99.06 73.66) (xy 99.06 87.63)
 		)
@@
 	(wire
 		(pts
-			(xy 99.06 73.66) (xy 124.46 73.66)
+			(xy 99.06 73.66) (xy 111.125 73.66)
 		)
 		(stroke
@@
 	(wire
 		(pts
+			(xy 104.14 59.69) (xy 111.125 59.69)
+		)
+		(stroke
+			(width 0)
+			(type default)
+		)
+	)
+	(wire
+		(pts
 			(xy 101.6 105.41) (xy 96.52 105.41)
 		)
@@
 		(pts
 			(xy 78.74 134.62) (xy 81.28 134.62)
+		)
+		(stroke
+			(width 0)
+			(type default)
+		)
+	)
+	(wire
+		(pts
+			(xy 111.125 73.66) (xy 124.46 73.66)
 		)
 		(stroke
@@
 		(effects
 			(font
+				(size 1.27 1.27)
+			)
+			(justify right)
+		)
+	)
+	(hierarchical_label "Injection_Backup_Fault"
+		(shape input)
+		(at 104.14 59.69 180)
+		(effects
+			(font

Commit message: Add files via upload
Changed lines of the file:
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@@
-		)
-	)
-	(label "Veh_Backup_Inject_Cmd"
-		(at 99.06 73.66 180)
-		(effects
-			(font
-				(size 1.016 1.016)
-			)
-			(justify right bottom)
 		)
 	)

Commit message: Add files via upload
Parts:
- R131, R132, R133: footprint (none) -> TRIM_3296W1103LF:TRIM_3296W1103LF
Changed lines of the file:
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@@
 			)
 		)
-		(property "Footprint" ""
+		(property "Footprint" "TRIM_3296W1103LF:TRIM_3296W1103LF"
 			(at 185.42 64.77 0)
 			(hide yes)
@@
 			)
 		)
-		(property "Footprint" ""
+		(property "Footprint" "TRIM_3296W1103LF:TRIM_3296W1103LF"
 			(at 185.42 101.6 0)
 			(hide yes)
@@
 			)
 		)
-		(property "Footprint" ""
+		(property "Footprint" "TRIM_3296W1103LF:TRIM_3296W1103LF"
 			(at 185.42 82.55 0)
 			(hide yes)

Commit message: Add files via upload
Parts:
- R131, R132, R133: footprint TRIM_3296W1103LF:TRIM_3296W1103LF -> (none)
Connections:
- net Injection_Backup_Fault renamed Veh_Backup_Inject_Cmd
Changed lines of the file:
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@@
-	)
-	(junction
-		(at 111.125 73.66)
-		(diameter 0)
-		(color 0 0 0 0)
 	)
 	(junction
@@
 	(wire
 		(pts
-			(xy 111.125 59.69) (xy 111.125 73.66)
-		)
-		(stroke
-			(width 0)
-			(type default)
-		)
-	)
-	(wire
-		(pts
 			(xy 99.06 73.66) (xy 99.06 87.63)
 		)
@@
 	(wire
 		(pts
-			(xy 99.06 73.66) (xy 111.125 73.66)
+			(xy 99.06 73.66) (xy 124.46 73.66)
 		)
 		(stroke
@@
 	(wire
 		(pts
-			(xy 104.14 59.69) (xy 111.125 59.69)
-		)
-		(stroke
-			(width 0)
-			(type default)
-		)
-	)
-	(wire
-		(pts
 			(xy 101.6 105.41) (xy 96.52 105.41)
 		)
@@
 		(pts
 			(xy 78.74 134.62) (xy 81.28 134.62)
-		)
-		(stroke
-			(width 0)
-			(type default)
-		)
-	)
-	(wire
-		(pts
-			(xy 111.125 73.66) (xy 124.46 73.66)
 		)
 		(stroke
@@
 			)
 			(justify left bottom)
+		)
+	)
+	(label "Veh_Backup_Inject_Cmd"
+		(at 99.06 73.66 180)
+		(effects
+			(font
+				(size 1.016 1.016)
+			)
+			(justify right bottom)
 		)
 	)
@@
 		(shape input)
 		(at 125.73 66.04 180)
-		(effects
-			(font
-				(size 1.27 1.27)
-			)
-			(justify right)
-		)
-	)
-	(hierarchical_label "Injection_Backup_Fault"
-		(shape input)
-		(at 104.14 59.69 180)
 		(effects
 			(font
@@
 			)
 		)
-		(property "Footprint" "TRIM_3296W1103LF:TRIM_3296W1103LF"
+		(property "Footprint" ""
 			(at 185.42 64.77 0)
 			(hide yes)
@@
 			)
 		)
-		(property "Footprint" "TRIM_3296W1103LF:TRIM_3296W1103LF"
+		(property "Footprint" ""
 			(at 185.42 101.6 0)
 			(hide yes)
@@
 			)
 		)
-		(property "Footprint" "TRIM_3296W1103LF:TRIM_3296W1103LF"
+		(property "Footprint" ""
 			(at 185.42 82.55 0)
 			(hide yes)

Commit message: Add files via upload
Parts:
- R122: value 3 Ohm - 5W -> 12 Ohm - 25W; footprint Resistor_THT:R_Axial_Power_L25.0mm_W9.0mm_P27.94mm -> TerminalBlock_Phoenix:TerminalBlock_Phoenix_PT-1,5-2-3.5-H_1x02_P3.50mm_Horizontal
- R123: value .05R Shunt -> 0.2 Ohm Shunt
- R131, R132, R133: footprint (none) -> TRIM_3296W1103LF:TRIM_3296W1103LF
Connections:
- net Veh_Backup_Inject_Cmd renamed Injection_Backup_Fault
Changed lines of the file:
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@@
+	)
+	(junction
+		(at 111.125 73.66)
+		(diameter 0)
+		(color 0 0 0 0)
 	)
 	(junction
@@
 	(wire
 		(pts
+			(xy 111.125 59.69) (xy 111.125 73.66)
+		)
+		(stroke
+			(width 0)
+			(type default)
+		)
+	)
+	(wire
+		(pts
 			(xy 99.06 73.66) (xy 99.06 87.63)
 		)
@@
 	(wire
 		(pts
-			(xy 99.06 73.66) (xy 124.46 73.66)
+			(xy 99.06 73.66) (xy 111.125 73.66)
 		)
 		(stroke
@@
 	(wire
 		(pts
+			(xy 104.14 59.69) (xy 111.125 59.69)
+		)
+		(stroke
+			(width 0)
+			(type default)
+		)
+	)
+	(wire
+		(pts
 			(xy 101.6 105.41) (xy 96.52 105.41)
 		)
@@
 		(pts
 			(xy 78.74 134.62) (xy 81.28 134.62)
+		)
+		(stroke
+			(width 0)
+			(type default)
+		)
+	)
+	(wire
+		(pts
+			(xy 111.125 73.66) (xy 124.46 73.66)
 		)
 		(stroke
@@
 			)
 			(justify left bottom)
-		)
-	)
-	(label "Veh_Backup_Inject_Cmd"
-		(at 99.06 73.66 180)
-		(effects
-			(font
-				(size 1.016 1.016)
-			)
-			(justify right bottom)
 		)
 	)
@@
 		(shape input)
 		(at 125.73 66.04 180)
+		(effects
+			(font
+				(size 1.27 1.27)
+			)
+			(justify right)
+		)
+	)
+	(hierarchical_label "Injection_Backup_Fault"
+		(shape input)
+		(at 104.14 59.69 180)
 		(effects
 			(font
@@
 			)
 		)
-		(property "Footprint" ""
+		(property "Footprint" "TRIM_3296W1103LF:TRIM_3296W1103LF"
 			(at 185.42 64.77 0)
 			(hide yes)
@@
 			)
 		)
-		(property "Value" ".05R Shunt"
+		(property "Value" "0.2 Ohm Shunt"
 			(at 64.77 146.05 0)
 			(show_name no)
@@
 			)
 		)
-		(property "Footprint" ""
+		(property "Footprint" "TRIM_3296W1103LF:TRIM_3296W1103LF"
 			(at 185.42 101.6 0)
 			(hide yes)
@@
 			)
 		)
-		(property "Value" "3 Ohm - 5W"
+		(property "Value" "12 Ohm - 25W"
 			(at 48.26 146.05 0)
 			(show_name no)
@@
 			)
 		)
-		(property "Footprint" "Resistor_THT:R_Axial_Power_L25.0mm_W9.0mm_P27.94mm"
+		(property "Footprint" "TerminalBlock_Phoenix:TerminalBlock_Phoenix_PT-1,5-2-3.5-H_1x02_P3.50mm_Horizontal"
 			(at 49.149 154.178 0)
 			(hide yes)
@@
 			)
 		)
-		(property "Description" "5W Resistor"
+		(property "Description" "25W Resistor"
 			(at 48.26 149.86 0)
 			(hide yes)
@@
 			)
 		)
-		(property "Footprint" ""
+		(property "Footprint" "TRIM_3296W1103LF:TRIM_3296W1103LF"
 			(at 185.42 82.55 0)
 			(hide yes)
