File: Vehicule_Backup.kicad_sch (KiCad schematic)
At the start: 16 parts, among them Q35 IRLZ44N, U9 LM339

Commit message: Add files via upload
Parts:
- R122: value 12 Ohm - 25W -> 3 Ohm - 5W; footprint TerminalBlock_Phoenix:TerminalBlock_Phoenix_PT-1,5-2-3.5-H_1x02_P3.50mm_Horizontal -> Resistor_THT:R_Axial_Power_L25.0mm_W9.0mm_P27.94mm
- R123: value 0.2 Ohm Shunt -> .05R Shunt
- R131, R132, R133: footprint TRIM_3296W1103LF:TRIM_3296W1103LF -> (none)
Connections:
- net Injection_Backup_Fault renamed Veh_Backup_Inject_Cmd
Changed lines of the file:
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@@
-	)
-	(junction
-		(at 111.125 73.66)
-		(diameter 0)
-		(color 0 0 0 0)
 	)
 	(junction
@@
 	(wire
 		(pts
-			(xy 111.125 59.69) (xy 111.125 73.66)
-		)
-		(stroke
-			(width 0)
-			(type default)
-		)
-	)
-	(wire
-		(pts
 			(xy 99.06 73.66) (xy 99.06 87.63)
 		)
@@
 	(wire
 		(pts
-			(xy 99.06 73.66) (xy 111.125 73.66)
+			(xy 99.06 73.66) (xy 124.46 73.66)
 		)
 		(stroke
@@
 	(wire
 		(pts
-			(xy 104.14 59.69) (xy 111.125 59.69)
-		)
-		(stroke
-			(width 0)
-			(type default)
-		)
-	)
-	(wire
-		(pts
 			(xy 101.6 105.41) (xy 96.52 105.41)
 		)
@@
 		(pts
 			(xy 78.74 134.62) (xy 81.28 134.62)
-		)
-		(stroke
-			(width 0)
-			(type default)
-		)
-	)
-	(wire
-		(pts
-			(xy 111.125 73.66) (xy 124.46 73.66)
 		)
 		(stroke
@@
 			)
 			(justify left bottom)
+		)
+	)
+	(label "Veh_Backup_Inject_Cmd"
+		(at 99.06 73.66 180)
+		(effects
+			(font
+				(size 1.016 1.016)
+			)
+			(justify right bottom)
 		)
 	)
@@
 		(shape input)
 		(at 125.73 66.04 180)
-		(effects
-			(font
-				(size 1.27 1.27)
-			)
-			(justify right)
-		)
-	)
-	(hierarchical_label "Injection_Backup_Fault"
-		(shape input)
-		(at 104.14 59.69 180)
 		(effects
 			(font
@@
 			)
 		)
-		(property "Footprint" "TRIM_3296W1103LF:TRIM_3296W1103LF"
+		(property "Footprint" ""
 			(at 185.42 64.77 0)
 			(hide yes)
@@
 			)
 		)
-		(property "Value" "0.2 Ohm Shunt"
+		(property "Value" ".05R Shunt"
 			(at 64.77 146.05 0)
 			(show_name no)
@@
 			)
 		)
-		(property "Footprint" "TRIM_3296W1103LF:TRIM_3296W1103LF"
+		(property "Footprint" ""
 			(at 185.42 101.6 0)
 			(hide yes)
@@
 			)
 		)
-		(property "Value" "12 Ohm - 25W"
+		(property "Value" "3 Ohm - 5W"
 			(at 48.26 146.05 0)
 			(show_name no)
@@
 			)
 		)
-		(property "Footprint" "TerminalBlock_Phoenix:TerminalBlock_Phoenix_PT-1,5-2-3.5-H_1x02_P3.50mm_Horizontal"
+		(property "Footprint" "Resistor_THT:R_Axial_Power_L25.0mm_W9.0mm_P27.94mm"
 			(at 49.149 154.178 0)
 			(hide yes)
@@
 			)
 		)
-		(property "Description" "25W Resistor"
+		(property "Description" "5W Resistor"
 			(at 48.26 149.86 0)
 			(hide yes)
@@
 			)
 		)
-		(property "Footprint" "TRIM_3296W1103LF:TRIM_3296W1103LF"
+		(property "Footprint" ""
 			(at 185.42 82.55 0)
 			(hide yes)

Commit message: Add files via upload
Parts:
- R131, R132, R133: footprint (none) -> TRIM_3296W1103LF:TRIM_3296W1103LF
Connections:
- net Veh_Backup_Inject_Cmd renamed Injection_Backup_Fault
Changed lines of the file:
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@@
+	)
+	(junction
+		(at 111.125 73.66)
+		(diameter 0)
+		(color 0 0 0 0)
 	)
 	(junction
@@
 	(wire
 		(pts
+			(xy 111.125 59.69) (xy 111.125 73.66)
+		)
+		(stroke
+			(width 0)
+			(type default)
+		)
+	)
+	(wire
+		(pts
 			(xy 99.06 73.66) (xy 99.06 87.63)
 		)
@@
 	(wire
 		(pts
-			(xy 99.06 73.66) (xy 124.46 73.66)
+			(xy 99.06 73.66) (xy 111.125 73.66)
 		)
 		(stroke
@@
 	(wire
 		(pts
+			(xy 104.14 59.69) (xy 111.125 59.69)
+		)
+		(stroke
+			(width 0)
+			(type default)
+		)
+	)
+	(wire
+		(pts
 			(xy 101.6 105.41) (xy 96.52 105.41)
 		)
@@
 		(pts
 			(xy 78.74 134.62) (xy 81.28 134.62)
+		)
+		(stroke
+			(width 0)
+			(type default)
+		)
+	)
+	(wire
+		(pts
+			(xy 111.125 73.66) (xy 124.46 73.66)
 		)
 		(stroke
@@
 			)
 			(justify left bottom)
-		)
-	)
-	(label "Veh_Backup_Inject_Cmd"
-		(at 99.06 73.66 180)
-		(effects
-			(font
-				(size 1.016 1.016)
-			)
-			(justify right bottom)
 		)
 	)
@@
 		(shape input)
 		(at 125.73 66.04 180)
+		(effects
+			(font
+				(size 1.27 1.27)
+			)
+			(justify right)
+		)
+	)
+	(hierarchical_label "Injection_Backup_Fault"
+		(shape input)
+		(at 104.14 59.69 180)
 		(effects
 			(font
@@
 			)
 		)
-		(property "Footprint" ""
+		(property "Footprint" "TRIM_3296W1103LF:TRIM_3296W1103LF"
 			(at 185.42 64.77 0)
 			(hide yes)
@@
 			)
 		)
-		(property "Footprint" ""
+		(property "Footprint" "TRIM_3296W1103LF:TRIM_3296W1103LF"
 			(at 185.42 101.6 0)
 			(hide yes)
@@
 			)
 		)
-		(property "Footprint" ""
+		(property "Footprint" "TRIM_3296W1103LF:TRIM_3296W1103LF"
 			(at 185.42 82.55 0)
 			(hide yes)

Commit message: Add files via upload
Parts:
- U9: footprint (none) -> Package_DIP:DIP-14_W7.62mm_Socket
Changed lines of the file:
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@@
 			)
 		)
-		(property "Footprint" ""
+		(property "Footprint" "Package_DIP:DIP-14_W7.62mm_Socket"
 			(at 87.63 102.87 0)
 			(hide yes)
@@
 			)
 		)
-		(property "Footprint" ""
+		(property "Footprint" "Package_DIP:DIP-14_W7.62mm_Socket"
 			(at 87.63 119.38 0)
 			(hide yes)
@@
 			)
 		)
-		(property "Footprint" ""
+		(property "Footprint" "Package_DIP:DIP-14_W7.62mm_Socket"
 			(at 87.63 85.09 0)
 			(hide yes)
@@
 			)
 		)
-		(property "Footprint" ""
+		(property "Footprint" "Package_DIP:DIP-14_W7.62mm_Socket"
 			(at 87.63 134.62 0)
 			(hide yes)
@@
 			)
 		)
-		(property "Footprint" ""
+		(property "Footprint" "Package_DIP:DIP-14_W7.62mm_Socket"
 			(at 85.09 152.4 0)
 			(hide yes)

Commit message: Add files via upload
Parts:
- U9: footprint Package_DIP:DIP-14_W7.62mm_Socket -> (none)
Changed lines of the file:
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@@
 			)
 		)
-		(property "Footprint" "Package_DIP:DIP-14_W7.62mm_Socket"
+		(property "Footprint" ""
 			(at 87.63 102.87 0)
 			(hide yes)
@@
 			)
 		)
-		(property "Footprint" "Package_DIP:DIP-14_W7.62mm_Socket"
+		(property "Footprint" ""
 			(at 87.63 119.38 0)
 			(hide yes)
@@
 			)
 		)
-		(property "Footprint" "Package_DIP:DIP-14_W7.62mm_Socket"
+		(property "Footprint" ""
 			(at 87.63 85.09 0)
 			(hide yes)
@@
 			)
 		)
-		(property "Footprint" "Package_DIP:DIP-14_W7.62mm_Socket"
+		(property "Footprint" ""
 			(at 87.63 134.62 0)
 			(hide yes)
@@
 			)
 		)
-		(property "Footprint" "Package_DIP:DIP-14_W7.62mm_Socket"
+		(property "Footprint" ""
 			(at 85.09 152.4 0)
 			(hide yes)

Commit message: Add files via upload
Parts:
- R122: value 3 Ohm - 5W -> 12 Ohm - 25W; footprint Resistor_THT:R_Axial_Power_L25.0mm_W9.0mm_P27.94mm -> TerminalBlock_Phoenix:TerminalBlock_Phoenix_PT-1,5-2-3.5-H_1x02_P3.50mm_Horizontal
- R123: value .05R Shunt -> 0.2 Ohm Shunt
Changed lines of the file:
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@@
 			)
 		)
-		(property "Value" ".05R Shunt"
+		(property "Value" "0.2 Ohm Shunt"
 			(at 64.77 146.05 0)
 			(show_name no)
@@
 			)
 		)
-		(property "Value" "3 Ohm - 5W"
+		(property "Value" "12 Ohm - 25W"
 			(at 48.26 146.05 0)
 			(show_name no)
@@
 			)
 		)
-		(property "Footprint" "Resistor_THT:R_Axial_Power_L25.0mm_W9.0mm_P27.94mm"
+		(property "Footprint" "TerminalBlock_Phoenix:TerminalBlock_Phoenix_PT-1,5-2-3.5-H_1x02_P3.50mm_Horizontal"
 			(at 49.149 154.178 0)
 			(hide yes)
@@
 			)
 		)
-		(property "Description" "5W Resistor"
+		(property "Description" "25W Resistor"
 			(at 48.26 149.86 0)
 			(hide yes)

Commit message: Add files via upload
Connections:
- net V_Ref: no longer OC7.2, OC8.2
- net Veh_Backup: now also R122.1; no longer Q35.2 (D)
- net Opto_Ouvert_Backup: now reaches R125.1, U9.1
- net Opto_Ouvert_Backup: now also OC8.2
- net Backup_Vehic_Shunt_Haut: now reaches R123.1, U9.11 (+), U9.6 (-)
- net Backup_Vehic_Shunt_Haut: now also Q35.3 (S); no longer R122.2
- net Opto_Court_Backup: now reaches R126.1, U9.13
- net Opto_Court_Backup: now also OC7.2
- removed net Q35_Source: Q35.3 (S), R122.1
- new net Q35_Drain: Q35.2 (D), R122.2
Other:
- note removed: "Backup_Vehic_Shunt_Haut"
- moved on the sheet: OC7, OC8, R122, R123, R127, R128, R129, R130, R131, R132, R133

Commit message: Add files via upload
Parts:
- U9: footprint (none) -> Package_DIP:DIP-14_W7.62mm_Socket
Changed lines of the file:
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@@
 			)
 		)
-		(property "Footprint" ""
+		(property "Footprint" "Package_DIP:DIP-14_W7.62mm_Socket"
 			(at 87.63 102.87 0)
 			(hide yes)
@@
 			)
 		)
-		(property "Footprint" ""
+		(property "Footprint" "Package_DIP:DIP-14_W7.62mm_Socket"
 			(at 87.63 119.38 0)
 			(hide yes)
@@
 			)
 		)
-		(property "Footprint" ""
+		(property "Footprint" "Package_DIP:DIP-14_W7.62mm_Socket"
 			(at 87.63 85.09 0)
 			(hide yes)
@@
 			)
 		)
-		(property "Footprint" ""
+		(property "Footprint" "Package_DIP:DIP-14_W7.62mm_Socket"
 			(at 87.63 134.62 0)
 			(hide yes)
@@
 			)
 		)
-		(property "Footprint" ""
+		(property "Footprint" "Package_DIP:DIP-14_W7.62mm_Socket"
 			(at 85.09 152.4 0)
 			(hide yes)

Commit message: Add files via upload
Other:
- note removed: "Injection"
