File: Vehicule_Tail.kicad_sch (KiCad schematic)
At the start: 16 parts, among them Q11 IRLZ44N, U2 LM339

Commit message: Add files via upload
Connections:
- net V_Ref: no longer Q11.1 (G)
- net Veh_Tail_Inject_Cmd: now reaches R26.1, U2.2
- net Veh_Tail_Inject_Cmd: now also Q11.1 (G)
Other:
- moved on the sheet: OC1, OC2, Q11, R21, R22, R23, R24, R25, R26, R27, R28, R29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

Commit message: Add files via upload
Connections:
- net Veh_Tail_Inject_Cmd renamed Injection_Tail_Fault
Changed lines of the file:
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@@
+	)
+	(junction
+		(at 121.92 57.15)
+		(diameter 0)
+		(color 0 0 0 0)
 	)
 	(junction
@@
 	(wire
 		(pts
+			(xy 121.92 45.72) (xy 121.92 57.15)
+		)
+		(stroke
+			(width 0)
+			(type default)
+		)
+	)
+	(wire
+		(pts
 			(xy 161.29 88.9) (xy 157.48 88.9)
 		)
@@
 	(wire
 		(pts
-			(xy 109.22 57.15) (xy 134.62 57.15)
-		)
-		(stroke
-			(width 0)
-			(type default)
-		)
-	)
-	(wire
-		(pts
 			(xy 190.5 44.45) (xy 195.58 44.45)
 		)
@@
 	(wire
 		(pts
+			(xy 109.22 57.15) (xy 121.92 57.15)
+		)
+		(stroke
+			(width 0)
+			(type default)
+		)
+	)
+	(wire
+		(pts
+			(xy 109.22 45.72) (xy 121.92 45.72)
+		)
+		(stroke
+			(width 0)
+			(type default)
+		)
+	)
+	(wire
+		(pts
 			(xy 88.9 68.58) (xy 91.44 68.58)
 		)
@@
 		(pts
 			(xy 135.89 49.53) (xy 140.97 49.53)
+		)
+		(stroke
+			(width 0)
+			(type default)
+		)
+	)
+	(wire
+		(pts
+			(xy 121.92 57.15) (xy 134.62 57.15)
 		)
 		(stroke
@@
 		(effects
 			(font
+				(size 1.27 1.27)
+			)
+			(justify right)
+		)
+	)
+	(hierarchical_label "Injection_Tail_Fault"
+		(shape input)
+		(at 109.22 45.72 180)
+		(effects
+			(font

Commit message: Add files via upload
Connections:
- net Injection_Tail_Fault renamed Veh_Tail_Inject_Cmd
Changed lines of the file:
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@@
-	)
-	(junction
-		(at 121.92 57.15)
-		(diameter 0)
-		(color 0 0 0 0)
 	)
 	(junction
@@
 	(wire
 		(pts
-			(xy 121.92 45.72) (xy 121.92 57.15)
-		)
-		(stroke
-			(width 0)
-			(type default)
-		)
-	)
-	(wire
-		(pts
 			(xy 161.29 88.9) (xy 157.48 88.9)
 		)
@@
 	(wire
 		(pts
+			(xy 109.22 57.15) (xy 134.62 57.15)
+		)
+		(stroke
+			(width 0)
+			(type default)
+		)
+	)
+	(wire
+		(pts
 			(xy 190.5 44.45) (xy 195.58 44.45)
 		)
@@
 	(wire
 		(pts
-			(xy 109.22 57.15) (xy 121.92 57.15)
-		)
-		(stroke
-			(width 0)
-			(type default)
-		)
-	)
-	(wire
-		(pts
-			(xy 109.22 45.72) (xy 121.92 45.72)
-		)
-		(stroke
-			(width 0)
-			(type default)
-		)
-	)
-	(wire
-		(pts
 			(xy 88.9 68.58) (xy 91.44 68.58)
 		)
@@
 		(pts
 			(xy 135.89 49.53) (xy 140.97 49.53)
-		)
-		(stroke
-			(width 0)
-			(type default)
-		)
-	)
-	(wire
-		(pts
-			(xy 121.92 57.15) (xy 134.62 57.15)
 		)
 		(stroke
@@
 		(effects
 			(font
-				(size 1.27 1.27)
-			)
-			(justify right)
-		)
-	)
-	(hierarchical_label "Injection_Tail_Fault"
-		(shape input)
-		(at 109.22 45.72 180)
-		(effects
-			(font

Commit message: Add files via upload
Parts:
- R23, R24, R25: footprint (none) -> TRIM_3296W1103LF:TRIM_3296W1103LF
Connections:
- net Veh_Tail_Inject_Cmd renamed Injection_Tail_Fault
Changed lines of the file:
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@@
+	)
+	(junction
+		(at 121.92 57.15)
+		(diameter 0)
+		(color 0 0 0 0)
 	)
 	(junction
@@
 	(wire
 		(pts
+			(xy 121.92 45.72) (xy 121.92 57.15)
+		)
+		(stroke
+			(width 0)
+			(type default)
+		)
+	)
+	(wire
+		(pts
 			(xy 161.29 88.9) (xy 157.48 88.9)
 		)
@@
 	(wire
 		(pts
-			(xy 109.22 57.15) (xy 134.62 57.15)
-		)
-		(stroke
-			(width 0)
-			(type default)
-		)
-	)
-	(wire
-		(pts
 			(xy 190.5 44.45) (xy 195.58 44.45)
 		)
@@
 	(wire
 		(pts
+			(xy 109.22 57.15) (xy 121.92 57.15)
+		)
+		(stroke
+			(width 0)
+			(type default)
+		)
+	)
+	(wire
+		(pts
+			(xy 109.22 45.72) (xy 121.92 45.72)
+		)
+		(stroke
+			(width 0)
+			(type default)
+		)
+	)
+	(wire
+		(pts
 			(xy 88.9 68.58) (xy 91.44 68.58)
 		)
@@
 		(pts
 			(xy 135.89 49.53) (xy 140.97 49.53)
+		)
+		(stroke
+			(width 0)
+			(type default)
+		)
+	)
+	(wire
+		(pts
+			(xy 121.92 57.15) (xy 134.62 57.15)
 		)
 		(stroke
@@
 	(label "Seuil_Ouvert"
 		(at 91.44 86.36 180)
-		(effects
-			(font
-				(size 1.27 1.27)
-			)
-			(justify right bottom)
-		)
-	)
-	(label "Veh_Tail_Inject_Cmd"
-		(at 109.22 57.15 180)
 		(effects
 			(font
@@
 		(shape input)
 		(at 135.89 49.53 180)
+		(effects
+			(font
+				(size 1.27 1.27)
+			)
+			(justify right)
+		)
+	)
+	(hierarchical_label "Injection_Tail_Fault"
+		(shape input)
+		(at 109.22 45.72 180)
 		(effects
 			(font
@@
 			)
 		)
-		(property "Footprint" ""
+		(property "Footprint" "TRIM_3296W1103LF:TRIM_3296W1103LF"
 			(at 195.58 66.04 0)
 			(hide yes)
@@
 			)
 		)
-		(property "Footprint" ""
+		(property "Footprint" "TRIM_3296W1103LF:TRIM_3296W1103LF"
 			(at 195.58 48.26 0)
 			(hide yes)
@@
 			)
 		)
-		(property "Footprint" ""
+		(property "Footprint" "TRIM_3296W1103LF:TRIM_3296W1103LF"
 			(at 195.58 85.09 0)
 			(hide yes)

Commit message: Add files via upload
Parts:
- U2: footprint (none) -> Package_DIP:DIP-14_W7.62mm_Socket
Changed lines of the file:
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@@
 			)
 		)
-		(property "Footprint" ""
+		(property "Footprint" "Package_DIP:DIP-14_W7.62mm_Socket"
 			(at 95.25 135.89 0)
 			(hide yes)
@@
 			)
 		)
-		(property "Footprint" ""
+		(property "Footprint" "Package_DIP:DIP-14_W7.62mm_Socket"
 			(at 97.79 102.87 0)
 			(hide yes)
@@
 			)
 		)
-		(property "Footprint" ""
+		(property "Footprint" "Package_DIP:DIP-14_W7.62mm_Socket"
 			(at 97.79 68.58 0)
 			(hide yes)
@@
 			)
 		)
-		(property "Footprint" ""
+		(property "Footprint" "Package_DIP:DIP-14_W7.62mm_Socket"
 			(at 97.79 86.36 0)
 			(hide yes)
@@
 			)
 		)
-		(property "Footprint" ""
+		(property "Footprint" "Package_DIP:DIP-14_W7.62mm_Socket"
 			(at 97.79 118.11 0)
 			(hide yes)

Commit message: Add files via upload
Parts:
- U2: footprint Package_DIP:DIP-14_W7.62mm_Socket -> (none)
Changed lines of the file:
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@@
 			)
 		)
-		(property "Footprint" "Package_DIP:DIP-14_W7.62mm_Socket"
+		(property "Footprint" ""
 			(at 95.25 135.89 0)
 			(hide yes)
@@
 			)
 		)
-		(property "Footprint" "Package_DIP:DIP-14_W7.62mm_Socket"
+		(property "Footprint" ""
 			(at 97.79 102.87 0)
 			(hide yes)
@@
 			)
 		)
-		(property "Footprint" "Package_DIP:DIP-14_W7.62mm_Socket"
+		(property "Footprint" ""
 			(at 97.79 68.58 0)
 			(hide yes)
@@
 			)
 		)
-		(property "Footprint" "Package_DIP:DIP-14_W7.62mm_Socket"
+		(property "Footprint" ""
 			(at 97.79 86.36 0)
 			(hide yes)
@@
 			)
 		)
-		(property "Footprint" "Package_DIP:DIP-14_W7.62mm_Socket"
+		(property "Footprint" ""
 			(at 97.79 118.11 0)
 			(hide yes)

Commit message: Add files via upload
Parts:
- R23, R24, R25: footprint TRIM_3296W1103LF:TRIM_3296W1103LF -> (none)
Connections:
- net Injection_Tail_Fault renamed Veh_Tail_Inject_Cmd
Changed lines of the file:
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@@
-	)
-	(junction
-		(at 121.92 57.15)
-		(diameter 0)
-		(color 0 0 0 0)
 	)
 	(junction
@@
 	(wire
 		(pts
-			(xy 121.92 45.72) (xy 121.92 57.15)
-		)
-		(stroke
-			(width 0)
-			(type default)
-		)
-	)
-	(wire
-		(pts
 			(xy 161.29 88.9) (xy 157.48 88.9)
 		)
@@
 	(wire
 		(pts
+			(xy 109.22 57.15) (xy 134.62 57.15)
+		)
+		(stroke
+			(width 0)
+			(type default)
+		)
+	)
+	(wire
+		(pts
 			(xy 190.5 44.45) (xy 195.58 44.45)
 		)
@@
 	(wire
 		(pts
-			(xy 109.22 57.15) (xy 121.92 57.15)
-		)
-		(stroke
-			(width 0)
-			(type default)
-		)
-	)
-	(wire
-		(pts
-			(xy 109.22 45.72) (xy 121.92 45.72)
-		)
-		(stroke
-			(width 0)
-			(type default)
-		)
-	)
-	(wire
-		(pts
 			(xy 88.9 68.58) (xy 91.44 68.58)
 		)
@@
 		(pts
 			(xy 135.89 49.53) (xy 140.97 49.53)
-		)
-		(stroke
-			(width 0)
-			(type default)
-		)
-	)
-	(wire
-		(pts
-			(xy 121.92 57.15) (xy 134.62 57.15)
 		)
 		(stroke
@@
 	(label "Seuil_Ouvert"
 		(at 91.44 86.36 180)
+		(effects
+			(font
+				(size 1.27 1.27)
+			)
+			(justify right bottom)
+		)
+	)
+	(label "Veh_Tail_Inject_Cmd"
+		(at 109.22 57.15 180)
 		(effects
 			(font
@@
 		(shape input)
 		(at 135.89 49.53 180)
-		(effects
-			(font
-				(size 1.27 1.27)
-			)
-			(justify right)
-		)
-	)
-	(hierarchical_label "Injection_Tail_Fault"
-		(shape input)
-		(at 109.22 45.72 180)
 		(effects
 			(font
@@
 			)
 		)
-		(property "Footprint" "TRIM_3296W1103LF:TRIM_3296W1103LF"
+		(property "Footprint" ""
 			(at 195.58 66.04 0)
 			(hide yes)
@@
 			)
 		)
-		(property "Footprint" "TRIM_3296W1103LF:TRIM_3296W1103LF"
+		(property "Footprint" ""
 			(at 195.58 48.26 0)
 			(hide yes)
@@
 			)
 		)
-		(property "Footprint" "TRIM_3296W1103LF:TRIM_3296W1103LF"
+		(property "Footprint" ""
 			(at 195.58 85.09 0)
 			(hide yes)

Commit message: Add files via upload
Parts:
- R21: value 3 Ohm - 5W -> 12 Ohm - 25W; footprint Resistor_THT:R_Axial_Power_L25.0mm_W9.0mm_P27.94mm -> TerminalBlock_Phoenix:TerminalBlock_Phoenix_PT-1,5-2-3.5-H_1x02_P3.50mm_Horizontal
- R22: value .05R Shunt -> 0.2 Ohm Shunt
- R23, R24, R25: footprint (none) -> TRIM_3296W1103LF:TRIM_3296W1103LF
Connections:
- net V_Ref: no longer OC1.2, OC2.2
- net Veh_Tail: now also R21.1; no longer Q11.2 (D)
- net at R27.1, U2.1: now also OC1.2
- net Tail_Vehic_Shunt_Haut: now reaches R22.1, U2.11 (+), U2.6 (-)
- net Tail_Vehic_Shunt_Haut: now also Q11.3 (S); no longer R21.2
- net at R28.1, U2.13: now also OC2.2
- removed net Q11_Source: Q11.3 (S), R21.1
- net Veh_Tail_Inject_Cmd renamed Injection_Tail_Fault
- new net Q11_Drain: Q11.2 (D), R21.2
Other:
- note removed: "Tail_Vehic_Shunt_Haut"
- moved on the sheet: R21, R22
