File: Vehicule_Tail.kicad_sch (KiCad schematic)
At the start: 16 parts, among them Q11 IRLZ44N, U2 LM339

Commit message: Add files via upload
Parts:
- R23, R24, R25: footprint (none) -> TRIM_3296W1103LF:TRIM_3296W1103LF
Changed lines of the file:
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@@
 			)
 		)
-		(property "Footprint" ""
+		(property "Footprint" "TRIM_3296W1103LF:TRIM_3296W1103LF"
 			(at 195.58 66.04 0)
 			(hide yes)
@@
 			)
 		)
-		(property "Footprint" ""
+		(property "Footprint" "TRIM_3296W1103LF:TRIM_3296W1103LF"
 			(at 195.58 48.26 0)
 			(hide yes)
@@
 			)
 		)
-		(property "Footprint" ""
+		(property "Footprint" "TRIM_3296W1103LF:TRIM_3296W1103LF"
 			(at 195.58 85.09 0)
 			(hide yes)

Commit message: Add files via upload
Parts:
- R21: value 3 Ohm - 5W -> 12 Ohm - 25W; footprint Resistor_THT:R_Axial_Power_L25.0mm_W9.0mm_P27.94mm -> TerminalBlock_Phoenix:TerminalBlock_Phoenix_PT-1,5-2-3.5-H_1x02_P3.50mm_Horizontal
- R22: value .05R Shunt -> 0.2 Ohm Shunt
Changed lines of the file:
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@@
 			)
 		)
-		(property "Value" "3 Ohm - 5W"
+		(property "Value" "12 Ohm - 25W"
 			(at 58.42 129.54 0)
 			(show_name no)
@@
 			)
 		)
-		(property "Footprint" "Resistor_THT:R_Axial_Power_L25.0mm_W9.0mm_P27.94mm"
+		(property "Footprint" "TerminalBlock_Phoenix:TerminalBlock_Phoenix_PT-1,5-2-3.5-H_1x02_P3.50mm_Horizontal"
 			(at 59.309 137.668 0)
 			(hide yes)
@@
 			)
 		)
-		(property "Description" "5W Resistor"
+		(property "Description" "25W Resistor"
 			(at 58.42 133.35 0)
 			(hide yes)
@@
 			)
 		)
-		(property "Value" ".05R Shunt"
+		(property "Value" "0.2 Ohm Shunt"
 			(at 74.93 129.54 0)
 			(show_name no)

Commit message: Add files via upload
Connections:
- net V_Ref: no longer OC1.2, OC2.2
- net Veh_Tail: now also R21.1; no longer Q11.2 (D), R37.1
- net at R27.1, U2.1: now also OC1.2
- net at U2.11 (+), U2.6 (-): no longer R21.2, R22.1
- net at R28.1, U2.13: now also OC2.2
- net Q11_Source renamed Tail_Vehic_Shunt_Haut
- net Tail_Vehic_Shunt_Haut: now also R22.1; no longer R21.1
- new net Q11_Drain: Q11.2 (D), R21.2, R37.1
Other:
- note removed: "Tail_Vehic_Shunt_Haut"
- moved on the sheet: R21, R22

Commit message: Add files via upload
Connections:
- net Q11_Drain: no longer R37.1
- net Tail_Vehic_Shunt_Haut: now also U2.11 (+), U2.6 (-)
- net Veh_Tail: now also R37.1
Changed lines of the file:
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@@
 	)
 	(junction
-		(at 140.97 49.53)
+		(at 67.31 97.79)
 		(diameter 0)
 		(color 0 0 0 0)
@@
 	(wire
 		(pts
+			(xy 67.31 97.79) (xy 67.31 102.87)
+		)
+		(stroke
+			(width 0)
+			(type default)
+		)
+	)
+	(wire
+		(pts
 			(xy 191.77 88.9) (xy 195.58 88.9)
 		)
@@
 	(wire
 		(pts
-			(xy 67.31 91.44) (xy 67.31 102.87)
+			(xy 67.31 91.44) (xy 67.31 97.79)
 		)
 		(stroke
@@
 	(wire
 		(pts
+			(xy 62.23 97.79) (xy 67.31 97.79)
+		)
+		(stroke
+			(width 0)
+			(type default)
+		)
+	)
+	(wire
+		(pts
 			(xy 161.29 88.9) (xy 157.48 88.9)
 		)
@@
 	(wire
 		(pts
-			(xy 140.97 49.53) (xy 144.78 49.53)
-		)
-		(stroke
-			(width 0)
-			(type default)
-		)
-	)
-	(wire
-		(pts
 			(xy 109.22 57.15) (xy 109.22 71.12)
 		)
@@
 	(wire
 		(pts
+			(xy 144.78 43.18) (xy 144.78 49.53)
+		)
+		(stroke
+			(width 0)
+			(type default)
+		)
+	)
+	(wire
+		(pts
 			(xy 109.22 91.44) (xy 109.22 88.9)
 		)
@@
 		(pts
 			(xy 109.22 110.49) (xy 140.97 110.49)
+		)
+		(stroke
+			(width 0)
+			(type default)
+		)
+	)
+	(wire
+		(pts
+			(xy 135.89 43.18) (xy 144.78 43.18)
 		)
 		(stroke
@@
 		)
 	)
+	(label "Tail_Vehic_Shunt_Haut"
+		(at 62.23 97.79 180)
+		(effects
+			(font
+				(size 1.27 1.27)
+			)
+			(justify right bottom)
+		)
+	)
 	(label "Seuil_Injection"
 		(at 199.39 48.26 0)
@@
 	(hierarchical_label "Veh_Tail"
 		(shape input)
+		(at 135.89 43.18 180)
+		(effects
+			(font
+				(size 1.27 1.27)
+			)
+			(justify right)
+		)
+	)
+	(hierarchical_label "Veh_Tail"
+		(shape input)
 		(at 54.61 156.21 180)
 		(effects
 			(font
-				(size 1.27 1.27)
-			)
-			(justify right)
-		)
-	)
-	(hierarchical_label "Veh_Tail"
-		(shape input)
-		(at 49.53 49.53 180)
-		(effects
-			(font

Commit message: Add files via upload
Parts:
- U2: footprint (none) -> Package_DIP:DIP-14_W7.62mm_Socket
Changed lines of the file:
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@@
 			)
 		)
-		(property "Footprint" ""
+		(property "Footprint" "Package_DIP:DIP-14_W7.62mm_Socket"
 			(at 95.25 135.89 0)
 			(hide yes)
@@
 			)
 		)
-		(property "Footprint" ""
+		(property "Footprint" "Package_DIP:DIP-14_W7.62mm_Socket"
 			(at 97.79 102.87 0)
 			(hide yes)
@@
 			)
 		)
-		(property "Footprint" ""
+		(property "Footprint" "Package_DIP:DIP-14_W7.62mm_Socket"
 			(at 97.79 68.58 0)
 			(hide yes)
@@
 			)
 		)
-		(property "Footprint" ""
+		(property "Footprint" "Package_DIP:DIP-14_W7.62mm_Socket"
 			(at 97.79 86.36 0)
 			(hide yes)
@@
 			)
 		)
-		(property "Footprint" ""
+		(property "Footprint" "Package_DIP:DIP-14_W7.62mm_Socket"
 			(at 97.79 118.11 0)
 			(hide yes)

Commit message: Add files via upload
Changed lines of the file:
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@@
 	(wire
 		(pts
-			(xy 154.94 35.56) (xy 88.9 35.56)
+			(xy 154.94 35.56) (xy 86.36 35.56)
 		)
 		(stroke
@@
 	(wire
 		(pts
-			(xy 88.9 68.58) (xy 91.44 68.58)
+			(xy 86.36 68.58) (xy 91.44 68.58)
 		)
 		(stroke
@@
 	(wire
 		(pts
-			(xy 88.9 35.56) (xy 88.9 68.58)
+			(xy 86.36 35.56) (xy 86.36 68.58)
 		)
 		(stroke
@@
 		)
 	)
+	(label "Injection_Tail_Fault"
+		(at 109.22 45.72 180)
+		(effects
+			(font
+				(size 1.27 1.27)
+			)
+			(justify right bottom)
+		)
+	)
 	(label "Seuil_Ouvert"
 		(at 91.44 86.36 180)
@@
 		)
 	)
-	(hierarchical_label "Injection_Tail_Fault"
-		(shape input)
-		(at 109.22 45.72 180)
-		(effects
-			(font
-				(size 1.27 1.27)
-			)
-			(justify right)
-		)
-	)

Commit message: Add files via upload
Parts:
- R26, R27, R28: value 4.7k -> 4.7kΩ
- R29, R30: value 1k -> 1kΩ
- R37: value 100k -> 100kΩ
- R38: value 10k -> 10kΩ
Changed lines of the file:
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@@
 			)
 		)
-		(property "Value" "1k"
+		(property "Value" "1kΩ"
 			(at 137.16 95.25 0)
 			(show_name no)
@@
 			)
 		)
-		(property "Value" "100k"
+		(property "Value" "100kΩ"
 			(at 148.59 45.72 0)
 			(show_name no)
@@
 			)
 		)
-		(property "Value" "4.7k"
+		(property "Value" "4.7kΩ"
 			(at 115.57 85.09 0)
 			(show_name no)
@@
 			)
 		)
-		(property "Value" "10k"
+		(property "Value" "10kΩ"
 			(at 160.02 45.72 0)
 			(show_name no)
@@
 			)
 		)
-		(property "Value" "4.7k"
+		(property "Value" "4.7kΩ"
 			(at 115.57 67.31 0)
 			(show_name no)
@@
 			)
 		)
-		(property "Value" "4.7k"
+		(property "Value" "4.7kΩ"
 			(at 115.57 101.6 0)
 			(show_name no)
@@
 			)
 		)
-		(property "Value" "1k"
+		(property "Value" "1kΩ"
 			(at 140.97 73.66 0)
 			(show_name no)
