File: Bloc_Test_Brake.kicad_sch (KiCad schematic)
At the start: 44 parts, among them Q13 2N7000, Q14 2N7000, Q15 2N7000, Q16 2N7000, Q17 2N7000, Q18 2N7000

Commit message: Add files via upload
Connections:
- net Fault_Actif: now reaches D44.1 (K), D45.1 (K), D48.1 (K), Q17.2 (G), R48.1
- net Vert_Enable: now reaches Q17.3 (D), R52.2
- net Vert_Enable: now also Q16.2 (G)
- net Bleu_Tail renamed Bleu_Brake
- net Court_Tail renamed Court_Brake
- net Not_Btn_Tail renamed Not_Btn_Brake
- net Ouvert_Tail renamed Ouvert_Brake
Other:
- note added: "Court_Brake (Porte OU #1)"
- note added: "Ouvet_Brake (Porte OU #2)"
- note added: "Porte ET #5 (Bleu_Brake)"
- note removed: "Court_Tail (Porte OU #1)"
- note removed: "Fault_Actif"
- note removed: "Ouvet_Tail (Porte OU #2)"
- note removed: "Porte ET #5 (Bleu_Tail)"
- note removed: "Vert_Enable"
- moved on the sheet: Q16, R49

Commit message: Add files via upload
Connections:
- net Court_T_Actif: now also D38.2 (A), D39.2 (A), R43.1
- net Court_V_Actif: now also D29.2 (A), D30.2 (A), R39.1
- net Ouvert_T_Actif: now also D35.2 (A), D36.2 (A), D37.2 (A), R42.1
- net Ouvert_V_Actif: now also D27.2 (A), D28.2 (A), R66.1
Other:
- moved on the sheet: D40, D41, R39, R42, R43, R44, R66

Commit message: Add files via upload
Connections:
- net Court_T_Actif renamed Court_T_Actif_Brake
- net Court_V_Actif renamed Court_V_Actif_Brake
- net Fault_Actif renamed Fault_Actif_Brake
- net Ouvert_T_Actif renamed Ouvert_T_Actif_Brake
- net Ouvert_V_Actif renamed Ouvert_V_Actif_Brake
- net Vert_Enable renamed Vert_Enale_Brake
Other:
- note added: "Ouvert_T_Actif_Brake (Porte ET #4 - 3 entrées)"
- note removed: "Ouvert_T_Actif (Porte ET #4 - 3 entrées)"
- moved on the sheet: D49, Q16, R49
Changed lines of the file:
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@@
 	)
 	(rectangle
-		(start 175.26 13.97)
-		(end 213.36 46.99)
+		(start 184.658 15.748)
+		(end 228.854 48.768)
 		(stroke
 			(width 0)
@@
 	)
 	(rectangle
-		(start 217.17 16.51)
-		(end 246.38 45.72)
+		(start 236.474 15.494)
+		(end 265.684 44.704)
 		(stroke
 			(width 0)
@@
 		)
 	)
-	(text "Ouvert_T_Actif\n(Porte ET #4 - 3 entrées)"
+	(text "Ouvert_T_Actif_Brake\n(Porte ET #4 - 3 entrées)"
 		(exclude_from_sim yes)
 		(at 97.79 55.88 0)
@@
 	(wire
 		(pts
-			(xy 195.58 36.83) (xy 195.58 39.37)
+			(xy 211.074 38.608) (xy 211.074 41.148)
 		)
 		(stroke
@@
 	(wire
 		(pts
-			(xy 195.58 39.37) (xy 191.77 39.37)
+			(xy 211.074 41.148) (xy 207.264 41.148)
 		)
 		(stroke
@@
 	(wire
 		(pts
-			(xy 195.58 22.86) (xy 196.85 22.86)
+			(xy 211.074 24.638) (xy 212.344 24.638)
 		)
 		(stroke
@@
 	(wire
 		(pts
-			(xy 195.58 26.67) (xy 195.58 22.86)
+			(xy 211.074 28.448) (xy 211.074 24.638)
 		)
 		(stroke
@@
 	)
 	(label "R_Lim_B"
-		(at 227.33 38.1 180)
+		(at 246.634 37.084 180)
 		(effects
 			(font
@@
 		)
 	)
-	(label "Ouvert_V_Actif"
+	(label "Ouvert_V_Actif_Brake"
 		(at 83.82 158.75 180)
 		(effects
@@
 	)
 	(label "R_Lim_R"
-		(at 227.33 27.94 180)
+		(at 246.634 26.924 180)
 		(effects
 			(font
@@
 	)
 	(label "R_Lim_G"
-		(at 227.33 33.02 180)
+		(at 246.634 32.004 180)
 		(effects
 			(font
@@
 		)
 	)
-	(label "Court_V_Actif"
+	(label "Court_V_Actif_Brake"
 		(at 45.72 158.75 180)
 		(effects
@@
 		)
 	)
-	(label "Court_T_Actif"
+	(label "Court_T_Actif_Brake"
 		(at 95.25 50.8 0)
 		(effects
@@
 		)
 	)
-	(label "Ouvert_V_Actif"
+	(label "Ouvert_V_Actif_Brake"
 		(at 49.53 93.98 0)
 		(effects
@@
 		)
 	)
-	(label "Vert_Enable"
+	(label "Vert_Enale_Brake"
 		(at 224.79 146.05 0)
 		(effects
@@
 		)
 	)
-	(label "Ouvert_T_Actif"
+	(label "Ouvert_T_Actif_Brake"
 		(at 83.82 170.18 180)
 		(effects
@@
 		)
 	)
-	(label "Vert_Enable"
-		(at 187.96 31.75 180)
+	(label "Vert_Enale_Brake"
+		(at 203.454 33.528 180)
 		(effects
 			(font
@@
 		)
 	)
-	(label "Court_T_Actif"
+	(label "Court_T_Actif_Brake"
 		(at 45.72 170.18 180)
 		(effects
@@
 		)
 	)
-	(label "Fault_Actif"
+	(label "Fault_Actif_Brake"
 		(at 198.12 120.65 0)
 		(effects
@@
 		)
 	)
-	(label "Court_V_Actif"
+	(label "Court_V_Actif_Brake"
 		(at 50.8 50.8 0)
 		(effects
@@
 		)
 	)
-	(label "Ouvert_T_Actif"
+	(label "Ouvert_T_Actif_Brake"
 		(at 93.98 102.87 0)
 		(effects
@@
 	)
 	(label "R_Lim_G"
-		(at 204.47 22.86 0)
+		(at 219.964 24.638 0)
 		(effects
 			(font
@@
 	(global_label "GND"
 		(shape input)
-		(at 191.77 39.37 180)
+		(at 207.264 41.148 180)
 		(fields_autoplaced yes)
 		(effects
@@
 		)
 		(property "Intersheetrefs" "${INTERSHEET_REFS}"
-			(at 184.9143 39.37 0)
+			(at 200.4083 41.148 0)
 			(hide yes)
 			(show_name no)
@@
 	(global_label "V_Ref"
 		(shape input)
-		(at 237.49 33.02 0)
+		(at 256.794 32.004 0)
 		(fields_autoplaced yes)
 		(effects
@@
 		)
 		(property "Intersheetrefs" "${INTERSHEET_REFS}"
-			(at 245.6157 33.02 0)
+			(at 264.9197 32.004 0)
 			(hide yes)
 			(show_name no)
@@
 	(symbol
 		(lib_id "PCM_SL_Resistors:330ohm")
-		(at 200.66 22.86 0)
+		(at 216.154 24.638 0)
 		(unit 1)
 		(body_style 1)
@@
 		(fields_autoplaced yes)
 		(property "Reference" "R49"
-			(at 200.66 16.51 0)
+			(at 216.154 18.288 0)
 			(show_name no)
 			(do_not_autoplace no)
@@
 		)
 		(property "Value" "330ohm"
-			(at 200.66 19.05 0)
+			(at 216.154 20.828 0)
 			(show_name no)
 			(do_not_autoplace no)
@@
 		)
 		(property "Footprint" "Resistor_THT:R_Axial_DIN0207_L6.3mm_D2.5mm_P10.16mm_Horizontal"
-			(at 201.549 27.178 0)
+			(at 217.043 28.956 0)
 			(hide yes)
 			(show_name no)
@@
 		)
 		(property "Datasheet" ""
-			(at 201.168 22.86 0)
+			(at 216.662 24.638 0)
 			(hide yes)
 			(show_name no)
@@
 		)
 		(property "Description" "330Ω, 1/4W Resistor"
-			(at 200.66 22.86 0)
+			(at 216.154 24.638 0)
 			(hide yes)
 			(show_name no)
@@
 	(symbol
 		(lib_id "Transistor_FET:2N7000")
-		(at 193.04 31.75 0)
+		(at 208.534 33.528 0)
 		(unit 1)
 		(body_style 1)
@@
 		(dnp no)
 		(property "Reference" "Q16"
-			(at 199.39 30.4799 0)
+			(at 214.884 32.2579 0)
 			(show_name no)
 			(do_not_autoplace no)
@@
 		)
 		(property "Value" "2N7000"
-			(at 198.12 33.02 0)
+			(at 213.614 34.798 0)
 			(show_name no)
 			(do_not_autoplace no)
@@
 		)
 		(property "Footprint" "Package_TO_SOT_THT:TO-92_Inline"
-			(at 198.12 33.655 0)
+			(at 213.614 35.433 0)
 			(hide yes)
 			(show_name no)
@@
 		)
 		(property "Datasheet" "https://www.vishay.com/docs/70226/70226.pdf"
-			(at 198.12 35.56 0)
+			(at 213.614 37.338 0)
 			(hide yes)
 			(show_name no)
@@
 		)
 		(property "Description" "0.2A Id, 200V Vds, N-Channel MOSFET, 2.6V Logic Level, TO-92"
-			(at 193.04 31.75 0)
+			(at 208.534 33.528 0)
 			(hide yes)
 			(show_name no)
@@
 	(symbol
 		(lib_id "Device:LED_ARGB")
-		(at 232.41 33.02 0)
+		(at 251.714 32.004 0)
 		(unit 1)
 		(body_style 1)
@@
 		(fields_autoplaced yes)
 		(property "Reference" "D49"
-			(at 232.41 19.05 0)
+			(at 251.714 18.034 0)
 			(show_name no)
 			(do_not_autoplace no)
@@
 		)
 		(property "Value" "LED_ARGB"
-			(at 232.41 21.59 0)
+			(at 251.714 20.574 0)
 			(show_name no)
 			(do_not_autoplace no)
@@
 		)
 		(property "Footprint" ""
-			(at 232.41 34.29 0)
+			(at 251.714 33.274 0)
 			(hide yes)
 			(show_name no)
@@
 		)
 		(property "Datasheet" ""
-			(at 232.41 34.29 0)
+			(at 251.714 33.274 0)
 			(hide yes)
 			(show_name no)
@@
 		)
 		(property "Description" "RGB LED, anode/red/green/blue"
-			(at 232.41 33.02 0)
+			(at 251.714 32.004 0)
 			(hide yes)
 			(show_name no)

Commit message: Add files via upload
Connections:
- net Vert_Enale_Brake: no longer Q16.2 (G)
- new net Vert_Enable_Brake: Q16.2 (G)
Changed lines of the file:
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@@
 		)
 	)
-	(label "Vert_Enale_Brake"
+	(label "Vert_Enable_Brake"
 		(at 203.454 33.528 180)
 		(effects

Commit message: Add files via upload
Connections:
- net Vert_Enale_Brake is gone; now on net Vert_Enable_Brake: Q17.3 (D), R52.2
Changed lines of the file:
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@@
 		)
 	)
-	(label "Vert_Enale_Brake"
+	(label "Vert_Enable_Brake"
 		(at 224.79 146.05 0)
 		(effects

Commit message: Add files via upload
Connections:
- net Court_T_Actif_Brake renamed Court_T_Actif
- net Court_V_Actif_Brake renamed Court_V_Actif
- net Fault_Actif_Brake renamed Fault_Actif
- net Ouvert_T_Actif_Brake renamed Ouvert_T_Actif
- net Ouvert_V_Actif_Brake renamed Ouvert_V_Actif
- net Vert_Enable_Brake renamed Vert_Enable
Other:
- note added: "Ouvert_T_Actif (Porte ET #4 - 3 entrées)"
- note removed: "Ouvert_T_Actif_Brake (Porte ET #4 - 3 entrées)"
- moved on the sheet: D49, Q16, R49
Changed lines of the file:
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@@
 	)
 	(rectangle
-		(start 184.658 15.748)
-		(end 228.854 48.768)
+		(start 175.26 13.97)
+		(end 213.36 46.99)
 		(stroke
 			(width 0)
@@
 	)
 	(rectangle
-		(start 236.474 15.494)
-		(end 265.684 44.704)
+		(start 217.17 16.51)
+		(end 246.38 45.72)
 		(stroke
 			(width 0)
@@
 		)
 	)
-	(text "Ouvert_T_Actif_Brake\n(Porte ET #4 - 3 entrées)"
+	(text "Ouvert_T_Actif\n(Porte ET #4 - 3 entrées)"
 		(exclude_from_sim yes)
 		(at 97.79 55.88 0)
@@
 	(wire
 		(pts
-			(xy 211.074 38.608) (xy 211.074 41.148)
+			(xy 195.58 36.83) (xy 195.58 39.37)
 		)
 		(stroke
@@
 	(wire
 		(pts
-			(xy 211.074 41.148) (xy 207.264 41.148)
+			(xy 195.58 39.37) (xy 191.77 39.37)
 		)
 		(stroke
@@
 	(wire
 		(pts
-			(xy 211.074 24.638) (xy 212.344 24.638)
+			(xy 195.58 22.86) (xy 196.85 22.86)
 		)
 		(stroke
@@
 	(wire
 		(pts
-			(xy 211.074 28.448) (xy 211.074 24.638)
+			(xy 195.58 26.67) (xy 195.58 22.86)
 		)
 		(stroke
@@
 	)
 	(label "R_Lim_B"
-		(at 246.634 37.084 180)
+		(at 227.33 38.1 180)
 		(effects
 			(font
@@
 		)
 	)
-	(label "Ouvert_V_Actif_Brake"
+	(label "Ouvert_V_Actif"
 		(at 83.82 158.75 180)
 		(effects
@@
 	)
 	(label "R_Lim_R"
-		(at 246.634 26.924 180)
+		(at 227.33 27.94 180)
 		(effects
 			(font
@@
 	)
 	(label "R_Lim_G"
-		(at 246.634 32.004 180)
+		(at 227.33 33.02 180)
 		(effects
 			(font
@@
 		)
 	)
-	(label "Court_V_Actif_Brake"
+	(label "Court_V_Actif"
 		(at 45.72 158.75 180)
 		(effects
@@
 		)
 	)
-	(label "Court_T_Actif_Brake"
+	(label "Court_T_Actif"
 		(at 95.25 50.8 0)
 		(effects
@@
 		)
 	)
-	(label "Ouvert_V_Actif_Brake"
+	(label "Ouvert_V_Actif"
 		(at 49.53 93.98 0)
 		(effects
@@
 		)
 	)
-	(label "Vert_Enable_Brake"
+	(label "Vert_Enable"
 		(at 224.79 146.05 0)
 		(effects
@@
 		)
 	)
-	(label "Ouvert_T_Actif_Brake"
+	(label "Ouvert_T_Actif"
 		(at 83.82 170.18 180)
 		(effects
@@
 		)
 	)
-	(label "Vert_Enable_Brake"
-		(at 203.454 33.528 180)
+	(label "Vert_Enable"
+		(at 187.96 31.75 180)
 		(effects
 			(font
@@
 		)
 	)
-	(label "Court_T_Actif_Brake"
+	(label "Court_T_Actif"
 		(at 45.72 170.18 180)
 		(effects
@@
 		)
 	)
-	(label "Fault_Actif_Brake"
+	(label "Fault_Actif"
 		(at 198.12 120.65 0)
 		(effects
@@
 		)
 	)
-	(label "Court_V_Actif_Brake"
+	(label "Court_V_Actif"
 		(at 50.8 50.8 0)
 		(effects
@@
 		)
 	)
-	(label "Ouvert_T_Actif_Brake"
+	(label "Ouvert_T_Actif"
 		(at 93.98 102.87 0)
 		(effects
@@
 	)
 	(label "R_Lim_G"
-		(at 219.964 24.638 0)
+		(at 204.47 22.86 0)
 		(effects
 			(font
@@
 	(global_label "GND"
 		(shape input)
-		(at 207.264 41.148 180)
+		(at 191.77 39.37 180)
 		(fields_autoplaced yes)
 		(effects
@@
 		)
 		(property "Intersheetrefs" "${INTERSHEET_REFS}"
-			(at 200.4083 41.148 0)
+			(at 184.9143 39.37 0)
 			(hide yes)
 			(show_name no)
@@
 	(global_label "V_Ref"
 		(shape input)
-		(at 256.794 32.004 0)
+		(at 237.49 33.02 0)
 		(fields_autoplaced yes)
 		(effects
@@
 		)
 		(property "Intersheetrefs" "${INTERSHEET_REFS}"
-			(at 264.9197 32.004 0)
+			(at 245.6157 33.02 0)
 			(hide yes)
 			(show_name no)
@@
 	(symbol
 		(lib_id "PCM_SL_Resistors:330ohm")
-		(at 216.154 24.638 0)
+		(at 200.66 22.86 0)
 		(unit 1)
 		(body_style 1)
@@
 		(fields_autoplaced yes)
 		(property "Reference" "R49"
-			(at 216.154 18.288 0)
+			(at 200.66 16.51 0)
 			(show_name no)
 			(do_not_autoplace no)
@@
 		)
 		(property "Value" "330ohm"
-			(at 216.154 20.828 0)
+			(at 200.66 19.05 0)
 			(show_name no)
 			(do_not_autoplace no)
@@
 		)
 		(property "Footprint" "Resistor_THT:R_Axial_DIN0207_L6.3mm_D2.5mm_P10.16mm_Horizontal"
-			(at 217.043 28.956 0)
+			(at 201.549 27.178 0)
 			(hide yes)
 			(show_name no)
@@
 		)
 		(property "Datasheet" ""
-			(at 216.662 24.638 0)
+			(at 201.168 22.86 0)
 			(hide yes)
 			(show_name no)
@@
 		)
 		(property "Description" "330Ω, 1/4W Resistor"
-			(at 216.154 24.638 0)
+			(at 200.66 22.86 0)
 			(hide yes)
 			(show_name no)
@@
 	(symbol
 		(lib_id "Transistor_FET:2N7000")
-		(at 208.534 33.528 0)
+		(at 193.04 31.75 0)
 		(unit 1)
 		(body_style 1)
@@
 		(dnp no)
 		(property "Reference" "Q16"
-			(at 214.884 32.2579 0)
+			(at 199.39 30.4799 0)
 			(show_name no)
 			(do_not_autoplace no)
@@
 		)
 		(property "Value" "2N7000"
-			(at 213.614 34.798 0)
+			(at 198.12 33.02 0)
 			(show_name no)
 			(do_not_autoplace no)
@@
 		)
 		(property "Footprint" "Package_TO_SOT_THT:TO-92_Inline"
-			(at 213.614 35.433 0)
+			(at 198.12 33.655 0)
 			(hide yes)
 			(show_name no)
@@
 		)
 		(property "Datasheet" "https://www.vishay.com/docs/70226/70226.pdf"
-			(at 213.614 37.338 0)
+			(at 198.12 35.56 0)
 			(hide yes)
 			(show_name no)
@@
 		)
 		(property "Description" "0.2A Id, 200V Vds, N-Channel MOSFET, 2.6V Logic Level, TO-92"
-			(at 208.534 33.528 0)
+			(at 193.04 31.75 0)
 			(hide yes)
 			(show_name no)
@@
 	(symbol
 		(lib_id "Device:LED_ARGB")
-		(at 251.714 32.004 0)
+		(at 232.41 33.02 0)
 		(unit 1)
 		(body_style 1)
@@
 		(fields_autoplaced yes)
 		(property "Reference" "D49"
-			(at 251.714 18.034 0)
+			(at 232.41 19.05 0)
 			(show_name no)
 			(do_not_autoplace no)
@@
 		)
 		(property "Value" "LED_ARGB"
-			(at 251.714 20.574 0)
+			(at 232.41 21.59 0)
 			(show_name no)
 			(do_not_autoplace no)
@@
 		)
 		(property "Footprint" ""
-			(at 251.714 33.274 0)
+			(at 232.41 34.29 0)
 			(hide yes)
 			(show_name no)
@@
 		)
 		(property "Datasheet" ""
-			(at 251.714 33.274 0)
+			(at 232.41 34.29 0)
 			(hide yes)
 			(show_name no)
@@
 		)
 		(property "Description" "RGB LED, anode/red/green/blue"
-			(at 251.714 32.004 0)
+			(at 232.41 33.02 0)
 			(hide yes)
 			(show_name no)

Commit message: Add files via upload
Connections:
- net Court_T_Actif renamed Court_T_Actif_Brake
- net Court_V_Actif renamed Court_V_Actif_Brake
- net Fault_Actif renamed Fault_Actif_Brake
- net Ouvert_T_Actif renamed Ouvert_T_Actif_Brake
- net Ouvert_V_Actif renamed Ouvert_V_Actif_Brake
- net Vert_Enable renamed Vert_Enable_Brake
Other:
- note added: "Ouvert_T_Actif_Brake (Porte ET #4 - 3 entrées)"
- note removed: "Ouvert_T_Actif (Porte ET #4 - 3 entrées)"
- moved on the sheet: D49, Q16, R49
Changed lines of the file:
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@@
 	)
 	(rectangle
-		(start 175.26 13.97)
-		(end 213.36 46.99)
+		(start 184.658 15.748)
+		(end 228.854 48.768)
 		(stroke
 			(width 0)
@@
 	)
 	(rectangle
-		(start 217.17 16.51)
-		(end 246.38 45.72)
+		(start 236.474 15.494)
+		(end 265.684 44.704)
 		(stroke
 			(width 0)
@@
 		)
 	)
-	(text "Ouvert_T_Actif\n(Porte ET #4 - 3 entrées)"
+	(text "Ouvert_T_Actif_Brake\n(Porte ET #4 - 3 entrées)"
 		(exclude_from_sim yes)
 		(at 97.79 55.88 0)
@@
 	(wire
 		(pts
-			(xy 195.58 36.83) (xy 195.58 39.37)
+			(xy 211.074 38.608) (xy 211.074 41.148)
 		)
 		(stroke
@@
 	(wire
 		(pts
-			(xy 195.58 39.37) (xy 191.77 39.37)
+			(xy 211.074 41.148) (xy 207.264 41.148)
 		)
 		(stroke
@@
 	(wire
 		(pts
-			(xy 195.58 22.86) (xy 196.85 22.86)
+			(xy 211.074 24.638) (xy 212.344 24.638)
 		)
 		(stroke
@@
 	(wire
 		(pts
-			(xy 195.58 26.67) (xy 195.58 22.86)
+			(xy 211.074 28.448) (xy 211.074 24.638)
 		)
 		(stroke
@@
 	)
 	(label "R_Lim_B"
-		(at 227.33 38.1 180)
+		(at 246.634 37.084 180)
 		(effects
 			(font
@@
 		)
 	)
-	(label "Ouvert_V_Actif"
+	(label "Ouvert_V_Actif_Brake"
 		(at 83.82 158.75 180)
 		(effects
@@
 	)
 	(label "R_Lim_R"
-		(at 227.33 27.94 180)
+		(at 246.634 26.924 180)
 		(effects
 			(font
@@
 	)
 	(label "R_Lim_G"
-		(at 227.33 33.02 180)
+		(at 246.634 32.004 180)
 		(effects
 			(font
@@
 		)
 	)
-	(label "Court_V_Actif"
+	(label "Court_V_Actif_Brake"
 		(at 45.72 158.75 180)
 		(effects
@@
 		)
 	)
-	(label "Court_T_Actif"
+	(label "Court_T_Actif_Brake"
 		(at 95.25 50.8 0)
 		(effects
@@
 		)
 	)
-	(label "Ouvert_V_Actif"
+	(label "Ouvert_V_Actif_Brake"
 		(at 49.53 93.98 0)
 		(effects
@@
 		)
 	)
-	(label "Vert_Enable"
+	(label "Vert_Enable_Brake"
 		(at 224.79 146.05 0)
 		(effects
@@
 		)
 	)
-	(label "Ouvert_T_Actif"
+	(label "Ouvert_T_Actif_Brake"
 		(at 83.82 170.18 180)
 		(effects
@@
 		)
 	)
-	(label "Vert_Enable"
-		(at 187.96 31.75 180)
+	(label "Vert_Enable_Brake"
+		(at 203.454 33.528 180)
 		(effects
 			(font
@@
 		)
 	)
-	(label "Court_T_Actif"
+	(label "Court_T_Actif_Brake"
 		(at 45.72 170.18 180)
 		(effects
@@
 		)
 	)
-	(label "Fault_Actif"
+	(label "Fault_Actif_Brake"
 		(at 198.12 120.65 0)
 		(effects
@@
 		)
 	)
-	(label "Court_V_Actif"
+	(label "Court_V_Actif_Brake"
 		(at 50.8 50.8 0)
 		(effects
@@
 		)
 	)
-	(label "Ouvert_T_Actif"
+	(label "Ouvert_T_Actif_Brake"
 		(at 93.98 102.87 0)
 		(effects
@@
 	)
 	(label "R_Lim_G"
-		(at 204.47 22.86 0)
+		(at 219.964 24.638 0)
 		(effects
 			(font
@@
 	(global_label "GND"
 		(shape input)
-		(at 191.77 39.37 180)
+		(at 207.264 41.148 180)
 		(fields_autoplaced yes)
 		(effects
@@
 		)
 		(property "Intersheetrefs" "${INTERSHEET_REFS}"
-			(at 184.9143 39.37 0)
+			(at 200.4083 41.148 0)
 			(hide yes)
 			(show_name no)
@@
 	(global_label "V_Ref"
 		(shape input)
-		(at 237.49 33.02 0)
+		(at 256.794 32.004 0)
 		(fields_autoplaced yes)
 		(effects
@@
 		)
 		(property "Intersheetrefs" "${INTERSHEET_REFS}"
-			(at 245.6157 33.02 0)
+			(at 264.9197 32.004 0)
 			(hide yes)
 			(show_name no)
@@
 	(symbol
 		(lib_id "PCM_SL_Resistors:330ohm")
-		(at 200.66 22.86 0)
+		(at 216.154 24.638 0)
 		(unit 1)
 		(body_style 1)
@@
 		(fields_autoplaced yes)
 		(property "Reference" "R49"
-			(at 200.66 16.51 0)
+			(at 216.154 18.288 0)
 			(show_name no)
 			(do_not_autoplace no)
@@
 		)
 		(property "Value" "330ohm"
-			(at 200.66 19.05 0)
+			(at 216.154 20.828 0)
 			(show_name no)
 			(do_not_autoplace no)
@@
 		)
 		(property "Footprint" "Resistor_THT:R_Axial_DIN0207_L6.3mm_D2.5mm_P10.16mm_Horizontal"
-			(at 201.549 27.178 0)
+			(at 217.043 28.956 0)
 			(hide yes)
 			(show_name no)
@@
 		)
 		(property "Datasheet" ""
-			(at 201.168 22.86 0)
+			(at 216.662 24.638 0)
 			(hide yes)
 			(show_name no)
@@
 		)
 		(property "Description" "330Ω, 1/4W Resistor"
-			(at 200.66 22.86 0)
+			(at 216.154 24.638 0)
 			(hide yes)
 			(show_name no)
@@
 	(symbol
 		(lib_id "Transistor_FET:2N7000")
-		(at 193.04 31.75 0)
+		(at 208.534 33.528 0)
 		(unit 1)
 		(body_style 1)
@@
 		(dnp no)
 		(property "Reference" "Q16"
-			(at 199.39 30.4799 0)
+			(at 214.884 32.2579 0)
 			(show_name no)
 			(do_not_autoplace no)
@@
 		)
 		(property "Value" "2N7000"
-			(at 198.12 33.02 0)
+			(at 213.614 34.798 0)
 			(show_name no)
 			(do_not_autoplace no)
@@
 		)
 		(property "Footprint" "Package_TO_SOT_THT:TO-92_Inline"
-			(at 198.12 33.655 0)
+			(at 213.614 35.433 0)
 			(hide yes)
 			(show_name no)
@@
 		)
 		(property "Datasheet" "https://www.vishay.com/docs/70226/70226.pdf"
-			(at 198.12 35.56 0)
+			(at 213.614 37.338 0)
 			(hide yes)
 			(show_name no)
@@
 		)
 		(property "Description" "0.2A Id, 200V Vds, N-Channel MOSFET, 2.6V Logic Level, TO-92"
-			(at 193.04 31.75 0)
+			(at 208.534 33.528 0)
 			(hide yes)
 			(show_name no)
@@
 	(symbol
 		(lib_id "Device:LED_ARGB")
-		(at 232.41 33.02 0)
+		(at 251.714 32.004 0)
 		(unit 1)
 		(body_style 1)
@@
 		(fields_autoplaced yes)
 		(property "Reference" "D49"
-			(at 232.41 19.05 0)
+			(at 251.714 18.034 0)
 			(show_name no)
 			(do_not_autoplace no)
@@
 		)
 		(property "Value" "LED_ARGB"
-			(at 232.41 21.59 0)
+			(at 251.714 20.574 0)
 			(show_name no)
 			(do_not_autoplace no)
@@
 		)
 		(property "Footprint" ""
-			(at 232.41 34.29 0)
+			(at 251.714 33.274 0)
 			(hide yes)
 			(show_name no)
@@
 		)
 		(property "Datasheet" ""
-			(at 232.41 34.29 0)
+			(at 251.714 33.274 0)
 			(hide yes)
 			(show_name no)
@@
 		)
 		(property "Description" "RGB LED, anode/red/green/blue"
-			(at 232.41 33.02 0)
+			(at 251.714 32.004 0)
 			(hide yes)
 			(show_name no)

Commit message: Add files via upload
Parts:
- added D173: 1N4148, PCM_Diode_THT_AKL:D_DO-35_SOD27_P7.62mm_Horizontal, symbol PCM_Diode_AKL:1N4148
Connections:
- net Btn_Brake_Etat: now also D173.1 (K)
- net Court_T_Actif_Brake: now also D173.2 (A)
Changed lines of the file:
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@@
 	(wire
 		(pts
+			(xy 144.78 158.75) (xy 147.32 158.75)
+		)
+		(stroke
+			(width 0)
+			(type default)
+		)
+	)
+	(wire
+		(pts
 			(xy 148.59 71.12) (xy 148.59 64.77)
 		)
@@
 	(wire
 		(pts
+			(xy 137.16 158.75) (xy 134.62 158.75)
+		)
+		(stroke
+			(width 0)
+			(type default)
+		)
+	)
+	(wire
+		(pts
 			(xy 148.59 46.99) (xy 144.78 46.99)
 		)
@@
 		)
 	)
+	(label "Court_T_Actif_Brake"
+		(at 134.62 158.75 180)
+		(effects
+			(font
+				(size 1.27 1.27)
+			)
+			(justify right bottom)
+		)
+	)
 	(label "R_Lim_R"
 		(at 246.634 26.924 180)
@@
 		)
 	)
+	(hierarchical_label "Btn_Brake_Etat"
+		(shape input)
+		(at 147.32 158.75 0)
+		(effects
+			(font
+				(size 1.27 1.27)
+			)
+			(justify left)
+		)
+	)
 	(hierarchical_label "Court_Brake_Trailer"
 		(shape input)
@@
 					(unit 1)
 				)
+			)
+		)
+	)
+	(symbol
+		(lib_id "PCM_Diode_AKL:1N4148")
+		(at 140.97 158.75 0)
+		(unit 1)
+		(body_style 1)
+		(exclude_from_sim no)
+		(in_bom yes)
+		(on_board yes)
+		(in_pos_files yes)
+		(dnp no)
+		(property "Reference" "D173"
+			(at 140.97 153.42 0)
+			(show_name no)
+			(do_not_autoplace no)
+			(effects
+				(font
+					(size 1.27 1.27)
+				)
+			)
+		)
+		(property "Value" "1N4148"
+			(at 140.97 155.7 0)
+			(show_name no)
+			(do_not_autoplace no)
+			(effects
+				(font
+					(size 1.27 1.27)
+				)
+			)
+		)
+		(property "Footprint" "PCM_Diode_THT_AKL:D_DO-35_SOD27_P7.62mm_Horizontal"
+			(at 140.97 158.75 0)
+			(hide yes)
+			(show_name no)
+			(do_not_autoplace no)
+			(effects
+				(font
+					(size 1.27 1.27)
+				)
+			)
+		)
+		(property "Datasheet" "https://datasheet.octopart.com/1N4148TR-ON-Semiconductor-datasheet-42765246.pdf"
+			(at 140.97 158.75 0)
+			(hide yes)
+			(show_name no)
+			(do_not_autoplace no)
+			(effects
+				(font
+					(size 1.27 1.27)
+				)
+			)
+		)
+		(property "Description" "DO-35 Diode, Small Signal, Fast Switching, 75V, 150mA, 4ns, Alternate KiCad Library"
+			(at 140.97 158.75 0)
+			(hide yes)
+			(show_name no)
+			(do_not_autoplace no)
+			(effects
+				(font
+					(size 1.27 1.27)
+				)
+			)
+		)
+		(pin "2"
+		)
+		(pin "1"
+		)
+		(instances
+			(project "TrailerDiagnosticSystem"
+				(path "/d4e407a7-3e32-4226-ae57-831ecdb3edf4/1c73cd0e-d554-4457-9021-54aac4b5c0a2/704733a3-8459-4f16-a041-c619adb87510"
+					(reference "D173")
+					(unit 1)
+				)
