File: Bloc_Test_Brake.kicad_sch (KiCad schematic)
At the start: 45 parts, among them Q13 2N7000, Q14 2N7000, Q15 2N7000, Q16 2N7000, Q17 2N7000, Q18 2N7000

Commit message: Add files via upload
Parts:
- R40, R44: value 4.7k -> 100kΩ
- R45, R48, R50: value 4.7k -> 470kΩ
Connections:
- net Bleu_Brake: now also D33.2 (A), D34.2 (A), R41.1
- net Court_Brake: now also D31.1 (K), D32.1 (K), R40.1
- net GND: no longer Q13.2 (G)
- net Mode_Trailer: now also D33.1 (K); no longer D33.2 (A)
- net Not_Btn_Brake: now also D34.1 (K); no longer D34.2 (A)
- net Ouvert_Brake: now also D40.1 (K), D41.1 (K), R44.2
- net Ouvert_Ou_Bleu_Brake: now reaches D42.1 (K), D43.1 (K), Q14.3 (D), R45.1
- net Ouvert_Ou_Bleu_Brake: now also Q13.2 (G)
Other:
- moved on the sheet: R40

Commit message: Add files via upload
Parts:
- R39, R41, R42, R43, R46, R52, R66: value 4.7k -> 4.7kΩ
- R47, R49, R51: value 330ohm -> 330Ω
Changed lines of the file:
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@@
 			)
 		)
-		(property "Value" "4.7k"
+		(property "Value" "4.7kΩ"
 			(at 55.88 132.08 0)
 			(show_name no)
@@
 			)
 		)
-		(property "Value" "4.7k"
+		(property "Value" "4.7kΩ"
 			(at 46.99 85.09 0)
 			(show_name no)
@@
 			)
 		)
-		(property "Value" "4.7k"
+		(property "Value" "4.7kΩ"
 			(at 91.44 42.926 0)
 			(show_name no)
@@
 			)
 		)
-		(property "Value" "330ohm"
+		(property "Value" "330Ω"
 			(at 216.154 20.828 0)
 			(show_name no)
@@
 			)
 		)
-		(property "Value" "330ohm"
+		(property "Value" "330Ω"
 			(at 153.67 69.85 0)
 			(show_name no)
@@
 			)
 		)
-		(property "Value" "4.7k"
+		(property "Value" "4.7kΩ"
 			(at 91.44 95.25 0)
 			(show_name no)
@@
 			)
 		)
-		(property "Value" "4.7k"
+		(property "Value" "4.7kΩ"
 			(at 228.6 152.4 0)
 			(show_name no)
@@
 			)
 		)
-		(property "Value" "330ohm"
+		(property "Value" "330Ω"
 			(at 220.98 63.5 0)
 			(show_name no)
@@
 			)
 		)
-		(property "Value" "4.7k"
+		(property "Value" "4.7kΩ"
 			(at 48.26 43.18 0)
 			(show_name no)
@@
 			)
 		)
-		(property "Value" "4.7k"
+		(property "Value" "4.7kΩ"
 			(at 146.05 106.68 0)
 			(show_name no)

Commit message: Add files via upload
Connections:
- net R_Lim_B renamed Fac_Brake_B
- net R_Lim_G renamed Fac_Brake_G
- net R_Lim_R renamed Fac_Brake_R
Other:
- moved on the sheet: Q16, R49
Changed lines of the file:
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@@
 	)
 	(junction
+		(at 219.71 24.13)
+		(diameter 0)
+		(color 0 0 0 0)
+	)
+	(junction
 		(at 149.86 115.57)
 		(diameter 0)
@@
 	)
 	(junction
+		(at 157.48 73.66)
+		(diameter 0)
+		(color 0 0 0 0)
+	)
+	(junction
 		(at 198.12 147.32)
 		(diameter 0)
@@
 	)
 	(junction
+		(at 224.79 67.31)
+		(diameter 0)
+		(color 0 0 0 0)
+	)
+	(junction
 		(at 58.42 170.18)
 		(diameter 0)
@@
 	(wire
 		(pts
+			(xy 158.75 68.58) (xy 157.48 68.58)
+		)
+		(stroke
+			(width 0)
+			(type default)
+		)
+	)
+	(wire
+		(pts
 			(xy 95.25 158.75) (xy 95.25 170.18)
 		)
@@
 	(wire
 		(pts
+			(xy 228.6 59.69) (xy 224.79 59.69)
+		)
+		(stroke
+			(width 0)
+			(type default)
+		)
+	)
+	(wire
+		(pts
 			(xy 43.18 179.07) (xy 46.99 179.07)
 		)
@@
 	(wire
 		(pts
+			(xy 224.79 59.69) (xy 224.79 67.31)
+		)
+		(stroke
+			(width 0)
+			(type default)
+		)
+	)
+	(wire
+		(pts
 			(xy 91.44 158.75) (xy 95.25 158.75)
 		)
@@
 	(wire
 		(pts
-			(xy 211.074 38.608) (xy 211.074 41.148)
+			(xy 210.82 38.1) (xy 210.82 40.64)
 		)
 		(stroke
@@
 	(wire
 		(pts
+			(xy 157.48 68.58) (xy 157.48 73.66)
+		)
+		(stroke
+			(width 0)
+			(type default)
+		)
+	)
+	(wire
+		(pts
 			(xy 64.77 124.46) (xy 59.69 124.46)
 		)
@@
 	(wire
 		(pts
+			(xy 220.98 19.05) (xy 219.71 19.05)
+		)
+		(stroke
+			(width 0)
+			(type default)
+		)
+	)
+	(wire
+		(pts
 			(xy 148.59 25.4) (xy 153.67 25.4)
 		)
@@
 	(wire
 		(pts
+			(xy 219.71 24.13) (xy 220.98 24.13)
+		)
+		(stroke
+			(width 0)
+			(type default)
+		)
+	)
+	(wire
+		(pts
 			(xy 134.62 81.28) (xy 137.16 81.28)
 		)
@@
 	(wire
 		(pts
+			(xy 228.6 67.31) (xy 224.79 67.31)
+		)
+		(stroke
+			(width 0)
+			(type default)
+		)
+	)
+	(wire
+		(pts
 			(xy 86.36 77.47) (xy 86.36 87.63)
 		)
@@
 	(wire
 		(pts
+			(xy 158.75 73.66) (xy 157.48 73.66)
+		)
+		(stroke
+			(width 0)
+			(type default)
+		)
+	)
+	(wire
+		(pts
 			(xy 209.55 146.05) (xy 224.79 146.05)
 		)
@@
 	(wire
 		(pts
-			(xy 211.074 41.148) (xy 207.264 41.148)
+			(xy 210.82 40.64) (xy 207.01 40.64)
 		)
 		(stroke
@@
 	(wire
 		(pts
-			(xy 211.074 24.638) (xy 212.344 24.638)
+			(xy 210.82 24.13) (xy 212.09 24.13)
 		)
 		(stroke
@@
 	(wire
 		(pts
-			(xy 211.074 28.448) (xy 211.074 24.638)
+			(xy 210.82 27.94) (xy 210.82 24.13)
+		)
+		(stroke
+			(width 0)
+			(type default)
+		)
+	)
+	(wire
+		(pts
+			(xy 219.71 19.05) (xy 219.71 24.13)
 		)
 		(stroke
@@
 	)
 	(label "R_Lim_B"
-		(at 246.634 37.084 180)
+		(at 246.38 36.83 180)
 		(effects
 			(font
@@
 	)
 	(label "R_Lim_R"
-		(at 246.634 26.924 180)
+		(at 246.38 26.67 180)
 		(effects
 			(font
@@
 	)
 	(label "R_Lim_G"
-		(at 246.634 32.004 180)
+		(at 246.38 31.75 180)
 		(effects
 			(font
@@
 	)
 	(label "Vert_Enable_Brake"
-		(at 203.454 33.528 180)
+		(at 203.2 33.02 180)
 		(effects
 			(font
@@
 	)
 	(label "R_Lim_R"
-		(at 224.79 67.31 0)
+		(at 228.6 67.31 0)
 		(effects
 			(font
@@
 	)
 	(label "R_Lim_B"
-		(at 157.48 73.66 0)
+		(at 158.75 73.66 0)
 		(effects
 			(font
@@
 	)
 	(label "R_Lim_G"
-		(at 219.964 24.638 0)
+		(at 220.98 24.13 0)
 		(effects
 			(font
@@
 	(global_label "GND"
 		(shape input)
-		(at 207.264 41.148 180)
+		(at 207.01 40.64 180)
 		(fields_autoplaced yes)
 		(effects
@@
 		)
 		(property "Intersheetrefs" "${INTERSHEET_REFS}"
-			(at 200.4083 41.148 0)
+			(at 200.1543 40.64 0)
 			(hide yes)
 			(show_name no)
@@
 		)
 	)
+	(global_label "Fac_Brake_B"
+		(shape input)
+		(at 158.75 68.58 0)
+		(fields_autoplaced yes)
+		(effects
+			(font
+				(size 1.27 1.27)
+			)
+			(justify left)
+		)
+		(property "Intersheetrefs" "${INTERSHEET_REFS}"
+			(at 173.5885 68.58 0)
+			(hide yes)
+			(show_name no)
+			(do_not_autoplace no)
+			(effects
+				(font
+					(size 1.27 1.27)
+				)
+				(justify left)
+			)
+		)
+	)
+	(global_label "Fac_Brake_R"
+		(shape input)
+		(at 228.6 59.69 0)
+		(fields_autoplaced yes)
+		(effects
+			(font
+				(size 1.27 1.27)
+			)
+			(justify left)
+		)
+		(property "Intersheetrefs" "${INTERSHEET_REFS}"
+			(at 243.4385 59.69 0)
+			(hide yes)
+			(show_name no)
+			(do_not_autoplace no)
+			(effects
+				(font
+					(size 1.27 1.27)
+				)
+				(justify left)
+			)
+		)
+	)
 	(global_label "V_Ref"
 		(shape input)
@@
 	(global_label "V_Ref"
 		(shape input)
-		(at 256.794 32.004 0)
+		(at 256.54 31.75 0)
 		(fields_autoplaced yes)
 		(effects
@@
 		)
 		(property "Intersheetrefs" "${INTERSHEET_REFS}"
-			(at 264.9197 32.004 0)
+			(at 264.6657 31.75 0)
 			(hide yes)
 			(show_name no)
@@
 		)
 	)
+	(global_label "Fac_Brake_G"
+		(shape input)
+		(at 220.98 19.05 0)
+		(fields_autoplaced yes)
+		(effects
+			(font
+				(size 1.27 1.27)
+			)
+			(justify left)
+		)
+		(property "Intersheetrefs" "${INTERSHEET_REFS}"
+			(at 235.8185 19.05 0)
+			(hide yes)
+			(show_name no)
+			(do_not_autoplace no)
+			(effects
+				(font
+					(size 1.27 1.27)
+				)
+				(justify left)
+			)
+		)
+	)
 	(hierarchical_label "Court_Brake_Vehic"
 		(shape input)
@@
 	(symbol
 		(lib_id "PCM_SL_Resistors:330ohm")
-		(at 216.154 24.638 0)
+		(at 215.9 24.13 0)
 		(unit 1)
 		(body_style 1)
@@
 		(fields_autoplaced yes)
 		(property "Reference" "R49"
-			(at 216.154 18.288 0)
+			(at 215.9 17.78 0)
 			(show_name no)
 			(do_not_autoplace no)
@@
 		)
 		(property "Value" "330Ω"
-			(at 216.154 20.828 0)
+			(at 215.9 20.32 0)
 			(show_name no)
 			(do_not_autoplace no)
@@
 		)
 		(property "Footprint" "Resistor_THT:R_Axial_DIN0207_L6.3mm_D2.5mm_P10.16mm_Horizontal"
-			(at 217.043 28.956 0)
+			(at 216.789 28.448 0)
 			(hide yes)
 			(show_name no)
@@
 		)
 		(property "Datasheet" ""
-			(at 216.662 24.638 0)
+			(at 216.408 24.13 0)
 			(hide yes)
 			(show_name no)
@@
 		)
 		(property "Description" "330Ω, 1/4W Resistor"
-			(at 216.154 24.638 0)
+			(at 215.9 24.13 0)
 			(hide yes)
 			(show_name no)
@@
 	(symbol
 		(lib_id "Transistor_FET:2N7000")
-		(at 208.534 33.528 0)
+		(at 208.28 33.02 0)
 		(unit 1)
 		(body_style 1)
@@
 		(dnp no)
 		(property "Reference" "Q16"
-			(at 214.884 32.2579 0)
+			(at 214.63 31.7499 0)
 			(show_name no)
 			(do_not_autoplace no)
@@
 		)
 		(property "Value" "2N7000"
-			(at 213.614 34.798 0)
+			(at 213.36 34.29 0)
 			(show_name no)
 			(do_not_autoplace no)
@@
 		)
 		(property "Footprint" "Package_TO_SOT_THT:TO-92_Inline"
-			(at 213.614 35.433 0)
+			(at 213.36 34.925 0)
 			(hide yes)
 			(show_name no)
@@
 		)
 		(property "Datasheet" "https://www.vishay.com/docs/70226/70226.pdf"
-			(at 213.614 37.338 0)
+			(at 213.36 36.83 0)
 			(hide yes)
 			(show_name no)
@@
 		)
 		(property "Description" "0.2A Id, 200V Vds, N-Channel MOSFET, 2.6V Logic Level, TO-92"
-			(at 208.534 33.528 0)
+			(at 208.28 33.02 0)
 			(hide yes)
 			(show_name no)
@@
 	(symbol
 		(lib_id "Device:LED_ARGB")
-		(at 251.714 32.004 0)
+		(at 251.46 31.75 0)
 		(unit 1)
 		(body_style 1)
@@
 		(fields_autoplaced yes)
 		(property "Reference" "D49"
-			(at 251.714 18.034 0)
+			(at 251.46 17.78 0)
 			(show_name no)
 			(do_not_autoplace no)
@@
 		)
 		(property "Value" "LED_ARGB"
-			(at 251.714 20.574 0)
+			(at 251.46 20.32 0)
 			(show_name no)
 			(do_not_autoplace no)
@@
 		)
 		(property "Footprint" ""
-			(at 251.714 33.274 0)
+			(at 251.46 33.02 0)
 			(hide yes)
 			(show_name no)
@@
 		)
 		(property "Datasheet" ""
-			(at 251.714 33.274 0)
+			(at 251.46 33.02 0)
 			(hide yes)
 			(show_name no)
@@
 		)
 		(property "Description" "RGB LED, anode/red/green/blue"
-			(at 251.714 32.004 0)
+			(at 251.46 31.75 0)
 			(hide yes)
 			(show_name no)
