File: Vehicule_Aux.kicad_sch (KiCad schematic)
At the start: 16 parts, among them Q43 IRLZ44N, U11 LM339

Commit message: Add files via upload
Connections:
- net Veh_Aux: no longer U11.5 (+)
- net at R162.2, R163.1: now also U11.5 (+)
Other:
- moved on the sheet: R163
Changed lines of the file:
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@@
 	)
 	(junction
-		(at 100.33 34.29)
+		(at 114.3 34.29)
 		(diameter 0)
 		(color 0 0 0 0)
@@
 	(wire
 		(pts
-			(xy 100.33 34.29) (xy 104.14 34.29)
+			(xy 95.25 34.29) (xy 104.14 34.29)
 		)
 		(stroke
@@
 	(wire
 		(pts
-			(xy 123.19 34.29) (xy 127 34.29)
+			(xy 124.46 34.29) (xy 128.27 34.29)
 		)
 		(stroke
@@
 	(wire
 		(pts
-			(xy 111.76 34.29) (xy 115.57 34.29)
+			(xy 111.76 34.29) (xy 114.3 34.29)
 		)
 		(stroke
@@
 	(wire
 		(pts
+			(xy 114.3 34.29) (xy 116.84 34.29)
+		)
+		(stroke
+			(width 0)
+			(type default)
+		)
+	)
+	(wire
+		(pts
 			(xy 102.87 90.17) (xy 78.74 90.17)
 		)
@@
 	(wire
 		(pts
+			(xy 114.3 34.29) (xy 114.3 40.64)
+		)
+		(stroke
+			(width 0)
+			(type default)
+		)
+	)
+	(wire
+		(pts
 			(xy 204.47 45.72) (xy 204.47 43.18)
 		)
@@
 	(wire
 		(pts
-			(xy 100.33 67.31) (xy 100.33 34.29)
-		)
-		(stroke
-			(width 0)
-			(type default)
-		)
-	)
-	(wire
-		(pts
-			(xy 95.25 34.29) (xy 100.33 34.29)
-		)
-		(stroke
-			(width 0)
-			(type default)
-		)
-	)
-	(wire
-		(pts
 			(xy 152.4 109.22) (xy 137.16 109.22)
 		)
@@
 	(wire
 		(pts
+			(xy 100.33 40.64) (xy 114.3 40.64)
+		)
+		(stroke
+			(width 0)
+			(type default)
+		)
+	)
+	(wire
+		(pts
 			(xy 152.4 97.79) (xy 152.4 99.06)
 		)
@@
 		(pts
 			(xy 152.4 63.5) (xy 170.18 63.5)
+		)
+		(stroke
+			(width 0)
+			(type default)
+		)
+	)
+	(wire
+		(pts
+			(xy 100.33 67.31) (xy 100.33 40.64)
 		)
 		(stroke
@@
 	(global_label "GND"
 		(shape input)
-		(at 127 34.29 0)
+		(at 128.27 34.29 0)
 		(fields_autoplaced yes)
 		(effects
@@
 		)
 		(property "Intersheetrefs" "${INTERSHEET_REFS}"
-			(at 133.8557 34.29 0)
+			(at 135.1257 34.29 0)
 			(hide yes)
 			(show_name no)
@@
 	(symbol
 		(lib_id "PCM_SL_Resistors:10k")
-		(at 119.38 34.29 0)
+		(at 120.65 34.29 0)
 		(unit 1)
 		(body_style 1)
@@
 		(fields_autoplaced yes)
 		(property "Reference" "R163"
-			(at 119.38 27.94 0)
+			(at 120.65 27.94 0)
 			(show_name no)
 			(do_not_autoplace no)
@@
 		)
 		(property "Value" "10k"
-			(at 119.38 30.48 0)
+			(at 120.65 30.48 0)
 			(show_name no)
 			(do_not_autoplace no)
@@
 		)
 		(property "Footprint" "Resistor_THT:R_Axial_DIN0207_L6.3mm_D2.5mm_P10.16mm_Horizontal"
-			(at 120.269 38.608 0)
+			(at 121.539 38.608 0)
 			(hide yes)
 			(show_name no)
@@
 		)
 		(property "Datasheet" ""
-			(at 119.888 34.29 0)
+			(at 121.158 34.29 0)
 			(hide yes)
 			(show_name no)
@@
 		)
 		(property "Description" "10kΩ, 1/4W Resistor"
-			(at 119.38 34.29 0)
-			(hide yes)
-			(show_name no)
+			(at 120.65 34.29 0)
+			(hide yes)
+			(show_name no)

Commit message: Add files via upload
Parts:
- added Q66: 2N7000, PCM_Package_TO_SOT_THT_AKL:TO-92_Inline_Wide_SGD, symbol PCM_Transistor_MOSFET_AKL:2N7000
- added R243: R100 Ohm, Resistor_THT:R_Axial_DIN0207_L6.3mm_D2.5mm_P10.16mm_Horizontal, symbol PCM_SL_Resistors:100k
- added SW10: TH_Aux, symbol Switch:SW_SPST_Temperature_NC
- R155: value 3 Ohm - 5W -> 4,7 Ohm - 50W; footprint Resistor_THT:R_Axial_Power_L25.0mm_W9.0mm_P27.94mm -> TerminalBlock_Phoenix:TerminalBlock_Phoenix_PT-1,5-2-3.5-H_1x02_P3.50mm_Horizontal
Connections:
- net GND: now also Q66.1 (S), SW10.2
- net Injection_Aux_Fault: now also Q66.3 (D)
- net V_Ref: now also R243.1
- new net: Q66.2 (G), R243.2, SW10.1

Commit message: Add files via upload
Parts:
- added LED1: LED_1.8mm_Amber, PCM_LED_THT_AKL:LED_D1.8mm_W3.3mm_H2.4mm, symbol PCM_LED_AKL:LED_1.8mm_Amber
- added Q67: 2N7000, PCM_Package_TO_SOT_THT_AKL:TO-92_Inline_Wide_SGD, symbol PCM_Transistor_MOSFET_AKL:2N7000
- added R244: R330 Ohm, Resistor_THT:R_Axial_DIN0207_L6.3mm_D2.5mm_P10.16mm_Horizontal, symbol PCM_SL_Resistors:100k
- R243: value R100 Ohm -> R100kΩ
Connections:
- net GND: now also Q67.1 (S)
- net V_Ref: now also LED1.2 (A)
- net at Q66.2 (G), R243.2, SW10.1: now also Q67.2 (G)
- new net: Q67.3 (D), R244.1
- new net: LED1.1 (K), R244.2

Commit message: Add files via upload
Parts:
- added C9: 4.7µF 63V, Capacitor_THT:C_Rect_L19.0mm_W7.0mm_P15.00mm_MKS4, symbol PCM_SL_Devices:Capacitor_NP
- R158: value 4.7k -> 330kΩ
Other:
- note added: "Protection contre surchauffe"
- moved on the sheet: LED1, OC10, OC9, Q43, Q66, Q67, R155, R156, R157, R158, R159, R160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

Commit message: Add files via upload
Parts:
- added R245, R246: 10k, Resistor_THT:R_Axial_DIN0207_L6.3mm_D2.5mm_P10.16mm_Horizontal, symbol PCM_SL_Resistors:10k
Connections:
- net GND: now also C9.2, R246.2; no longer U11.9 (+)
- net V_Ref: now also R245.1; no longer OC10.2, OC9.2, R158.2, R159.2, U11.8 (-)
- net To_C9_1: now reaches C9.1
- net To_C9_1: now also R158.1, U11.1, U11.9 (+)
- net To_U11_14: now reaches U11.14
- net To_U11_14: now also OC10.2
- new net: R245.2, R246.1, U11.8 (-)
- new net: OC9.2, R159.2
- no-connect marks 1 -> 0
Other:
- moved on the sheet: OC9, R160

Commit message: Add files via upload
Connections:
- net V_Ref: now also R158.2, R159.2
- net at R159.1, U11.13: now also OC9.2
Changed lines of the file:
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@@
 		(color 0 0 0 0)
 	)
+	(junction
+		(at 64.77 100.33)
+		(diameter 0)
+		(color 0 0 0 0)
+	)
 	(wire
 		(pts
@@
 	(wire
 		(pts
+			(xy 74.93 83.82) (xy 77.47 83.82)
+		)
+		(stroke
+			(width 0)
+			(type default)
+		)
+	)
+	(wire
+		(pts
 			(xy 116.84 106.68) (xy 113.03 106.68)
 		)
@@
 	(wire
 		(pts
+			(xy 64.77 100.33) (xy 62.23 100.33)
+		)
+		(stroke
+			(width 0)
+			(type default)
+		)
+	)
+	(wire
+		(pts
 			(xy 147.32 64.77) (xy 151.13 64.77)
 		)
@@
 	(wire
 		(pts
-			(xy 74.93 100.33) (xy 74.93 105.41)
+			(xy 74.93 100.33) (xy 77.47 100.33)
 		)
 		(stroke
@@
 	(wire
 		(pts
-			(xy 67.31 100.33) (xy 62.23 100.33)
+			(xy 67.31 100.33) (xy 64.77 100.33)
 		)
 		(stroke
@@
 	(wire
 		(pts
-			(xy 74.93 105.41) (xy 105.41 105.41)
+			(xy 64.77 100.33) (xy 64.77 105.41)
 		)
 		(stroke
@@
 		(pts
 			(xy 113.03 106.68) (xy 113.03 105.41)
+		)
+		(stroke
+			(width 0)
+			(type default)
+		)
+	)
+	(wire
+		(pts
+			(xy 64.77 105.41) (xy 105.41 105.41)
 		)
 		(stroke
@@
 		)
 	)
+	(global_label "V_Ref"
+		(shape input)
+		(at 77.47 83.82 0)
+		(fields_autoplaced yes)
+		(effects
+			(font
+				(size 1.27 1.27)
+			)
+			(justify left)
+		)
+		(property "Intersheetrefs" "${INTERSHEET_REFS}"
+			(at 85.5957 83.82 0)
+			(hide yes)
+			(show_name no)
+			(do_not_autoplace no)
+			(effects
+				(font
+					(size 1.27 1.27)
+				)
+				(justify left)
+			)
+		)
+	)
 	(global_label "GND"
 		(shape input)
@@
 			)
 		)
+	)
+	(global_label "V_Ref"
+		(shape input)
+		(at 77.47 100.33 0)
+		(fields_autoplaced yes)
+		(effects
+			(font
+				(size 1.27 1.27)
+			)
+			(justify left)
+		)
+		(property "Intersheetrefs" "${INTERSHEET_REFS}"
+			(at 85.5957 100.33 0)
+			(hide yes)
+			(show_name no)
+			(do_not_autoplace no)
+			(effects
+				(font
+					(size 1.27 1.27)
+				)
+				(justify left)
+			)
+		)

Commit message: Add files via upload
Changed lines of the file:
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@@
-	)
-	(junction
-		(at 64.77 87.63)
-		(diameter 0)
-		(color 0 0 0 0)
 	)
 	(junction
@@
 	(wire
 		(pts
-			(xy 64.77 87.63) (xy 64.77 91.44)
-		)
-		(stroke
-			(width 0)
-			(type default)
-		)
-	)
-	(wire
-		(pts
 			(xy 130.81 147.32) (xy 134.62 147.32)
 		)
@@
 		(pts
 			(xy 96.52 59.69) (xy 114.3 59.69)
-		)
-		(stroke
-			(width 0)
-			(type default)
-		)
-	)
-	(wire
-		(pts
-			(xy 68.58 91.44) (xy 64.77 91.44)
 		)
 		(stroke
@@
 		)
 	)
-	(label "To_U11_9"
+	(label "To_C9_1"
 		(at 44.45 113.03 180)
 		(effects
@@
 		(effects
 			(font
-				(size 1.27 1.27)
-			)
-			(justify left bottom)
-		)
-	)
-	(label "To_U11_9"
-		(at 68.58 91.44 0)
-		(effects
-			(font

Commit message: Add files via upload
Other:
- note removed: "Aux_Vehic_Shunt_Haut"
- moved on the sheet: C9, LED1, OC10, OC9, Q43, Q66, Q67, R155, R156, R157, R158, R159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
