File: Vehicule_Aux.kicad_sch (KiCad schematic)
At the start: 25 parts, among them Q43 IRLZ44N, Q66 2N7000, Q67 2N7000, SW10 TH_Aux, U11 LM339

Commit message: Add files via upload
Parts:
- U11: footprint (none) -> Package_DIP:DIP-14_W7.62mm_Socket
Changed lines of the file:
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@@
 			)
 		)
-		(property "Footprint" ""
+		(property "Footprint" "Package_DIP:DIP-14_W7.62mm_Socket"
 			(at 67.31 93.98 0)
 			(hide yes)
@@
 			)
 		)
-		(property "Footprint" ""
+		(property "Footprint" "Package_DIP:DIP-14_W7.62mm_Socket"
 			(at 67.31 77.47 0)
 			(hide yes)
@@
 			)
 		)
-		(property "Footprint" ""
+		(property "Footprint" "Package_DIP:DIP-14_W7.62mm_Socket"
 			(at 67.31 110.49 0)
 			(hide yes)
@@
 			)
 		)
-		(property "Footprint" ""
+		(property "Footprint" "Package_DIP:DIP-14_W7.62mm_Socket"
 			(at 63.5 130.81 0)
 			(hide yes)
@@
 			)
 		)
-		(property "Footprint" ""
+		(property "Footprint" "Package_DIP:DIP-14_W7.62mm_Socket"
 			(at 67.31 57.15 0)
 			(hide yes)

Commit message: Add files via upload
Parts:
- SW10: footprint (none) -> TerminalBlock_Phoenix:TerminalBlock_Phoenix_PT-1,5-2-3.5-H_1x02_P3.50mm_Horizontal
Changed lines of the file:
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@@
 			)
 		)
-		(property "Footprint" ""
+		(property "Footprint" "TerminalBlock_Phoenix:TerminalBlock_Phoenix_PT-1,5-2-3.5-H_1x02_P3.50mm_Horizontal"
 			(at 281.94 53.34 0)
 			(hide yes)

Commit message: Add files via upload
Other:
- note removed: "Court-circuit"
- note removed: "Injection"
- note removed: "Ouvvert"
Changed lines of the file:
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@@
-		)
-	)
-	(text "Injection"
-		(exclude_from_sim no)
-		(at 68.58 54.61 0)
-		(effects
-			(font
-				(size 0.762 0.762)
-			)
-		)
-	)
-	(text "Court-circuit\n"
-		(exclude_from_sim no)
-		(at 72.39 91.44 0)
-		(effects
-			(font
-				(size 0.762 0.762)
-			)
 		)
 	)
@@
 			(font
 				(size 1.27 1.27)
-			)
-		)
-	)
-	(text "Ouvvert\n"
-		(exclude_from_sim no)
-		(at 72.39 74.93 0)
-		(effects
-			(font
-				(size 0.762 0.762)
 			)
 		)
@@
 	)
 	(junction
-		(at 90.805 45.72)
+		(at 78.74 45.72)
+		(diameter 0)
+		(color 0 0 0 0)
+	)
+	(junction
+		(at 36.83 82.55)
 		(diameter 0)
 		(color 0 0 0 0)
@@
 	)
 	(junction
-		(at 36.83 82.55)
-		(diameter 0)
-		(color 0 0 0 0)
-	)
-	(junction
 		(at 270.51 55.88)
 		(diameter 0)
@@
 	(wire
 		(pts
-			(xy 36.83 21.59) (xy 36.83 82.55)
+			(xy 34.29 20.32) (xy 34.29 82.55)
 		)
 		(stroke
@@
 	(wire
 		(pts
+			(xy 34.29 82.55) (xy 36.83 82.55)
+		)
+		(stroke
+			(width 0)
+			(type default)
+		)
+	)
+	(wire
+		(pts
 			(xy 270.51 55.88) (xy 270.51 88.9)
 		)
@@
 	(wire
 		(pts
-			(xy 124.46 21.59) (xy 36.83 21.59)
+			(xy 124.46 20.32) (xy 34.29 20.32)
 		)
 		(stroke
@@
 	(wire
 		(pts
-			(xy 78.74 83.82) (xy 78.74 80.01)
+			(xy 78.74 85.09) (xy 78.74 80.01)
 		)
 		(stroke
@@
 	(wire
 		(pts
-			(xy 82.55 40.64) (xy 90.805 40.64)
-		)
-		(stroke
-			(width 0)
-			(type default)
-		)
-	)
-	(wire
-		(pts
 			(xy 228.6 99.06) (xy 232.41 99.06)
 		)
@@
 	(wire
 		(pts
-			(xy 78.74 83.82) (xy 82.55 83.82)
-		)
-		(stroke
-			(width 0)
-			(type default)
-		)
-	)
-	(wire
-		(pts
-			(xy 90.805 45.72) (xy 104.14 45.72)
-		)
-		(stroke
-			(width 0)
-			(type default)
-		)
-	)
-	(wire
-		(pts
-			(xy 124.46 52.07) (xy 124.46 21.59)
+			(xy 78.74 85.09) (xy 82.55 85.09)
+		)
+		(stroke
+			(width 0)
+			(type default)
+		)
+	)
+	(wire
+		(pts
+			(xy 124.46 52.07) (xy 124.46 20.32)
 		)
 		(stroke
@@
 	(wire
 		(pts
-			(xy 78.74 45.72) (xy 90.805 45.72)
+			(xy 78.74 45.72) (xy 104.14 45.72)
 		)
 		(stroke
@@
 	(wire
 		(pts
-			(xy 90.805 40.64) (xy 90.805 45.72)
+			(xy 78.74 38.1) (xy 78.74 45.72)
 		)
 		(stroke
@@
 	)
 	(label "To_C9_1"
-		(at 82.55 83.82 0)
+		(at 82.55 85.09 0)
 		(effects
 			(font
@@
 		)
 	)
+	(label "Injection_Aux_Fault"
+		(at 78.74 38.1 180)
+		(effects
+			(font
+				(size 1.27 1.27)
+			)
+			(justify right bottom)
+		)
+	)
 	(label "Seuil_Injection_Aux"
 		(at 60.96 62.23 180)
@@
 		(shape input)
 		(at 96.52 36.83 180)
-		(effects
-			(font
-				(size 1.27 1.27)
-			)
-			(justify right)
-		)
-	)
-	(hierarchical_label "Injection_Aux_Fault"
-		(shape input)
-		(at 82.55 40.64 180)
 		(effects
 			(font
@@
 		(property "Etiquette" "R_Aux_PU_C"
 			(at 85.09 94.234 0)
-			(show_name no)
-			(do_not_autoplace no)
+			(hide yes)
+			(show_name no)
+			(do_not_autoplace no)

Commit message: Add files via upload
Other:
- note removed: "Non_Utilisé"
- moved on the sheet: R156
Changed lines of the file:
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@@
-		)
-	)
-	(text "Non_Utilisé"
-		(exclude_from_sim no)
-		(at 71.12 107.95 0)
-		(effects
-			(font
-				(size 0.762 0.762)
-			)
 		)
 	)
@@
 	)
 	(junction
-		(at 36.83 93.98)
-		(diameter 0)
-		(color 0 0 0 0)
-	)
-	(junction
 		(at 59.69 115.57)
 		(diameter 0)
@@
 	)
 	(junction
-		(at 36.83 82.55)
+		(at 34.29 93.98)
 		(diameter 0)
 		(color 0 0 0 0)
@@
 	)
 	(junction
+		(at 34.29 82.55)
+		(diameter 0)
+		(color 0 0 0 0)
+	)
+	(junction
 		(at 58.42 30.48)
 		(diameter 0)
@@
 	(wire
 		(pts
-			(xy 34.29 82.55) (xy 36.83 82.55)
+			(xy 34.29 82.55) (xy 60.96 82.55)
 		)
 		(stroke
@@
 	(wire
 		(pts
-			(xy 36.83 93.98) (xy 36.83 128.27)
+			(xy 34.29 93.98) (xy 34.29 128.27)
 		)
 		(stroke
@@
 	(wire
 		(pts
-			(xy 36.83 128.27) (xy 31.75 128.27)
+			(xy 34.29 128.27) (xy 29.21 128.27)
 		)
 		(stroke
@@
 	(wire
 		(pts
-			(xy 36.83 82.55) (xy 36.83 93.98)
+			(xy 34.29 82.55) (xy 34.29 93.98)
 		)
 		(stroke
@@
 	(wire
 		(pts
-			(xy 36.83 82.55) (xy 60.96 82.55)
-		)
-		(stroke
-			(width 0)
-			(type default)
-		)
-	)
-	(wire
-		(pts
 			(xy 273.05 73.66) (xy 273.05 55.88)
 		)
@@
 	(wire
 		(pts
-			(xy 36.83 93.98) (xy 60.96 93.98)
-		)
-		(stroke
-			(width 0)
-			(type default)
-		)
-	)
-	(wire
-		(pts
 			(xy 148.59 82.55) (xy 148.59 85.09)
 		)
@@
 		(pts
 			(xy 107.95 36.83) (xy 110.49 36.83)
+		)
+		(stroke
+			(width 0)
+			(type default)
+		)
+	)
+	(wire
+		(pts
+			(xy 34.29 93.98) (xy 60.96 93.98)
 		)
 		(stroke
@@
 		)
 	)
+	(label "Injection_Aux_Fault"
+		(at 288.29 63.5 0)
+		(effects
+			(font
+				(size 1.27 1.27)
+			)
+			(justify left bottom)
+		)
+	)
 	(label "To_U11_14"
 		(at 142.24 85.09 180)
@@
 	(global_label "GND"
 		(shape input)
-		(at 24.13 128.27 180)
+		(at 21.59 128.27 180)
 		(fields_autoplaced yes)
 		(effects
@@
 		)
 		(property "Intersheetrefs" "${INTERSHEET_REFS}"
-			(at 20.0163 128.27 0)
+			(at 17.4763 128.27 0)
 			(hide yes)
 			(show_name no)
@@
 				(justify right)
 			)
-		)
-	)
-	(hierarchical_label "Injection_Aux_Fault"
-		(shape input)
-		(at 288.29 63.5 0)
-		(effects
-			(font
-				(size 1.27 1.27)
-			)
-			(justify left)
 		)
 	)
@@
 	(symbol
 		(lib_id "PCM_SL_Devices:Resistor_5W")
-		(at 27.94 128.27 0)
+		(at 25.4 128.27 0)
 		(mirror y)
 		(unit 1)
@@
 		(fields_autoplaced yes)
 		(property "Reference" "R156"
-			(at 27.94 121.92 0)
+			(at 25.4 121.92 0)
 			(show_name no)
 			(do_not_autoplace no)
@@
 		)
 		(property "Value" ".05R Shunt"
-			(at 27.94 124.46 0)
+			(at 25.4 124.46 0)
 			(show_name no)
 			(do_not_autoplace no)
@@
 		)
 		(property "Footprint" "Resistor_THT:R_Axial_Power_L25.0mm_W9.0mm_P27.94mm"
-			(at 27.051 132.588 0)
+			(at 24.511 132.588 0)
 			(hide yes)
 			(show_name no)
@@
 		)
 		(property "Datasheet" ""
-			(at 27.432 128.27 0)
+			(at 24.892 128.27 0)
 			(hide yes)
 			(show_name no)
@@
 		)
 		(property "Description" "5W Resistor"
-			(at 27.94 128.27 0)
-			(hide yes)
-			(show_name no)
+			(at 25.4 128.27 0)
+			(hide yes)
+			(show_name no)

Commit message: Add files via upload
Parts:
- R157, R159: value 4.7k -> 4.7kΩ
- R160, R161: value 1k -> 1kΩ
- R162: value 100k -> 100kΩ
- R163, R245, R246: value 10k -> 10kΩ
- R244: value R330 Ohm -> R330Ω
Changed lines of the file:
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@@
 			)
 		)
-		(property "Value" "10k"
+		(property "Value" "10kΩ"
 			(at 54.61 119.38 0)
 			(show_name no)
@@
 			)
 		)
-		(property "Value" "1k"
+		(property "Value" "1kΩ"
 			(at 139.7 67.31 0)
 			(show_name no)
@@
 			)
 		)
-		(property "Value" "10k"
+		(property "Value" "10kΩ"
 			(at 64.77 26.67 0)
 			(show_name no)
@@
 			)
 		)
-		(property "Value" "4.7k"
+		(property "Value" "4.7kΩ"
 			(at 85.09 92.71 0)
 			(show_name no)
@@
 			)
 		)
-		(property "Value" "R330 Ohm"
+		(property "Value" "R330Ω"
 			(at 236.22 96.52 0)
 			(show_name no)
@@
 			)
 		)
-		(property "Value" "1k"
+		(property "Value" "1kΩ"
 			(at 144.78 91.44 0)
 			(show_name no)
@@
 			)
 		)
-		(property "Value" "10k"
+		(property "Value" "10kΩ"
 			(at 82.55 118.11 0)
 			(show_name no)
@@
 			)
 		)
-		(property "Value" "4.7k"
+		(property "Value" "4.7kΩ"
 			(at 85.09 55.88 0)
 			(show_name no)
@@
 			)
 		)
-		(property "Value" "100k"
+		(property "Value" "100kΩ"
 			(at 52.07 26.67 0)
 			(show_name no)

Commit message: Add files via upload
Parts:
- R243: value R100kΩ -> 100kΩ
- R244: value R330Ω -> 330Ω
Changed lines of the file:
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@@
 			)
 		)
-		(property "Value" "R330Ω"
+		(property "Value" "330Ω"
 			(at 236.22 96.52 0)
 			(show_name no)
@@
 			)
 		)
-		(property "Value" "R100kΩ"
+		(property "Value" "100kΩ"
 			(at 264.16 51.054 0)
 			(show_name no)
@@
 		(property "Etiquette" "R_Surch_Aux"
 			(at 264.16 53.34 0)
-			(show_name no)
-			(do_not_autoplace no)
+			(hide yes)
+			(show_name no)
+			(do_not_autoplace no)
