File: Vehicule_Right.kicad_sch (KiCad schematic)
At the start: 16 parts, among them Q27 IRLZ44N, U7 LM339

Commit message: Add files via upload
Connections:
- net V_Ref: no longer Q27.1 (G)
- net Veh_Right_Inject_Cmd: now reaches R91.1, U7.2
- net Veh_Right_Inject_Cmd: now also Q27.1 (G)
Changed lines of the file:
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@@
 	)
 	(junction
-		(at 138.43 69.85)
+		(at 124.46 69.85)
 		(diameter 0)
 		(color 0 0 0 0)
@@
 	(wire
 		(pts
+			(xy 124.46 69.85) (xy 121.92 69.85)
+		)
+		(stroke
+			(width 0)
+			(type default)
+		)
+	)
+	(wire
+		(pts
 			(xy 176.53 88.9) (xy 176.53 87.63)
 		)
@@
 	(wire
 		(pts
-			(xy 149.86 55.88) (xy 138.43 55.88)
-		)
-		(stroke
-			(width 0)
-			(type default)
-		)
-	)
-	(wire
-		(pts
 			(xy 167.64 110.49) (xy 163.83 110.49)
 		)
@@
 	(wire
 		(pts
-			(xy 138.43 55.88) (xy 138.43 69.85)
-		)
-		(stroke
-			(width 0)
-			(type default)
-		)
-	)
-	(wire
-		(pts
 			(xy 82.55 101.6) (xy 106.68 101.6)
 		)
@@
 	(wire
 		(pts
+			(xy 124.46 55.88) (xy 149.86 55.88)
+		)
+		(stroke
+			(width 0)
+			(type default)
+		)
+	)
+	(wire
+		(pts
 			(xy 82.55 90.17) (xy 82.55 101.6)
 		)
@@
 	(wire
 		(pts
-			(xy 142.24 69.85) (xy 138.43 69.85)
-		)
-		(stroke
-			(width 0)
-			(type default)
-		)
-	)
-	(wire
-		(pts
 			(xy 156.21 59.69) (xy 156.21 63.5)
 		)
@@
 	(wire
 		(pts
+			(xy 124.46 55.88) (xy 124.46 69.85)
+		)
+		(stroke
+			(width 0)
+			(type default)
+		)
+	)
+	(wire
+		(pts
 			(xy 144.78 87.63) (xy 165.1 87.63)
 		)
@@
 	(wire
 		(pts
-			(xy 138.43 69.85) (xy 134.62 69.85)
+			(xy 134.62 69.85) (xy 142.24 69.85)
 		)
 		(stroke
@@
 	(wire
 		(pts
-			(xy 127 69.85) (xy 121.92 69.85)
+			(xy 127 69.85) (xy 124.46 69.85)
 		)
 		(stroke
@@
 			)
 			(justify right bottom)
+		)
+	)
+	(label "Veh_Right_Inject_Cmd"
+		(at 124.46 55.88 180)
+		(effects
+			(font
+				(size 1.016 1.016)
+			)
+			(justify right bottom)

Commit message: Add files via upload
Changed lines of the file:
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@@
-	(wire
-		(pts
-			(xy 172.72 77.47) (xy 171.45 77.47)
-		)
-		(stroke
-			(width 0)
-			(type default)
-		)
-	)
 	(wire
 		(pts
@@
 		(pts
 			(xy 167.64 111.76) (xy 167.64 110.49)
+		)
+		(stroke
+			(width 0)
+			(type default)
+		)
+	)
+	(wire
+		(pts
+			(xy 172.72 77.47) (xy 176.53 77.47)
 		)
 		(stroke
@@
 	(hierarchical_label "Ouvert_Right_Vehic"
 		(shape input)
-		(at 172.72 77.47 0)
-		(effects
-			(font
+		(at 176.53 77.47 0)
+		(effects
+			(font

Commit message: Add files via upload
Parts:
- R100, R98, R99: footprint (none) -> TRIM_3296W1103LF:TRIM_3296W1103LF
- R89: value 3 Ohm - 5W -> 12 Ohm - 25W; footprint Resistor_THT:R_Axial_Power_L25.0mm_W9.0mm_P27.94mm -> TerminalBlock_Phoenix:TerminalBlock_Phoenix_PT-1,5-2-3.5-H_1x02_P3.50mm_Horizontal
- R90: value .05R Shunt -> 0.2 Ohm Shunt
Connections:
- net Veh_Right_Inject_Cmd renamed Injection_Right_Fault
Changed lines of the file:
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@@
+	)
+	(junction
+		(at 134.62 55.88)
+		(diameter 0)
+		(color 0 0 0 0)
 	)
 	(junction
@@
 	(wire
 		(pts
+			(xy 134.62 55.88) (xy 149.86 55.88)
+		)
+		(stroke
+			(width 0)
+			(type default)
+		)
+	)
+	(wire
+		(pts
 			(xy 124.46 69.85) (xy 121.92 69.85)
 		)
@@
 	(wire
 		(pts
+			(xy 134.62 47.625) (xy 134.62 55.88)
+		)
+		(stroke
+			(width 0)
+			(type default)
+		)
+	)
+	(wire
+		(pts
 			(xy 207.01 87.63) (xy 210.82 87.63)
 		)
@@
 	(wire
 		(pts
-			(xy 124.46 55.88) (xy 149.86 55.88)
+			(xy 124.46 55.88) (xy 134.62 55.88)
 		)
 		(stroke
@@
 		(pts
 			(xy 156.21 48.26) (xy 156.21 49.53)
+		)
+		(stroke
+			(width 0)
+			(type default)
+		)
+	)
+	(wire
+		(pts
+			(xy 128.27 47.625) (xy 134.62 47.625)
 		)
 		(stroke
@@
 			(font
 				(size 1.27 1.27)
-			)
-			(justify right bottom)
-		)
-	)
-	(label "Veh_Right_Inject_Cmd"
-		(at 124.46 55.88 180)
-		(effects
-			(font
-				(size 1.016 1.016)
 			)
 			(justify right bottom)
@@
 				(justify right)
 			)
+		)
+	)
+	(hierarchical_label "Injection_Right_Fault"
+		(shape input)
+		(at 128.27 47.625 180)
+		(effects
+			(font
+				(size 1.27 1.27)
+			)
+			(justify right)
 		)
 	)
@@
 			)
 		)
-		(property "Value" "3 Ohm - 5W"
+		(property "Value" "12 Ohm - 25W"
 			(at 73.66 128.27 0)
 			(show_name no)
@@
 			)
 		)
-		(property "Footprint" "Resistor_THT:R_Axial_Power_L25.0mm_W9.0mm_P27.94mm"
+		(property "Footprint" "TerminalBlock_Phoenix:TerminalBlock_Phoenix_PT-1,5-2-3.5-H_1x02_P3.50mm_Horizontal"
 			(at 74.549 136.398 0)
 			(hide yes)
@@
 			)
 		)
-		(property "Description" "5W Resistor"
+		(property "Description" "25W Resistor"
 			(at 73.66 132.08 0)
 			(hide yes)
@@
 			)
 		)
-		(property "Footprint" ""
+		(property "Footprint" "TRIM_3296W1103LF:TRIM_3296W1103LF"
 			(at 210.82 64.77 0)
 			(hide yes)
@@
 			)
 		)
-		(property "Footprint" ""
+		(property "Footprint" "TRIM_3296W1103LF:TRIM_3296W1103LF"
 			(at 210.82 46.99 0)
 			(hide yes)
@@
 			)
 		)
-		(property "Footprint" ""
+		(property "Footprint" "TRIM_3296W1103LF:TRIM_3296W1103LF"
 			(at 210.82 83.82 0)
 			(hide yes)
@@
 			)
 		)
-		(property "Value" ".05R Shunt"
+		(property "Value" "0.2 Ohm Shunt"
 			(at 90.17 128.27 0)
 			(show_name no)

Commit message: Add files via upload
Parts:
- R100, R98, R99: footprint TRIM_3296W1103LF:TRIM_3296W1103LF -> (none)
- R89: value 12 Ohm - 25W -> 3 Ohm - 5W; footprint TerminalBlock_Phoenix:TerminalBlock_Phoenix_PT-1,5-2-3.5-H_1x02_P3.50mm_Horizontal -> Resistor_THT:R_Axial_Power_L25.0mm_W9.0mm_P27.94mm
- R90: value 0.2 Ohm Shunt -> .05R Shunt
Connections:
- net Injection_Right_Fault renamed Veh_Right_Inject_Cmd
Changed lines of the file:
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@@
-	)
-	(junction
-		(at 134.62 55.88)
-		(diameter 0)
-		(color 0 0 0 0)
 	)
 	(junction
@@
 	(wire
 		(pts
-			(xy 134.62 55.88) (xy 149.86 55.88)
-		)
-		(stroke
-			(width 0)
-			(type default)
-		)
-	)
-	(wire
-		(pts
 			(xy 124.46 69.85) (xy 121.92 69.85)
 		)
@@
 	(wire
 		(pts
-			(xy 134.62 47.625) (xy 134.62 55.88)
-		)
-		(stroke
-			(width 0)
-			(type default)
-		)
-	)
-	(wire
-		(pts
 			(xy 207.01 87.63) (xy 210.82 87.63)
 		)
@@
 	(wire
 		(pts
-			(xy 124.46 55.88) (xy 134.62 55.88)
+			(xy 124.46 55.88) (xy 149.86 55.88)
 		)
 		(stroke
@@
 		(pts
 			(xy 156.21 48.26) (xy 156.21 49.53)
-		)
-		(stroke
-			(width 0)
-			(type default)
-		)
-	)
-	(wire
-		(pts
-			(xy 128.27 47.625) (xy 134.62 47.625)
 		)
 		(stroke
@@
 			(font
 				(size 1.27 1.27)
+			)
+			(justify right bottom)
+		)
+	)
+	(label "Veh_Right_Inject_Cmd"
+		(at 124.46 55.88 180)
+		(effects
+			(font
+				(size 1.016 1.016)
 			)
 			(justify right bottom)
@@
 				(justify right)
 			)
-		)
-	)
-	(hierarchical_label "Injection_Right_Fault"
-		(shape input)
-		(at 128.27 47.625 180)
-		(effects
-			(font
-				(size 1.27 1.27)
-			)
-			(justify right)
 		)
 	)
@@
 			)
 		)
-		(property "Value" "12 Ohm - 25W"
+		(property "Value" "3 Ohm - 5W"
 			(at 73.66 128.27 0)
 			(show_name no)
@@
 			)
 		)
-		(property "Footprint" "TerminalBlock_Phoenix:TerminalBlock_Phoenix_PT-1,5-2-3.5-H_1x02_P3.50mm_Horizontal"
+		(property "Footprint" "Resistor_THT:R_Axial_Power_L25.0mm_W9.0mm_P27.94mm"
 			(at 74.549 136.398 0)
 			(hide yes)
@@
 			)
 		)
-		(property "Description" "25W Resistor"
+		(property "Description" "5W Resistor"
 			(at 73.66 132.08 0)
 			(hide yes)
@@
 			)
 		)
-		(property "Footprint" "TRIM_3296W1103LF:TRIM_3296W1103LF"
+		(property "Footprint" ""
 			(at 210.82 64.77 0)
 			(hide yes)
@@
 			)
 		)
-		(property "Footprint" "TRIM_3296W1103LF:TRIM_3296W1103LF"
+		(property "Footprint" ""
 			(at 210.82 46.99 0)
 			(hide yes)
@@
 			)
 		)
-		(property "Footprint" "TRIM_3296W1103LF:TRIM_3296W1103LF"
+		(property "Footprint" ""
 			(at 210.82 83.82 0)
 			(hide yes)
@@
 			)
 		)
-		(property "Value" "0.2 Ohm Shunt"
+		(property "Value" ".05R Shunt"
 			(at 90.17 128.27 0)
 			(show_name no)

Commit message: Add files via upload
Parts:
- R100, R98, R99: footprint (none) -> TRIM_3296W1103LF:TRIM_3296W1103LF
Connections:
- net Veh_Right_Inject_Cmd renamed Injection_Right_Fault
Changed lines of the file:
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@@
+	)
+	(junction
+		(at 134.62 55.88)
+		(diameter 0)
+		(color 0 0 0 0)
 	)
 	(junction
@@
 	(wire
 		(pts
+			(xy 134.62 55.88) (xy 149.86 55.88)
+		)
+		(stroke
+			(width 0)
+			(type default)
+		)
+	)
+	(wire
+		(pts
 			(xy 124.46 69.85) (xy 121.92 69.85)
 		)
@@
 	(wire
 		(pts
+			(xy 134.62 47.625) (xy 134.62 55.88)
+		)
+		(stroke
+			(width 0)
+			(type default)
+		)
+	)
+	(wire
+		(pts
 			(xy 207.01 87.63) (xy 210.82 87.63)
 		)
@@
 	(wire
 		(pts
-			(xy 124.46 55.88) (xy 149.86 55.88)
+			(xy 124.46 55.88) (xy 134.62 55.88)
 		)
 		(stroke
@@
 		(pts
 			(xy 156.21 48.26) (xy 156.21 49.53)
+		)
+		(stroke
+			(width 0)
+			(type default)
+		)
+	)
+	(wire
+		(pts
+			(xy 128.27 47.625) (xy 134.62 47.625)
 		)
 		(stroke
@@
 		)
 	)
-	(label "Veh_Right_Inject_Cmd"
-		(at 124.46 55.88 180)
-		(effects
-			(font
-				(size 1.016 1.016)
-			)
-			(justify right bottom)
-		)
-	)
 	(label "Seuil_Ouvert_Right"
 		(at 214.63 64.77 0)
@@
 				(justify right)
 			)
+		)
+	)
+	(hierarchical_label "Injection_Right_Fault"
+		(shape input)
+		(at 128.27 47.625 180)
+		(effects
+			(font
+				(size 1.27 1.27)
+			)
+			(justify right)
 		)
 	)
@@
 			)
 		)
-		(property "Footprint" ""
+		(property "Footprint" "TRIM_3296W1103LF:TRIM_3296W1103LF"
 			(at 210.82 64.77 0)
 			(hide yes)
@@
 			)
 		)
-		(property "Footprint" ""
+		(property "Footprint" "TRIM_3296W1103LF:TRIM_3296W1103LF"
 			(at 210.82 46.99 0)
 			(hide yes)
@@
 			)
 		)
-		(property "Footprint" ""
+		(property "Footprint" "TRIM_3296W1103LF:TRIM_3296W1103LF"
 			(at 210.82 83.82 0)
 			(hide yes)

Commit message: Add files via upload
Parts:
- R89: value 3 Ohm - 5W -> 12 Ohm - 25W; footprint Resistor_THT:R_Axial_Power_L25.0mm_W9.0mm_P27.94mm -> TerminalBlock_Phoenix:TerminalBlock_Phoenix_PT-1,5-2-3.5-H_1x02_P3.50mm_Horizontal
- R90: value .05R Shunt -> 0.2 Ohm Shunt
Changed lines of the file:
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@@
 			)
 		)
-		(property "Value" "3 Ohm - 5W"
+		(property "Value" "12 Ohm - 25W"
 			(at 73.66 128.27 0)
 			(show_name no)
@@
 			)
 		)
-		(property "Footprint" "Resistor_THT:R_Axial_Power_L25.0mm_W9.0mm_P27.94mm"
+		(property "Footprint" "TerminalBlock_Phoenix:TerminalBlock_Phoenix_PT-1,5-2-3.5-H_1x02_P3.50mm_Horizontal"
 			(at 74.549 136.398 0)
 			(hide yes)
@@
 			)
 		)
-		(property "Description" "5W Resistor"
+		(property "Description" "25W Resistor"
 			(at 73.66 132.08 0)
 			(hide yes)
@@
 			)
 		)
-		(property "Value" ".05R Shunt"
+		(property "Value" "0.2 Ohm Shunt"
 			(at 90.17 128.27 0)
 			(show_name no)

Commit message: Add files via upload
Other:
- note removed: "Right_Vehic_Shunt_Haut"
Changed lines of the file:
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@@
-		)
-	)
-	(text "Right_Vehic_Shunt_Haut"
-		(exclude_from_sim no)
-		(at 80.264 105.664 90)
-		(effects
-			(font
-				(size 0.762 0.762)
-			)
 		)
 	)
@@
 	)
 	(junction
+		(at 139.7 109.22)
+		(diameter 0)
+		(color 0 0 0 0)
+	)
+	(junction
 		(at 82.55 101.6)
 		(diameter 0)
@@
 		(color 0 0 0 0)
 	)
-	(junction
-		(at 140.97 109.22)
-		(diameter 0)
-		(color 0 0 0 0)
-	)
 	(no_connect
 		(at 121.92 119.38)
@@
 	(wire
 		(pts
+			(xy 139.7 104.14) (xy 142.24 104.14)
+		)
+		(stroke
+			(width 0)
+			(type default)
+		)
+	)
+	(wire
+		(pts
 			(xy 176.53 88.9) (xy 176.53 87.63)
 		)
@@
 	(wire
 		(pts
-			(xy 134.62 47.625) (xy 134.62 55.88)
+			(xy 134.62 48.26) (xy 134.62 55.88)
 		)
 		(stroke
@@
 	(wire
 		(pts
+			(xy 102.87 106.68) (xy 106.68 106.68)
+		)
+		(stroke
+			(width 0)
+			(type default)
+		)
+	)
+	(wire
+		(pts
 			(xy 170.18 34.29) (xy 104.14 34.29)
 		)
@@
 	(wire
 		(pts
-			(xy 140.97 104.14) (xy 140.97 109.22)
+			(xy 139.7 104.14) (xy 139.7 109.22)
 		)
 		(stroke
@@
 	(wire
 		(pts
+			(xy 102.87 85.09) (xy 106.68 85.09)
+		)
+		(stroke
+			(width 0)
+			(type default)
+		)
+	)
+	(wire
+		(pts
 			(xy 82.55 132.08) (xy 86.36 132.08)
 		)
@@
 	(wire
 		(pts
+			(xy 139.7 109.22) (xy 156.21 109.22)
+		)
+		(stroke
+			(width 0)
+			(type default)
+		)
+	)
+	(wire
+		(pts
 			(xy 151.13 48.26) (xy 156.21 48.26)
 		)
@@
 	(wire
 		(pts
-			(xy 128.27 47.625) (xy 134.62 47.625)
+			(xy 128.27 48.26) (xy 134.62 48.26)
 		)
 		(stroke
@@
 	(wire
 		(pts
-			(xy 134.62 109.22) (xy 140.97 109.22)
+			(xy 102.87 72.39) (xy 106.68 72.39)
+		)
+		(stroke
+			(width 0)
+			(type default)
+		)
+	)
+	(wire
+		(pts
+			(xy 134.62 109.22) (xy 139.7 109.22)
 		)
 		(stroke
@@
 		(pts
 			(xy 156.21 48.26) (xy 160.02 48.26)
-		)
-		(stroke
-			(width 0)
-			(type default)
-		)
-	)
-	(wire
-		(pts
-			(xy 156.21 109.22) (xy 140.97 109.22)
 		)
 		(stroke
@@
 	)
 	(label "Seuil_Ouvert_Right"
-		(at 106.68 85.09 180)
+		(at 102.87 85.09 180)
 		(effects
 			(font
@@
 	)
 	(label "Seuil_Injection_Right"
-		(at 106.68 72.39 180)
+		(at 102.87 72.39 180)
 		(effects
 			(font
@@
 	)
 	(label "Seuil_Court_Right"
-		(at 106.68 106.68 180)
+		(at 102.87 106.68 180)
 		(effects
 			(font
@@
 		)
 	)
+	(global_label "V_Ref"
+		(shape input)
+		(at 142.24 104.14 0)
+		(fields_autoplaced yes)
+		(effects
+			(font
+				(size 1.27 1.27)
+			)
+			(justify left)
+		)
+		(property "Intersheetrefs" "${INTERSHEET_REFS}"
+			(at 150.3657 104.14 0)
+			(hide yes)
+			(show_name no)
+			(do_not_autoplace no)
+			(effects
+				(font
+					(size 1.27 1.27)
+				)
+				(justify left)
+			)
+		)
+	)
 	(global_label "GND"
 		(shape input)
@@
 	(global_label "V_Ref"
 		(shape input)
-		(at 140.97 104.14 0)
-		(fields_autoplaced yes)
-		(effects
-			(font
-				(size 1.27 1.27)
-			)
-			(justify left)
-		)
-		(property "Intersheetrefs" "${INTERSHEET_REFS}"
-			(at 149.0957 104.14 0)
-			(hide yes)
-			(show_name no)
-			(do_not_autoplace no)
-			(effects
-				(font
-					(size 1.27 1.27)
-				)
-				(justify left)
-			)
-		)
-	)
-	(global_label "V_Ref"
-		(shape input)
 		(at 105.41 121.92 180)
 		(fields_autoplaced yes)
@@
 	(hierarchical_label "Injection_Right_Fault"
 		(shape input)
-		(at 128.27 47.625 180)
+		(at 128.27 48.26 180)
 		(effects
 			(font
@@
 		(property "Etiquette" "R_Right_LED_Ouvert"
 			(at 156.21 74.168 0)
-			(show_name no)
-			(do_not_autoplace no)
+			(hide yes)
+			(show_name no)
+			(do_not_autoplace no)

Commit message: Add files via upload
Connections:
- net V_Ref: no longer OC5.2, OC6.2
- net Veh_Right: now also R89.1; no longer Q27.2 (D)
- net Right_Vehic_Shunt_Haut: now reaches R90.1, U7.11 (+), U7.6 (-)
- net Right_Vehic_Shunt_Haut: now also Q27.3 (S); no longer R89.2
- net Opto_Ouvert_Right: now reaches R92.1, U7.1
- net Opto_Ouvert_Right: now also OC6.2
- net Opto_Court_Right: now reaches R93.1, U7.13
- net Opto_Court_Right: now also OC5.2
- removed net Q27_Source: Q27.3 (S), R89.1
- new net Q27_Drain: Q27.2 (D), R89.2
Other:
- note added: "Right_Vehic_Shunt_Haut"
