File: Bloc_Test_Right.kicad_sch (KiCad schematic)
At the start: 44 parts, among them Q29 2N7000, Q30 2N7000, Q31 2N7000, Q32 2N7000, Q33 2N7000, Q34 2N7000

Commit message: Add files via upload
Changed lines of the file:
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@@
-	)
-	(junction
-		(at 91.44 86.36)
-		(diameter 0)
-		(color 0 0 0 0)
 	)
 	(junction
@@
 	)
 	(junction
-		(at 52.07 86.36)
-		(diameter 0)
-		(color 0 0 0 0)
-	)
-	(junction
 		(at 64.77 53.34)
 		(diameter 0)
@@
 	(wire
 		(pts
-			(xy 50.8 86.36) (xy 52.07 86.36)
-		)
-		(stroke
-			(width 0)
-			(type default)
-		)
-	)
-	(wire
-		(pts
 			(xy 156.21 50.8) (xy 162.56 50.8)
 		)
@@
 		)
 		(stroke
-			(width 0)
-			(type default)
-		)
-	)
-	(wire
-		(pts
-			(xy 90.17 86.36) (xy 91.44 86.36)
-		)
-		(stroke

Commit message: Add files via upload
Changed lines of the file:
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@@
+	(wire
+		(pts
+			(xy 40.64 170.18) (xy 43.18 170.18)
+		)
+		(stroke
+			(width 0)
+			(type default)
+		)
+	)
 	(wire
 		(pts
@@
 	(wire
 		(pts
-			(xy 34.29 104.14) (xy 55.88 104.14)
+			(xy 35.56 104.14) (xy 55.88 104.14)
 		)
 		(stroke
@@
 		(pts
 			(xy 102.87 149.86) (xy 102.87 156.21)
+		)
+		(stroke
+			(width 0)
+			(type default)
+		)
+	)
+	(wire
+		(pts
+			(xy 99.06 168.91) (xy 101.6 168.91)
 		)
 		(stroke
@@
 	)
 	(label "Vert_Enable_Right"
-		(at 99.06 168.91 0)
+		(at 101.6 168.91 0)
 		(effects
 			(font
@@
 	)
 	(label "Ouvert_Ou_Bleu_Right"
-		(at 40.64 170.18 0)
+		(at 43.18 170.18 0)
 		(effects
 			(font
@@
 	)
 	(label "Ouvert_Right"
-		(at 34.29 104.14 180)
-		(effects
-			(font
+		(at 35.56 104.14 180)
+		(effects
+			(font

Commit message: Add files via upload
Parts:
- added D177: 1N4148, PCM_Diode_THT_AKL:D_DO-35_SOD27_P7.62mm_Horizontal, symbol PCM_Diode_AKL:1N4148
Connections:
- net Btn_Right_Etat: now also D177.1 (K)
- net Court_T_Actif_Right: now also D177.2 (A)

Commit message: Add files via upload
Parts:
- removed D177: 1N4148, PCM_Diode_THT_AKL:D_DO-35_SOD27_P7.62mm_Horizontal, symbol PCM_Diode_AKL:1N4148
