File: Trailer_Backup.kicad_sch (KiCad schematic)
At the start: 16 parts, among them Q27 IRLZ44N, U7 LM339

Commit message: Add files via upload
Parts:
- removed OC5, OC6: PC817, PCM_Package_DIP_AKL:DIP-4_W7.62mm_LongPads, symbol PCM_Optocoupler_AKL:PC817
- removed Q27: IRLZ44N, PCM_Package_TO_SOT_THT_AKL:TO-220-3_Vertical_GDS, symbol PCM_Transistor_MOSFET_AKL:IRLZ44N
- removed R100, R98, R99: Potentiometer, symbol Simulation_SPICE:Potentiometer
- removed R89: 3 Ohm - 5W, Resistor_THT:R_Axial_Power_L25.0mm_W9.0mm_P27.94mm, symbol PCM_SL_Devices:Resistor_5W
- removed R90: .05R Shunt, Resistor_THT:R_Axial_Power_L25.0mm_W9.0mm_P27.94mm, symbol PCM_SL_Devices:Resistor_5W
- removed R91, R92, R93: 4.7k, Resistor_THT:R_Axial_DIN0207_L6.3mm_D2.5mm_P10.16mm_Horizontal, symbol PCM_SL_Resistors:4.7k
- removed R94, R95: 1k, Resistor_THT:R_Axial_DIN0207_L6.3mm_D2.5mm_P10.16mm_Horizontal, symbol PCM_SL_Resistors:4.7k
- removed R96: 100k, Resistor_THT:R_Axial_DIN0207_L6.3mm_D2.5mm_P10.16mm_Horizontal, symbol PCM_SL_Resistors:100k
- removed R97: 10k, Resistor_THT:R_Axial_DIN0207_L6.3mm_D2.5mm_P10.16mm_Horizontal, symbol PCM_SL_Resistors:10k
- removed U7: LM339, symbol Comparator:LM339
- added D98: SMBJ33A, PCM_Diode_SMD_AKL:D_SMB, symbol PCM_Diode_TVS_AKL:SMBJ33A
- added F5: Polyfuse, symbol Device:Polyfuse
- added Q36: IRLZ44N, PCM_Package_TO_SOT_THT_AKL:TO-220-3_Vertical_GDS, symbol PCM_Transistor_MOSFET_AKL:IRLZ44N
- added R134: 10k, Resistor_THT:R_Axial_DIN0207_L6.3mm_D2.5mm_P10.16mm_Horizontal, symbol PCM_SL_Resistors:10k
- added R135: .1 ohm, Resistor_THT:R_Axial_DIN0207_L6.3mm_D2.5mm_P10.16mm_Horizontal, symbol PCM_SL_Resistors:4.7k
- added R136, R137: Potentiometer, symbol Simulation_SPICE:Potentiometer
- added R138, R139: 4.7k, Resistor_THT:R_Axial_DIN0207_L6.3mm_D2.5mm_P10.16mm_Horizontal, symbol PCM_SL_Resistors:4.7k
- added SW6: SW_SPST, symbol Switch:SW_SPST
- added U10: LM339, symbol Comparator:LM339
Connections:
- net GND: now also D98.2 (A), R134.2, R136.3, R137.3, U10.12 (V-), U10.5 (+), U10.9 (+)
- net V_Ref: now also R136.1, R137.1, R138.2, R139.2, SW6.1 (A), U10.3 (V+), U10.4 (-), U10.8 (-)
- new net: R136.2, U10.7 (+)
- new net: R137.2, U10.11 (+)
- new net Backup_Trailer_Shunt_Haut: Q36.3 (S), R135.2, U10.10 (-), U10.6 (-)
- new net Btn_Backup_Etat: Q36.1 (G), R134.1, SW6.2 (B)
- new net Court_Backup_Trailer: R139.1, U10.13
- new net Ouvert_Backup_Trailer: R138.1, U10.1
- new net Q36.2_Drain: F5.2, Q36.2 (D)
- new net Trail_Backup: D98.1 (K), R135.1
- new net V_Arm_Trailer: F5.1
- no-connect marks 1 -> 2
Other:
- note removed: "Court-circuit"
- note removed: "Injection"
- note removed: "Non_Utilisé"
- note removed: "Ouvvert"
- note removed: "Right_Vehic_Shunt_Haut"

Commit message: Add files via upload
Parts:
- R135: footprint Resistor_THT:R_Axial_DIN0207_L6.3mm_D2.5mm_P10.16mm_Horizontal -> PCM_SL_Devices:Resistor_5W
Changed lines of the file:
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@@
 			)
 		)
-		(property "Footprint" "Resistor_THT:R_Axial_DIN0207_L6.3mm_D2.5mm_P10.16mm_Horizontal"
+		(property "Footprint" "PCM_SL_Devices:Resistor_5W"
 			(at 94.869 65.278 0)
 			(hide yes)

Commit message: Add files via upload
Parts:
- R135: footprint PCM_SL_Devices:Resistor_5W -> Resistor_THT:R_Axial_Power_L25.0mm_W9.0mm_P27.94mm
Changed lines of the file:
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@@
 			)
 		)
-		(property "Footprint" "PCM_SL_Devices:Resistor_5W"
+		(property "Footprint" "Resistor_THT:R_Axial_Power_L25.0mm_W9.0mm_P27.94mm"
 			(at 94.869 65.278 0)
 			(hide yes)

Commit message: Add files via upload
Parts:
- R136, R137: footprint (none) -> TRIM_3296W1103LF:TRIM_3296W1103LF
Changed lines of the file:
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@@
 			)
 		)
-		(property "Footprint" ""
+		(property "Footprint" "TRIM_3296W1103LF:TRIM_3296W1103LF"
 			(at 100.33 50.8 0)
 			(hide yes)
@@
 			)
 		)
-		(property "Footprint" ""
+		(property "Footprint" "TRIM_3296W1103LF:TRIM_3296W1103LF"
 			(at 111.76 72.39 0)
 			(hide yes)

Commit message: Add files via upload
Parts:
- R135: footprint Resistor_THT:R_Axial_Power_L25.0mm_W9.0mm_P27.94mm -> Resistor_THT:R_Axial_DIN0207_L6.3mm_D2.5mm_P10.16mm_Horizontal
- R136, R137: footprint TRIM_3296W1103LF:TRIM_3296W1103LF -> (none)
Changed lines of the file:
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@@
 			)
 		)
-		(property "Footprint" "Resistor_THT:R_Axial_Power_L25.0mm_W9.0mm_P27.94mm"
+		(property "Footprint" "Resistor_THT:R_Axial_DIN0207_L6.3mm_D2.5mm_P10.16mm_Horizontal"
 			(at 94.869 65.278 0)
 			(hide yes)
@@
 			)
 		)
-		(property "Footprint" "TRIM_3296W1103LF:TRIM_3296W1103LF"
+		(property "Footprint" ""
 			(at 100.33 50.8 0)
 			(hide yes)
@@
 			)
 		)
-		(property "Footprint" "TRIM_3296W1103LF:TRIM_3296W1103LF"
+		(property "Footprint" ""
 			(at 111.76 72.39 0)
 			(hide yes)

Commit message: Add files via upload
Parts:
- R135: footprint Resistor_THT:R_Axial_DIN0207_L6.3mm_D2.5mm_P10.16mm_Horizontal -> Resistor_THT:R_Axial_Power_L25.0mm_W9.0mm_P27.94mm
- R136, R137: footprint (none) -> TRIM_3296W1103LF:TRIM_3296W1103LF
Changed lines of the file:
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@@
 			)
 		)
-		(property "Footprint" "Resistor_THT:R_Axial_DIN0207_L6.3mm_D2.5mm_P10.16mm_Horizontal"
+		(property "Footprint" "Resistor_THT:R_Axial_Power_L25.0mm_W9.0mm_P27.94mm"
 			(at 94.869 65.278 0)
 			(hide yes)
@@
 			)
 		)
-		(property "Footprint" ""
+		(property "Footprint" "TRIM_3296W1103LF:TRIM_3296W1103LF"
 			(at 100.33 50.8 0)
 			(hide yes)
@@
 			)
 		)
-		(property "Footprint" ""
+		(property "Footprint" "TRIM_3296W1103LF:TRIM_3296W1103LF"
 			(at 111.76 72.39 0)
 			(hide yes)

Commit message: Add files via upload
Parts:
- removed Q36: IRLZ44N, PCM_Package_TO_SOT_THT_AKL:TO-220-3_Vertical_GDS, symbol PCM_Transistor_MOSFET_AKL:IRLZ44N
- removed R134: 10k, Resistor_THT:R_Axial_DIN0207_L6.3mm_D2.5mm_P10.16mm_Horizontal, symbol PCM_SL_Resistors:10k
- removed R135: .1 ohm, Resistor_THT:R_Axial_Power_L25.0mm_W9.0mm_P27.94mm, symbol PCM_SL_Resistors:4.7k
- added D178: MUR1520G, Package_TO_SOT_THT:TO-220-2_Vertical, symbol Device:D
- added DZ6: 1N5242B, PCM_Diode_THT_AKL:D_DO-35_SOD27_P7.62mm_Horizontal_Zener, symbol PCM_Diode_Zener_AKL:1N5242B
- added Q36: IRF4905PBF, Package_TO_SOT_THT:TO-220-3_Vertical, symbol Transistor_FET:IRF4905
- added Q77: 2N7000, PCM_Package_TO_SOT_THT_AKL:TO-92_Inline_Wide_SGD, symbol PCM_Transistor_MOSFET_AKL:2N7000
- added Q78: 2N3906, PCM_Package_TO_SOT_THT_AKL:TO-92_Inline_Wide_EBC, symbol PCM_Transistor_BJT_AKL:2N3906
- added R134: 10k, Resistor_THT:R_Axial_DIN0207_L6.3mm_D2.5mm_P10.16mm_Horizontal, symbol PCM_SL_Resistors:4.7k
- added R135: 12 Ohm - 1W, Resistor_THT:R_Axial_DIN0414_L11.9mm_D4.5mm_P15.24mm_Horizontal, symbol PCM_SL_Devices:Resistor_5W
- added R281, R283: 1k, Resistor_THT:R_Axial_DIN0207_L6.3mm_D2.5mm_P10.16mm_Horizontal, symbol PCM_SL_Resistors:1k
- added R282, R284, R287: 10k, Resistor_THT:R_Axial_DIN0207_L6.3mm_D2.5mm_P10.16mm_Horizontal, symbol PCM_SL_Resistors:10k
- added R285: 2.7k, Resistor_THT:R_Axial_DIN0207_L6.3mm_D2.5mm_P10.16mm_Horizontal, symbol PCM_SL_Resistors:2.7k
- added R286: 39kΩ, Resistor_THT:R_Axial_DIN0207_L6.3mm_D2.5mm_P10.16mm_Horizontal, symbol PCM_SL_Resistors:10k
- R136: Etiquette Pot_Backup_Ouvert -> (none)
- R137: Etiquette Pot2_Backup_Court -> (none)
Connections:
- net Btn_Backup_Etat: now also Q77.2 (G), R134.2
- net GND: now also R137.1, Q77.1 (S), R134.1, R285.2, R287.2; no longer R137.3
- net Trail_Backup: now also D178.1 (K), R135.2, R283.1, R286.2
- net V_Ref: now also R137.3; no longer R137.1
- net Backup_Trailer_Shunt_Haut renamed Court_Sense_Backup
- net Court_Sense_Backup: now also R286.1, R287.1; no longer U10.6 (-)
- net Q36.2_Drain: no longer names the net of F5.2
- net Q36.2_Drain: now also DZ6.1 (K), Q36.3 (S), R282.2
- new net: DZ6.2 (A), Q36.1 (G), R281.2, R282.1
- new net: D178.2 (A), Q36.2 (D), Q78.1 (E), R135.1
- new net: Q77.3 (D), R281.1
- new net: Q78.2 (B), R283.2
- new net: Q78.3 (C), R284.1
- new net I_Present_Backup: R284.2, R285.1, U10.6 (-)

Commit message: Add files via upload
Parts:
- D98: value SMBJ33A -> P6KE39A; footprint PCM_Diode_SMD_AKL:D_SMB -> PCM_Diode_THT_AKL:D_DO-15_P10.16mm_Horizontal_Zener; symbol PCM_Diode_TVS_AKL:SMBJ33A -> PCM_Diode_TVS_AKL:P6KE39A
Changed lines of the file:
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@@
 	)
 	(symbol
-		(lib_id "PCM_Diode_TVS_AKL:SMBJ33A")
+		(lib_id "PCM_Diode_TVS_AKL:P6KE39A")
 		(at 199.39 109.22 0)
 		(unit 1)
@@
 			)
 		)
-		(property "Value" "SMBJ33A"
+		(property "Value" "P6KE39A"
 			(at 199.39 105.41 0)
 			(show_name no)
@@
 			)
 		)
-		(property "Footprint" "PCM_Diode_SMD_AKL:D_SMB"
+		(property "Footprint" "PCM_Diode_THT_AKL:D_DO-15_P10.16mm_Horizontal_Zener"
 			(at 199.39 109.22 0)
 			(hide yes)
@@
 			)
 		)
-		(property "Datasheet" "https://www.tme.eu/Document/0b6222bec7e12d83185b51d73cb6a54d/SMBJ_ser.pdf"
+		(property "Datasheet" "https://www.tme.eu/Document/6b488a936123e1f9ccf03f4f9186b150/P6KE_ser.pdf"
 			(at 199.39 109.22 0)
 			(hide yes)
@@
 			)
 		)
-		(property "Description" "SMB Unidirectional TVS diode, 33V, 600W, Alternate KiCAD Library"
+		(property "Description" "DO-15 Unidirectional TVS diode, 39V, 600W, Alternate KiCAD Library"
 			(at 199.39 109.22 0)
 			(hide yes)
