File: Trailer_Backup.kicad_sch (KiCad schematic)
At the start: 22 parts, among them Q36 IRF4905PBF, Q77 2N7000, Q78 2N3906, SW6 SW_SPST, U10 LM339

Commit message: Add files via upload
Parts:
- F5: value Polyfuse -> MF-R700
- U10: footprint (none) -> Package_DIP:DIP-14_W7.62mm_Socket
Changed lines of the file:
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@@
 			)
 		)
-		(property "Footprint" ""
+		(property "Footprint" "Package_DIP:DIP-14_W7.62mm_Socket"
 			(at 233.68 62.23 0)
 			(hide yes)
@@
 			)
 		)
-		(property "Footprint" ""
+		(property "Footprint" "Package_DIP:DIP-14_W7.62mm_Socket"
 			(at 233.68 40.64 0)
 			(hide yes)
@@
 			)
 		)
-		(property "Footprint" ""
+		(property "Footprint" "Package_DIP:DIP-14_W7.62mm_Socket"
 			(at 234.95 104.14 0)
 			(hide yes)
@@
 			)
 		)
-		(property "Footprint" ""
+		(property "Footprint" "Package_DIP:DIP-14_W7.62mm_Socket"
 			(at 233.68 83.82 0)
 			(hide yes)
@@
 			)
 		)
-		(property "Value" "Polyfuse"
+		(property "Value" "MF-R700"
 			(at 115.57 74.93 90)
 			(show_name no)
@@
 			)
 		)
-		(property "Footprint" ""
+		(property "Footprint" "Package_DIP:DIP-14_W7.62mm_Socket"
 			(at 236.22 128.27 0)
 			(hide yes)

Commit message: Add files via upload
Parts:
- F5: footprint (none) -> PTC_Bourns_MF-R:PTC_Bourns_MF-R_P10.20mm_W24.2mm
Changed lines of the file:
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@@
 			)
 		)
-		(property "Footprint" ""
+		(property "Footprint" "PTC_Bourns_MF-R:PTC_Bourns_MF-R_P10.20mm_W24.2mm"
 			(at 110.49 77.47 0)
 			(hide yes)

Commit message: Add files via upload
Parts:
- SW6: value SW_SPST -> SW_SPDT; symbol Switch:SW_SPST -> Switch:SW_SPDT
Other:
- moved on the sheet: R134
Changed lines of the file:
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@@
 	)
 	(junction
-		(at 97.79 73.66)
+		(at 68.58 76.2)
 		(diameter 0)
 		(color 0 0 0 0)
 	)
 	(junction
-		(at 245.11 64.77)
+		(at 97.79 73.66)
 		(diameter 0)
 		(color 0 0 0 0)
 	)
 	(junction
-		(at 68.58 76.2)
+		(at 245.11 64.77)
 		(diameter 0)
 		(color 0 0 0 0)
@@
 	(wire
 		(pts
-			(xy 52.07 63.5) (xy 55.88 63.5)
+			(xy 52.07 60.96) (xy 55.88 60.96)
 		)
 		(stroke
@@
 	(wire
 		(pts
-			(xy 57.15 76.2) (xy 68.58 76.2)
+			(xy 62.23 76.2) (xy 68.58 76.2)
 		)
 		(stroke
@@
 	(wire
 		(pts
+			(xy 54.61 76.2) (xy 52.07 76.2)
+		)
+		(stroke
+			(width 0)
+			(type default)
+		)
+	)
+	(wire
+		(pts
 			(xy 224.79 80.01) (xy 224.79 83.82)
 		)
@@
 	(global_label "V_Ref"
 		(shape input)
-		(at 52.07 63.5 180)
+		(at 52.07 60.96 180)
 		(fields_autoplaced yes)
 		(effects
@@
 		)
 		(property "Intersheetrefs" "${INTERSHEET_REFS}"
-			(at 43.9443 63.5 0)
+			(at 43.9443 60.96 0)
 			(hide yes)
 			(show_name no)
@@
 	(global_label "GND"
 		(shape input)
-		(at 49.53 76.2 180)
+		(at 52.07 76.2 180)
 		(fields_autoplaced yes)
 		(effects
@@
 		)
 		(property "Intersheetrefs" "${INTERSHEET_REFS}"
-			(at 42.6743 76.2 0)
+			(at 45.2143 76.2 0)
 			(hide yes)
 			(show_name no)
@@
 	)
 	(symbol
-		(lib_id "Switch:SW_SPST")
+		(lib_id "Switch:SW_SPDT")
 		(at 60.96 63.5 0)
+		(mirror y)
 		(unit 1)
 		(body_style 1)
@@
 		(in_pos_files yes)
 		(dnp no)
-		(fields_autoplaced yes)
 		(property "Reference" "SW6"
-			(at 60.96 57.15 0)
+			(at 60.96 56.388 0)
 			(show_name no)
 			(do_not_autoplace no)
@@
 			)
 		)
-		(property "Value" "SW_SPST"
-			(at 60.96 59.69 0)
+		(property "Value" "SW_SPDT"
+			(at 60.96 58.42 0)
 			(show_name no)
 			(do_not_autoplace no)
@@
 			)
 		)
-		(property "Description" "Single Pole Single Throw (SPST) switch"
+		(property "Description" "Switch, single pole double throw"
 			(at 60.96 63.5 0)
 			(hide yes)
@@
 		(pin "2"
 		)
+		(pin "3"
+		)
 		(instances
 			(project "TrailerDiagnosticSystem"
@@
 	(symbol
 		(lib_id "PCM_SL_Resistors:4.7k")
-		(at 53.34 76.2 0)
+		(at 58.42 76.2 0)
 		(unit 1)
 		(body_style 1)
@@
 		(fields_autoplaced yes)
 		(property "Reference" "R134"
-			(at 53.34 69.85 0)
+			(at 58.42 69.85 0)
 			(show_name no)
 			(do_not_autoplace no)
@@
 		)
 		(property "Value" "10k"
-			(at 53.34 72.39 0)
+			(at 58.42 72.39 0)
 			(show_name no)
 			(do_not_autoplace no)
@@
 		)
 		(property "Footprint" "Resistor_THT:R_Axial_DIN0207_L6.3mm_D2.5mm_P10.16mm_Horizontal"
-			(at 54.229 80.518 0)
+			(at 59.309 80.518 0)
 			(hide yes)
 			(show_name no)
@@
 		)
 		(property "Datasheet" ""
-			(at 53.848 76.2 0)
+			(at 58.928 76.2 0)
 			(hide yes)
 			(show_name no)
@@
 		)
 		(property "Description" "10kΩ, 1/4W Resistor"
-			(at 53.34 76.2 0)
+			(at 58.42 76.2 0)
 			(hide yes)
 			(show_name no)

Commit message: Add files via upload
Connections:
- net GND: now also SW6.3 (C)
Changed lines of the file:
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@@
+	(wire
+		(pts
+			(xy 52.07 66.04) (xy 55.88 66.04)
+		)
+		(stroke
+			(width 0)
+			(type default)
+		)
+	)
 	(wire
 		(pts
@@
 			)
 		)
+	)
+	(global_label "GND"
+		(shape input)
+		(at 52.07 66.04 180)
+		(fields_autoplaced yes)
+		(effects
+			(font
+				(size 1.27 1.27)
+			)
+			(justify right)
+		)
+		(property "Intersheetrefs" "${INTERSHEET_REFS}"
+			(at 45.2143 66.04 0)
+			(hide yes)
+			(show_name no)
+			(do_not_autoplace no)
+			(effects
+				(font
+					(size 1.27 1.27)
+				)
+				(justify right)
+			)
+		)

Commit message: Add files via upload
Parts:
- R134, R282, R284, R287: value 10k -> 10kΩ
- R138, R139: value 4.7k -> 4.7kΩ
- R281, R283: value 1k -> 1kΩ
- R285: value 2.7k -> 2.7kΩ
Changed lines of the file:
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@@
 			)
 		)
-		(property "Value" "10k"
+		(property "Value" "10kΩ"
 			(at 102.87 71.12 0)
 			(show_name no)
@@
 			)
 		)
-		(property "Value" "4.7k"
+		(property "Value" "4.7kΩ"
 			(at 250.19 82.55 0)
 			(show_name no)
@@
 			)
 		)
-		(property "Value" "1k"
+		(property "Value" "1kΩ"
 			(at 163.83 78.74 0)
 			(show_name no)
@@
 			)
 		)
-		(property "Value" "1k"
+		(property "Value" "1kΩ"
 			(at 91.44 59.69 0)
 			(show_name no)
@@
 			)
 		)
-		(property "Value" "2.7k"
+		(property "Value" "2.7kΩ"
 			(at 135.89 90.17 0)
 			(show_name no)
@@
 			)
 		)
-		(property "Value" "10k"
+		(property "Value" "10kΩ"
 			(at 182.88 88.9 0)
 			(show_name no)
@@
 			)
 		)
-		(property "Value" "4.7k"
+		(property "Value" "4.7kΩ"
 			(at 250.19 60.96 0)
 			(show_name no)
@@
 			)
 		)
-		(property "Value" "10k"
+		(property "Value" "10kΩ"
 			(at 152.4 40.64 0)
 			(show_name no)
@@
 			)
 		)
-		(property "Value" "10k"
+		(property "Value" "10kΩ"
 			(at 58.42 72.39 0)
 			(show_name no)

Commit message: Add files via upload
Connections:
- net Btn_Backup_Etat renamed Fac_Btn_Backup
Changed lines of the file:
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@@
+	)
+	(junction
+		(at 68.58 63.5)
+		(diameter 0)
+		(color 0 0 0 0)
 	)
 	(junction
@@
 	(wire
 		(pts
+			(xy 71.12 59.69) (xy 68.58 59.69)
+		)
+		(stroke
+			(width 0)
+			(type default)
+		)
+	)
+	(wire
+		(pts
 			(xy 77.47 73.66) (xy 77.47 76.2)
 		)
@@
 		(pts
 			(xy 217.17 85.09) (xy 220.98 85.09)
+		)
+		(stroke
+			(width 0)
+			(type default)
+		)
+	)
+	(wire
+		(pts
+			(xy 68.58 59.69) (xy 68.58 63.5)
 		)
 		(stroke
@@
 			)
 		)
+	)
+	(global_label "Fac_Btn_Backup"
+		(shape input)
+		(at 71.12 59.69 0)
+		(fields_autoplaced yes)
+		(effects
+			(font
+				(size 1.27 1.27)
+			)
+			(justify left)
+		)
+		(property "Intersheetrefs" "${INTERSHEET_REFS}"
+			(at 89.345 59.69 0)
+			(hide yes)
+			(show_name no)
+			(do_not_autoplace no)
+			(effects
+				(font
+					(size 1.27 1.27)
+				)
+				(justify left)
+			)
+		)
