File: MassDetection.kicad_sch (KiCad schematic)
At the start: 8 parts, among them U15 LM339

Commit message: Add files via upload
Parts:
- U15: footprint Package_DIP:DIP-14_W7.62mm_Socket -> (none)
Changed lines of the file:
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@@
 			)
 		)
-		(property "Footprint" "Package_DIP:DIP-14_W7.62mm_Socket"
+		(property "Footprint" ""
 			(at 59.69 93.98 0)
 			(hide yes)
@@
 			)
 		)
-		(property "Footprint" "Package_DIP:DIP-14_W7.62mm_Socket"
+		(property "Footprint" ""
 			(at 55.88 130.81 0)
 			(hide yes)
@@
 			)
 		)
-		(property "Footprint" "Package_DIP:DIP-14_W7.62mm_Socket"
+		(property "Footprint" ""
 			(at 59.69 111.76 0)
 			(hide yes)
@@
 			)
 		)
-		(property "Footprint" "Package_DIP:DIP-14_W7.62mm_Socket"
+		(property "Footprint" ""
 			(at 59.69 57.15 0)
 			(hide yes)
@@
 			)
 		)
-		(property "Footprint" "Package_DIP:DIP-14_W7.62mm_Socket"
+		(property "Footprint" ""
 			(at 59.69 76.2 0)
 			(hide yes)

Commit message: Add files via upload
Parts:
- removed D149, D150: 1N4148, PCM_Diode_THT_AKL:D_DO-35_SOD27_P7.62mm_Horizontal, symbol PCM_Diode_AKL:1N4148
- removed D151: LED_2x5mm_Horizontal_Red, PCM_LED_THT_AKL:LED_Rectangular_W5.0mm_H2.0mm_Horizontal_O3.81mm_Z1.0mm, symbol PCM_LED_AKL:LED_2x5mm_Horizontal_Red
- removed R211: 330Ω, Resistor_THT:R_Axial_DIN0207_L6.3mm_D2.5mm_P10.16mm_Horizontal, symbol PCM_SL_Resistors:330ohm
- added C12: SR205E104MARAP1, SR205E104MARAP1:CAPRR254W50L508T317H508, symbol SR205E104MARAP1:SR205E104MARAP1
- added R211, R301, R302: 10k, Resistor_THT:R_Axial_DIN0207_L6.3mm_D2.5mm_P10.16mm_Horizontal, symbol PCM_SL_Resistors:10k
- added R303, R307: 330k, Resistor_THT:R_Axial_DIN0207_L6.3mm_D2.5mm_P10.16mm_Horizontal, symbol PCM_SL_Resistors:330k
- added R304: 62k, Resistor_THT:R_Axial_DIN0207_L6.3mm_D2.5mm_P10.16mm_Horizontal, symbol PCM_SL_Resistors:62k
- added R305, R306: 82k, Resistor_THT:R_Axial_DIN0207_L6.3mm_D2.5mm_P10.16mm_Horizontal, symbol PCM_SL_Resistors:82k
- U15: footprint (none) -> Package_DIP:DIP-14_W7.62mm_Socket
Connections:
- net GND: now also R208.2, R209.2, C12.2, R211.2, R306.2; no longer R208.1, R210.1, U15.7 (+), U15.9 (+)
- net Masse_Fault: now also U15.14, R302.2; no longer U15.2
- net Masse_Sense: now also R209.1, R210.2, R210.3, U15.4 (-), C12.1, R303.2, R304.2, R305.2, R307.2; no longer R208.2
- net V_Ref: now also R301.1, R302.1, R304.1, R305.1; no longer R209.1, U15.6 (-), U15.8 (-)
- removed net Seuil_Masse: R209.2, R210.2, R210.3, U15.4 (-)
- new net Fenetre_Ok: R301.2, U15.2, U15.8 (-)
- new net Pince_Trail: R211.1, R307.1
- new net Pince_Veh: R208.1, R303.1
- new net Seuil_Bas: R210.1, R306.1, U15.9 (+)
- no-connect marks 3 -> 1
Other:
- moved on the sheet: R208, R210, U15A, U15B, U15C, U15D, U15E
