File: MassDetection.kicad_sch (KiCad schematic)
At the start: 13 parts, among them U15 LM339

Commit message: Add files via upload
Parts:
- R211, R301, R302: value 10k -> 10kΩ
- R303, R307: value 330k -> 330kΩ
- R304: value 62k -> 62kΩ
- R305, R306: value 82k -> 82kΩ
Changed lines of the file:
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@@
 			)
 		)
-		(property "Value" "82k"
+		(property "Value" "82kΩ"
 			(at 163.83 96.52 0)
 			(show_name no)
@@
 			)
 		)
-		(property "Value" "10k"
+		(property "Value" "10kΩ"
 			(at 163.83 135.89 0)
 			(show_name no)
@@
 			)
 		)
-		(property "Value" "10k"
+		(property "Value" "10kΩ"
 			(at 163.83 121.92 0)
 			(show_name no)
@@
 			)
 		)
-		(property "Value" "10k"
+		(property "Value" "10kΩ"
 			(at 163.83 48.26 0)
 			(show_name no)
@@
 			)
 		)
-		(property "Value" "62k"
+		(property "Value" "62kΩ"
 			(at 163.83 71.12 0)
 			(show_name no)
@@
 			)
 		)
-		(property "Value" "330k"
+		(property "Value" "330kΩ"
 			(at 163.83 58.42 0)
 			(show_name no)
@@
 			)
 		)
-		(property "Value" "82k"
+		(property "Value" "82kΩ"
 			(at 163.83 109.22 0)
 			(show_name no)
@@
 			)
 		)
-		(property "Value" "330k"
+		(property "Value" "330kΩ"
 			(at 163.83 35.56 0)
 			(show_name no)

Commit message: Add files via upload
Parts:
- R208: value 10KΩ -> 10kΩ
- R209: value 100KΩ -> 100kΩ
Changed lines of the file:
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@@
 			)
 		)
-		(property "Value" "100KΩ"
+		(property "Value" "100kΩ"
 			(at 163.83 83.82 0)
 			(show_name no)
@@
 			)
 		)
-		(property "Value" "10KΩ"
+		(property "Value" "10kΩ"
 			(at 163.83 22.86 0)
 			(show_name no)
