File: Limite_Pack_Int.kicad_sch (KiCad schematic)
At the start: 18 parts, among them Q79 2N3906, Q80 2N3904, Q81 2N7000, Q82 2N3906

Commit message: Add files via upload
Changed lines of the file:
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@@
+	)
+	(junction
+		(at 135.89 45.72)
+		(diameter 0)
+		(color 0 0 0 0)
 	)
 	(junction
@@
 	)
 	(junction
-		(at 135.89 45.72)
-		(diameter 0)
-		(color 0 0 0 0)
-	)
-	(junction
 		(at 172.72 57.15)
 		(diameter 0)
@@
 	(wire
 		(pts
-			(xy 135.89 41.91) (xy 135.89 45.72)
-		)
-		(stroke
-			(width 0)
-			(type default)
-		)
-	)
-	(wire
-		(pts
 			(xy 92.71 83.82) (xy 92.71 64.77)
 		)
@@
 	(wire
 		(pts
+			(xy 148.59 73.66) (xy 148.59 45.72)
+		)
+		(stroke
+			(width 0)
+			(type default)
+		)
+	)
+	(wire
+		(pts
 			(xy 135.89 64.77) (xy 135.89 62.23)
 		)
@@
 	(wire
 		(pts
-			(xy 133.35 41.91) (xy 135.89 41.91)
-		)
-		(stroke
-			(width 0)
-			(type default)
-		)
-	)
-	(wire
-		(pts
 			(xy 170.18 57.15) (xy 172.72 57.15)
 		)
@@
 	(wire
 		(pts
-			(xy 139.7 73.66) (xy 143.51 73.66)
+			(xy 139.7 73.66) (xy 148.59 73.66)
+		)
+		(stroke
+			(width 0)
+			(type default)
+		)
+	)
+	(wire
+		(pts
+			(xy 148.59 45.72) (xy 135.89 45.72)
 		)
 		(stroke
@@
 			(width 0)
 			(type default)
-		)
-	)
-	(label "Q82.1"
-		(at 143.51 73.66 0)
-		(effects
-			(font
-				(size 1.27 1.27)
-			)
-			(justify left bottom)
 		)
 	)
@@
 		(effects
 			(font
-				(size 1.27 1.27)
-			)
-			(justify right bottom)
-		)
-	)
-	(label "Q82.1"
-		(at 133.35 41.91 180)
-		(effects
-			(font

Commit message: Add files via upload
Parts:
- R290: value 1.5k -> 1.5kΩ
- R291: value 1k -> 1kΩ
- R292, R296, R297, R298: value 100k -> 100kΩ
- R293: value 18k -> 18kΩ
- R294: value 39k -> 39kΩ
- R299, R300: value 10k -> 10kΩ
Changed lines of the file:
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@@
 			)
 		)
-		(property "Value" "100k"
+		(property "Value" "100kΩ"
 			(at 135.89 69.85 0)
 			(show_name no)
@@
 			)
 		)
-		(property "Value" "18k"
+		(property "Value" "18kΩ"
 			(at 105.41 80.01 0)
 			(show_name no)
@@
 			)
 		)
-		(property "Value" "1k"
+		(property "Value" "1kΩ"
 			(at 105.41 21.59 0)
 			(show_name no)
@@
 			)
 		)
-		(property "Value" "100k"
+		(property "Value" "100kΩ"
 			(at 179.07 53.34 0)
 			(show_name no)
@@
 			)
 		)
-		(property "Value" "10k"
+		(property "Value" "10kΩ"
 			(at 166.37 53.34 0)
 			(show_name no)
@@
 			)
 		)
-		(property "Value" "1.5k"
+		(property "Value" "1.5kΩ"
 			(at 63.5 27.94 0)
 			(show_name no)
@@
 			)
 		)
-		(property "Value" "39k"
+		(property "Value" "39kΩ"
 			(at 105.41 91.44 0)
 			(show_name no)
@@
 			)
 		)
-		(property "Value" "100k"
+		(property "Value" "100kΩ"
 			(at 81.28 60.96 0)
 			(show_name no)
@@
 			)
 		)
-		(property "Value" "100k"
+		(property "Value" "100kΩ"
 			(at 66.04 49.53 0)
 			(show_name no)
@@
 			)
 		)
-		(property "Value" "10k"
+		(property "Value" "10kΩ"
 			(at 119.38 53.34 0)
 			(show_name no)
