File: Bloc_Test_Backup.kicad_sch (KiCad schematic)
At the start: 44 parts, among them Q29 2N7000, Q30 2N7000, Q31 2N7000, Q32 2N7000, Q33 2N7000, Q34 2N7000

Commit message: Add files via upload
Parts:
- removed D75, D76, D77, D78, D79, D80, D81, D82, D83, D84, D85, D86, D87, D88, D89, D90, D91, D92, D93, D94, D95, D96: 1N4148, PCM_Diode_THT_AKL:D_DO-35_SOD27_P7.62mm_Horizontal, symbol PCM_Diode_AKL:1N4148
- removed D97: LED_ARGB, symbol Device:LED_ARGB
- removed Q29, Q30, Q31, Q32, Q33, Q34: 2N7000, Package_TO_SOT_THT:TO-92_Inline, symbol Transistor_FET:2N7000
- removed R107, R108, R109, R110, R111, R112, R113, R114, R115, R116, R117, R118: 4.7k, Resistor_THT:R_Axial_DIN0207_L6.3mm_D2.5mm_P10.16mm_Horizontal, symbol PCM_SL_Resistors:4.7k
- removed R119, R120, R121: 330ohm, Resistor_THT:R_Axial_DIN0207_L6.3mm_D2.5mm_P10.16mm_Horizontal, symbol PCM_SL_Resistors:330ohm
- added D100, D101, D102, D103, D104, D105, D106, D107, D108, D109, D110, D111, D112, D113, D114, D115, D116, D117, D118, D119, D120, D99: 1N4148, PCM_Diode_THT_AKL:D_DO-35_SOD27_P7.62mm_Horizontal, symbol PCM_Diode_AKL:1N4148
- added D121: LED_ARGB, symbol Device:LED_ARGB
- added Q37, Q38, Q39, Q40, Q41, Q42: 2N7000, Package_TO_SOT_THT:TO-92_Inline, symbol Transistor_FET:2N7000
- added R140, R141, R142, R143, R144, R145, R146, R147, R148, R149, R150, R151: 4.7k, Resistor_THT:R_Axial_DIN0207_L6.3mm_D2.5mm_P10.16mm_Horizontal, symbol PCM_SL_Resistors:4.7k
- added R152, R153, R154: 330ohm, Resistor_THT:R_Axial_DIN0207_L6.3mm_D2.5mm_P10.16mm_Horizontal, symbol PCM_SL_Resistors:330ohm
Connections:
- net GND: now also Q37.1 (S), Q38.1 (S), Q39.1 (S), Q40.1 (S), Q41.1 (S), Q42.1 (S), R141.1, R142.1, R144.2, R145.1, R148.1, R151.2
- net Mode_Trailer: now also D106.1 (K), D117.1 (K), D119.1 (K)
- net Mode_Vehicule: now also D100.1 (K), D113.1 (K)
- net V_Ref: now also D121.1 (A), R140.2, R143.2, R146.1, R147.2, R149.2, R150.1
- new net: Q42.3 (D), R154.1
- new net: Q40.3 (D), R152.1
- new net: D121.2 (RK), R152.2
- new net: Q41.3 (D), R153.1
- new net: D121.3 (GK), R153.2
- new net: D121.4 (BK), R154.2
- new net Bleu_Backup: D102.2 (A), D111.2 (A), D119.2 (A), D120.2 (A), R151.1
- new net Btn_Backup_Etat: D118.1 (K), Q39.2 (G)
- new net Court_Backup: D107.1 (K), D108.1 (K), D109.2 (A), D114.2 (A), Q37.2 (G), R145.2
- new net Court_Backup_Trailer: D105.1 (K)
- new net Court_Backup_Vehic: D99.1 (K)
- new net Court_T_Actif_Backup: D105.2 (A), D106.2 (A), D108.2 (A), R143.1
- new net Court_V_Actif_Backup: D100.2 (A), D107.2 (A), D99.2 (A), R140.1
- new net Fault_Actif_Backup: D109.1 (K), D110.1 (K), D111.1 (K), Q38.2 (G), R144.1
- new net Not_Btn_Backup: D120.1 (K), Q39.3 (D), R150.2
- new net Ouvert_Backup: D101.2 (A), D103.1 (K), D104.1 (K), D110.2 (A), D115.2 (A), R142.2
- new net Ouvert_Backup_Trailer: D116.1 (K)
- new net Ouvert_Backup_Vehic: D112.1 (K)
- new net Ouvert_Ou_Bleu_Backup: D101.1 (K), D102.1 (K), Q37.3 (D), Q42.2 (G), R141.2
- new net Ouvert_T_Actif_Backup: D104.2 (A), D116.2 (A), D117.2 (A), D118.2 (A), R149.1
- new net Ouvert_V_Actif_Backup: D103.2 (A), D112.2 (A), D113.2 (A), R147.1
- new net Rouge_Enable_Backup: D114.1 (K), D115.1 (K), Q40.2 (G), R148.2
- new net Vert_Enable_Backup: Q38.3 (D), Q41.2 (G), R146.2
Other:
- note added: "1ère Porte "ET" (Court_V_Actif_Backup)"
- note added: "1ère Porte "OU" (Ouvert_Backup)"
- note added: "2ième Porte "ET" (Court_T_Actif_Backup)"
- note added: "2ième Porte "OU" (Court_Backup)"
- note added: "3ième Porte "ET" (Ouvert_V_Actif_Backup)"
- note added: "4ième Porte "ET" (Ouvert_T_Actif_Backup)"
- note added: "5ième Porte "ET" (Bleu_Backup)"
- note added: "Inverseur (Dépendance de Bleu_Backup)"
- note added: "Porte OU Fault_Actif_Backup (3 entrées) + inverseur vert"
- note added: "Porte OU Ouvert_Ou_Bleu_Backup + override"
- note added: "Porte OU Rouge_Enable_Backup"
- note removed: "1ère Porte "ET" (Court_V_Actif_Right)"
- note removed: "1ère Porte "OU" (Ouvert_Right)"
- note removed: "2ième Porte "ET" (Court_T_Actif_Right)"
- note removed: "2ième Porte "OU" (Court_Right)"
- note removed: "3ième Porte "ET" (Ouvert_V_Actif_Right)"
- note removed: "4ième Porte "ET" (Ouvert_T_Actif_Right)"
- note removed: "5ième Porte "ET" (Bleu_Right)"
- note removed: "Inverseur (Dépendance de Bleu_Right)"
- note removed: "Porte OU Fault_Actif_Right (3 entrées) + inverseur vert"
- note removed: "Porte OU Ouvert_Ou_Bleu_Right + override"
- note removed: "Porte OU Rouge_Enable_Right"

Commit message: Add files via upload
Changed lines of the file:
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@@
 	)
 	(junction
-		(at 52.07 86.36)
+		(at 229.87 55.88)
+		(diameter 0)
+		(color 0 0 0 0)
+	)
+	(junction
+		(at 102.87 156.21)
+		(diameter 0)
+		(color 0 0 0 0)
+	)
+	(junction
+		(at 106.68 45.72)
+		(diameter 0)
+		(color 0 0 0 0)
+	)
+	(junction
+		(at 26.67 44.45)
+		(diameter 0)
+		(color 0 0 0 0)
+	)
+	(junction
+		(at 148.59 58.42)
+		(diameter 0)
+		(color 0 0 0 0)
+	)
+	(junction
+		(at 148.59 41.91)
+		(diameter 0)
+		(color 0 0 0 0)
+	)
+	(junction
+		(at 148.59 50.8)
+		(diameter 0)
+		(color 0 0 0 0)
+	)
+	(junction
+		(at 106.68 55.88)
+		(diameter 0)
+		(color 0 0 0 0)
+	)
+	(junction
+		(at 99.06 176.53)
+		(diameter 0)
+		(color 0 0 0 0)
+	)
+	(junction
+		(at 64.77 44.45)
+		(diameter 0)
+		(color 0 0 0 0)
+	)
+	(junction
+		(at 102.87 140.97)
+		(diameter 0)
+		(color 0 0 0 0)
+	)
+	(junction
+		(at 157.48 152.4)
 		(diameter 0)
 		(color 0 0 0 0)
@@
 	)
 	(junction
-		(at 229.87 55.88)
-		(diameter 0)
-		(color 0 0 0 0)
-	)
-	(junction
-		(at 102.87 156.21)
-		(diameter 0)
-		(color 0 0 0 0)
-	)
-	(junction
-		(at 106.68 45.72)
-		(diameter 0)
-		(color 0 0 0 0)
-	)
-	(junction
-		(at 26.67 44.45)
-		(diameter 0)
-		(color 0 0 0 0)
-	)
-	(junction
-		(at 148.59 58.42)
-		(diameter 0)
-		(color 0 0 0 0)
-	)
-	(junction
-		(at 148.59 41.91)
-		(diameter 0)
-		(color 0 0 0 0)
-	)
-	(junction
-		(at 148.59 50.8)
-		(diameter 0)
-		(color 0 0 0 0)
-	)
-	(junction
-		(at 106.68 55.88)
-		(diameter 0)
-		(color 0 0 0 0)
-	)
-	(junction
-		(at 99.06 176.53)
-		(diameter 0)
-		(color 0 0 0 0)
-	)
-	(junction
-		(at 64.77 44.45)
-		(diameter 0)
-		(color 0 0 0 0)
-	)
-	(junction
-		(at 102.87 140.97)
-		(diameter 0)
-		(color 0 0 0 0)
-	)
-	(junction
-		(at 157.48 152.4)
-		(diameter 0)
-		(color 0 0 0 0)
-	)
-	(junction
 		(at 49.53 151.13)
 		(diameter 0)
@@
 	)
 	(junction
-		(at 91.44 86.36)
-		(diameter 0)
-		(color 0 0 0 0)
-	)
-	(junction
 		(at 157.48 142.24)
 		(diameter 0)
@@
 	(wire
 		(pts
-			(xy 50.8 86.36) (xy 52.07 86.36)
-		)
-		(stroke
-			(width 0)
-			(type default)
-		)
-	)
-	(wire
-		(pts
 			(xy 156.21 33.02) (xy 161.29 33.02)
 		)
@@
 	(wire
 		(pts
+			(xy 55.88 86.36) (xy 55.88 97.79)
+		)
+		(stroke
+			(width 0)
+			(type default)
+		)
+	)
+	(wire
+		(pts
 			(xy 137.16 152.4) (xy 144.78 152.4)
 		)
@@
 	(wire
 		(pts
-			(xy 90.17 86.36) (xy 91.44 86.36)
-		)
-		(stroke
-			(width 0)
-			(type default)
-		)
-	)
-	(wire
-		(pts
 			(xy 95.25 77.47) (xy 91.44 77.47)
 		)
@@
 	(wire
 		(pts
-			(xy 55.88 86.36) (xy 52.07 86.36)
-		)
-		(stroke
-			(width 0)
-			(type default)
-		)
-	)
-	(wire
-		(pts
 			(xy 26.67 53.34) (xy 27.94 53.34)
 		)
@@
 	(wire
 		(pts
-			(xy 55.88 86.36) (xy 55.88 97.79)
-		)
-		(stroke
+			(xy 52.07 86.36) (xy 55.88 86.36)
+		)
+		(stroke

Commit message: Add files via upload
Parts:
- added D179: 1N4148, PCM_Diode_THT_AKL:D_DO-35_SOD27_P7.62mm_Horizontal, symbol PCM_Diode_AKL:1N4148
Connections:
- net Btn_Backup_Etat: now also D179.1 (K)
- net Court_T_Actif_Backup: now also D179.2 (A)
Changed lines of the file:
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@@
 	(wire
 		(pts
+			(xy 148.59 187.96) (xy 151.13 187.96)
+		)
+		(stroke
+			(width 0)
+			(type default)
+		)
+	)
+	(wire
+		(pts
 			(xy 71.12 97.79) (xy 83.82 97.79)
 		)
@@
 	(wire
 		(pts
+			(xy 140.97 187.96) (xy 138.43 187.96)
+		)
+		(stroke
+			(width 0)
+			(type default)
+		)
+	)
+	(wire
+		(pts
 			(xy 73.66 53.34) (xy 77.47 53.34)
 		)
@@
 		)
 	)
+	(label "Court_T_Actif_Backup"
+		(at 138.43 187.96 180)
+		(effects
+			(font
+				(size 1.27 1.27)
+			)
+			(justify right bottom)
+		)
+	)
 	(label "Ouvert_Backup"
 		(at 34.29 132.08 180)
@@
 		)
 	)
+	(hierarchical_label "Btn_Backup_Etat"
+		(shape input)
+		(at 151.13 187.96 0)
+		(effects
+			(font
+				(size 1.27 1.27)
+			)
+			(justify left)
+		)
+	)
 	(symbol
 		(lib_id "PCM_Diode_AKL:1N4148")
@@
 					(unit 1)
 				)
+			)
+		)
+	)
+	(symbol
+		(lib_id "PCM_Diode_AKL:1N4148")
+		(at 144.78 187.96 0)
+		(unit 1)
+		(body_style 1)
+		(exclude_from_sim no)
+		(in_bom yes)
+		(on_board yes)
+		(in_pos_files yes)
+		(dnp no)
+		(property "Reference" "D179"
+			(at 144.78 182.63 0)
+			(show_name no)
+			(do_not_autoplace no)
+			(effects
+				(font
+					(size 1.27 1.27)
+				)
+			)
+		)
+		(property "Value" "1N4148"
+			(at 144.78 184.91 0)
+			(show_name no)
+			(do_not_autoplace no)
+			(effects
+				(font
+					(size 1.27 1.27)
+				)
+			)
+		)
+		(property "Footprint" "PCM_Diode_THT_AKL:D_DO-35_SOD27_P7.62mm_Horizontal"
+			(at 144.78 187.96 0)
+			(hide yes)
+			(show_name no)
+			(do_not_autoplace no)
+			(effects
+				(font
+					(size 1.27 1.27)
+				)
+			)
+		)
+		(property "Datasheet" "https://datasheet.octopart.com/1N4148TR-ON-Semiconductor-datasheet-42765246.pdf"
+			(at 144.78 187.96 0)
+			(hide yes)
+			(show_name no)
+			(do_not_autoplace no)
+			(effects
+				(font
+					(size 1.27 1.27)
+				)
+			)
+		)
+		(property "Description" "DO-35 Diode, Small Signal, Fast Switching, 75V, 150mA, 4ns, Alternate KiCad Library"
+			(at 144.78 187.96 0)
+			(hide yes)
+			(show_name no)
+			(do_not_autoplace no)
+			(effects
+				(font
+					(size 1.27 1.27)
+				)
+			)
+		)
+		(pin "2"
+		)
+		(pin "1"
+		)
+		(instances
+			(project "TrailerDiagnosticSystem"
+				(path "/d4e407a7-3e32-4226-ae57-831ecdb3edf4/b4ff831c-304a-4222-b9bb-487c614afe45/3c1e0037-3393-4d0b-90ae-4005503ff1f2"
+					(reference "D179")
+					(unit 1)
+				)

Commit message: Add files via upload
Parts:
- R141, R144, R148: value 4.7k -> 470kΩ
- R142, R145: value 4.7k -> 100k
Connections:
- net GND: no longer R151.2
- net V_Ref: now also R151.2
Changed lines of the file:
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@@
 		)
 	)
-	(global_label "GND"
+	(global_label "V_Ref"
 		(shape input)
 		(at 242.57 55.88 0)
@@
 		)
 		(property "Intersheetrefs" "${INTERSHEET_REFS}"
-			(at 249.4257 55.88 0)
+			(at 250.6957 55.88 0)
 			(hide yes)
 			(show_name no)
@@
 			)
 		)
-		(property "Value" "4.7k"
+		(property "Value" "100k"
 			(at 87.63 95.25 0)
 			(show_name no)
@@
 			)
 		)
-		(property "Value" "4.7k"
+		(property "Value" "470kΩ"
 			(at 148.59 149.86 0)
 			(show_name no)
@@
 			)
 		)
-		(property "Value" "4.7k"
+		(property "Value" "470kΩ"
 			(at 40.64 148.59 0)
 			(show_name no)
@@
 			)
 		)
-		(property "Value" "4.7k"
+		(property "Value" "100k"
 			(at 48.26 95.25 0)
 			(show_name no)
@@
 			)
 		)
-		(property "Value" "4.7k"
+		(property "Value" "470kΩ"
 			(at 86.36 153.67 0)
 			(show_name no)

Commit message: Add files via upload
Parts:
- R140, R143, R146, R147, R149, R150, R151: value 4.7k -> 4.7kΩ
- R142, R145: value 100k -> 100kΩ
- R152, R153, R154: value 330ohm -> 330Ω
Changed lines of the file:
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@@
 			)
 		)
-		(property "Value" "100k"
+		(property "Value" "100kΩ"
 			(at 87.63 95.25 0)
 			(show_name no)
@@
 			)
 		)
-		(property "Value" "4.7k"
+		(property "Value" "4.7kΩ"
 			(at 31.75 50.8 0)
 			(show_name no)
@@
 			)
 		)
-		(property "Value" "4.7k"
+		(property "Value" "4.7kΩ"
 			(at 152.4 55.88 0)
 			(show_name no)
@@
 			)
 		)
-		(property "Value" "330ohm"
+		(property "Value" "330Ω"
 			(at 234.95 98.044 0)
 			(show_name no)
@@
 			)
 		)
-		(property "Value" "100k"
+		(property "Value" "100kΩ"
 			(at 48.26 95.25 0)
 			(show_name no)
@@
 			)
 		)
-		(property "Value" "330ohm"
+		(property "Value" "330Ω"
 			(at 234.95 119.634 0)
 			(show_name no)
@@
 			)
 		)
-		(property "Value" "4.7k"
+		(property "Value" "4.7kΩ"
 			(at 69.85 50.8 0)
 			(show_name no)
@@
 			)
 		)
-		(property "Value" "4.7k"
+		(property "Value" "4.7kΩ"
 			(at 95.25 173.99 0)
 			(show_name no)
@@
 			)
 		)
-		(property "Value" "4.7k"
+		(property "Value" "4.7kΩ"
 			(at 110.49 53.34 0)
 			(show_name no)
@@
 			)
 		)
-		(property "Value" "4.7k"
+		(property "Value" "4.7kΩ"
 			(at 205.74 40.64 0)
 			(show_name no)
@@
 			)
 		)
-		(property "Value" "4.7k"
+		(property "Value" "4.7kΩ"
 			(at 233.68 53.34 0)
 			(show_name no)
@@
 			)
 		)
-		(property "Value" "330ohm"
+		(property "Value" "330Ω"
 			(at 234.95 139.954 0)
 			(show_name no)

Commit message: Add files via upload
Connections:
- net Fac_Backup_R: now reaches D121.2 (RK), R152.2
- net Fac_Backup_G: now reaches D121.3 (GK), R153.2
- net Fac_Backup_B: now reaches D121.4 (BK), R154.2
Changed lines of the file:
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@@
+	)
+	(junction
+		(at 240.03 100.33)
+		(diameter 0)
+		(color 0 0 0 0)
 	)
 	(junction
@@
 	)
 	(junction
+		(at 240.03 121.92)
+		(diameter 0)
+		(color 0 0 0 0)
+	)
+	(junction
 		(at 229.87 55.88)
 		(diameter 0)
@@
 	)
 	(junction
+		(at 240.03 142.24)
+		(diameter 0)
+		(color 0 0 0 0)
+	)
+	(junction
 		(at 64.77 53.34)
 		(diameter 0)
@@
 	(wire
 		(pts
+			(xy 243.84 97.79) (xy 240.03 97.79)
+		)
+		(stroke
+			(width 0)
+			(type default)
+		)
+	)
+	(wire
+		(pts
 			(xy 156.21 58.42) (xy 161.29 58.42)
 		)
@@
 	(wire
 		(pts
+			(xy 240.03 97.79) (xy 240.03 100.33)
+		)
+		(stroke
+			(width 0)
+			(type default)
+		)
+	)
+	(wire
+		(pts
+			(xy 240.03 121.92) (xy 260.35 121.92)
+		)
+		(stroke
+			(width 0)
+			(type default)
+		)
+	)
+	(wire
+		(pts
 			(xy 34.29 104.14) (xy 55.88 104.14)
 		)
@@
 	(wire
 		(pts
+			(xy 243.84 139.7) (xy 240.03 139.7)
+		)
+		(stroke
+			(width 0)
+			(type default)
+		)
+	)
+	(wire
+		(pts
 			(xy 156.21 33.02) (xy 161.29 33.02)
 		)
@@
 	(wire
 		(pts
+			(xy 243.84 119.38) (xy 240.03 119.38)
+		)
+		(stroke
+			(width 0)
+			(type default)
+		)
+	)
+	(wire
+		(pts
 			(xy 35.56 53.34) (xy 39.37 53.34)
 		)
@@
 	(wire
 		(pts
-			(xy 257.81 119.38) (xy 257.81 142.24)
+			(xy 240.03 100.33) (xy 264.16 100.33)
+		)
+		(stroke
+			(width 0)
+			(type default)
+		)
+	)
+	(wire
+		(pts
+			(xy 261.62 119.38) (xy 261.62 142.24)
 		)
 		(stroke
@@
 	(wire
 		(pts
-			(xy 238.76 121.92) (xy 251.46 121.92)
+			(xy 238.76 121.92) (xy 240.03 121.92)
 		)
 		(stroke
@@
 	(wire
 		(pts
+			(xy 240.03 119.38) (xy 240.03 121.92)
+		)
+		(stroke
+			(width 0)
+			(type default)
+		)
+	)
+	(wire
+		(pts
 			(xy 72.39 34.29) (xy 76.2 34.29)
 		)
@@
 	(wire
 		(pts
-			(xy 251.46 114.3) (xy 251.46 121.92)
+			(xy 260.35 114.3) (xy 260.35 121.92)
 		)
 		(stroke
@@
 	(wire
 		(pts
-			(xy 238.76 100.33) (xy 264.16 100.33)
+			(xy 238.76 100.33) (xy 240.03 100.33)
 		)
 		(stroke
@@
 	(wire
 		(pts
-			(xy 251.46 114.3) (xy 264.16 114.3)
+			(xy 260.35 114.3) (xy 264.16 114.3)
 		)
 		(stroke
@@
 	(wire
 		(pts
+			(xy 240.03 139.7) (xy 240.03 142.24)
+		)
+		(stroke
+			(width 0)
+			(type default)
+		)
+	)
+	(wire
+		(pts
 			(xy 34.29 34.29) (xy 38.1 34.29)
 		)
@@
 	(wire
 		(pts
-			(xy 238.76 142.24) (xy 257.81 142.24)
+			(xy 238.76 142.24) (xy 240.03 142.24)
 		)
 		(stroke
@@
 	(wire
 		(pts
-			(xy 257.81 119.38) (xy 264.16 119.38)
+			(xy 261.62 119.38) (xy 264.16 119.38)
 		)
 		(stroke
@@
 		(pts
 			(xy 55.88 77.47) (xy 55.88 86.36)
+		)
+		(stroke
+			(width 0)
+			(type default)
+		)
+	)
+	(wire
+		(pts
+			(xy 240.03 142.24) (xy 261.62 142.24)
 		)
 		(stroke
@@
 		)
 	)
+	(global_label "Fac_Backup_B"
+		(shape input)
+		(at 243.84 139.7 0)
+		(fields_autoplaced yes)
+		(effects
+			(font
+				(size 1.27 1.27)
+			)
+			(justify left)
+		)
+		(property "Intersheetrefs" "${INTERSHEET_REFS}"
+			(at 260.1903 139.7 0)
+			(hide yes)
+			(show_name no)
+			(do_not_autoplace no)
+			(effects
+				(font
+					(size 1.27 1.27)
+				)
+				(justify left)
+			)
+		)
+	)
 	(global_label "GND"
 		(shape input)
@@
 		)
 	)
+	(global_label "Fac_Backup_G"
+		(shape input)
+		(at 243.84 119.38 0)
+		(fields_autoplaced yes)
+		(effects
+			(font
+				(size 1.27 1.27)
+			)
+			(justify left)
+		)
+		(property "Intersheetrefs" "${INTERSHEET_REFS}"
+			(at 260.1903 119.38 0)
+			(hide yes)
+			(show_name no)
+			(do_not_autoplace no)
+			(effects
+				(font
+					(size 1.27 1.27)
+				)
+				(justify left)
+			)
+		)
+	)
 	(global_label "GND"
 		(shape input)
@@
 			(hide yes)
 			(show_name no)
+			(do_not_autoplace no)
+			(effects
+				(font
+					(size 1.27 1.27)
+				)
+				(justify left)
+			)
+		)
+	)
+	(global_label "Fac_Backup_R"
+		(shape input)
+		(at 243.84 97.79 0)
+		(fields_autoplaced yes)
+		(effects
+			(font
+				(size 1.27 1.27)
+			)
+			(justify left)
+		)
+		(property "Intersheetrefs" "${INTERSHEET_REFS}"
+			(at 260.1903 97.79 0)
+			(hide yes)
+			(show_name no)
