File: Bloc_Test_Left.kicad_sch (KiCad schematic)
At the start: 0 parts

Commit message: Add files via upload
Parts:
- added D51, D52, D53, D54, D55, D56, D57, D58, D59, D60, D61, D62, D63, D64, D65, D66, D67, D68, D69, D70, D71, D72: 1N4148, PCM_Diode_THT_AKL:D_DO-35_SOD27_P7.62mm_Horizontal, symbol PCM_Diode_AKL:1N4148
- added D73: LED_ARGB, symbol Device:LED_ARGB
- added Q21, Q22, Q23, Q24, Q25, Q26: 2N7000, Package_TO_SOT_THT:TO-92_Inline, symbol Transistor_FET:2N7000
- added R74, R75, R76, R77, R78, R79, R80, R81, R82, R83, R84, R85: 4.7k, Resistor_THT:R_Axial_DIN0207_L6.3mm_D2.5mm_P10.16mm_Horizontal, symbol PCM_SL_Resistors:4.7k
- added R86, R87, R88: 330ohm, Resistor_THT:R_Axial_DIN0207_L6.3mm_D2.5mm_P10.16mm_Horizontal, symbol PCM_SL_Resistors:330ohm
Connections:
- net Btn_Left_Etat: now also D59.1 (K), Q21.2 (G)
- net Court_Left_Trailer: now also D53.1 (K)
- net Court_Left_Vehic: now also D51.1 (K)
- net Ouvert_Left_Trailer: now also D57.1 (K)
- net Ouvert_Left_Vehic: now also D55.1 (K)
- new net: Q24.3 (D), R86.1
- new net: Q26.3 (D), R88.1
- new net: D73.4 (BK), R88.2
- new net: D73.2 (RK), R86.2
- new net: Q25.3 (D), R87.1
- new net: D73.3 (GK), R87.2
- new net Bleu_Left: D64.2 (A), D65.2 (A), D67.2 (A), D70.2 (A), R81.1
- new net Court_Left: D62.1 (K), D63.1 (K), D68.2 (A), D71.2 (A), Q22.2 (G), R79.2
- new net Court_T_Actif_Left: D53.2 (A), D54.2 (A), D63.2 (A), R75.1
- new net Court_V_Actif_Left: D51.2 (A), D52.2 (A), D62.2 (A), R74.1
- new net Fault_Actif_Left: D68.1 (K), D69.1 (K), D70.1 (K), Q23.2 (G), R83.1
- new net GND: Q21.1 (S), Q22.1 (S), Q23.1 (S), Q24.1 (S), Q25.1 (S), Q26.1 (S), R78.1, R79.1, R81.2, R82.1, R83.2, R85.1
- new net Mode_Trailer: D54.1 (K), D58.1 (K), D64.1 (K)
- new net Mode_Vehicule: D52.1 (K), D56.1 (K)
- new net Not_Btn_Left: D65.1 (K), Q21.3 (D), R80.2
- new net Ouvert_Left: D60.1 (K), D61.1 (K), D66.2 (A), D69.2 (A), D72.2 (A), R78.2
- new net Ouvert_Ou_Bleu_Left: D66.1 (K), D67.1 (K), Q22.3 (D), Q26.2 (G), R82.2
- new net Ouvert_T_Actif_Left: D57.2 (A), D58.2 (A), D59.2 (A), D61.2 (A), R77.1
- new net Ouvert_V_Actif_Left: D55.2 (A), D56.2 (A), D60.2 (A), R76.1
- new net Rouge_Enable_Left: D71.1 (K), D72.1 (K), Q24.2 (G), R85.2
- new net V_Ref: D73.1 (A), R74.2, R75.2, R76.2, R77.2, R80.1, R84.1
- new net Vert_Enable_Left: Q23.3 (D), Q25.2 (G), R84.2
Other:
- note added: "1ère Porte "ET" (Court_V_Actif_Left)"
- note added: "1ère Porte "OU" (Ouvert_Left)"
- note added: "2ième Porte "ET" (Court_T_Actif_Left)"
- note added: "2ième Porte "OU" (Court_Left)"
- note added: "3ième Porte "ET" (Ouvert_V_Actif_Left)"
- note added: "4ième Porte "ET" (Ouvert_T_Actif_Left)"
- note added: "5ième Porte "ET" (Bleu_Left)"
- note added: "====================================== NIVEAU 3 =================="
- note added: "=========================================== NIVEAU 2 ================================================="
- note added: "========================================================================== NIVEAU 1 =========================================================================="
- note added: "Inverseur (Dépendance de Bleu_Left)"
- note added: "Porte OU Fault_Actif_Left (3 entrées) + inverseur vert"
- note added: "Porte OU Ouvert_Ou_Bleu_Left + override"
- note added: "Porte OU Rouge_Enable_Left"

Commit message: Add files via upload
Parts:
- added D175: 1N4148, PCM_Diode_THT_AKL:D_DO-35_SOD27_P7.62mm_Horizontal, symbol PCM_Diode_AKL:1N4148
Connections:
- net Btn_Left_Etat: now also D175.1 (K)
- net Court_T_Actif_Left: now also D175.2 (A)
Other:
- moved on the sheet: D65, R81, R84
Changed lines of the file:
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@@
 	)
 	(junction
+		(at 97.79 171.45)
+		(diameter 0)
+		(color 0 0 0 0)
+	)
+	(junction
 		(at 105.41 44.45)
 		(diameter 0)
@@
 	)
 	(junction
-		(at 97.79 175.26)
-		(diameter 0)
-		(color 0 0 0 0)
-	)
-	(junction
-		(at 228.6 44.45)
-		(diameter 0)
-		(color 0 0 0 0)
-	)
-	(junction
 		(at 48.26 139.7)
 		(diameter 0)
@@
 	)
 	(junction
-		(at 228.6 54.61)
-		(diameter 0)
-		(color 0 0 0 0)
-	)
-	(junction
 		(at 25.4 52.07)
 		(diameter 0)
@@
 	)
 	(junction
+		(at 228.6 54.61)
+		(diameter 0)
+		(color 0 0 0 0)
+	)
+	(junction
 		(at 63.5 43.18)
 		(diameter 0)
@@
 	)
 	(junction
+		(at 228.6 44.45)
+		(diameter 0)
+		(color 0 0 0 0)
+	)
+	(junction
 		(at 105.41 54.61)
 		(diameter 0)
@@
 	(wire
 		(pts
-			(xy 113.03 33.02) (xy 116.84 33.02)
+			(xy 97.79 166.37) (xy 101.6 166.37)
 		)
 		(stroke
@@
 	(wire
 		(pts
-			(xy 25.4 33.02) (xy 25.4 43.18)
+			(xy 97.79 166.37) (xy 97.79 171.45)
 		)
 		(stroke
@@
 	(wire
 		(pts
-			(xy 48.26 130.81) (xy 44.45 130.81)
+			(xy 113.03 33.02) (xy 116.84 33.02)
 		)
 		(stroke
@@
 	(wire
 		(pts
-			(xy 97.79 167.64) (xy 97.79 175.26)
+			(xy 25.4 33.02) (xy 25.4 43.18)
+		)
+		(stroke
+			(width 0)
+			(type default)
+		)
+	)
+	(wire
+		(pts
+			(xy 48.26 130.81) (xy 44.45 130.81)
 		)
 		(stroke
@@
 	(wire
 		(pts
-			(xy 236.22 44.45) (xy 241.3 44.45)
+			(xy 97.79 171.45) (xy 97.79 175.26)
+		)
+		(stroke
+			(width 0)
+			(type default)
+		)
+	)
+	(wire
+		(pts
+			(xy 240.03 44.45) (xy 241.3 44.45)
 		)
 		(stroke
@@
 	(wire
 		(pts
+			(xy 148.59 187.96) (xy 151.13 187.96)
+		)
+		(stroke
+			(width 0)
+			(type default)
+		)
+	)
+	(wire
+		(pts
 			(xy 82.55 139.7) (xy 88.9 139.7)
 		)
@@
 	(wire
 		(pts
+			(xy 232.41 44.45) (xy 228.6 44.45)
+		)
+		(stroke
+			(width 0)
+			(type default)
+		)
+	)
+	(wire
+		(pts
 			(xy 101.6 148.59) (xy 101.6 154.94)
 		)
@@
 	(wire
 		(pts
+			(xy 232.41 54.61) (xy 228.6 54.61)
+		)
+		(stroke
+			(width 0)
+			(type default)
+		)
+	)
+	(wire
+		(pts
 			(xy 29.21 96.52) (xy 43.18 96.52)
 		)
@@
 	(wire
 		(pts
-			(xy 236.22 54.61) (xy 241.3 54.61)
+			(xy 240.03 54.61) (xy 242.57 54.61)
 		)
 		(stroke
@@
 	(wire
 		(pts
+			(xy 140.97 187.96) (xy 138.43 187.96)
+		)
+		(stroke
+			(width 0)
+			(type default)
+		)
+	)
+	(wire
+		(pts
 			(xy 54.61 85.09) (xy 54.61 96.52)
 		)
@@
 	(wire
 		(pts
-			(xy 83.82 175.26) (xy 90.17 175.26)
+			(xy 83.82 171.45) (xy 90.17 171.45)
 		)
 		(stroke
@@
 	)
 	(label "Vert_Enable_Left"
-		(at 97.79 167.64 0)
+		(at 101.6 166.37 0)
 		(effects
 			(font
@@
 		)
 	)
+	(label "Court_T_Actif_Left"
+		(at 138.43 187.96 180)
+		(effects
+			(font
+				(size 1.27 1.27)
+			)
+			(justify right bottom)
+		)
+	)
 	(label "Court_Left"
 		(at 140.97 132.08 180)
@@
 	(global_label "GND"
 		(shape input)
-		(at 241.3 54.61 0)
+		(at 242.57 54.61 0)
 		(fields_autoplaced yes)
 		(effects
@@
 		)
 		(property "Intersheetrefs" "${INTERSHEET_REFS}"
-			(at 248.1557 54.61 0)
+			(at 249.4257 54.61 0)
 			(hide yes)
 			(show_name no)
@@
 	(global_label "V_Ref"
 		(shape input)
-		(at 83.82 175.26 180)
+		(at 83.82 171.45 180)
 		(fields_autoplaced yes)
 		(effects
@@
 		)
 		(property "Intersheetrefs" "${INTERSHEET_REFS}"
-			(at 75.6943 175.26 0)
+			(at 75.6943 171.45 0)
 			(hide yes)
 			(show_name no)
@@
 		)
 	)
+	(hierarchical_label "Btn_Left_Etat"
+		(shape input)
+		(at 151.13 187.96 0)
+		(effects
+			(font
+				(size 1.27 1.27)
+			)
+			(justify left)
+		)
+	)
 	(hierarchical_label "Court_Left_Vehic"
 		(shape input)
@@
 	(symbol
 		(lib_id "PCM_Diode_AKL:1N4148")
-		(at 232.41 44.45 0)
+		(at 236.22 44.45 0)
 		(unit 1)
 		(body_style 1)
@@
 		(dnp no)
 		(property "Reference" "D65"
-			(at 232.41 39.116 0)
+			(at 236.22 39.116 0)
 			(show_name no)
 			(do_not_autoplace no)
@@
 		)
 		(property "Value" "1N4148"
-			(at 232.41 41.402 0)
+			(at 236.22 41.402 0)
 			(show_name no)
 			(do_not_autoplace no)
@@
 		)
 		(property "Footprint" "PCM_Diode_THT_AKL:D_DO-35_SOD27_P7.62mm_Horizontal"
-			(at 232.41 44.45 0)
+			(at 236.22 44.45 0)
 			(hide yes)
 			(show_name no)
@@
 		)
 		(property "Datasheet" "https://datasheet.octopart.com/1N4148TR-ON-Semiconductor-datasheet-42765246.pdf"
-			(at 232.41 44.45 0)
+			(at 236.22 44.45 0)
 			(hide yes)
 			(show_name no)
@@
 		)
 		(property "Description" "DO-35 Diode, Small Signal, Fast Switching, 75V, 150mA, 4ns, Alternate KiCad Library"
-			(at 232.41 44.45 0)
+			(at 236.22 44.45 0)
 			(hide yes)
 			(show_name no)
@@
 	(symbol
 		(lib_id "PCM_SL_Resistors:4.7k")
-		(at 93.98 175.26 0)
+		(at 93.98 171.45 0)
 		(unit 1)
 		(body_style 1)
@@
 		(dnp no)
 		(property "Reference" "R84"
-			(at 94.234 170.434 0)
+			(at 94.234 166.624 0)
 			(show_name no)
 			(do_not_autoplace no)
@@
 		)
 		(property "Value" "4.7k"
-			(at 93.98 172.72 0)
+			(at 93.98 168.91 0)
 			(show_name no)
 			(do_not_autoplace no)
@@
 		)
 		(property "Footprint" "Resistor_THT:R_Axial_DIN0207_L6.3mm_D2.5mm_P10.16mm_Horizontal"
-			(at 94.869 179.578 0)
+			(at 94.869 175.768 0)
 			(hide yes)
 			(show_name no)
@@
 		)
 		(property "Datasheet" ""
-			(at 94.488 175.26 0)
+			(at 94.488 171.45 0)
 			(hide yes)
 			(show_name no)
@@
 		)
 		(property "Description" "4.7kΩ, 1/4W Resistor"
-			(at 93.98 175.26 0)
+			(at 93.98 171.45 0)
 			(hide yes)
 			(show_name no)
@@
 	(symbol
 		(lib_id "PCM_SL_Resistors:4.7k")
-		(at 232.41 54.61 0)
+		(at 236.22 54.61 0)
 		(unit 1)
 		(body_style 1)
@@
 		(dnp no)
 		(property "Reference" "R81"
-			(at 232.664 49.784 0)
+			(at 236.474 49.784 0)
 			(show_name no)
 			(do_not_autoplace no)
@@
 		)
 		(property "Value" "4.7k"
-			(at 232.41 52.07 0)
+			(at 236.22 52.07 0)
 			(show_name no)
 			(do_not_autoplace no)
@@
 		)
 		(property "Footprint" "Resistor_THT:R_Axial_DIN0207_L6.3mm_D2.5mm_P10.16mm_Horizontal"
-			(at 233.299 58.928 0)
+			(at 237.109 58.928 0)
 			(hide yes)
 			(show_name no)
@@
 		)
 		(property "Datasheet" ""
-			(at 232.918 54.61 0)
+			(at 236.728 54.61 0)
 			(hide yes)
 			(show_name no)
@@
 		)
 		(property "Description" "4.7kΩ, 1/4W Resistor"
-			(at 232.41 54.61 0)
+			(at 236.22 54.61 0)
 			(hide yes)
 			(show_name no)
@@
 					(unit 1)
 				)
+			)
+		)
+	)
+	(symbol
+		(lib_id "PCM_Diode_AKL:1N4148")
+		(at 144.78 187.96 0)
+		(unit 1)
+		(body_style 1)
+		(exclude_from_sim no)
+		(in_bom yes)
+		(on_board yes)
+		(in_pos_files yes)
+		(dnp no)
+		(property "Reference" "D175"
+			(at 144.78 182.63 0)
+			(show_name no)
+			(do_not_autoplace no)
+			(effects
+				(font
+					(size 1.27 1.27)
+				)
+			)
+		)
+		(property "Value" "1N4148"
+			(at 144.78 184.91 0)
+			(show_name no)
+			(do_not_autoplace no)
+			(effects
+				(font
+					(size 1.27 1.27)
+				)
+			)
+		)
+		(property "Footprint" "PCM_Diode_THT_AKL:D_DO-35_SOD27_P7.62mm_Horizontal"
+			(at 144.78 187.96 0)
+			(hide yes)
+			(show_name no)
+			(do_not_autoplace no)
+			(effects
+				(font
+					(size 1.27 1.27)
+				)
+			)
+		)
+		(property "Datasheet" "https://datasheet.octopart.com/1N4148TR-ON-Semiconductor-datasheet-42765246.pdf"
+			(at 144.78 187.96 0)
+			(hide yes)
+			(show_name no)
+			(do_not_autoplace no)
+			(effects
+				(font
+					(size 1.27 1.27)
+				)
+			)
+		)
+		(property "Description" "DO-35 Diode, Small Signal, Fast Switching, 75V, 150mA, 4ns, Alternate KiCad Library"
+			(at 144.78 187.96 0)
+			(hide yes)
+			(show_name no)
+			(do_not_autoplace no)
+			(effects
+				(font
+					(size 1.27 1.27)
+				)
+			)
+		)
+		(pin "2"
+		)
+		(pin "1"
+		)
+		(instances
+			(project "TrailerDiagnosticSystem"
+				(path "/d4e407a7-3e32-4226-ae57-831ecdb3edf4/d158d25b-993e-468a-8f69-95ddcf9272e8/f7963cc6-1c2c-440a-87f5-49a6c6c4b196"
+					(reference "D175")
+					(unit 1)
+				)

Commit message: Add files via upload
Parts:
- R78, R79: value 4.7k -> 100k
- R82, R83, R85: value 4.7k -> 470kΩ
Connections:
- net GND: no longer R81.2
- net V_Ref: now also R81.2
Changed lines of the file:
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@@
 	(global_label "GND"
 		(shape input)
-		(at 242.57 54.61 0)
-		(fields_autoplaced yes)
-		(effects
-			(font
-				(size 1.27 1.27)
-			)
-			(justify left)
-		)
-		(property "Intersheetrefs" "${INTERSHEET_REFS}"
-			(at 249.4257 54.61 0)
-			(hide yes)
-			(show_name no)
-			(do_not_autoplace no)
-			(effects
-				(font
-					(size 1.27 1.27)
-				)
-				(justify left)
-			)
-		)
-	)
-	(global_label "GND"
-		(shape input)
 		(at 97.79 189.23 0)
 		(fields_autoplaced yes)
@@
 	(global_label "V_Ref"
 		(shape input)
+		(at 242.57 54.61 0)
+		(fields_autoplaced yes)
+		(effects
+			(font
+				(size 1.27 1.27)
+			)
+			(justify left)
+		)
+		(property "Intersheetrefs" "${INTERSHEET_REFS}"
+			(at 250.6957 54.61 0)
+			(hide yes)
+			(show_name no)
+			(do_not_autoplace no)
+			(effects
+				(font
+					(size 1.27 1.27)
+				)
+				(justify left)
+			)
+		)
+	)
+	(global_label "V_Ref"
+		(shape input)
 		(at 83.82 171.45 180)
 		(fields_autoplaced yes)
@@
 			)
 		)
-		(property "Value" "4.7k"
+		(property "Value" "100k"
 			(at 46.99 93.98 0)
 			(show_name no)
@@
 			)
 		)
-		(property "Value" "4.7k"
+		(property "Value" "470kΩ"
 			(at 147.32 148.59 0)
 			(show_name no)
@@
 			)
 		)
-		(property "Value" "4.7k"
+		(property "Value" "470kΩ"
 			(at 85.09 152.4 0)
 			(show_name no)
@@
 			)
 		)
-		(property "Value" "4.7k"
+		(property "Value" "100k"
 			(at 86.36 93.98 0)
 			(show_name no)
@@
 			)
 		)
-		(property "Value" "4.7k"
+		(property "Value" "470kΩ"
 			(at 39.37 147.32 0)
 			(show_name no)

Commit message: Add files via upload
Parts:
- R74, R75, R76, R77, R80, R81, R84: value 4.7k -> 4.7kΩ
- R78, R79: value 100k -> 100kΩ
- R86, R87, R88: value 330ohm -> 330Ω
Changed lines of the file:
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@@
 			)
 		)
-		(property "Value" "100k"
+		(property "Value" "100kΩ"
 			(at 46.99 93.98 0)
 			(show_name no)
@@
 			)
 		)
-		(property "Value" "4.7k"
+		(property "Value" "4.7kΩ"
 			(at 93.98 168.91 0)
 			(show_name no)
@@
 			)
 		)
-		(property "Value" "4.7k"
+		(property "Value" "4.7kΩ"
 			(at 204.47 39.37 0)
 			(show_name no)
@@
 			)
 		)
-		(property "Value" "330ohm"
+		(property "Value" "330Ω"
 			(at 233.68 138.684 0)
 			(show_name no)
@@
 			)
 		)
-		(property "Value" "4.7k"
+		(property "Value" "4.7kΩ"
 			(at 236.22 52.07 0)
 			(show_name no)
@@
 			)
 		)
-		(property "Value" "330ohm"
+		(property "Value" "330Ω"
 			(at 233.68 96.774 0)
 			(show_name no)
@@
 			)
 		)
-		(property "Value" "330ohm"
+		(property "Value" "330Ω"
 			(at 233.68 118.364 0)
 			(show_name no)
@@
 			)
 		)
-		(property "Value" "100k"
+		(property "Value" "100kΩ"
 			(at 86.36 93.98 0)
 			(show_name no)
@@
 			)
 		)
-		(property "Value" "4.7k"
+		(property "Value" "4.7kΩ"
 			(at 30.48 49.53 0)
 			(show_name no)
@@
 			)
 		)
-		(property "Value" "4.7k"
+		(property "Value" "4.7kΩ"
 			(at 109.22 52.07 0)
 			(show_name no)
@@
 			)
 		)
-		(property "Value" "4.7k"
+		(property "Value" "4.7kΩ"
 			(at 151.13 54.61 0)
 			(show_name no)
@@
 			)
 		)
-		(property "Value" "4.7k"
+		(property "Value" "4.7kΩ"
 			(at 68.58 49.53 0)
 			(show_name no)

Commit message: Add files via upload
Connections:
- net Fac_Left_B: now reaches D73.4 (BK), R88.2
- net Fac_Left_R: now reaches D73.2 (RK), R86.2
- net Fac_Left_G: now reaches D73.3 (GK), R87.2
Changed lines of the file:
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@@
+	)
+	(junction
+		(at 237.49 140.97)
+		(diameter 0)
+		(color 0 0 0 0)
 	)
 	(junction
@@
 	)
 	(junction
+		(at 237.49 120.65)
+		(diameter 0)
+		(color 0 0 0 0)
+	)
+	(junction
 		(at 54.61 85.09)
 		(diameter 0)
@@
 	)
 	(junction
+		(at 237.49 99.06)
+		(diameter 0)
+		(color 0 0 0 0)
+	)
+	(junction
 		(at 48.26 139.7)
 		(diameter 0)
@@
 	(wire
 		(pts
+			(xy 241.3 93.98) (xy 237.49 93.98)
+		)
+		(stroke
+			(width 0)
+			(type default)
+		)
+	)
+	(wire
+		(pts
 			(xy 50.8 85.09) (xy 54.61 85.09)
 		)
@@
 	(wire
 		(pts
+			(xy 237.49 137.16) (xy 237.49 140.97)
+		)
+		(stroke
+			(width 0)
+			(type default)
+		)
+	)
+	(wire
+		(pts
 			(xy 54.61 96.52) (xy 50.8 96.52)
 		)
@@
 	(wire
 		(pts
+			(xy 242.57 137.16) (xy 237.49 137.16)
+		)
+		(stroke
+			(width 0)
+			(type default)
+		)
+	)
+	(wire
+		(pts
 			(xy 229.87 111.76) (xy 231.14 111.76)
 		)
@@
 	(wire
 		(pts
+			(xy 241.3 118.11) (xy 237.49 118.11)
+		)
+		(stroke
+			(width 0)
+			(type default)
+		)
+	)
+	(wire
+		(pts
 			(xy 229.87 109.22) (xy 229.87 111.76)
 		)
@@
 	(wire
 		(pts
-			(xy 250.19 113.03) (xy 262.89 113.03)
+			(xy 255.27 113.03) (xy 262.89 113.03)
 		)
 		(stroke
@@
 	(wire
 		(pts
-			(xy 237.49 120.65) (xy 250.19 120.65)
+			(xy 237.49 120.65) (xy 255.27 120.65)
 		)
 		(stroke
@@
 	(wire
 		(pts
+			(xy 237.49 93.98) (xy 237.49 99.06)
+		)
+		(stroke
+			(width 0)
+			(type default)
+		)
+	)
+	(wire
+		(pts
 			(xy 25.4 59.69) (xy 27.94 59.69)
 		)
@@
 	(wire
 		(pts
-			(xy 250.19 113.03) (xy 250.19 120.65)
+			(xy 255.27 113.03) (xy 255.27 120.65)
 		)
 		(stroke
@@
 		(pts
 			(xy 63.5 52.07) (xy 64.77 52.07)
+		)
+		(stroke
+			(width 0)
+			(type default)
+		)
+	)
+	(wire
+		(pts
+			(xy 237.49 118.11) (xy 237.49 120.65)
 		)
 		(stroke
@@
 		)
 	)
+	(global_label "Fac_Left_R"
+		(shape input)
+		(at 241.3 93.98 0)
+		(fields_autoplaced yes)
+		(effects
+			(font
+				(size 1.27 1.27)
+			)
+			(justify left)
+		)
+		(property "Intersheetrefs" "${INTERSHEET_REFS}"
+			(at 254.3847 93.98 0)
+			(hide yes)
+			(show_name no)
+			(do_not_autoplace no)
+			(effects
+				(font
+					(size 1.27 1.27)
+				)
+				(justify left)
+			)
+		)
+	)
 	(global_label "GND"
 		(shape input)
@@
 		)
 	)
+	(global_label "Fac_Left_G"
+		(shape input)
+		(at 241.3 118.11 0)
+		(fields_autoplaced yes)
+		(effects
+			(font
+				(size 1.27 1.27)
+			)
+			(justify left)
+		)
+		(property "Intersheetrefs" "${INTERSHEET_REFS}"
+			(at 254.3847 118.11 0)
+			(hide yes)
+			(show_name no)
+			(do_not_autoplace no)
+			(effects
+				(font
+					(size 1.27 1.27)
+				)
+				(justify left)
+			)
+		)
+	)
 	(global_label "GND"
 		(shape input)
@@
 			(hide yes)
 			(show_name no)
+			(do_not_autoplace no)
+			(effects
+				(font
+					(size 1.27 1.27)
+				)
+				(justify left)
+			)
+		)
+	)
+	(global_label "Fac_Left_B"
+		(shape input)
+		(at 242.57 137.16 0)
+		(fields_autoplaced yes)
+		(effects
+			(font
+				(size 1.27 1.27)
+			)
+			(justify left)
+		)
+		(property "Intersheetrefs" "${INTERSHEET_REFS}"
+			(at 255.6547 137.16 0)
+			(hide yes)
+			(show_name no)
