File: mode_coherence.kicad_sch (KiCad schematic)
At the start: 11 parts, among them Q2 2N3904, Q3 2N3904, Q4 2N3904, SW2 SW_DPDT_x2

Commit message: Add files via upload
Changed lines of the file:
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@@
-		)
-	)
-	(label "V_Ref"
-		(at 26.67 41.91 180)
-		(effects
-			(font
-				(size 1.27 1.27)
-			)
-			(justify right bottom)
 		)
 	)
@@
 			(hide yes)
 			(show_name no)
+			(do_not_autoplace no)
+			(effects
+				(font
+					(size 1.27 1.27)
+				)
+				(justify right)
+			)
+		)
+	)
+	(global_label "V_Ref"
+		(shape input)
+		(at 26.67 41.91 180)
+		(fields_autoplaced yes)
+		(effects
+			(font
+				(size 1.27 1.27)
+			)
+			(justify right)
+		)
+		(property "Intersheetrefs" "${INTERSHEET_REFS}"
+			(at 18.5443 41.91 0)
+			(hide yes)
+			(show_name no)

Commit message: Add files via upload
Parts:
- removed Q3: 2N3904, PCM_Package_TO_SOT_THT_AKL:TO-92_Inline_Wide_EBC, symbol PCM_Transistor_BJT_AKL:2N3904
- removed R4: 10k, Resistor_THT:R_Axial_DIN0207_L6.3mm_D2.5mm_P10.16mm_Horizontal, symbol PCM_SL_Resistors:10k
- added D181: 1N4148, PCM_Diode_THT_AKL:D_DO-35_SOD27_P7.62mm_Horizontal, symbol PCM_Diode_AKL:1N4148
- added Q83: 2N7000, PCM_Package_TO_SOT_THT_AKL:TO-92_Inline_Wide_SGD, symbol PCM_Transistor_MOSFET_AKL:2N7000
- added R310, R311, R312: 10k, Resistor_THT:R_Axial_DIN0207_L6.3mm_D2.5mm_P10.16mm_Horizontal, symbol PCM_SL_Resistors:10k
- added R313: 100k, Resistor_THT:R_Axial_DIN0207_L6.3mm_D2.5mm_P10.16mm_Horizontal, symbol PCM_SL_Resistors:100k
- added R4: 4.7k, Resistor_THT:R_Axial_DIN0207_L6.3mm_D2.5mm_P10.16mm_Horizontal, symbol PCM_SL_Resistors:4.7k
- R3: value 10k -> 4.7k; symbol PCM_SL_Resistors:10k -> PCM_SL_Resistors:4.7k
Connections:
- net Alerte_Incoherence: now also D2.1 (K), D181.1 (K); no longer Q2.3 (C)
- net Detect_Trailer: now also R311.2, R312.1; no longer D2.2 (A)
- net Detect_Vehicule: now also R310.2
- net GND: now also SW2.4 (A), Q83.1 (S), R313.2; no longer R1.2
- net Mode_Trailer: now also SW2.5 (B), Q83.2 (G), R4.1; no longer SW2.6 (C)
- net Mode_Vehicule: now also D1.1 (K), Q83.3 (D); no longer D1.2 (A), SW2.4 (A)
- net V_Ref: now also R1.2, SW2.6 (C), R310.1, R311.1; no longer SW2.5 (B)
- net at Q4.3 (C): now also D181.2 (A), R4.2
- new net: Q2.2 (B), R312.2
- new net Incoh_T: D1.2 (A), D2.2 (A), Q2.3 (C), R3.2, R313.1
Other:
- moved on the sheet: D1, D2, Q2, Q4, R1, R2, R3, R5

Commit message: Add files via upload
Connections:
- net Alerte_Incoherence: now also R313.1
- net Incoh_T: no longer R313.1
Other:
- moved on the sheet: D1, D181, D2, Q2, Q4, Q83, R1, R2, R3, R310, R311, R312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

Commit message: Add files via upload
Changed lines of the file:
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@@
-	(hierarchical_label "Alerte_Incoherence"
-		(shape input)
-		(at 39.37 109.22 180)
-		(effects
-			(font
-				(size 1.27 1.27)
-			)
-			(justify right)
-		)
-	)
 	(hierarchical_label "Alerte_Incoherence"
 		(shape input)

Commit message: Add files via upload
Parts:
- R1, R2, R310, R311, R312, R5: value 10k -> 10kΩ
- R3, R4: value 4.7k -> 4.7kΩ
- R313: value 100k -> 100kΩ
Changed lines of the file:
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@@
 			)
 		)
-		(property "Value" "4.7k"
+		(property "Value" "4.7kΩ"
 			(at 129.54 90.17 0)
 			(show_name no)
@@
 			)
 		)
-		(property "Value" "10k"
+		(property "Value" "10kΩ"
 			(at 34.29 135.89 0)
 			(show_name no)
@@
 			)
 		)
-		(property "Value" "100k"
+		(property "Value" "100kΩ"
 			(at 46.99 102.87 0)
 			(show_name no)
@@
 			)
 		)
-		(property "Value" "4.7k"
+		(property "Value" "4.7kΩ"
 			(at 29.21 92.71 0)
 			(show_name no)
@@
 			)
 		)
-		(property "Value" "10k"
+		(property "Value" "10kΩ"
 			(at 45.72 124.46 0)
 			(show_name no)
@@
 			)
 		)
-		(property "Value" "10k"
+		(property "Value" "10kΩ"
 			(at 132.08 130.81 0)
 			(show_name no)
@@
 			)
 		)
-		(property "Value" "10k"
+		(property "Value" "10kΩ"
 			(at 128.27 72.39 0)
 			(show_name no)
@@
 			)
 		)
-		(property "Value" "10k"
+		(property "Value" "10kΩ"
 			(at 95.25 115.57 0)
 			(show_name no)
@@
 			)
 		)
-		(property "Value" "10k"
+		(property "Value" "10kΩ"
 			(at 132.08 105.41 0)
 			(show_name no)

Commit message: Add files via upload
Parts:
- added J6: Conn_02x02_Top_Bottom, Connector_Molex:Molex_Mega-Fit_76829-0004_2x02_P5.70mm_Vertical, symbol Connector_Generic:Conn_02x02_Top_Bottom
Connections:
- net V12_Rail: now also J6.1 (Pin_1), J6.3 (Pin_3)
- net V_Arm_Trailer: now also J6.2 (Pin_2), J6.4 (Pin_4)
Changed lines of the file:
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@@
+	(wire
+		(pts
+			(xy 29.21 30.48) (xy 33.02 30.48)
+		)
+		(stroke
+			(width 0)
+			(type default)
+		)
+	)
 	(wire
 		(pts
@@
 	(wire
 		(pts
+			(xy 29.21 33.02) (xy 33.02 33.02)
+		)
+		(stroke
+			(width 0)
+			(type default)
+		)
+	)
+	(wire
+		(pts
 			(xy 121.92 92.71) (xy 125.73 92.71)
 		)
@@
 	(wire
 		(pts
+			(xy 45.72 30.48) (xy 49.53 30.48)
+		)
+		(stroke
+			(width 0)
+			(type default)
+		)
+	)
+	(wire
+		(pts
 			(xy 78.74 165.1) (xy 78.74 168.91)
 		)
@@
 		(pts
 			(xy 43.18 83.82) (xy 39.37 83.82)
+		)
+		(stroke
+			(width 0)
+			(type default)
+		)
+	)
+	(wire
+		(pts
+			(xy 45.72 33.02) (xy 49.53 33.02)
 		)
 		(stroke
@@
 		)
 	)
+	(global_label "V_Arm_Trailer"
+		(shape input)
+		(at 29.21 33.02 180)
+		(fields_autoplaced yes)
+		(effects
+			(font
+				(size 1.27 1.27)
+			)
+			(justify right)
+		)
+		(property "Intersheetrefs" "${INTERSHEET_REFS}"
+			(at 13.5853 33.02 0)
+			(hide yes)
+			(show_name no)
+			(do_not_autoplace no)
+			(effects
+				(font
+					(size 1.27 1.27)
+				)
+				(justify right)
+			)
+		)
+	)
 	(global_label "V_Ref"
 		(shape input)
@@
 		)
 	)
+	(global_label "V_Arm_Trailer"
+		(shape input)
+		(at 49.53 33.02 0)
+		(fields_autoplaced yes)
+		(effects
+			(font
+				(size 1.27 1.27)
+			)
+			(justify left)
+		)
+		(property "Intersheetrefs" "${INTERSHEET_REFS}"
+			(at 65.1547 33.02 0)
+			(hide yes)
+			(show_name no)
+			(do_not_autoplace no)
+			(effects
+				(font
+					(size 1.27 1.27)
+				)
+				(justify left)
+			)
+		)
+	)
 	(hierarchical_label "Detect_Vehicule"
 		(shape input)
@@
 		)
 	)
+	(hierarchical_label "V12_Rail"
+		(shape input)
+		(at 29.21 30.48 180)
+		(effects
+			(font
+				(size 1.27 1.27)
+			)
+			(justify right)
+		)
+	)
 	(hierarchical_label "Detect_Trailer"
 		(shape input)
@@
 		(shape input)
 		(at 55.88 95.25 0)
+		(effects
+			(font
+				(size 1.27 1.27)
+			)
+			(justify left)
+		)
+	)
+	(hierarchical_label "V12_Rail"
+		(shape input)
+		(at 49.53 30.48 0)
 		(effects
 			(font
@@
 		(exclude_from_sim no)
 		(in_bom yes)
-		(on_board yes)
+		(on_board no)
 		(in_pos_files yes)
 		(dnp no)
@@
 		(exclude_from_sim no)
 		(in_bom yes)
-		(on_board yes)
+		(on_board no)
 		(in_pos_files yes)
 		(dnp no)
@@
 					(unit 1)
 				)
+			)
+		)
+	)
+	(symbol
+		(lib_id "Connector_Generic:Conn_02x02_Top_Bottom")
+		(at 38.1 30.48 0)
+		(unit 1)
+		(body_style 1)
+		(exclude_from_sim no)
+		(in_bom yes)
+		(on_board yes)
+		(in_pos_files yes)
+		(dnp no)
+		(fields_autoplaced yes)
+		(property "Reference" "J6"
+			(at 39.37 24.13 0)
+			(show_name no)
+			(do_not_autoplace no)
+			(effects
+				(font
+					(size 1.27 1.27)
+				)
+			)
+		)
+		(property "Value" "Conn_02x02_Top_Bottom"
+			(at 39.37 26.67 0)
+			(show_name no)
+			(do_not_autoplace no)
+			(effects
+				(font
+					(size 1.27 1.27)
+				)
+			)
+		)
+		(property "Footprint" "Connector_Molex:Molex_Mega-Fit_76829-0004_2x02_P5.70mm_Vertical"
+			(at 38.1 30.48 0)
+			(hide yes)
+			(show_name no)
+			(do_not_autoplace no)
+			(effects
+				(font
+					(size 1.27 1.27)
+				)
+			)
+		)
+		(property "Datasheet" ""
+			(at 38.1 30.48 0)
+			(hide yes)
+			(show_name no)
+			(do_not_autoplace no)
+			(effects
+				(font
+					(size 1.27 1.27)
+				)
+			)
+		)
+		(property "Description" "Generic connector, double row, 02x02, top/bottom pin numbering scheme (row 1: 1...pins_per_row, row2: pins_per_row+1 ... num_pins), script generated (kicad-library-utils/schlib/autogen/connector/)"
+			(at 38.1 30.48 0)
+			(hide yes)
+			(show_name no)
+			(do_not_autoplace no)
+			(effects
+				(font
+					(size 1.27 1.27)
+				)
+			)
+		)
+		(pin "4"
+		)
+		(pin "1"
+		)
+		(pin "2"
+		)
+		(pin "3"
+		)
+		(instances
+			(project "TrailerDiagnosticSystem"
+				(path "/d4e407a7-3e32-4226-ae57-831ecdb3edf4/d808f71c-7914-43fb-8ac9-96d92cd6294f"
+					(reference "J6")
+					(unit 1)
+				)

Commit message: Add files via upload
Parts:
- SW2: value SW_DPDT_x2 -> Cole Hersee 5592
Changed lines of the file:
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@@
 			)
 		)
-		(property "Value" "SW_DPDT_x2"
+		(property "Value" "Cole Hersee 5592"
 			(at 35.56 63.5 0)
 			(hide yes)
@@
 			)
 		)
-		(property "Value" "SW_DPDT_x2"
+		(property "Value" "Cole Hersee 5592"
 			(at 35.56 55.88 0)
 			(show_name no)
