File: Facade/Facade.kicad_sch (KiCad schematic)
At the start: 0 parts

Commit message: Add files via upload
Other:
- added sheet Bottom_Zone (Bottom_Zone.kicad_sch)
- added sheet Center_Zone (Center_Zone.kicad_sch)
- added sheet Top_Zone (Top_Zone.kicad_sch)
- title: (none) -> Trailer Diagnostic System - Façade
Changed lines of the file:
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@@
 	(generator "eeschema")
 	(generator_version "10.0")
-	(paper "A4")
+	(paper "USLedger")
+	(title_block
+		(title "Trailer Diagnostic System - Façade")
+		(date "2026-10-18")
+	)
+	(sheet
+		(at 30.988 19.304)
+		(size 376.682 74.168)
+		(exclude_from_sim no)
+		(in_bom yes)
+		(on_board yes)
+		(dnp no)
+		(fields_autoplaced yes)
+		(stroke
+			(width 0.1524)
+			(type solid)
+		)
+		(fill
+			(color 0 0 0 0)
+		)
+		(property "Sheetname" "Top_Zone"
+			(at 30.988 18.5924 0)
+			(show_name no)
+			(do_not_autoplace no)
+			(effects
+				(font
+					(size 1.27 1.27)
+				)
+				(justify left bottom)
+			)
+		)
+		(property "Sheetfile" "Top_Zone.kicad_sch"
+			(at 30.988 94.0566 0)
+			(show_name no)
+			(do_not_autoplace no)
+			(effects
+				(font
+					(size 1.27 1.27)
+				)
+				(justify left top)
+			)
+		)
+		(instances
+			(project "Facade"
+				(path "/a22adf74-3f4e-45d1-a847-1db98a43facb"
+					(page "2")
+				)
+			)
+		)
+	)
+	(sheet
+		(at 32.004 106.172)
+		(size 376.936 55.372)
+		(exclude_from_sim no)
+		(in_bom yes)
+		(on_board yes)
+		(dnp no)
+		(fields_autoplaced yes)
+		(stroke
+			(width 0.1524)
+			(type solid)
+		)
+		(fill
+			(color 0 0 0 0)
+		)
+		(property "Sheetname" "Center_Zone"
+			(at 32.004 105.4604 0)
+			(show_name no)
+			(do_not_autoplace no)
+			(effects
+				(font
+					(size 1.27 1.27)
+				)
+				(justify left bottom)
+			)
+		)
+		(property "Sheetfile" "Center_Zone.kicad_sch"
+			(at 32.004 162.1286 0)
+			(show_name no)
+			(do_not_autoplace no)
+			(effects
+				(font
+					(size 1.27 1.27)
+				)
+				(justify left top)
+			)
+		)
+		(instances
+			(project "Facade"
+				(path "/a22adf74-3f4e-45d1-a847-1db98a43facb"
+					(page "3")
+				)
+			)
+		)
+	)
+	(sheet
+		(at 32.766 170.688)
+		(size 375.666 49.53)
+		(exclude_from_sim no)
+		(in_bom yes)
+		(on_board yes)
+		(dnp no)
+		(fields_autoplaced yes)
+		(stroke
+			(width 0.1524)
+			(type solid)
+		)
+		(fill
+			(color 0 0 0 0)
+		)
+		(property "Sheetname" "Bottom_Zone"
+			(at 32.766 169.9764 0)
+			(show_name no)
+			(do_not_autoplace no)
+			(effects
+				(font
+					(size 1.27 1.27)
+				)
+				(justify left bottom)
+			)
+		)
+		(property "Sheetfile" "Bottom_Zone.kicad_sch"
+			(at 32.766 220.8026 0)
+			(show_name no)
+			(do_not_autoplace no)
+			(effects
+				(font
+					(size 1.27 1.27)
+				)
+				(justify left top)
+			)
+		)
+		(instances
+			(project "Facade"
+				(path "/a22adf74-3f4e-45d1-a847-1db98a43facb"
+					(page "4")
+				)
+			)
+		)
+	)
 	(sheet_instances
 		(path "/"
