File: Facade/Facade.kicad_pcb (KiCad board)
At the start: 2 copper layers, 28 parts, among them J20 Conn_01x03 (Fils soudés), J21 Conn_01x03 (Fils soudés), J22 Conn_01x03 (Fils soudés), J23 Conn_01x03 (Fils soudés), J24 Conn_01x03 (Fils soudés), J25 Conn_01x03 (Fils soudés), J26 Conn_01x06 (Fils soudés), J27 Conn_01x05 (Fils soudés), J28 Conn_01x03 (Fils soudés), J7 Conn_02x07_Odd_Even, J8 Conn_02x17_Odd_Even, J9 Conn_02x13_Odd_Even

Commit message: Add files via upload
Parts:
- J20, J21, J22, J23, J24, J25, J28: value Conn_01x03 (Fils soudés) -> Micro-Fit 3.0 1x03; footprint Connector_Wire:SolderWire-0.5sqmm_1x03_P4.6mm_D0.9mm_OD2.1mm_Relief -> Connector_Molex:Molex_Micro-Fit_3.0_43650-0315_1x03_P3.00mm_Vertical
- J26: value Conn_01x06 (Fils soudés) -> Micro-Fit 3.0 1x06; footprint Connector_Wire:SolderWire-0.5sqmm_1x06_P4.6mm_D0.9mm_OD2.1mm_Relief -> Connector_Molex:Molex_Micro-Fit_3.0_43650-0615_1x06_P3.00mm_Vertical
- J27: value Conn_01x05 (Fils soudés) -> Micro-Fit 3.0 1x05; footprint Connector_Wire:SolderWire-0.5sqmm_1x05_P4.6mm_D0.9mm_OD2.1mm_Relief -> Connector_Molex:Molex_Micro-Fit_3.0_43650-0515_1x05_P3.00mm_Vertical
