File: Facade/Center_Zone.kicad_sch (KiCad schematic)
At the start: 19 parts, among them J20 Conn_01x03 (Fils soudés), J21 Conn_01x03 (Fils soudés), J22 Conn_01x03 (Fils soudés), J23 Conn_01x03 (Fils soudés), J24 Conn_01x03 (Fils soudés), J25 Conn_01x03 (Fils soudés), J8 Conn_02x17_Odd_Even, SW3 Bouton verouillable, SW4 Bouton verouillable, SW5 Bouton verouillable, SW6 Bouton verouillable, SW7 Bouton verouillable, SW8 Bouton verouillable

Commit message: Add files via upload
Parts:
- J20: footprint Connector_Wire:SolderWire-…_1x03_… (fil 0,25 à 0,5 mm²) -> Connector_Wire:SolderWire-0.5sqmm_1x03_P4.6mm_D0.9mm_OD2.1mm_Relief
- SW3, SW4, SW5, SW6, SW7, SW8: value Bouton verouillable -> Bouton verrouillable; footprint openinput:SW_Micro_Switch -> (none)
Changed lines of the file:
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@@
 			)
 		)
-		(property "Value" "Bouton verouillable"
+		(property "Value" "Bouton verrouillable"
 			(at 230.378 45.466 90)
 			(show_name no)
@@
 			)
 		)
-		(property "Footprint" "openinput:SW_Micro_Switch"
+		(property "Footprint" ""
 			(at 205.74 45.72 0)
 			(hide yes)
@@
 			)
 		)
-		(property "Value" "Bouton verouillable"
+		(property "Value" "Bouton verrouillable"
 			(at 212.852 116.84 90)
 			(show_name no)
@@
 			)
 		)
-		(property "Footprint" "openinput:SW_Micro_Switch"
+		(property "Footprint" ""
 			(at 204.47 115.57 0)
 			(hide yes)
@@
 			)
 		)
-		(property "Value" "Bouton verouillable"
+		(property "Value" "Bouton verrouillable"
 			(at 210.82 161.036 90)
 			(show_name no)
@@
 			)
 		)
-		(property "Footprint" "openinput:SW_Micro_Switch"
+		(property "Footprint" ""
 			(at 204.47 160.02 0)
 			(hide yes)
@@
 			)
 		)
-		(property "Value" "Bouton verouillable"
+		(property "Value" "Bouton verrouillable"
 			(at 211.328 140.97 90)
 			(show_name no)
@@
 			)
 		)
-		(property "Footprint" "openinput:SW_Micro_Switch"
+		(property "Footprint" ""
 			(at 204.47 139.7 0)
 			(hide yes)
@@
 			)
 		)
-		(property "Footprint" "Connector_Wire:SolderWire-…_1x03_… (fil 0,25 à 0,5 mm²)"
+		(property "Footprint" "Connector_Wire:SolderWire-0.5sqmm_1x03_P4.6mm_D0.9mm_OD2.1mm_Relief"
 			(at 57.15 76.2 0)
 			(hide yes)
@@
 			)
 		)
-		(property "Value" "Bouton verouillable"
+		(property "Value" "Bouton verrouillable"
 			(at 211.836 66.802 90)
 			(show_name no)
@@
 			)
 		)
-		(property "Footprint" "openinput:SW_Micro_Switch"
+		(property "Footprint" ""
 			(at 205.74 66.04 0)
 			(hide yes)
@@
 			)
 		)
-		(property "Value" "Bouton verouillable"
+		(property "Value" "Bouton verrouillable"
 			(at 211.582 92.456 90)
 			(show_name no)
@@
 			)
 		)
-		(property "Footprint" "openinput:SW_Micro_Switch"
+		(property "Footprint" ""
 			(at 205.74 91.44 0)
 			(hide yes)

Commit message: Add files via upload
Parts:
- D121, D145, D26, D49, D73, D97: value LED_ARGB -> RGB 5mm; now in the parts list
- J20, J21, SW3, SW4, SW5, SW6, SW7, SW8: now in the parts list
- J22, J23, J24, J25: now left out of the parts list
- J8: footprint (none) -> Connector_IDC:IDC-Header_2x17_P2.54mm_Latch_Vertical
Changed lines of the file:
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@@
 		(body_style 1)
 		(exclude_from_sim no)
-		(in_bom yes)
+		(in_bom no)
 		(on_board yes)
 		(in_pos_files yes)
@@
 		(body_style 1)
 		(exclude_from_sim no)
-		(in_bom no)
+		(in_bom yes)
 		(on_board yes)
 		(in_pos_files yes)
@@
 			)
 		)
-		(property "Value" "LED_ARGB"
+		(property "Value" "RGB 5mm"
 			(at 261.62 33.02 0)
 			(show_name no)
@@
 		(body_style 1)
 		(exclude_from_sim no)
-		(in_bom yes)
+		(in_bom no)
 		(on_board yes)
 		(in_pos_files yes)
@@
 		(body_style 1)
 		(exclude_from_sim no)
-		(in_bom no)
+		(in_bom yes)
 		(on_board no)
 		(in_pos_files yes)
@@
 		(body_style 1)
 		(exclude_from_sim no)
-		(in_bom no)
+		(in_bom yes)
 		(on_board yes)
 		(in_pos_files yes)
@@
 			)
 		)
-		(property "Footprint" ""
+		(property "Footprint" "Connector_IDC:IDC-Header_2x17_P2.54mm_Latch_Vertical"
 			(at 134.62 113.03 0)
 			(hide yes)
@@
 		(body_style 1)
 		(exclude_from_sim no)
-		(in_bom no)
+		(in_bom yes)
 		(on_board yes)
 		(in_pos_files yes)
@@
 			)
 		)
-		(property "Value" "LED_ARGB"
+		(property "Value" "RGB 5mm"
 			(at 260.35 165.1 0)
 			(show_name no)
@@
 		(body_style 1)
 		(exclude_from_sim no)
-		(in_bom no)
+		(in_bom yes)
 		(on_board yes)
 		(in_pos_files yes)
@@
 			)
 		)
-		(property "Value" "LED_ARGB"
+		(property "Value" "RGB 5mm"
 			(at 261.62 139.7 0)
 			(show_name no)
@@
 		(body_style 1)
 		(exclude_from_sim no)
-		(in_bom no)
+		(in_bom yes)
 		(on_board no)
 		(in_pos_files yes)
@@
 		(body_style 1)
 		(exclude_from_sim no)
-		(in_bom yes)
+		(in_bom no)
 		(on_board yes)
 		(in_pos_files yes)
@@
 		(body_style 1)
 		(exclude_from_sim no)
-		(in_bom no)
+		(in_bom yes)
 		(on_board no)
 		(in_pos_files yes)
@@
 		(body_style 1)
 		(exclude_from_sim no)
-		(in_bom no)
+		(in_bom yes)
 		(on_board yes)
 		(in_pos_files yes)
@@
 			)
 		)
-		(property "Value" "LED_ARGB"
+		(property "Value" "RGB 5mm"
 			(at 261.62 113.03 0)
 			(show_name no)
@@
 		(body_style 1)
 		(exclude_from_sim no)
-		(in_bom no)
+		(in_bom yes)
 		(on_board no)
 		(in_pos_files yes)
@@
 		(body_style 1)
 		(exclude_from_sim no)
-		(in_bom no)
+		(in_bom yes)
 		(on_board yes)
 		(in_pos_files yes)
@@
 		(body_style 1)
 		(exclude_from_sim no)
-		(in_bom yes)
+		(in_bom no)
 		(on_board yes)
 		(in_pos_files yes)
@@
 		(body_style 1)
 		(exclude_from_sim no)
-		(in_bom no)
+		(in_bom yes)
 		(on_board yes)
 		(in_pos_files yes)
@@
 			)
 		)
-		(property "Value" "LED_ARGB"
+		(property "Value" "RGB 5mm"
 			(at 261.62 86.36 0)
 			(show_name no)
@@
 		(body_style 1)
 		(exclude_from_sim no)
-		(in_bom no)
+		(in_bom yes)
 		(on_board no)
 		(in_pos_files yes)
@@
 		(body_style 1)
 		(exclude_from_sim no)
-		(in_bom no)
+		(in_bom yes)
 		(on_board yes)
 		(in_pos_files yes)
@@
 			)
 		)
-		(property "Value" "LED_ARGB"
+		(property "Value" "RGB 5mm"
 			(at 261.62 59.69 0)
 			(show_name no)
@@
 		(body_style 1)
 		(exclude_from_sim no)
-		(in_bom no)
+		(in_bom yes)
 		(on_board no)
 		(in_pos_files yes)

Commit message: Add files via upload
Parts:
- D121, D145, D26, D49, D73, D97: footprint Connector_IDC:IDC-Header_2x17_P2.54mm_Latch_Vertical -> LED_THT:LED_D5.0mm-4_RGB; now left out of the parts list
- SW3, SW4, SW5, SW6, SW7, SW8: now left out of the parts list
Changed lines of the file:
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@@
 		(body_style 1)
 		(exclude_from_sim no)
-		(in_bom yes)
+		(in_bom no)
 		(on_board yes)
 		(in_pos_files yes)
@@
 			)
 		)
-		(property "Footprint" "Connector_IDC:IDC-Header_2x17_P2.54mm_Latch_Vertical"
+		(property "Footprint" "LED_THT:LED_D5.0mm-4_RGB"
 			(at 261.62 45.72 0)
 			(hide yes)
@@
 		(body_style 1)
 		(exclude_from_sim no)
-		(in_bom yes)
+		(in_bom no)
 		(on_board no)
 		(in_pos_files yes)
@@
 		(body_style 1)
 		(exclude_from_sim no)
-		(in_bom yes)
+		(in_bom no)
 		(on_board yes)
 		(in_pos_files yes)
@@
 			)
 		)
-		(property "Footprint" "Connector_IDC:IDC-Header_2x17_P2.54mm_Latch_Vertical"
+		(property "Footprint" "LED_THT:LED_D5.0mm-4_RGB"
 			(at 260.35 177.8 0)
 			(hide yes)
@@
 		(body_style 1)
 		(exclude_from_sim no)
-		(in_bom yes)
+		(in_bom no)
 		(on_board yes)
 		(in_pos_files yes)
@@
 			)
 		)
-		(property "Footprint" "Connector_IDC:IDC-Header_2x17_P2.54mm_Latch_Vertical"
+		(property "Footprint" "LED_THT:LED_D5.0mm-4_RGB"
 			(at 261.62 152.4 0)
 			(hide yes)
@@
 		(body_style 1)
 		(exclude_from_sim no)
-		(in_bom yes)
+		(in_bom no)
 		(on_board no)
 		(in_pos_files yes)
@@
 		(body_style 1)
 		(exclude_from_sim no)
-		(in_bom yes)
+		(in_bom no)
 		(on_board no)
 		(in_pos_files yes)
@@
 		(body_style 1)
 		(exclude_from_sim no)
-		(in_bom yes)
+		(in_bom no)
 		(on_board yes)
 		(in_pos_files yes)
@@
 			)
 		)
-		(property "Footprint" "Connector_IDC:IDC-Header_2x17_P2.54mm_Latch_Vertical"
+		(property "Footprint" "LED_THT:LED_D5.0mm-4_RGB"
 			(at 261.62 125.73 0)
 			(hide yes)
@@
 		(body_style 1)
 		(exclude_from_sim no)
-		(in_bom yes)
+		(in_bom no)
 		(on_board no)
 		(in_pos_files yes)
@@
 		(body_style 1)
 		(exclude_from_sim no)
-		(in_bom yes)
+		(in_bom no)
 		(on_board yes)
 		(in_pos_files yes)
@@
 			)
 		)
-		(property "Footprint" "Connector_IDC:IDC-Header_2x17_P2.54mm_Latch_Vertical"
+		(property "Footprint" "LED_THT:LED_D5.0mm-4_RGB"
 			(at 261.62 99.06 0)
 			(hide yes)
@@
 		(body_style 1)
 		(exclude_from_sim no)
-		(in_bom yes)
+		(in_bom no)
 		(on_board no)
 		(in_pos_files yes)
@@
 		(body_style 1)
 		(exclude_from_sim no)
-		(in_bom yes)
+		(in_bom no)
 		(on_board yes)
 		(in_pos_files yes)
@@
 			)
 		)
-		(property "Footprint" "Connector_IDC:IDC-Header_2x17_P2.54mm_Latch_Vertical"
+		(property "Footprint" "LED_THT:LED_D5.0mm-4_RGB"
 			(at 261.62 72.39 0)
 			(hide yes)
@@
 		(body_style 1)
 		(exclude_from_sim no)
-		(in_bom yes)
+		(in_bom no)
 		(on_board no)
 		(in_pos_files yes)

Commit message: Add files via upload
Parts:
- J20, J21: now left out of the parts list
Changed lines of the file:
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@@
 		(body_style 1)
 		(exclude_from_sim no)
-		(in_bom yes)
+		(in_bom no)
 		(on_board yes)
 		(in_pos_files yes)
@@
 		(body_style 1)
 		(exclude_from_sim no)
-		(in_bom yes)
-		(on_board yes)
-		(in_pos_files yes)
+		(in_bom no)
+		(on_board yes)
+		(in_pos_files yes)

Commit message: Add files via upload
Parts:
- J20, J21, J22, J23, J24, J25: value Conn_01x03 (Fils soudés) -> Micro-Fit 3.0 1x03; footprint Connector_Wire:SolderWire-0.5sqmm_1x03_P4.6mm_D0.9mm_OD2.1mm_Relief -> Connector_Molex:Molex_Micro-Fit_3.0_43650-0315_1x03_P3.00mm_Vertical
- SW3, SW4, SW5, SW6, SW7, SW8: value Bouton verrouillable -> 82-5153.2000
Changed lines of the file:
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@@
 	(wire
 		(pts
-			(xy 154.94 62.23) (xy 148.59 62.23)
-		)
-		(stroke
-			(width 0)
-			(type default)
-		)
-	)
-	(wire
-		(pts
 			(xy 142.24 133.35) (xy 144.78 133.35)
 		)
@@
 	(wire
 		(pts
-			(xy 148.59 92.71) (xy 142.24 92.71)
+			(xy 142.24 92.71) (xy 152.4 92.71)
 		)
 		(stroke
@@
 	(wire
 		(pts
-			(xy 148.59 62.23) (xy 148.59 92.71)
-		)
-		(stroke
-			(width 0)
-			(type default)
-		)
-	)
-	(wire
-		(pts
 			(xy 266.7 151.13) (xy 271.78 151.13)
 		)
@@
 	)
 	(label "V_Ref"
-		(at 154.94 62.23 0)
+		(at 152.4 92.71 0)
 		(effects
 			(font
@@
 			)
 		)
-		(property "Value" "Conn_01x03 (Fils soudés)"
+		(property "Value" "Micro-Fit 3.0 1x03"
 			(at 59.69 109.2199 0)
 			(show_name no)
@@
 			)
 		)
-		(property "Footprint" "Connector_Wire:SolderWire-0.5sqmm_1x03_P4.6mm_D0.9mm_OD2.1mm_Relief"
+		(property "Footprint" "Connector_Molex:Molex_Micro-Fit_3.0_43650-0315_1x03_P3.00mm_Vertical"
 			(at 57.15 107.95 0)
 			(hide yes)
@@
 			)
 		)
-		(property "Value" "Conn_01x03 (Fils soudés)"
+		(property "Value" "Micro-Fit 3.0 1x03"
 			(at 59.69 129.5399 0)
 			(show_name no)
@@
 			)
 		)
-		(property "Footprint" "Connector_Wire:SolderWire-0.5sqmm_1x03_P4.6mm_D0.9mm_OD2.1mm_Relief"
+		(property "Footprint" "Connector_Molex:Molex_Micro-Fit_3.0_43650-0315_1x03_P3.00mm_Vertical"
 			(at 57.15 128.27 0)
 			(hide yes)
@@
 			)
 		)
-		(property "Value" "Bouton verrouillable"
+		(property "Value" "82-5153.2000"
 			(at 230.378 45.466 90)
 			(show_name no)
@@
 			)
 		)
-		(property "Value" "Conn_01x03 (Fils soudés)"
+		(property "Value" "Micro-Fit 3.0 1x03"
 			(at 59.69 88.8999 0)
 			(show_name no)
@@
 			)
 		)
-		(property "Footprint" "Connector_Wire:SolderWire-0.5sqmm_1x03_P4.6mm_D0.9mm_OD2.1mm_Relief"
+		(property "Footprint" "Connector_Molex:Molex_Micro-Fit_3.0_43650-0315_1x03_P3.00mm_Vertical"
 			(at 57.15 87.63 0)
 			(hide yes)
@@
 			)
 		)
-		(property "Value" "Bouton verrouillable"
+		(property "Value" "82-5153.2000"
 			(at 212.852 116.84 90)
 			(show_name no)
@@
 			)
 		)
-		(property "Value" "Conn_01x03 (Fils soudés)"
+		(property "Value" "Micro-Fit 3.0 1x03"
 			(at 59.69 99.0599 0)
 			(show_name no)
@@
 			)
 		)
-		(property "Footprint" "Connector_Wire:SolderWire-0.5sqmm_1x03_P4.6mm_D0.9mm_OD2.1mm_Relief"
+		(property "Footprint" "Connector_Molex:Molex_Micro-Fit_3.0_43650-0315_1x03_P3.00mm_Vertical"
 			(at 57.15 97.79 0)
 			(hide yes)
@@
 			)
 		)
-		(property "Value" "Bouton verrouillable"
+		(property "Value" "82-5153.2000"
 			(at 210.82 161.036 90)
 			(show_name no)
@@
 			)
 		)
-		(property "Value" "Bouton verrouillable"
+		(property "Value" "82-5153.2000"
 			(at 211.328 140.97 90)
 			(show_name no)
@@
 			)
 		)
-		(property "Value" "Conn_01x03 (Fils soudés)"
+		(property "Value" "Micro-Fit 3.0 1x03"
 			(at 59.69 77.4699 0)
 			(show_name no)
@@
 			)
 		)
-		(property "Footprint" "Connector_Wire:SolderWire-0.5sqmm_1x03_P4.6mm_D0.9mm_OD2.1mm_Relief"
+		(property "Footprint" "Connector_Molex:Molex_Micro-Fit_3.0_43650-0315_1x03_P3.00mm_Vertical"
 			(at 57.15 76.2 0)
 			(hide yes)
@@
 			)
 		)
-		(property "Value" "Conn_01x03 (Fils soudés)"
+		(property "Value" "Micro-Fit 3.0 1x03"
 			(at 59.69 119.3799 0)
 			(show_name no)
@@
 			)
 		)
-		(property "Footprint" "Connector_Wire:SolderWire-0.5sqmm_1x03_P4.6mm_D0.9mm_OD2.1mm_Relief"
+		(property "Footprint" "Connector_Molex:Molex_Micro-Fit_3.0_43650-0315_1x03_P3.00mm_Vertical"
 			(at 57.15 118.11 0)
 			(hide yes)
@@
 			)
 		)
-		(property "Value" "Bouton verrouillable"
+		(property "Value" "82-5153.2000"
 			(at 211.836 66.802 90)
 			(show_name no)
@@
 			)
 		)
-		(property "Value" "Bouton verrouillable"
+		(property "Value" "82-5153.2000"
 			(at 211.582 92.456 90)
 			(show_name no)

Commit message: Add files via upload
Parts:
- SW3, SW4, SW5, SW6, SW7, SW8: value 82-5153.2000 -> 82-4153.2000
Changed lines of the file:
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@@
 			)
 		)
-		(property "Value" "82-5153.2000"
+		(property "Value" "82-4153.2000"
 			(at 230.378 45.466 90)
 			(show_name no)
@@
 			)
 		)
-		(property "Value" "82-5153.2000"
+		(property "Value" "82-4153.2000"
 			(at 212.852 116.84 90)
 			(show_name no)
@@
 			)
 		)
-		(property "Value" "82-5153.2000"
+		(property "Value" "82-4153.2000"
 			(at 210.82 161.036 90)
 			(show_name no)
@@
 			)
 		)
-		(property "Value" "82-5153.2000"
+		(property "Value" "82-4153.2000"
 			(at 211.328 140.97 90)
 			(show_name no)
@@
 			)
 		)
-		(property "Value" "82-5153.2000"
+		(property "Value" "82-4153.2000"
 			(at 211.836 66.802 90)
 			(show_name no)
@@
 			)
 		)
-		(property "Value" "82-5153.2000"
+		(property "Value" "82-4153.2000"
 			(at 211.582 92.456 90)
 			(show_name no)
