File: Facade/Top_Zone.kicad_sch (KiCad schematic)
At the start: 0 parts

Commit message: Add files via upload
Parts:
- added D25: OSX10201-GYR1, OSX10201-GYR1:DIP760W45P254L2550H815Q20B, symbol OSX10201-GYR1:OSX10201-GYR1
- added J26: Conn_01x06, Connector_Wire:SolderWire-0.5sqmm_1x06_P4.6mm_D0.9mm_OD2.1mm_Relief, symbol Connector_Generic:Conn_01x06
- added J27: Conn_01x05, Connector_Wire:SolderWire-0.5sqmm_1x05_P4.6mm_D0.9mm_OD2.1mm_Relief, symbol Connector_Generic:Conn_01x05
- added J28: Conn_01x03, Connector_Wire:SolderWire-0.5sqmm_1x03_P4.6mm_D0.9mm_OD2.1mm_Relief, symbol Connector_Generic:Conn_01x03
- added J9: Conn_02x13_Odd_Even, Connector_IDC:IDC-Header_2x13_P2.54mm_Latch_Vertical, symbol Connector_Generic:Conn_02x13_Odd_Even
- added SW2: SW_DPDT_x2, symbol Switch:SW_DPDT_x2
- added SW9: CKS1503, symbol Switch:SW_Rotary_1x12
Connections:
- new net D25.11: D25.11, J9.17 (Pin_17)
- new net D25.12: D25.12, J9.18 (Pin_18)
- new net D25.13: D25.13, J9.19 (Pin_19)
- new net D25.14: D25.14, J9.20 (Pin_20)
- new net D25.15: D25.15, J9.21 (Pin_21)
- new net D25.16: D25.16, J9.22 (Pin_22)
- new net D25.17: D25.17, J9.23 (Pin_23)
- new net D25.18: D25.18, J9.24 (Pin_24)
- new net D25.19: D25.19, J9.25 (Pin_25)
- new net D25.20: D25.20, J9.26 (Pin_26)
- new net GND: J28.1 (Pin_1), J9.1 (Pin_1), J9.3 (Pin_3), SW2.4 (A)
- new net J26.1: J26.1 (Pin_1), J9.4 (Pin_4), SW9.1
- new net J26.2: J26.2 (Pin_2), J9.5 (Pin_5), SW9.2
- new net J26.3: J26.3 (Pin_3), J9.6 (Pin_6), SW9.3
- new net J26.4: J26.4 (Pin_4), J9.7 (Pin_7), SW9.4
- new net J26.5: J26.5 (Pin_5), J9.8 (Pin_8), SW9.5
- new net J26.6: J26.6 (Pin_6), J9.9 (Pin_9), SW9.6
- new net J27.1: J27.1 (Pin_1), J9.10 (Pin_10), SW9.7
- new net J27.2: J27.2 (Pin_2), J9.11 (Pin_11), SW9.8
- new net J27.3: J27.3 (Pin_3), J9.12 (Pin_12), SW9.9
- new net J27.4: J27.4 (Pin_4), J9.13 (Pin_13), SW9.10
- new net J27.5: J27.5 (Pin_5), J9.2 (Pin_2), SW9.13
- new net J28.2: J28.2 (Pin_2), J9.14 (Pin_14), SW2.5 (B)
- new net J28.3: J28.3 (Pin_3), J9.15 (Pin_15), SW2.6 (C)
- new net VLed_Jauge: D25.1, D25.10, D25.2, D25.3, D25.4, D25.5, D25.6, D25.7, D25.8, D25.9, J9.16 (Pin_16)
- no-connect marks 0 -> 2

Commit message: Add files via upload
Parts:
- J26: value Conn_01x06 -> Conn_01x06 (Fils soudés)
- J27: value Conn_01x05 -> Conn_01x05 (Fils soudés)
- J28: value Conn_01x03 -> Conn_01x03 (Fils soudés)
- SW2: now left out of the parts list
Changed lines of the file:
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@@
 		(exclude_from_sim no)
 		(in_bom no)
-		(on_board yes)
+		(on_board no)
 		(in_pos_files yes)
 		(dnp no)
@@
 			)
 		)
-		(property "Value" "Conn_01x05"
+		(property "Value" "Conn_01x05 (Fils soudés)"
 			(at 69.85 102.8699 0)
 			(show_name no)
@@
 		(body_style 1)
 		(exclude_from_sim no)
-		(in_bom yes)
-		(on_board yes)
+		(in_bom no)
+		(on_board no)
 		(in_pos_files yes)
 		(dnp no)
@@
 			)
 		)
-		(property "Value" "Conn_01x06"
+		(property "Value" "Conn_01x06 (Fils soudés)"
 			(at 70.358 120.396 0)
 			(show_name no)
@@
 			)
 		)
-		(property "Value" "Conn_01x03"
+		(property "Value" "Conn_01x03 (Fils soudés)"
 			(at 69.85 86.3599 0)
 			(show_name no)

Commit message: Add files via upload
Parts:
- J26: value Conn_01x06 (Fils soudés) -> Micro-Fit 3.0 1x06; footprint Connector_Wire:SolderWire-0.5sqmm_1x06_P4.6mm_D0.9mm_OD2.1mm_Relief -> Connector_Molex:Molex_Micro-Fit_3.0_43650-0615_1x06_P3.00mm_Vertical
- J27: value Conn_01x05 (Fils soudés) -> Micro-Fit 3.0 1x05; footprint Connector_Wire:SolderWire-0.5sqmm_1x05_P4.6mm_D0.9mm_OD2.1mm_Relief -> Connector_Molex:Molex_Micro-Fit_3.0_43650-0515_1x05_P3.00mm_Vertical
- J28: value Conn_01x03 (Fils soudés) -> Micro-Fit 3.0 1x03; footprint Connector_Wire:SolderWire-0.5sqmm_1x03_P4.6mm_D0.9mm_OD2.1mm_Relief -> Connector_Molex:Molex_Micro-Fit_3.0_43650-0315_1x03_P3.00mm_Vertical
Changed lines of the file:
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@@
 			)
 		)
-		(property "Value" "Conn_01x05 (Fils soudés)"
+		(property "Value" "Micro-Fit 3.0 1x05"
 			(at 69.85 102.8699 0)
 			(show_name no)
@@
 			)
 		)
-		(property "Footprint" "Connector_Wire:SolderWire-0.5sqmm_1x05_P4.6mm_D0.9mm_OD2.1mm_Relief"
+		(property "Footprint" "Connector_Molex:Molex_Micro-Fit_3.0_43650-0515_1x05_P3.00mm_Vertical"
 			(at 67.31 101.6 0)
 			(hide yes)
@@
 			)
 		)
-		(property "Value" "Conn_01x06 (Fils soudés)"
+		(property "Value" "Micro-Fit 3.0 1x06"
 			(at 70.358 120.396 0)
 			(show_name no)
@@
 			)
 		)
-		(property "Footprint" "Connector_Wire:SolderWire-0.5sqmm_1x06_P4.6mm_D0.9mm_OD2.1mm_Relief"
+		(property "Footprint" "Connector_Molex:Molex_Micro-Fit_3.0_43650-0615_1x06_P3.00mm_Vertical"
 			(at 67.31 118.11 0)
 			(hide yes)
@@
 			)
 		)
-		(property "Value" "Conn_01x03 (Fils soudés)"
+		(property "Value" "Micro-Fit 3.0 1x03"
 			(at 69.85 86.3599 0)
 			(show_name no)
@@
 			)
 		)
-		(property "Footprint" "Connector_Wire:SolderWire-0.5sqmm_1x03_P4.6mm_D0.9mm_OD2.1mm_Relief"
+		(property "Footprint" "Connector_Molex:Molex_Micro-Fit_3.0_43650-0315_1x03_P3.00mm_Vertical"
 			(at 67.31 85.09 0)
 			(hide yes)

Commit message: Add files via upload
Parts:
- SW2: value SW_DPDT_x2 -> Cole Hersee 5592
Changed lines of the file:
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@@
 			)
 		)
-		(property "Value" "SW_DPDT_x2"
+		(property "Value" "Cole Hersee 5592"
 			(at 67.31 59.69 0)
 			(hide yes)
